File: 2015/Hardware/PT_2015_PB_MAIN_Rev1.sch (EAGLE design)
At the start: 46 parts, among them Q1 Q_INA28, Q2 Q_INA28, Q4 Q_ACS711LC, Q5 Q_ACS711LC, Q6 Q_IRFS7437PbF

Commit message: Added the LT1910 for the MOSFET driver
Also I copied and pasted all of the primary voltage busses.
Parts:
- added C16, C17, C18, C19, C20, C21, C22: (no value), resistor:C-USC1206
- added Q10, Q12, Q14, Q16, Q18, Q3, Q8: Q_INA28, MRDT-2014-All:Q_INA28
- added Q11, Q13, Q15, Q17, Q19, Q7, Q9: Q_IRFS7437PbF, MRDT-2015-PowerBoard:Q_IRF7437SMD
- added R10, R11, R12, R13, R14, R15, R9: (no value), MRDT-2014-All:R_FC4L110R001JER
- added U$10, U$11, U$12, U$13, U$6, U$7, U$8, U$9: LT1910, Jake:LT1910
Connections:
- new net N$43: U$6.IN
- new net N$44: Q3.+IN, R9.SENSE2
- new net N$45: Q3.-IN, R9.SENSE1
- new net N$46: Q7.D, R9.1, U$7.SENSE, U$7.V+
- new net N$47: Q7.S
- new net N$48: Q7.G, U$7.GATE
- new net N$49: U$7.IN
- new net N$50: Q8.+IN, R10.SENSE2
- new net N$51: Q8.-IN, R10.SENSE1
- new net N$52: Q9.D, R10.1, U$8.SENSE, U$8.V+
- new net N$53: Q9.S
- new net N$54: Q9.G, U$8.GATE
- new net N$55: U$8.IN
- new net N$56: Q10.+IN, R11.SENSE2
- new net N$57: Q10.-IN, R11.SENSE1
- new net N$58: Q11.D, R11.1, U$9.SENSE, U$9.V+
- new net N$59: Q11.S
- new net N$60: Q11.G, U$9.GATE
- new net N$61: U$9.IN
- new net N$62: Q12.+IN, R12.SENSE2
- new net N$63: Q12.-IN, R12.SENSE1
- new net N$64: Q13.D, R12.1, U$10.SENSE, U$10.V+
- new net N$65: Q13.S
- new net N$66: Q13.G, U$10.GATE
- new net N$67: U$10.IN
- new net N$68: Q14.+IN, R13.SENSE2
- new net N$69: Q14.-IN, R13.SENSE1
- new net N$70: Q15.D, R13.1, U$11.SENSE, U$11.V+
- new net N$71: Q15.S
- new net N$72: Q15.G, U$11.GATE
- new net N$73: U$11.IN
- new net N$74: Q16.+IN, R14.SENSE2
- new net N$75: Q16.-IN, R14.SENSE1
- new net N$76: Q17.D, R14.1, U$12.SENSE, U$12.V+
- new net N$77: Q17.S
- new net N$78: Q17.G, U$12.GATE
- new net N$79: U$12.IN
- new net N$80: Q18.+IN, R15.SENSE2
- new net N$81: Q18.-IN, R15.SENSE1
- new net N$82: Q19.D, R15.1, U$13.SENSE, U$13.V+
- new net N$83: Q19.S
- new net N$84: Q19.G, U$13.GATE
- new net N$85: U$13.IN
- net +5V: now also C16.1, C17.1, C18.1, C19.1, C20.1, C21.1, C22.1, Q10.REF2, Q10.V+, Q12.REF2, Q12.V+, Q14.REF2, Q14.V+, Q16.REF2, Q16.V+, Q18.REF2, Q18.V+, Q3.REF2, Q3.V+, Q8.REF2, Q8.V+
- net GND: now also C16.2, C17.2, C18.2, C19.2, C20.2, C21.2, C22.2, Q10.GND, Q10.REF1, Q12.GND, Q12.REF1, Q14.GND, Q14.REF1, Q16.GND, Q16.REF1, Q18.GND, Q18.REF1, Q3.GND, Q3.REF1, Q8.GND, Q8.REF1, U$10.GND, U$11.GND, U$12.GND, U$13.GND, U$6.GND, U$7.GND, U$8.GND, U$9.GND
- net N$40: now also U$6.SENSE, U$6.V+
- net N$42: now also U$6.GATE
- net V_BATT: now also R10.2, R11.2, R12.2, R13.2, R14.2, R15.2, R9.2

Commit message: Removed Primary voltage busses
I was overeager with my copying and pasting. I removed the busses so I
could keep working on them.
Parts:
- removed C17, C18, C19, C20, C21, C22: (no value), resistor:C-USC1206
- removed Q10, Q12, Q14, Q16, Q18, Q3, Q8: Q_INA28, MRDT-2014-All:Q_INA28
- removed Q11, Q13, Q15, Q17, Q19, Q7, Q9: Q_IRFS7437PbF, MRDT-2015-PowerBoard:Q_IRF7437SMD
- removed R10, R11, R12, R13, R14, R15, R9: (no value), MRDT-2014-All:R_FC4L110R001JER
- removed U$10, U$11, U$12, U$13, U$7, U$8, U$9: LT1910, Jake:LT1910
Connections:
- removed net N$44: Q3.+IN, R9.SENSE2
- removed net N$45: Q3.-IN, R9.SENSE1
- removed net N$46: Q7.D, R9.1, U$7.SENSE, U$7.V+
- removed net N$47: Q7.S
- removed net N$48: Q7.G, U$7.GATE
- removed net N$49: U$7.IN
- removed net N$50: Q8.+IN, R10.SENSE2
- removed net N$51: Q8.-IN, R10.SENSE1
- removed net N$52: Q9.D, R10.1, U$8.SENSE, U$8.V+
- removed net N$53: Q9.S
- removed net N$54: Q9.G, U$8.GATE
- removed net N$55: U$8.IN
- removed net N$56: Q10.+IN, R11.SENSE2
- removed net N$57: Q10.-IN, R11.SENSE1
- removed net N$58: Q11.D, R11.1, U$9.SENSE, U$9.V+
- removed net N$59: Q11.S
- removed net N$60: Q11.G, U$9.GATE
- removed net N$61: U$9.IN
- removed net N$62: Q12.+IN, R12.SENSE2
- removed net N$63: Q12.-IN, R12.SENSE1
- removed net N$64: Q13.D, R12.1, U$10.SENSE, U$10.V+
- removed net N$65: Q13.S
- removed net N$66: Q13.G, U$10.GATE
- removed net N$67: U$10.IN
- removed net N$68: Q14.+IN, R13.SENSE2
- removed net N$69: Q14.-IN, R13.SENSE1
- removed net N$70: Q15.D, R13.1, U$11.SENSE, U$11.V+
- removed net N$71: Q15.S
- removed net N$72: Q15.G, U$11.GATE
- removed net N$73: U$11.IN
- removed net N$74: Q16.+IN, R14.SENSE2
- removed net N$75: Q16.-IN, R14.SENSE1
- removed net N$76: Q17.D, R14.1, U$12.SENSE, U$12.V+
- removed net N$77: Q17.S
- removed net N$78: Q17.G, U$12.GATE
- removed net N$79: U$12.IN
- removed net N$80: Q18.+IN, R15.SENSE2
- removed net N$81: Q18.-IN, R15.SENSE1
- removed net N$82: Q19.D, R15.1, U$13.SENSE, U$13.V+
- removed net N$83: Q19.S
- removed net N$84: Q19.G, U$13.GATE
- removed net N$85: U$13.IN
- net +5V: no longer C16.1, C17.1, C18.1, C19.1, C20.1, C21.1, C22.1, Q10.REF2, Q10.V+, Q12.REF2, Q12.V+, Q14.REF2, Q14.V+, Q16.REF2, Q16.V+, Q18.REF2, Q18.V+, Q3.REF2, Q3.V+, Q8.REF2, Q8.V+
- net GND: now also C16.1; no longer C16.2, C17.2, C18.2, C19.2, C20.2, C21.2, C22.2, Q10.GND, Q10.REF1, Q12.GND, Q12.REF1, Q14.GND, Q14.REF1, Q16.GND, Q16.REF1, Q18.GND, Q18.REF1, Q3.GND, Q3.REF1, Q8.GND, Q8.REF1, U$10.GND, U$11.GND, U$12.GND, U$13.GND, U$7.GND, U$8.GND, U$9.GND
- net N$40: now also C16.2
- net V_BATT: no longer R10.2, R11.2, R12.2, R13.2, R14.2, R15.2, R9.2
Other:
- moved on the sheet: C16

Commit message: Additional 5V bus and Motor Controller Connection
Changed the 5V bus to a non-critical bus, and added a low-power
critical 5V bus that breaks off of the 12V critical bus for the
motherboard.

Additionally, a pluggable screw terminal was added to the motor
controller bus, and values were updated everywhere
Parts:
- added C17: 47µF, resistor:C-USC1206
- added MOTOR_1: H_20020618-M02, MRDT-2015-PowerBoard:H_20020618-M02
- added OKI-78SR-5/1.5-W36H: Q_OKI-78SR, MRDT-2015-PowerBoard:Q_OKI-78SR
- C16: value (none) -> 10µF
- C5: value (none) -> .1µF
- R1: value (none) -> .001Ω
- renumbered VADER-5V-CRIT to VADER-5V-EXT
Connections:
- net N$33 renamed 5V-EXT
- net N$38 renamed 12V-AUX
- removed net N$37: C8.1, Q5.IP-
- new net 12V-CRIT: C8.1, OKI-78SR-5/1.5-W36H.VI, Q5.IP-
- new net 5V-CRIT: C17.1, OKI-78SR-5/1.5-W36H.VO
- net GND: now also C17.2, MOTOR_1.L, OKI-78SR-5/1.5-W36H.GND
- net N$41: now also MOTOR_1.R
Changed lines of the file:
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@@
 <part name="SIDEOUS-12V" library="MRDT-2015-PowerBoard" deviceset="UQW-12/20-T48NBS" device=""/>
 <part name="PALPATINE-12V" library="MRDT-2015-PowerBoard" deviceset="UQW-12/20-T48NBS" device=""/>
-<part name="VADER-5V-CRIT" library="MRDT-2015-PowerBoard" deviceset="Q_PTN78020" device="" value="Q_PTN78020WAH"/>
+<part name="VADER-5V-EXT" library="MRDT-2015-PowerBoard" deviceset="Q_PTN78020" device="" value="Q_PTN78020WAH"/>
 <part name="DOOKU-12V-CRIT" library="MRDT-2015-PowerBoard" deviceset="Q_PTN78020" device="" value="Q_PTN78020WAH"/>
 <part name="GND2" library="SparkFun-Aesthetics" deviceset="GND" device=""/>
@@
 <part name="C3" library="MRDT-2014-All" deviceset="C_POL" device="12.5MM_NORMAL" value="1mF"/>
 <part name="C4" library="MRDT-2014-All" deviceset="C_POL" device="12.5MM_NORMAL" value="1mF"/>
-<part name="R1" library="MRDT-2014-All" deviceset="R_FC4L110R001JER" device=""/>
+<part name="R1" library="MRDT-2014-All" deviceset="R_FC4L110R001JER" device="" value=".001Ω"/>
 <part name="Q1" library="MRDT-2014-All" deviceset="Q_INA28" device=""/>
 <part name="SUPPLY1" library="SparkFun-Aesthetics" deviceset="V_BATT" device=""/>
 <part name="GND1" library="SparkFun-Aesthetics" deviceset="GND" device=""/>
-<part name="C5" library="resistor" deviceset="C-US" device="C1206"/>
+<part name="C5" library="resistor" deviceset="C-US" device="C1206" value=".1µF"/>
 <part name="P+1" library="supply1" deviceset="+5V" device=""/>
 <part name="P+2" library="supply1" deviceset="+5V" device=""/>
@@
 <part name="U$6" library="Jake" deviceset="LT1910" device=""/>
 <part name="GND27" library="SparkFun-Aesthetics" deviceset="GND" device=""/>
-<part name="C16" library="resistor" deviceset="C-US" device="C1206"/>
+<part name="C16" library="resistor" deviceset="C-US" device="C1206" value="10µF"/>
 <part name="GND28" library="SparkFun-Aesthetics" deviceset="GND" device=""/>
+<part name="MOTOR_1" library="MRDT-2015-PowerBoard" deviceset="H_20020618-M02*" device=""/>
+<part name="GND29" library="SparkFun-Aesthetics" deviceset="GND" device=""/>
+<part name="OKI-78SR-5/1.5-W36H" library="MRDT-2015-PowerBoard" deviceset="Q_OKI-78SR" device=""/>
+<part name="GND30" library="SparkFun-Aesthetics" deviceset="GND" device=""/>
+<part name="C17" library="resistor" deviceset="C-US" device="C1206" value="47µF"/>
 </parts>
 <sheets>
@@
 <instance part="SIDEOUS-12V" gate="G$1" x="63.5" y="73.66"/>
 <instance part="PALPATINE-12V" gate="G$1" x="63.5" y="43.18"/>
-<instance part="VADER-5V-CRIT" gate="G$1" x="45.72" y="12.7"/>
+<instance part="VADER-5V-EXT" gate="G$1" x="45.72" y="12.7"/>
 <instance part="DOOKU-12V-CRIT" gate="G$1" x="45.72" y="134.62"/>
 <instance part="GND2" gate="1" x="2.54" y="10.16"/>
@@
 <instance part="C16" gate="G$1" x="-205.74" y="152.4"/>
 <instance part="GND28" gate="1" x="-213.36" y="160.02"/>
+<instance part="MOTOR_1" gate="G$1" x="-205.74" y="96.52"/>
+<instance part="GND29" gate="1" x="-218.44" y="93.98"/>
+<instance part="OKI-78SR-5/1.5-W36H" gate="G$1" x="218.44" y="129.54"/>
+<instance part="GND30" gate="1" x="220.98" y="116.84"/>
+<instance part="C17" gate="G$1" x="236.22" y="127"/>
 </instances>
 <busses>
@@
 </segment>
 <segment>
-<pinref part="VADER-5V-CRIT" gate="G$1" pin="GND"/>
+<pinref part="VADER-5V-EXT" gate="G$1" pin="GND"/>
 <pinref part="GND2" gate="1" pin="GND"/>
 <wire x1="40.64" y1="12.7" x2="35.56" y2="12.7" width="0.1524" layer="91"/>
@@
 </segment>
 <segment>
-<pinref part="VADER-5V-CRIT" gate="G$1" pin="GND1"/>
+<pinref part="VADER-5V-EXT" gate="G$1" pin="GND1"/>
 <pinref part="GND13" gate="1" pin="GND"/>
 </segment>
@@
 <pinref part="GND28" gate="1" pin="GND"/>
 <wire x1="-213.36" y1="167.64" x2="-213.36" y2="162.56" width="0.1524" layer="91"/>
+</segment>
+<segment>
+<pinref part="MOTOR_1" gate="G$1" pin="L"/>
+<pinref part="GND29" gate="1" pin="GND"/>
+<wire x1="-215.9" y1="99.06" x2="-218.44" y2="99.06" width="0.1524" layer="91"/>
+<wire x1="-218.44" y1="99.06" x2="-218.44" y2="96.52" width="0.1524" layer="91"/>
+</segment>
+<segment>
+<pinref part="OKI-78SR-5/1.5-W36H" gate="G$1" pin="GND"/>
+<pinref part="GND30" gate="1" pin="GND"/>
+<wire x1="220.98" y1="121.92" x2="220.98" y2="119.38" width="0.1524" layer="91"/>
+<pinref part="C17" gate="G$1" pin="2"/>
+<wire x1="236.22" y1="121.92" x2="236.22" y2="119.38" width="0.1524" layer="91"/>
+<wire x1="236.22" y1="119.38" x2="220.98" y2="119.38" width="0.1524" layer="91"/>
 </segment>
 </net>
@@
 <pinref part="L8" gate="G$1" pin="5"/>
 <wire x1="30.48" y1="-5.08" x2="30.48" y2="-2.54" width="0.1524" layer="91"/>
-<pinref part="VADER-5V-CRIT" gate="G$1" pin="VIN"/>
+<pinref part="VADER-5V-EXT" gate="G$1" pin="VIN"/>
 <wire x1="40.64" y1="0" x2="35.56" y2="0" width="0.1524" layer="91"/>
 <junction x="30.48" y="-5.08"/>
@@
 <pinref part="L4" gate="G$1" pin="1"/>
 <wire x1="101.6" y1="5.08" x2="101.6" y2="2.54" width="0.1524" layer="91"/>
-<pinref part="VADER-5V-CRIT" gate="G$1" pin="VOUT"/>
+<pinref part="VADER-5V-EXT" gate="G$1" pin="VOUT"/>
 <wire x1="101.6" y1="2.54" x2="101.6" y2="0" width="0.1524" layer="91"/>
 <wire x1="101.6" y1="0" x2="101.6" y2="-2.54" width="0.1524" layer="91"/>
@@
 <junction x="101.6" y="-2.54"/>
 <wire x1="91.44" y1="0" x2="93.98" y2="0" width="0.1524" layer="91"/>
-<pinref part="VADER-5V-CRIT" gate="G$1" pin="SENSE"/>
+<pinref part="VADER-5V-EXT" gate="G$1" pin="SENSE"/>
 <wire x1="93.98" y1="0" x2="101.6" y2="0" width="0.1524" layer="91"/>
 <wire x1="73.66" y1="-10.16" x2="73.66" y2="-12.7" width="0.1524" layer="91"/>
@@
 <net name="N$35" class="0">
 <segment>
-<pinref part="VADER-5V-CRIT" gate="G$1" pin="ADJUST"/>
+<pinref part="VADER-5V-EXT" gate="G$1" pin="ADJUST"/>
 <wire x1="66.04" y1="-10.16" x2="66.04" y2="-12.7" width="0.1524" layer="91"/>
 <pinref part="R8" gate="G$1" pin="2"/>
 </segment>
 </net>
-<net name="N$33" class="0">
-<segment>
-<wire x1="172.72" y1="-2.54" x2="182.88" y2="-2.54" width="0.1524" layer="91"/>
+<net name="5V-EXT" class="0">
+<segment>
+<wire x1="172.72" y1="-2.54" x2="246.38" y2="-2.54" width="0.1524" layer="91"/>
 <pinref part="C12" gate="G$1" pin="1"/>
 <wire x1="172.72" y1="-5.08" x2="172.72" y2="-2.54" width="0.1524" layer="91"/>
@@
 <wire x1="137.16" y1="10.16" x2="137.16" y2="-2.54" width="0.1524" layer="91"/>
 <wire x1="137.16" y1="-2.54" x2="172.72" y2="-2.54" width="0.1524" layer="91"/>
+<label x="246.38" y="-2.54" size="1.27" layer="95" xref="yes"/>
 </segment>
 </net>
@@
 </segment>
 </net>
-<net name="N$37" class="0">
+<net name="12V-CRIT" class="0">
 <segment>
 <pinref part="Q5" gate="G$1" pin="IP-"/>
@@
 <wire x1="177.8" y1="111.76" x2="205.74" y2="111.76" width="0.1524" layer="91"/>
 <wire x1="177.8" y1="109.22" x2="177.8" y2="111.76" width="0.1524" layer="91"/>
+<wire x1="205.74" y1="111.76" x2="248.92" y2="111.76" width="0.1524" layer="91"/>
+<wire x1="205.74" y1="111.76" x2="205.74" y2="129.54" width="0.1524" layer="91"/>
+<pinref part="OKI-78SR-5/1.5-W36H" gate="G$1" pin="VI"/>
+<wire x1="205.74" y1="129.54" x2="210.82" y2="129.54" width="0.1524" layer="91"/>
+<label x="248.92" y="111.76" size="1.27" layer="95" xref="yes"/>
 </segment>
 </net>
@@
 </segment>
 </net>
-<net name="N$38" class="0">
+<net name="12V-AUX" class="0">
 <segment>
 <pinref part="R2" gate="G$1" pin="1"/>
-<wire x1="157.48" y1="53.34" x2="170.18" y2="53.34" width="0.1524" layer="91"/>
-<wire x1="170.18" y1="53.34" x2="170.18" y2="48.26" width="0.1524" layer="91"/>
-<wire x1="170.18" y1="48.26" x2="205.74" y2="48.26" width="0.1524" layer="91"/>
+<wire x1="157.48" y1="53.34" x2="246.38" y2="53.34" width="0.1524" layer="91"/>
+<label x="246.38" y="53.34" size="1.27" layer="95" xref="yes"/>
 </segment>
 </net>
@@
 <segment>
 <pinref part="Q6" gate="G$1" pin="S"/>
-<wire x1="-193.04" y1="119.38" x2="-193.04" y2="101.6" width="0.1524" layer="91"/>
+<wire x1="-193.04" y1="119.38" x2="-193.04" y2="99.06" width="0.1524" layer="91"/>
+<pinref part="MOTOR_1" gate="G$1" pin="R"/>
+<wire x1="-195.58" y1="99.06" x2="-193.04" y2="99.06" width="0.1524" layer="91"/>
 </segment>
 </net>
@@
 </segment>
 </net>
+<net name="5V-CRIT" class="0">
+<segment>
+<pinref part="OKI-78SR-5/1.5-W36H" gate="G$1" pin="VO"/>
+<wire x1="231.14" y1="129.54" x2="236.22" y2="129.54" width="0.1524" layer="91"/>
+<pinref part="C17" gate="G$1" pin="1"/>
+<junction x="236.22" y="129.54"/>
+<wire x1="236.22" y1="129.54" x2="248.92" y2="129.54" width="0.1524" layer="91"/>
+<label x="248.92" y="129.54" size="1.27" layer="95" xref="yes"/>
+</segment>
+</net>
