File: 2015/Hardware/PT_2015_PB_MAIN_Rev1.brd (EAGLE design)
At the start: 120.3 x 80 mm, 136 parts, among them Q1 Q_INA28, Q10 Q_INA28, Q11 Q_IRFS7437PbF, Q12 2N7002, Q13 Q_INA28, Q14 Q_IRFS7437PbF, Q15 Q_INA28, Q16 Q_IRFS7437PbF, Q17 Q_INA28, Q18 Q_IRFS7437PbF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

Commit message: I did stuff
hey check it out
Parts:
- moved 12V-AUX 407.6 mm to (223.5, 154.9), turned to 90 degrees
- moved LED2 396.1 mm to (218.4, 74.9)
- moved R2 389.7 mm to (233.7, 86.4)
- moved 12V-CRIT 388.5 mm to (218.4, 55.9)
- moved R26 353.9 mm to (165.1, 12.7), turned to 90 degrees
- moved R28 338.1 mm to (142.2, 12.7), turned to 90 degrees
- moved C13 337.0 mm to (180.3, 95.2)
- moved R10 330.3 mm to (214.6, 87.6)
- moved L8 320.0 mm to (166.4, 81.3)
- moved R25 317.9 mm to (176.5, 48.3), turned to 90 degrees
- moved Q17 312.5 mm to (166.4, 48.3), turned to 270 degrees
- moved U$12 312.2 mm to (166.4, 29.2), turned to 270 degrees
- moved R24 309.5 mm to (119.4, 12.7), turned to 90 degrees
- moved R27 306.9 mm to (153.7, 48.3), turned to 90 degrees
- moved Q19 306.6 mm to (143.5, 48.3), turned to 270 degrees
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Routing:
- added copper zone on layer 16, net GND
- added copper zone on layer 1, net V_BATT
Other:
- board size 120.3 x 80 mm -> 199.4 x 152.4 mm

Commit message: Into sex
is happen
Parts:
- moved U$4 273.1 mm to (237.5, 26.7), turned to 90 degrees
- moved R4 252.8 mm to (194.3, 43.2), turned to 90 degrees
- moved C14 247.9 mm to (295.9, 21.0)
- moved L5 247.9 mm to (295.9, 14.6)
- moved C21 247.9 mm to (303.5, 69.2)
- moved L1 247.9 mm to (290.8, 66.7)
- moved Q5 247.9 mm to (290.8, 74.3)
- moved DOOKU-12V-CRIT 247.6 mm to (294.6, 43.8)
- moved OKI-78SR-5/1.5-W36H 243.9 mm to (271.8, 52.7)
- moved R6 240.2 mm to (222.9, 22.9), turned to 270 degrees
- moved R5 233.2 mm to (222.9, 29.8), turned to 270 degrees
- moved 5V-INT 222.8 mm to (254.0, 84.5)
- moved U$3 219.9 mm to (215.3, 26.7), turned to 270 degrees
- moved U$1 215.0 mm to (205.7, 26.7), turned to 270 degrees
- moved R3 204.0 mm to (194.3, 50.8), turned to 90 degrees
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Routing:
- net M1-IMEAS: track 0.00 -> 255.7 mm
- net M1-SIG: track 0.00 -> 234.6 mm
- net M2-IMEAS: track 0.00 -> 229.8 mm
- net +5V: track 0.00 -> 224.5 mm
- net M2-SIG: track 0.00 -> 208.7 mm
- net M4-IMEAS: track 0.00 -> 203.8 mm
- net M4-SIG: track 0.00 -> 182.7 mm
- net M5-IMEAS: track 0.00 -> 177.9 mm
- net M5-SIG: track 0.00 -> 156.8 mm
- net M6-IMEAS: track 0.00 -> 152.0 mm
- net M6-SIG: track 0.00 -> 130.9 mm
- net M3-IMEAS: track 0.00 -> 126.1 mm
- net M3-SIG: track 0.00 -> 104.9 mm
- net AUX_P-IMEAS: track 0.00 -> 100.1 mm
- net GND: track 0.00 -> 94.7 mm, vias 0 -> 24
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- added copper zone on layer 1, net N$28
- added copper zone on layer 1, net N$29
- added copper zone on layer 1, net N$4
- added copper zone on layer 1, net N$40
- added copper zone on layer 1, net N$41
- added copper zone on layer 1, net N$44
- added copper zone on layer 1, net N$45
- added copper zone on layer 1, net N$54
- added copper zone on layer 1, net N$55
- added copper zone on layer 1, net N$60
- added copper zone on layer 1, net N$61
- added copper zone on layer 1, net N$66
- added copper zone on layer 1, net N$67
- added copper zone on layer 1, net N$72
- added copper zone on layer 1, net N$73
- added copper zone on layer 1, net N$78
- added copper zone on layer 1, net N$79
Other:
- board size 199.4 x 152.4 mm -> 241.3 x 151.8 mm

Commit message: Erectile Function
;)
Connections:
- net 12V-IMEAS: now also U$1.32; no longer U$1.22
- net 12V-SIG: now also U$1.2; no longer U$1.25
- net 5V-IMEAS: now also U$1.30; no longer U$1.23
- net ARM_P-IMEAS: now also U$1.19; no longer U$1.32
- net ARM_P-SIG: now also U$1.13; no longer U$1.27
- net AUX_P-IMEAS: now also U$1.20; no longer U$1.28
- net AUX_P-SIG: now also U$1.12; no longer U$1.26
- net CRIT-IMEAS: now also U$1.31; no longer U$1.21
- net M1-IMEAS: now also U$1.29; no longer U$1.20
- net M1-SIG: now also U$1.27; no longer U$1.2
- net M2-IMEAS: now also U$1.28; no longer U$1.19
- net M2-SIG: now also U$1.26; no longer U$1.5
- net M3-IMEAS: now also Q8.5, U$1.24; no longer Q15.5, U$1.1
- net M3-SIG: now also U$1.25, U$8.4; no longer U$1.6, U$11.4
- net M4-IMEAS: now also Q10.5, U$1.23; no longer Q8.5, U$1.31
- net M4-SIG: now also U$1.5, U$9.4; no longer U$1.8, U$8.4
- net M5-IMEAS: now also Q13.5, U$1.22; no longer Q10.5, U$1.30
- net M5-SIG: now also U$1.6, U$10.4; no longer U$1.12, U$9.4
- net M6-IMEAS: now also Q15.5, U$1.21; no longer Q13.5, U$1.29
- net M6-SIG: now also U$1.8, U$11.4; no longer U$1.13, U$10.4
- net PRIMARY-VMEAS: now also U$1.1; no longer U$1.24
Routing:
- net M3-SIG: track 104.9 -> 194.7 mm
- net M3-IMEAS: track 126.1 -> 210.8 mm
- net M6-IMEAS: track 152.0 -> 129.2 mm
- net M1-SIG: track 234.6 -> 256.7 mm
- net M5-IMEAS: track 177.9 -> 156.4 mm
- net AUX_P-SIG: track 79.0 -> 99.7 mm
- net M4-IMEAS: track 203.8 -> 183.6 mm
- net ARM_P-SIG: track 53.1 -> 72.5 mm
- net M1-IMEAS: track 255.7 -> 272.8 mm
- net M2-IMEAS: track 229.8 -> 245.6 mm
- net M2-SIG: track 208.7 -> 220.1 mm
- net M4-SIG: track 182.7 -> 185.4 mm
- net AUX_P-IMEAS: track 100.1 -> 102.0 mm
- net M5-SIG: track 156.8 -> 158.3 mm
- net M6-SIG: track 130.9 -> 130.0 mm
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
Commit message: This is a literal sexual experience at this point
I'm going to need protection
Parts:
- moved LED3 280.3 mm to (235.6, 55.9), turned to 270 degrees
- moved C8 214.6 mm to (229.9, 50.2), turned to 270 degrees
- moved R7 184.8 mm to (196.2, 65.4), turned to 90 degrees
- moved R11 174.7 mm to (231.8, 55.9), turned to 90 degrees
- moved L3 155.8 mm to (219.7, 36.2)
- moved C18 152.4 mm to (224.2, 37.5), turned to 90 degrees
- moved L5 128.5 mm to (184.2, 78.1), turned to 270 degrees
- moved U$5 123.5 mm to (226.1, 58.4), turned to 90 degrees
- moved C14 116.0 mm to (196.8, 81.3), turned to 90 degrees
- moved C9 115.4 mm to (223.5, 58.4), turned to 90 degrees
- moved LED4 111.3 mm to (228.0, 70.5)
- moved LED2 103.3 mm to (228.6, 111.8)
- moved 5V-EXT 101.8 mm to (233.7, 77.5)
- moved DOOKU-12V-CRIT 95.2 mm to (201.9, 65.4), turned to 270 degrees
- moved U$2 94.3 mm to (71.1, 169.5)
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Connections:
- net 12V-CRIT: now also Q5.1; no longer Q5.4
- net 5V-IMEAS: now also U$1.31; no longer U$1.30
- net ARM_P-IMEAS: now also U$1.20; no longer U$1.19
- net AUX_P-IMEAS: now also U$1.21; no longer U$1.20
- net CRIT-IMEAS: now also U$1.1; no longer U$1.31
- net M1-IMEAS: now also U$1.30; no longer U$1.29
- net M2-IMEAS: now also U$1.29; no longer U$1.28
- net M3-IMEAS: now also U$1.28; no longer U$1.24
- net M4-IMEAS: now also U$1.24; no longer U$1.23
- net M5-IMEAS: now also U$1.23; no longer U$1.22
- net M6-IMEAS: now also U$1.22; no longer U$1.21
- net N$10: now also Q5.4; no longer Q5.1
- net PRIMARY-VMEAS: now also U$1.19; no longer U$1.1
Routing:
- net +5V: track 224.5 -> 314.5 mm
- net N$36: track 0.00 -> 57.1 mm
- net PRIMARY-VMEAS: track 0.00 -> 41.5 mm
- net 12V-CRIT: track 0.00 -> 39.2 mm
- net CRIT-IMEAS: track 0.00 -> 37.7 mm
- net N$3: track 0.00 -> 28.9 mm
- net N$20: track 0.00 -> 24.2 mm
- net N$8: track 0.00 -> 23.2 mm
- net N$10: track 0.00 -> 20.1 mm
- net N$15: track 0.00 -> 15.9 mm
- net GND: track 94.7 -> 108.6 mm, vias 24 -> 36
- net N$14: track 0.00 -> 13.3 mm
- net N$21: track 0.00 -> 12.6 mm
- net N$18: track 0.00 -> 10.3 mm
- net RXD: track 0.00 -> 10.3 mm
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- added copper zone on layer 1, net N$5
- added copper zone on layer 1, net N$6
- added copper zone on layer 1, net N$7
Other:
- board size 241.3 x 151.8 mm -> 241.9 x 137.2 mm

Commit message: Speaking of sexual experiences...
It is bed time. Cleaned up the ugly pour. Work will resume tomorrow.
Parts:
- moved C20 59.3 mm to (165.7, 138.4)
- moved C27 59.3 mm to (140.3, 147.3)
- moved C29 59.3 mm to (134.0, 147.3)
- moved C31 59.3 mm to (154.3, 158.8)
- moved C10 59.3 mm to (186.1, 138.4)
- moved C11 59.3 mm to (181.0, 138.4)
- moved C12 59.3 mm to (102.2, 147.3)
- moved C19 59.3 mm to (170.8, 138.4)
- moved C23 59.3 mm to (153.0, 147.3)
- moved C25 59.3 mm to (146.7, 147.3)
- moved C33 59.3 mm to (121.3, 147.3)
- moved C35 59.3 mm to (112.4, 153.0)
- moved C5 59.3 mm to (159.4, 147.3)
- moved C6 59.3 mm to (196.2, 138.4)
- moved C7 59.3 mm to (97.2, 147.3)
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Routing:
- net N$3: track 28.9 -> 35.8 mm
- net N$35: track 3.88 -> 5.11 mm
- net GND: track 108.6 -> 109.3 mm
Other:
- board size 241.9 x 137.2 mm -> 241.3 x 127.6 mm

Commit message: Initial Powerboard Layout Completed.
Board layout finished. Passed DRC with zero airwires and 51 approved
errors (GND via overlap with SMD pads). One single ground plane cut was
used. Board will be rerouted for smaller size.
Parts:
- C6: value (none) -> .1µF
- moved C5 184.4 mm to (6.35, 44.5)
- moved C7 169.9 mm to (211.5, 21.6), turned to 270 degrees
- moved C23 161.0 mm to (29.2, 44.5)
- moved R13 144.0 mm to (230.5, 33.7)
- moved C12 140.2 mm to (232.4, 95.2), turned to 90 degrees
- moved C25 139.8 mm to (52.1, 44.5)
- moved C27 121.9 mm to (74.9, 44.5)
- moved LED5 121.2 mm to (235.6, 33.7)
- moved C31 119.2 mm to (120.7, 44.5)
- moved U$2 118.8 mm to (226.1, 87.6), turned to 270 degrees
- moved C35 113.0 mm to (143.5, 44.5)
- moved C33 112.3 mm to (166.4, 44.5)
- moved C29 109.1 mm to (97.8, 44.5)
- moved R15 108.6 mm to (65.4, 86.4), turned to 180 degrees
- moved C11 66.3 mm to (222.9, 87.0), turned to 270 degrees
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Connections:
- net 12V-AUX: now also R2.2; no longer R2.1
- net N$11: now also R2.1; no longer R2.2
Routing:
- net 12V-SIG: track 0.00 -> 412.4 mm
- net +5V: track 314.5 -> 474.8 mm
- net 12V-IMEAS: track 0.00 -> 160.1 mm
- net 5V-IMEAS: track 0.00 -> 122.4 mm
- net N$4: track 0.00 -> 46.2 mm
- net GND: track 109.3 -> 138.2 mm, vias 36 -> 51
- net N$15: track 15.9 -> 42.1 mm
- net 5V-EXT: track 0.00 -> 22.7 mm
- net N$16: track 0.00 -> 21.8 mm
- net N$3: track 35.8 -> 18.3 mm
- net N$36: track 57.1 -> 43.3 mm
- net N$114: track 0.00 -> 9.28 mm
- net N$50: track 0.00 -> 4.11 mm
- net N$12: track 0.00 -> 3.07 mm
- net N$46: track 0.00 -> 2.96 mm
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- added copper zone on layer 1, net 12V-AUX
- added copper zone on layer 1, net N$11
- removed copper zone on layer 1, net N$4
