File: 2015/Hardware/PT_2015_PB_MAIN_Rev2.sch (EAGLE design)
At the start: 137 parts, among them Q1 Q_ACS711LC_SKETCH, Q11 Q_IRFS7437PbF, Q12 2N7002, Q14 Q_IRFS7437PbF, Q16 Q_IRFS7437PbF, Q18 Q_FDT86102LZ, Q20 Q_IRFS7437PbF, Q4 Q_ACS711LC, Q5 Q_ACS711LC, Q6 Q_IRFS7437PbF, Q7 Q_IRFS7437PbF, Q9 Q_IRFS7437PbF

Commit message: Added LEDs, a buzzer, and adjusted traces
Parts:
- added LED13, LED14: (no value), SparkFun-LED:LED-FKIT-1206
- added R1, R2: 1k Ohm, SparkFun-Passives:RESISTOR1206
- added SG1: BUZZERSMD2, SparkFun-Electromechanical:BUZZERSMD2
Connections:
- new net BUZZ_BUZZ_MOTHERFUCKER: SG1.2, U$1.D11~
- new net INFO_LED_1: R1.1, U$1.MISO
- new net INFO_LED_2: R2.1, U$1.MOSI
- new net N$11: LED13.A, R1.2
- new net N$32: LED14.A, R2.2
- net AUX_P-IMEAS: now also U$1.D8/A8; no longer U$1.D5~
- net AUX_P-SIG: now also U$1.SCK; no longer U$1.D11~
- net GND: now also LED13.C, LED14.C, SG1.1
- net M1-SIG: now also U$1.PE2; no longer U$1.D10~/A10
- net M2-SIG: now also U$1.D13~; no longer U$1.D9~/A9
- net M3-SIG: now also U$1.D5~; no longer U$1.D8/A8
- net M5-IMEAS: now also U$1.D10~/A10; no longer U$1.PE2
- net M6-IMEAS: now also U$1.D9~/A9; no longer U$1.D13~
- net N$5: now also L6.9
Changed lines of the file:
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@@
 <part name="D1" library="diode" deviceset="15KEXX" device="" value="1.5KE36A"/>
 <part name="D2" library="diode" deviceset="15KEXX" device="" value="1.5KE36A"/>
+<part name="LED13" library="SparkFun-LED" deviceset="LED" device="-FKIT-1206"/>
+<part name="LED14" library="SparkFun-LED" deviceset="LED" device="-FKIT-1206"/>
+<part name="R1" library="SparkFun-Passives" deviceset="RESISTOR" device="1206" value="1k Ohm"/>
+<part name="R2" library="SparkFun-Passives" deviceset="RESISTOR" device="1206" value="1k Ohm"/>
+<part name="GND91" library="SparkFun-Aesthetics" deviceset="GND" device=""/>
+<part name="GND92" library="SparkFun-Aesthetics" deviceset="GND" device=""/>
+<part name="SG1" library="SparkFun-Electromechanical" deviceset="BUZZER" device="SMD2"/>
+<part name="GND93" library="SparkFun-Aesthetics" deviceset="GND" device=""/>
 </parts>
 <sheets>
@@
 <instance part="D1" gate="1" x="86.36" y="175.26" rot="R90"/>
 <instance part="D2" gate="1" x="78.74" y="175.26" rot="R90"/>
+<instance part="LED13" gate="G$1" x="-276.86" y="-167.64"/>
+<instance part="LED14" gate="G$1" x="-264.16" y="-167.64"/>
+<instance part="R1" gate="G$1" x="-276.86" y="-157.48" rot="R270"/>
+<instance part="R2" gate="G$1" x="-264.16" y="-157.48" rot="R270"/>
+<instance part="GND91" gate="1" x="-276.86" y="-180.34"/>
+<instance part="GND92" gate="1" x="-264.16" y="-180.34"/>
+<instance part="SG1" gate="G$1" x="-297.18" y="-165.1"/>
+<instance part="GND93" gate="1" x="-289.56" y="-180.34" rot="MR0"/>
 </instances>
 <busses>
@@
 <pinref part="GND90" gate="1" pin="GND"/>
 </segment>
+<segment>
+<pinref part="LED13" gate="G$1" pin="C"/>
+<pinref part="GND91" gate="1" pin="GND"/>
+<wire x1="-276.86" y1="-177.8" x2="-276.86" y2="-172.72" width="0.1524" layer="91"/>
+</segment>
+<segment>
+<pinref part="LED14" gate="G$1" pin="C"/>
+<pinref part="GND92" gate="1" pin="GND"/>
+<wire x1="-264.16" y1="-177.8" x2="-264.16" y2="-172.72" width="0.1524" layer="91"/>
+</segment>
+<segment>
+<pinref part="SG1" gate="G$1" pin="1"/>
+<wire x1="-297.18" y1="-167.64" x2="-297.18" y2="-172.72" width="0.1524" layer="91"/>
+<wire x1="-297.18" y1="-172.72" x2="-289.56" y2="-172.72" width="0.1524" layer="91"/>
+<wire x1="-289.56" y1="-172.72" x2="-289.56" y2="-177.8" width="0.1524" layer="91"/>
+<pinref part="GND93" gate="1" pin="GND"/>
+</segment>
 </net>
 <net name="V_BATT" class="0">
@@
 <pinref part="L6" gate="G$1" pin="5"/>
 <wire x1="27.94" y1="55.88" x2="27.94" y2="53.34" width="0.1524" layer="91"/>
+<junction x="27.94" y="53.34"/>
+<junction x="27.94" y="55.88"/>
+<junction x="27.94" y="45.72"/>
 </segment>
 <segment>
@@
 <pinref part="L6" gate="G$1" pin="8"/>
 <pinref part="L6" gate="G$1" pin="10"/>
-<wire x1="38.1" y1="55.88" x2="38.1" y2="50.8" width="0.1524" layer="91"/>
+<wire x1="38.1" y1="55.88" x2="38.1" y2="53.34" width="0.1524" layer="91"/>
+<pinref part="L6" gate="G$1" pin="9"/>
+<junction x="38.1" y="53.34"/>
+<wire x1="38.1" y1="53.34" x2="38.1" y2="50.8" width="0.1524" layer="91"/>
+<junction x="38.1" y="50.8"/>
+<junction x="38.1" y="45.72"/>
+<junction x="38.1" y="55.88"/>
 </segment>
 </net>
@@
 </segment>
 <segment>
-<pinref part="U$1" gate="G$1" pin="PE2"/>
-<wire x1="-175.26" y1="-83.82" x2="-170.18" y2="-83.82" width="0.1524" layer="91"/>
-<label x="-170.18" y="-83.82" size="1.27" layer="95" xref="yes"/>
+<label x="-162.56" y="-68.58" size="1.27" layer="95" xref="yes"/>
+<pinref part="U$1" gate="G$1" pin="D10~/A10"/>
+<wire x1="-162.56" y1="-68.58" x2="-175.26" y2="-68.58" width="0.1524" layer="91"/>
 </segment>
 </net>
@@
 </segment>
 <segment>
-<pinref part="U$1" gate="G$1" pin="D13~"/>
-<wire x1="-175.26" y1="-78.74" x2="-170.18" y2="-78.74" width="0.1524" layer="91"/>
-<label x="-170.18" y="-78.74" size="1.27" layer="95" xref="yes"/>
+<label x="-162.56" y="-63.5" size="1.27" layer="95" xref="yes"/>
+<pinref part="U$1" gate="G$1" pin="D9~/A9"/>
+<wire x1="-162.56" y1="-63.5" x2="-175.26" y2="-63.5" width="0.1524" layer="91"/>
 </segment>
 </net>
@@
 </segment>
 <segment>
-<pinref part="U$1" gate="G$1" pin="D5~"/>
-<wire x1="-175.26" y1="-73.66" x2="-170.18" y2="-73.66" width="0.1524" layer="91"/>
-<label x="-170.18" y="-73.66" size="1.27" layer="95" xref="yes"/>
+<label x="-162.56" y="-58.42" size="1.27" layer="95" xref="yes"/>
+<pinref part="U$1" gate="G$1" pin="D8/A8"/>
+<wire x1="-162.56" y1="-58.42" x2="-175.26" y2="-58.42" width="0.1524" layer="91"/>
 </segment>
 </net>
@@
 </segment>
 <segment>
-<pinref part="U$1" gate="G$1" pin="D10~/A10"/>
-<wire x1="-175.26" y1="-68.58" x2="-162.56" y2="-68.58" width="0.1524" layer="91"/>
-<label x="-162.56" y="-68.58" size="1.27" layer="95" xref="yes"/>
+<label x="-162.56" y="-83.82" size="1.27" layer="95" xref="yes"/>
+<pinref part="U$1" gate="G$1" pin="PE2"/>
+<wire x1="-162.56" y1="-83.82" x2="-175.26" y2="-83.82" width="0.1524" layer="91"/>
 </segment>
 </net>
@@
 </segment>
 <segment>
-<label x="-160.02" y="-63.5" size="1.27" layer="95" xref="yes"/>
-<pinref part="U$1" gate="G$1" pin="D9~/A9"/>
-<wire x1="-175.26" y1="-63.5" x2="-160.02" y2="-63.5" width="0.1524" layer="91"/>
+<label x="-162.56" y="-78.74" size="1.27" layer="95" xref="yes"/>
+<pinref part="U$1" gate="G$1" pin="D13~"/>
+<wire x1="-162.56" y1="-78.74" x2="-175.26" y2="-78.74" width="0.1524" layer="91"/>
 </segment>
 </net>
@@
 </segment>
 <segment>
-<label x="-160.02" y="-58.42" size="1.27" layer="95" xref="yes"/>
-<pinref part="U$1" gate="G$1" pin="D8/A8"/>
-<wire x1="-175.26" y1="-58.42" x2="-160.02" y2="-58.42" width="0.1524" layer="91"/>
+<label x="-162.56" y="-73.66" size="1.27" layer="95" xref="yes"/>
+<pinref part="U$1" gate="G$1" pin="D5~"/>
+<wire x1="-162.56" y1="-73.66" x2="-175.26" y2="-73.66" width="0.1524" layer="91"/>
 </segment>
 </net>
@@
 </segment>
 <segment>
-<pinref part="U$1" gate="G$1" pin="D11~"/>
-<wire x1="-215.9" y1="-83.82" x2="-220.98" y2="-83.82" width="0.1524" layer="91"/>
-<label x="-220.98" y="-83.82" size="1.27" layer="95" rot="R180" xref="yes"/>
+<wire x1="-215.9" y1="-99.06" x2="-220.98" y2="-99.06" width="0.1524" layer="91"/>
+<label x="-220.98" y="-99.06" size="1.27" layer="95" rot="R180" xref="yes"/>
+<pinref part="U$1" gate="G$1" pin="SCK"/>
 </segment>
 </net>
@@
 </segment>
 </net>
+<net name="N$11" class="0">
+<segment>
+<pinref part="R1" gate="G$1" pin="2"/>
+<pinref part="LED13" gate="G$1" pin="A"/>
+<wire x1="-276.86" y1="-162.56" x2="-276.86" y2="-165.1" width="0.1524" layer="91"/>
+</segment>
+</net>
+<net name="N$32" class="0">
+<segment>
+<pinref part="R2" gate="G$1" pin="2"/>
+<pinref part="LED14" gate="G$1" pin="A"/>
+<wire x1="-264.16" y1="-165.1" x2="-264.16" y2="-162.56" width="0.1524" layer="91"/>
+</segment>
+</net>
+<net name="BUZZ_BUZZ_MOTHERFUCKER" class="0">
+<segment>
+<wire x1="-215.9" y1="-83.82" x2="-220.98" y2="-83.82" width="0.1524" layer="91"/>
+<label x="-220.98" y="-83.82" size="1.27" layer="95" rot="R180" xref="yes"/>
+<pinref part="U$1" gate="G$1" pin="D11~"/>
+</segment>
+<segment>
+<wire x1="-294.64" y1="-170.18" x2="-289.56" y2="-170.18" width="0.1524" layer="91"/>
+<wire x1="-289.56" y1="-170.18" x2="-289.56" y2="-147.32" width="0.1524" layer="91"/>
+<label x="-289.56" y="-147.32" size="1.27" layer="95" rot="R180" xref="yes"/>
+<pinref part="SG1" gate="G$1" pin="2"/>
+<wire x1="-294.64" y1="-170.18" x2="-294.64" y2="-167.64" width="0.1524" layer="91"/>
+</segment>
+</net>
+<net name="INFO_LED_1" class="0">
+<segment>
+<wire x1="-215.9" y1="-88.9" x2="-220.98" y2="-88.9" width="0.1524" layer="91"/>
+<label x="-220.98" y="-88.9" size="1.27" layer="95" rot="R180" xref="yes"/>
+<pinref part="U$1" gate="G$1" pin="MISO"/>
+</segment>
+<segment>
+<pinref part="R1" gate="G$1" pin="1"/>
+<wire x1="-276.86" y1="-152.4" x2="-276.86" y2="-147.32" width="0.1524" layer="91"/>
+<label x="-276.86" y="-147.32" size="1.27" layer="95" rot="R180" xref="yes"/>
+<label x="-276.86" y="-147.32" size="1.27" layer="95" rot="R180" xref="yes"/>
+</segment>
+</net>
+<net name="INFO_LED_2" class="0">
+<segment>
+<pinref part="U$1" gate="G$1" pin="MOSI"/>
+<wire x1="-215.9" y1="-93.98" x2="-220.98" y2="-93.98" width="0.1524" layer="91"/>
+<label x="-220.98" y="-93.98" size="1.27" layer="95" rot="R180" xref="yes"/>
+</segment>
+<segment>
+<pinref part="R2" gate="G$1" pin="1"/>
+<wire x1="-264.16" y1="-152.4" x2="-264.16" y2="-147.32" width="0.1524" layer="91"/>
+<label x="-264.16" y="-147.32" size="1.27" layer="95" rot="R180" xref="yes"/>
+</segment>
+</net>

Commit message: Fixed some values
Parts:
- C10, C15: value (none) -> 2.2µF
- C8: value 47µf -> 10µf
- R3: value 70kΩ -> 60kΩ
Changed lines of the file:
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@@
 <?xml version="1.0" encoding="utf-8"?>
 <!DOCTYPE eagle SYSTEM "eagle.dtd">
-<eagle version="6.5.0">
+<eagle version="7.0.0">
 <drawing>
 <settings>
@@
 <part name="SUPPLY7" library="SparkFun-Aesthetics" deviceset="V_BATT" device=""/>
 <part name="GND18" library="SparkFun-Aesthetics" deviceset="GND" device=""/>
-<part name="R3" library="resistor" deviceset="R-US_" device="R1206" value="70kΩ"/>
+<part name="R3" library="resistor" deviceset="R-US_" device="R1206" value="60kΩ"/>
 <part name="R4" library="resistor" deviceset="R-US_" device="R1206" value="10kΩ"/>
 <part name="C11" library="resistor" deviceset="C-US" device="C1206"/>
 <part name="C12" library="resistor" deviceset="C-US" device="C1206" value="47µf"/>
 <part name="C13" library="resistor" deviceset="C-US" device="C1206" value="2.2µF"/>
-<part name="C15" library="resistor" deviceset="C-US" device="C1206"/>
+<part name="C15" library="resistor" deviceset="C-US" device="C1206" value="2.2µF"/>
 <part name="R8" library="resistor" deviceset="R-US_" device="R1206" value="21kΩ"/>
 <part name="GND19" library="SparkFun-Aesthetics" deviceset="GND" device=""/>
@@
 <part name="GND22" library="SparkFun-Aesthetics" deviceset="GND" device=""/>
 <part name="C7" library="resistor" deviceset="C-US" device="C1206" value="1uF"/>
-<part name="C8" library="resistor" deviceset="C-US" device="C1206" value="47µf"/>
+<part name="C8" library="resistor" deviceset="C-US" device="C1206" value="10µf"/>
 <part name="GND23" library="SparkFun-Aesthetics" deviceset="GND" device=""/>
 <part name="GND24" library="SparkFun-Aesthetics" deviceset="GND" device=""/>
@@
 <part name="C9" library="resistor" deviceset="C-US" device="C1206"/>
 <part name="GND25" library="SparkFun-Aesthetics" deviceset="GND" device=""/>
-<part name="C10" library="resistor" deviceset="C-US" device="C1206"/>
+<part name="C10" library="resistor" deviceset="C-US" device="C1206" value="2.2µF"/>
 <part name="C14" library="resistor" deviceset="C-US" device="C1206" value="2.2µF"/>
 <part name="GND9" library="SparkFun-Aesthetics" deviceset="GND" device=""/>

Commit message: Added new Inductor for Pi Filter ***NEEDS FINISH
Pi Filter now uses Fair-Rite 2773019447 Inductor.
THE FOOTPRINT HAS CHANGED! I ONLY HAVE THE LITE VERSION OF EAGLE, SO IT
IS NOT LAYED OUT PROPERLY YET!!
Parts:
- L3: device resistor:L-USL3216C -> rcl:L-USL4532C
Changed lines of the file:
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@@
 <part name="GND30" library="SparkFun-Aesthetics" deviceset="GND" device=""/>
 <part name="C17" library="resistor" deviceset="C-US" device="C1206" value="47µF"/>
-<part name="L3" library="resistor" deviceset="L-US" device="L3216C"/>
+<part name="L3" library="rcl" deviceset="L-US" device="L4532C"/>
 <part name="C18" library="resistor" deviceset="C-US" device="C1206" value="47µF"/>
 <part name="GND31" library="SparkFun-Aesthetics" deviceset="GND" device=""/>

Commit message: DFM revisions
Working on preparing the board for a new print.
Parts:
- removed L1, L4, L5, L8: L_29F0429, MRDT-2014-All:L_29F0429
- removed L2, L6: L_29F0429, MRDT-2015-PowerBoard:L_29F0429
- added C46: 330µF, resistor:CPOL-USE5-8.5
- 12V-AUX, AUX_P, MOTOR_1, MOTOR_2, MOTOR_3, MOTOR_4, MOTOR_5, MOTOR_6: value H_20020618-M02 -> H_20020618-M02HORIZ; device MRDT-2015-PowerBoard:H_20020618-M02 -> MRDT-2015-PowerBoard:H_20020618-M02HORIZ
- C10, C15: value 2.2µF -> 10µF
- C11, C9: value (none) -> 10uF
- C13, C14: value 2.2µF -> 1µF
- C19, C20: value (none) -> 47uF
- C27, C31, C35, C37, C38, C40, C42: device resistor:C-USC0805 -> resistor:C-USC1206
- L3: device rcl:L-USL4532C -> resistor:L-USL8530M
- R12, R13: value 1kΩ -> 330
- R15: value (none) -> 1k
- R16, R18, R20, R22, R24, R26, R28, R9: value 1kΩ -> 5kΩ
Connections:
- removed net N$10: C9.1, L1.5, L1.6, L1.7, L1.8, Q5.IP-, U$5.C
- removed net N$15: C22.+, L4.1, L4.2, L4.3, L4.4, VADER-5V-EXT.SENSE, VADER-5V-EXT.VOUT
- removed net N$48: LED3.A, R11.2
- removed net N$50: LED4.A, R12.2
- removed net N$52: LED5.A, R13.2
- removed net N$8: C14.2, DOOKU-12V-CRIT.VIN, L5.5, L5.6, L5.7, L5.8
- net +5V: now also LED5.A; no longer R13.1
- net 12V-CRIT: now also LED3.A; no longer R11.1
- net 5V-EXT: now also LED4.A; no longer R12.1
- net GND: now also C46.-, R11.2, R12.2, R13.2; no longer LED3.C, LED4.C, LED5.C
- net N$16: now also C22.+, VADER-5V-EXT.SENSE, VADER-5V-EXT.VOUT; no longer L4.5, L4.6, L4.7, L4.8
- net N$3: now also LED3.C, R11.1; no longer C13.2, L8.5, L8.6, L8.7, L8.8, VADER-5V-EXT.VIN
- net N$36: now also C9.1, Q5.IP-, U$5.C; no longer L1.1, L1.2, L1.3, L1.4
- net N$5: now also LED4.C, R12.1; no longer L6.10, L6.6, L6.7, L6.8, L6.9, PALPATINE-12V.+VIN
- net N$6: now also LED5.C, R13.1; no longer L2.10, L2.6, L2.7, L2.8, L2.9, SIDEOUS-12V.+VIN
- net N$7: now also C46.+
- net V_BATT: now also C13.2, C14.2, DOOKU-12V-CRIT.VIN, PALPATINE-12V.+VIN, SIDEOUS-12V.+VIN, VADER-5V-EXT.VIN; no longer L2.1, L2.2, L2.3, L2.4, L2.5, L5.1, L5.2, L5.3, L5.4, L6.1, L6.2, L6.3, L6.4, L6.5, L8.1, L8.2, L8.3, L8.4
Other:
- note removed: "I don't know what values to use for this Pi-Filter yet!!!"
- moved on the sheet: C45, LED3, LED4, LED5, R11, R12, R13
