File: 2015/Hardware/DumbBoard/PT_2015_DB_MAIN_Rev1.sch (EAGLE design)
At the start: 69 parts, among them Q12 2N7002

Commit message: Dumb Board - Attempt 2
Fixed schematic and rerouted
Parts:
- removed Q12: 2N7002, SparkFun-DiscreteSemi:MOSFET-NCHANNEL2N7002PW
- removed R15: (no value), resistor:R-US_R1206
- added C17, C18: 47µF, resistor:C-USC1206
- added L3: (no value), resistor:L-USL3216C
- added OKI-78SR-5/1.5-W36H: Q_OKI-78SR, MRDT-2015-PowerBoard:Q_OKI-78SR
Connections:
- removed net 12V-SIG: R15.2
- removed net N$114: Q12.G, R15.1
- removed net N$4: PALPATINE-12V.REMOTE, Q12.D, SIDEOUS-12V.REMOTE
- new net N$100: C17.1, L3.1, OKI-78SR-5/1.5-W36H.VO
- net +5V: now also C18.1, L3.2; no longer C11.1, C20.1, C9.1, L1.5, L1.6, L1.7, L1.8, L2.5, L2.6, L2.7, L2.8, L4.5, L4.6, L4.7, L4.8, U$2.C, U$5.C
- net 12V-AUX: now also C20.1, L2.5, L2.6, L2.7, L2.8
- net 12V-CRIT: now also C9.1, L1.5, L1.6, L1.7, L1.8, OKI-78SR-5/1.5-W36H.VI, U$5.C
- net 5V-EXT: now also C11.1, L4.5, L4.6, L4.7, L4.8, U$2.C
- net GND: now also C17.2, C18.2, OKI-78SR-5/1.5-W36H.GND; no longer Q12.S

Commit message: More Changes
Removed LED’s and increased V_BATT polygon pour
Parts:
- removed LED1, LED10, LED11, LED12, LED6, LED7, LED8, LED9: (no value), SparkFun-LED:LED1206
- removed R16, R18, R20, R22, R24, R26, R28, R9: 1kΩ, SparkFun-Passives:RESISTOR1206
Connections:
- removed net N$31: LED6.A, R16.2
- removed net N$39: LED1.A, R9.2
- removed net N$49: LED7.A, R18.2
- removed net N$57: LED8.A, R20.2
- removed net N$63: LED9.A, R22.2
- removed net N$69: LED10.A, R24.2
- removed net N$75: LED11.A, R26.2
- removed net N$81: LED12.A, R28.2
- net GND: no longer LED1.C, LED10.C, LED11.C, LED12.C, LED6.C, LED7.C, LED8.C, LED9.C
- net V_BATT: no longer R16.1, R18.1, R20.1, R22.1, R24.1, R26.1, R28.1, R9.1
