File: 2015/ATmega32u4 Breakout/32u4 board.sch (EAGLE design)
At the start: 19 parts, among them X1 MINI-USB-UX60A-MB-5ST

Commit message: I fix'd the part values
This only took one bottle of wine. Can I graduate now?
Parts:
- C18, C19: value 0.1uF -> 18pF
- C6: value 0.1uF -> 1uF
- R1: value (none) -> 1k
Changed lines of the file:
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@@
 <?xml version="1.0" encoding="utf-8"?>
 <!DOCTYPE eagle SYSTEM "eagle.dtd">
-<eagle version="7.0.0">
+<eagle version="6.5.0">
 <drawing>
 <settings>
@@
 <part name="R19" library="SparkFun-Passives" deviceset="RESISTOR" device="0603-RES" value="22"/>
 <part name="R23" library="SparkFun-Passives" deviceset="RESISTOR" device="0603-RES" value="22"/>
-<part name="C6" library="SparkFun-Capacitors" deviceset="0.1UF-25V(+80/-20%)(0603)" device="" value="0.1uF"/>
+<part name="C6" library="SparkFun-Capacitors" deviceset="0.1UF-25V(+80/-20%)(0603)" device="" value="1uF"/>
 <part name="MH2029" library="resistor" deviceset="L-US" device="L2012C" value="MH2029-300Y"/>
 <part name="C20" library="SparkFun-Capacitors" deviceset="0.1UF-25V(+80/-20%)(0603)" device="" value="0.1uF"/>
@@
 <part name="S1" library="SparkFun-Electromechanical" deviceset="SWITCH-MOMENTARY-2" device="SMD"/>
 <part name="GND3" library="supply1" deviceset="GND" device=""/>
-<part name="C18" library="SparkFun-Capacitors" deviceset="0.1UF-25V(+80/-20%)(0603)" device="" value="0.1uF"/>
-<part name="C19" library="SparkFun-Capacitors" deviceset="0.1UF-25V(+80/-20%)(0603)" device="" value="0.1uF"/>
+<part name="C18" library="SparkFun-Capacitors" deviceset="0.1UF-25V(+80/-20%)(0603)" device="" value="18pF"/>
+<part name="C19" library="SparkFun-Capacitors" deviceset="0.1UF-25V(+80/-20%)(0603)" device="" value="18pF"/>
 <part name="GND30" library="supply1" deviceset="GND" device=""/>
 <part name="GND31" library="supply1" deviceset="GND" device=""/>
@@
 <part name="GND26" library="supply1" deviceset="GND" device=""/>
 <part name="LED1" library="adafruit" deviceset="LED" device="CHIPLED_0603"/>
-<part name="R1" library="SparkFun-Resistors" deviceset="RESISTOR" device="0603"/>
+<part name="R1" library="SparkFun-Resistors" deviceset="RESISTOR" device="0603" value="1k"/>
 <part name="GND4" library="supply1" deviceset="GND" device=""/>
 </parts>
@@
 <pinref part="C21" gate="G$1" pin="1"/>
 <wire x1="195.58" y1="195.58" x2="193.04" y2="195.58" width="0.1524" layer="91"/>
-<wire x1="195.58" y1="195.58" x2="195.58" y2="187.96" width="0.1524" layer="91"/>
-<wire x1="195.58" y1="187.96" x2="193.04" y2="187.96" width="0.1524" layer="91"/>
-<label x="193.04" y="187.96" size="1.27" layer="95" rot="R180" xref="yes"/>
+<wire x1="195.58" y1="195.58" x2="195.58" y2="185.42" width="0.1524" layer="91"/>
+<label x="195.58" y="185.42" size="1.27" layer="95" rot="R180" xref="yes"/>
 <junction x="195.58" y="195.58"/>
 </segment>

Commit message: Added a solder jumper between VCC and VBUS
Parts:
- added SJ1: SOLDERJUMPERNO, SparkFun-Retired:SOLDERJUMPERNO
Connections:
- net VBUS: now also SJ1.1
- net VCC: now also SJ1.2
Changed lines of the file:
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@@
 <?xml version="1.0" encoding="utf-8"?>
 <!DOCTYPE eagle SYSTEM "eagle.dtd">
-<eagle version="6.5.0">
+<eagle version="7.2.0">
 <drawing>
 <settings>
@@
 <part name="R1" library="SparkFun-Resistors" deviceset="RESISTOR" device="0603" value="1k"/>
 <part name="GND4" library="supply1" deviceset="GND" device=""/>
+<part name="SJ1" library="SparkFun-Retired" deviceset="SOLDERJUMPER" device="NO" value="SOLDERJUMPERNO"/>
 </parts>
 <sheets>
@@
 <instance part="R1" gate="G$1" x="182.88" y="236.22"/>
 <instance part="GND4" gate="1" x="172.72" y="236.22" rot="R270"/>
+<instance part="SJ1" gate="1" x="238.76" y="238.76"/>
 </instances>
 <busses>
@@
 <label x="279.4" y="251.46" size="1.27" layer="95" rot="R180" xref="yes"/>
 </segment>
+<segment>
+<pinref part="SJ1" gate="1" pin="1"/>
+<wire x1="233.68" y1="238.76" x2="231.14" y2="238.76" width="0.1524" layer="91"/>
+<wire x1="231.14" y1="238.76" x2="231.14" y2="241.3" width="0.1524" layer="91"/>
+<label x="231.14" y="241.3" size="1.778" layer="95" rot="R90" xref="yes"/>
+</segment>
 </net>
 <net name="VCC" class="0">
@@
 <label x="279.4" y="246.38" size="1.27" layer="95" rot="R180" xref="yes"/>
 </segment>
-</net>
+<segment>
+<pinref part="SJ1" gate="1" pin="2"/>
+<wire x1="243.84" y1="238.76" x2="246.38" y2="238.76" width="0.1524" layer="91"/>
+<wire x1="246.38" y1="238.76" x2="246.38" y2="241.3" width="0.1524" layer="91"/>
+<label x="246.38" y="241.3" size="1.778" layer="95" rot="R90" xref="yes"/>
+</segment>
+</net>

Commit message: Added poly fuse
Parts:
- added F1: PTCSMD, SparkFun-PowerIC:PTCSMD
Connections:
- new net N$2: F1.2, X1.1
- net VBUS: now also F1.1; no longer X1.1
Changed lines of the file:
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@@
 <part name="GND4" library="supply1" deviceset="GND" device=""/>
 <part name="SJ1" library="SparkFun-Retired" deviceset="SOLDERJUMPER" device="NO" value="SOLDERJUMPERNO"/>
+<part name="F1" library="SparkFun-PowerIC" deviceset="PTC" device="SMD"/>
 </parts>
 <sheets>
@@
 <instance part="GND4" gate="1" x="172.72" y="236.22" rot="R270"/>
 <instance part="SJ1" gate="1" x="238.76" y="238.76"/>
+<instance part="F1" gate="G$1" x="266.7" y="20.32"/>
 </instances>
 <busses>
@@
 <label x="248.92" y="20.32" size="1.27" layer="95" rot="R180" xref="yes"/>
 <wire x1="248.92" y1="20.32" x2="261.62" y2="20.32" width="0.1524" layer="91"/>
-<wire x1="261.62" y1="20.32" x2="276.86" y2="20.32" width="0.1524" layer="91"/>
-<pinref part="X1" gate="G$1" pin="1"/>
+<pinref part="F1" gate="G$1" pin="1"/>
 <junction x="261.62" y="20.32"/>
 </segment>
@@
 </segment>
 </net>
+<net name="N$2" class="0">
+<segment>
+<pinref part="X1" gate="G$1" pin="1"/>
+<pinref part="F1" gate="G$1" pin="2"/>
+<wire x1="274.32" y1="20.32" x2="276.86" y2="20.32" width="0.1524" layer="91"/>
+</segment>
+</net>
