File: 2017/PT_2017_PB_4lyr_Rev1.sch (EAGLE design)
At the start: 150 parts, among them Q12 2N7002

Commit message: Added fuse blocks and bus bar mounting holes
Fuse blocks for the 12V buses. Swapped temporary anderson connectors
with holes to mount bus bars to connect PB to patch panel.
Parts:
- added U$14, U$30, U$31, U$32: ATC_FUSE_BLOCK, MRDT-Hardware:ATC_FUSE_BLOCK
- added U$33: BUS_BAR_MOUNTING_HOLE, MRDT-Connectors:BUS_BAR_MOUNTING_HOLE
- added U$34, U$35: MOUNTING_HOLE#8, MRDT-Hardware:MOUNTING_HOLE#8
- U$16, U$17, U$18, U$25: value APP_2POS_CONFIG12V_VERT -> BUS_BAR_MOUNTING_HOLE; device MRDT-Connectors:APP_2POS_CONFIG12V_VERT -> MRDT-Connectors:BUS_BAR_MOUNTING_HOLE
Connections:
- new net N$18: RICK-12V.+VOUT, U$31.IN, U$32.IN
- new net N$21: DARYL-12V.+VOUT, U$30.IN
- new net N$23: MICHONNE-12V.+VOUT, U$14.IN
- new net N$9: C23.1, FET-R1.S, U$32.OUT, U$4.IN
- net 12V-AUX-ACT: now also U$17.12V; no longer U$17VCC.P$1
- net 12V-AUX-ARM: now also U$18.12V; no longer U$16VCC.P$1
- net 12V-AUX-COM: now also U$33.12V; no longer U$25VCC.P$1
- net 12V-AUX-LOGIC: now also U$16.12V; no longer U$18VCC.P$1
- net GND: now also U$25.12V; no longer U$16GND.P$1, U$17GND.P$1, U$18GND.P$1, U$25GND.P$1
- net N$1: now also U$30.OUT; no longer DARYL-12V.+VOUT
- net N$13: now also U$31.OUT; no longer C23.1, FET-R1.S, RICK-12V.+VOUT, U$4.IN
- net N$2: now also U$14.OUT; no longer MICHONNE-12V.+VOUT
Other:
- moved on the sheet: C19, C20

Commit message: Rearranged 5V & 3.3V Regulators
Also changed the horizontal RJ45 jack to a vertical jack.
Parts:
- removed U$5: RJ45FCI-54602-908LF, MRDT-2015-General:RJ45FCI-54602-908LF
- added U$41: MRDT_LOGO, MRDT-2015-General:MRDT_LOGO
- added U$42: RJ45KEYSTONE-949, MRDT-2015-General:RJ45KEYSTONE-949
Connections:
- net GND: now also U$42.7, U$42.8; no longer U$5.7, U$5.8
- net REC+1: now also U$42.1; no longer U$5.1
- net REC-1: now also U$42.2; no longer U$5.2
- net TRANS+1: now also U$42.3; no longer U$5.3
- net TRANS-1: now also U$42.6; no longer U$5.6
Changed lines of the file:
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@@
 <part name="GND79" library="SparkFun-Aesthetics" deviceset="GND" device=""/>
 <part name="U$1" library="MRDT-2015-General" deviceset="TIVA-C-CONNECTED" device=""/>
-<part name="U$5" library="MRDT-2015-General" deviceset="RJ45" device="FCI-54602-908LF"/>
 <part name="U$8" library="MRDT-Hardware" deviceset="MOUNTING_HOLE" device="#8"/>
 <part name="U$10" library="MRDT-Hardware" deviceset="MOUNTING_HOLE" device="#8"/>
@@
 <part name="U$34" library="MRDT-Hardware" deviceset="MOUNTING_HOLE" device="#8"/>
 <part name="U$35" library="MRDT-Hardware" deviceset="MOUNTING_HOLE" device="#8"/>
+<part name="U$41" library="MRDT-2015-General" deviceset="MRDT_LOGO" device=""/>
+<part name="U$42" library="MRDT-2015-General" deviceset="RJ45" device="KEYSTONE-949"/>
 </parts>
 <sheets>
@@
 <instance part="GND79" gate="1" x="612.14" y="139.7"/>
 <instance part="U$1" gate="G$1" x="-63.5" y="-210.82"/>
-<instance part="U$5" gate="G$1" x="152.4" y="-185.42"/>
 <instance part="U$8" gate="G$1" x="0" y="27.94"/>
 <instance part="U$10" gate="G$1" x="0" y="20.32"/>
@@
 <instance part="U$34" gate="G$1" x="12.7" y="35.56"/>
 <instance part="U$35" gate="G$1" x="0" y="35.56"/>
+<instance part="U$41" gate="G$1" x="0" y="43.18"/>
+<instance part="U$42" gate="G$1" x="152.4" y="-185.42"/>
 </instances>
 <busses>
@@
 <pinref part="GND15" gate="1" pin="GND"/>
 <wire x1="160.02" y1="-177.8" x2="160.02" y2="-175.26" width="0.1524" layer="91"/>
-<pinref part="U$5" gate="G$1" pin="8"/>
+<pinref part="U$42" gate="G$1" pin="8"/>
 <wire x1="160.02" y1="-175.26" x2="160.02" y2="-165.1" width="0.1524" layer="91"/>
 <junction x="160.02" y="-175.26"/>
-<pinref part="U$5" gate="G$1" pin="7"/>
+<pinref part="U$42" gate="G$1" pin="7"/>
 </segment>
 <segment>
@@
 <pinref part="U$24" gate="G$1" pin="A"/>
 <wire x1="177.8" y1="-193.04" x2="160.02" y2="-193.04" width="0.1524" layer="91"/>
-<pinref part="U$5" gate="G$1" pin="1"/>
+<pinref part="U$42" gate="G$1" pin="1"/>
 </segment>
 </net>
@@
 <wire x1="187.96" y1="-185.42" x2="190.5" y2="-185.42" width="0.1524" layer="91"/>
 <wire x1="175.26" y1="-190.5" x2="160.02" y2="-190.5" width="0.1524" layer="91"/>
-<pinref part="U$5" gate="G$1" pin="2"/>
+<pinref part="U$42" gate="G$1" pin="2"/>
 </segment>
 </net>
@@
 <wire x1="187.96" y1="-175.26" x2="190.5" y2="-175.26" width="0.1524" layer="91"/>
 <wire x1="170.18" y1="-187.96" x2="160.02" y2="-187.96" width="0.1524" layer="91"/>
-<pinref part="U$5" gate="G$1" pin="3"/>
+<pinref part="U$42" gate="G$1" pin="3"/>
 </segment>
 </net>
@@
 <wire x1="160.02" y1="-180.34" x2="177.8" y2="-180.34" width="0.1524" layer="91"/>
 <junction x="177.8" y="-180.34"/>
-<pinref part="U$5" gate="G$1" pin="6"/>
-</segment>
-</net>
+<pinref part="U$42" gate="G$1" pin="6"/>
+</segment>
+</net>

Commit message: Spaced Out 12V Busses
Components easier to solder and fuses are easier to reach.
Parts:
- removed U$17, U$18, U$25, U$33: BUS_BAR_MOUNTING_HOLE, MRDT-Connectors:BUS_BAR_MOUNTING_HOLE
- added J1, J2, J3, J4: APP_2POS_CONFIG12V_VERT, MRDT-Connectors:APP_2POS_CONFIG12V_VERT
- added U$5: MOUNTING_HOLE#8, MRDT-Hardware:MOUNTING_HOLE#8
- U$16: value BUS_BAR_MOUNTING_HOLE -> MOUNTING_HOLE#8; device MRDT-Connectors:BUS_BAR_MOUNTING_HOLE -> MRDT-Hardware:MOUNTING_HOLE#8
Connections:
- net ARM-12V-SIG renamed EXTRA-12V-SIG
- removed net 12V-AUX-ARM: R10.1, U$11.IP-, U$18.12V
- new net 12V-AUX-EXTRA: J4VCC.P$1, R10.1, U$11.IP-
- net 12V-AUX-ACT: now also J3VCC.P$1; no longer U$17.12V
- net 12V-AUX-COM: now also J1VCC.P$1; no longer U$33.12V
- net 12V-AUX-LOGIC: now also J2VCC.P$1; no longer U$16.12V
- net GND: now also J1GND.P$1, J2GND.P$1, J3GND.P$1, J4GND.P$1; no longer U$25.12V

Commit message: Added Fan Power/Control
Parts:
- added Q1: 2N7002PW, SparkFun-DiscreteSemi:MOSFET-NCHANNEL2N7002PW
- added X1: 22-23-2021, con-molex:22-23-2021
Connections:
- new net FAN_CTL_1: Q1.G, U$1.PE4
- new net N$66: Q1.D, X1-1.S
- net 5V: now also X1-2.S
- net GND: now also Q1.S
Other:
- note added: "Fan Power/Control"
- moved on the sheet: C18, C21, C22, C47, C48, C49, C5, C7, C8

Commit message: Fixed All Vias
Moved vias away from pads to prevent solder bridging and unrouted
dead-end traces resulting from pulling traces to other layers.
Parts:
- removed FET-M1: Q_IRFS7437PbF, MRDT-2015-PowerBoard:Q_IRF7437SMD
- added Q13: 2N7002PW, SparkFun-DiscreteSemi:MOSFET-NCHANNEL2N7002PW
- Q1: value 2N7002PW -> Q_IRFS7437PbF; device SparkFun-DiscreteSemi:MOSFET-NCHANNEL2N7002PW -> MRDT-2015-PowerBoard:Q_IRF7437SMD
- renumbered ACS714-M1 to U8, ACS714-M2 to U9, ACS714-M3 to U10, ACS714-M4 to U11, ACS714-M5 to U13, ACS714-M6 to U14, ACS714-M7 to U15, ACS714CAP-M1 to C.8, ACS714CAP-M2 to C.9, ACS714CAP-M3 to C.10, ACS714CAP-M4 to C.11, ACS714CAP-M5 to C.12, ACS714CAP-M6 to C.13, ACS714CAP-M7 to C.14, BB-8-5V to 3.3V-OKI, BB-8-5V1 to 5V-OKI, C1 to C.51, C10 to C.38, C11 to C.33, C12 to C.32, C13 to C.36, C14 to C.24, C15 to C.40, C16 to C.29, C17 to C.28, C18 to C.44, C19 to C.34, C2 to C.52, C20 to C.35, C21 to C.47, C22 to C.50, C23 to C.37, C24 to C.25, C25 to C.41, C26 to C.31, C27 to C.30, C3 to C.53, C4 to C.54, C43 to C.39, C45 to C.27, C46 to C.26, C47 to C.43, C48 to C.46, C49 to C.49, C5 to C.42, C6 to C.23, C7 to C.45, C8 to C.48, C9 to C.22, DARYL-12V to NEMO-12V, FET-D to Q9, FET-M to Q8, FET-M2 to Q2, FET-M3 to Q3, FET-M4 to Q4, FET-M5 to Q5, FET-M6 to Q6, FET-M7 to Q7, FET-R1 to Q11, FET-R2 to Q10, FILTERCAP-M1 to C.1, FILTERCAP-M2 to C.2, FILTERCAP-M3 to C.3, FILTERCAP-M4 to C.4, FILTERCAP-M5 to C.5, FILTERCAP-M6 to C.6, FILTERCAP-M7 to C.7, LED-M1 to LED-1, LED-M2 to LED-2, LED-M3 to LED-3, LED-M4 to LED-4, LED-M5 to LED-5, LED-M6 to LED-6, LED-M7 to LED-7, LED1 to LED-9, LED2 to LED-8, LED3 to LED-10, LEDRES-M1 to R.1, LEDRES-M2 to R.2, LEDRES-M3 to R.3, LEDRES-M4 to R.4, LEDRES-M5 to R.5, LEDRES-M6 to R.6, LEDRES-M7 to R.7, LT1910-M1 to U1, LT1910-M2 to U2, LT1910-M3 to U3, LT1910-M4 to U4, LT1910-M5 to U5, LT1910-M6 to U6, LT1910-M7 to U7, LT1910CAP-M1 to C.15, LT1910CAP-M2 to C.16, LT1910CAP-M3 to C.17, LT1910CAP-M4 to C.18, LT1910CAP-M5 to C.19, LT1910CAP-M6 to C.20, LT1910CAP-M7 to C.21, MICHONNE-12V to DORY-12V, R1 to R.9, R10 to R.8, R15 to R.15, R2 to R.13, R3 to R.16, R4 to R.17, R5 to R.14, R6 to R.10, R7 to R.12, R8 to R.11, RICK-12V to MARLIN-12V, U$11 to U20, U$12 to U22, U$13 to U18, U$2 to U23, U$21 to U21, U$24 to U24, U$4 to U19, U$42 to RJ45, U$6 to U17, U$9 to U16
Connections:
- net DRAIN-M1: now also Q1.D; no longer FET-M1.D
- net FAN_CTL_1: now also Q13.G; no longer Q1.G
- net GATE-M1: now also Q1.G; no longer FET-M1.G
- net GND: now also Q13.S; no longer Q1.S
- net N$66: now also Q13.D; no longer Q1.D
- net SOURCE-M1: now also Q1.S; no longer FET-M1.S
Other:
- note added: "Extra 12V"
- note removed: "Arm 12V"
