File: BLDC_Motor_Controller_2016_Rev1.sch (EAGLE design)
At the start: 101 parts, among them J3 APP_2POS_CONFIG5V_HORIZ, Q1 MOSFET-NCHANNELFQP30N06L, Q2 MOSFET-NCHANNELFQP30N06L, Q3 MOSFET-NCHANNELFQP30N06L, Q4 MOSFET-NCHANNELFQP30N06L, Q5 MOSFET-NCHANNELFQP30N06L, Q6 MOSFET-NCHANNELFQP30N06L, Q7 MOSFET-PCHANNEL, Q8 MOSFET-PCHANNEL

Commit message: Routed separate sense resistor ground traces using short
Parts:
- added SH1, SH2: SHORT-HT5, shorts-old:SHORT-HT5
Connections:
- net GND: now also C21.2, C24.2, R13.1, R18.1, SH1.P$2, SH2.P$2
- net SP1: now also SH2.P$1; no longer C21.2, R13.1
- net SP2: now also SH1.P$1; no longer C24.2, R18.1
Changed lines of the file:
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@@
 <part name="GND37" library="SparkFun-Aesthetics" deviceset="GND" device=""/>
 <part name="C39" library="SparkFun-Passives" deviceset="CAP_POL" device="PTH4" value="220u"/>
+<part name="SH1" library="shorts-old" deviceset="SHORT-H" device="T5"/>
+<part name="SH2" library="shorts-old" deviceset="SHORT-H" device="T5"/>
 </parts>
 <sheets>
@@
 <instance part="GND37" gate="1" x="-147.32" y="-101.6"/>
 <instance part="C39" gate="G$1" x="-83.82" y="-121.92"/>
+<instance part="SH1" gate="G$1" x="93.98" y="-73.66"/>
+<instance part="SH2" gate="G$1" x="93.98" y="7.62"/>
 </instances>
 <busses>
@@
 <pinref part="GND36" gate="1" pin="GND"/>
 <wire x1="-88.9" y1="-88.9" x2="-91.44" y2="-88.9" width="0.1524" layer="91"/>
+</segment>
+<segment>
+<pinref part="GND17" gate="1" pin="GND"/>
+<wire x1="142.24" y1="-73.66" x2="142.24" y2="-78.74" width="0.1524" layer="91"/>
+<pinref part="R18" gate="G$1" pin="1"/>
+<junction x="142.24" y="-73.66"/>
+<wire x1="142.24" y1="-73.66" x2="129.54" y2="-73.66" width="0.1524" layer="91"/>
+<pinref part="C24" gate="G$1" pin="2"/>
+<wire x1="129.54" y1="-71.12" x2="129.54" y2="-73.66" width="0.1524" layer="91"/>
+<junction x="129.54" y="-73.66"/>
+<wire x1="129.54" y1="-73.66" x2="96.52" y2="-73.66" width="0.1524" layer="91"/>
+<pinref part="SH1" gate="G$1" pin="P$2"/>
+</segment>
+<segment>
+<pinref part="GND14" gate="1" pin="GND"/>
+<wire x1="142.24" y1="7.62" x2="142.24" y2="2.54" width="0.1524" layer="91"/>
+<pinref part="R13" gate="G$1" pin="1"/>
+<junction x="142.24" y="7.62"/>
+<wire x1="142.24" y1="7.62" x2="129.54" y2="7.62" width="0.1524" layer="91"/>
+<pinref part="C21" gate="G$1" pin="2"/>
+<wire x1="129.54" y1="10.16" x2="129.54" y2="7.62" width="0.1524" layer="91"/>
+<junction x="129.54" y="7.62"/>
+<wire x1="129.54" y1="7.62" x2="96.52" y2="7.62" width="0.1524" layer="91"/>
+<pinref part="SH2" gate="G$1" pin="P$2"/>
 </segment>
 </net>
@@
 <net name="SP1" class="0">
 <segment>
-<wire x1="142.24" y1="7.62" x2="142.24" y2="2.54" width="0.1524" layer="91"/>
-<wire x1="142.24" y1="7.62" x2="129.54" y2="7.62" width="0.1524" layer="91"/>
-<pinref part="GND14" gate="1" pin="GND"/>
-<pinref part="C21" gate="G$1" pin="2"/>
-<wire x1="129.54" y1="10.16" x2="129.54" y2="7.62" width="0.1524" layer="91"/>
-<wire x1="129.54" y1="7.62" x2="81.28" y2="7.62" width="0.1524" layer="91"/>
-<junction x="129.54" y="7.62"/>
+<wire x1="91.44" y1="7.62" x2="81.28" y2="7.62" width="0.1524" layer="91"/>
 <wire x1="81.28" y1="7.62" x2="81.28" y2="-45.72" width="0.1524" layer="91"/>
 <pinref part="U$1" gate="G$1" pin="SP1"/>
 <wire x1="81.28" y1="-45.72" x2="17.78" y2="-45.72" width="0.1524" layer="91"/>
-<pinref part="R13" gate="G$1" pin="1"/>
-<junction x="142.24" y="7.62"/>
+<pinref part="SH2" gate="G$1" pin="P$1"/>
 </segment>
 </net>
 <net name="SP2" class="0">
 <segment>
-<wire x1="142.24" y1="-73.66" x2="142.24" y2="-78.74" width="0.1524" layer="91"/>
-<wire x1="142.24" y1="-73.66" x2="129.54" y2="-73.66" width="0.1524" layer="91"/>
-<pinref part="GND17" gate="1" pin="GND"/>
-<pinref part="C24" gate="G$1" pin="2"/>
-<wire x1="129.54" y1="-71.12" x2="129.54" y2="-73.66" width="0.1524" layer="91"/>
-<wire x1="129.54" y1="-73.66" x2="63.5" y2="-73.66" width="0.1524" layer="91"/>
+<wire x1="91.44" y1="-73.66" x2="63.5" y2="-73.66" width="0.1524" layer="91"/>
 <wire x1="63.5" y1="-73.66" x2="63.5" y2="-55.88" width="0.1524" layer="91"/>
-<junction x="129.54" y="-73.66"/>
 <pinref part="U$1" gate="G$1" pin="SP2"/>
 <wire x1="63.5" y1="-55.88" x2="17.78" y2="-55.88" width="0.1524" layer="91"/>
-<pinref part="R18" gate="G$1" pin="1"/>
-<junction x="142.24" y="-73.66"/>
-</segment>
-</net>
+<pinref part="SH1" gate="G$1" pin="P$1"/>
+</segment>
+</net>

Commit message: Swapped MAX3077 for MAX3078
Parts:
- removed U$3: MAX3077, MRDT-2015-General:MAX3077
- added U$10: MAX3078E, MRDT-ICs:MAX3078E
Connections:
- new net DE: U$10.DE, U$2.PD6
- new net NRE: U$10.NRE, U$2.PC7
- net GND: no longer U$3.GND
- net N$34: now also U$10.A; no longer U$3.B, U$3.Z
- net N$36: now also U$10.B; no longer U$3.A, U$3.Y
- net RX: now also U$10.RO; no longer U$3.RO
- net TX: now also U$10.DI; no longer U$3.DI
- net VCC: now also U$10.VCC; no longer U$3.VCC
Changed lines of the file:
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@@
 <?xml version="1.0" encoding="utf-8"?>
 <!DOCTYPE eagle SYSTEM "eagle.dtd">
-<eagle version="7.3.0">
+<eagle version="7.4.0">
 <drawing>
 <settings>
@@
 <part name="J3" library="MRDT-Connectors" deviceset="APP_2POS_CONFIG" device="5V_HORIZ"/>
 <part name="C38" library="SparkFun-Passives" deviceset="CAP_POL" device="PTH4" value="220u"/>
-<part name="U$3" library="MRDT-2015-General" deviceset="MAX3077" device=""/>
 <part name="R30" library="SparkFun-Passives" deviceset="RESISTOR" device="0805-RES" value="120"/>
 <part name="U$4" library="Molex-SL" deviceset="5PIN" device=""/>
@@
 <part name="SH1" library="shorts-old" deviceset="SHORT-H" device="T5"/>
 <part name="SH2" library="shorts-old" deviceset="SHORT-H" device="T5"/>
+<part name="U$10" library="MRDT-ICs" deviceset="MAX3078E" device=""/>
 </parts>
 <sheets>
@@
 <instance part="J3" gate="VCC" x="256.54" y="-45.72"/>
 <instance part="C38" gate="G$1" x="-73.66" y="-121.92"/>
-<instance part="U$3" gate="G$1" x="-121.92" y="-96.52"/>
 <instance part="R30" gate="G$1" x="-101.6" y="-81.28"/>
 <instance part="U$4" gate="G$1" x="-81.28" y="-91.44"/>
 <instance part="GND36" gate="1" x="-93.98" y="-88.9" rot="R270"/>
-<instance part="GND37" gate="1" x="-147.32" y="-101.6"/>
+<instance part="GND37" gate="1" x="-111.76" y="-93.98"/>
 <instance part="C39" gate="G$1" x="-83.82" y="-121.92"/>
 <instance part="SH1" gate="G$1" x="93.98" y="-73.66"/>
 <instance part="SH2" gate="G$1" x="93.98" y="7.62"/>
+<instance part="U$10" gate="G$1" x="-124.46" y="-81.28"/>
 </instances>
 <busses>
@@
 </segment>
 <segment>
-<pinref part="U$3" gate="G$1" pin="GND"/>
 <pinref part="GND37" gate="1" pin="GND"/>
-<wire x1="-144.78" y1="-93.98" x2="-147.32" y2="-93.98" width="0.1524" layer="91"/>
-<wire x1="-147.32" y1="-93.98" x2="-147.32" y2="-99.06" width="0.1524" layer="91"/>
+<wire x1="-114.3" y1="-88.9" x2="-111.76" y2="-88.9" width="0.1524" layer="91"/>
+<wire x1="-111.76" y1="-88.9" x2="-111.76" y2="-91.44" width="0.1524" layer="91"/>
 </segment>
 <segment>
@@
 </segment>
 <segment>
-<pinref part="U$3" gate="G$1" pin="VCC"/>
-<wire x1="-144.78" y1="-78.74" x2="-147.32" y2="-78.74" width="0.1524" layer="91"/>
-<wire x1="-147.32" y1="-78.74" x2="-147.32" y2="-73.66" width="0.1524" layer="91"/>
-<label x="-147.32" y="-73.66" size="1.778" layer="95" rot="R90" xref="yes"/>
+<wire x1="-114.3" y1="-73.66" x2="-111.76" y2="-73.66" width="0.1524" layer="91"/>
+<wire x1="-111.76" y1="-73.66" x2="-111.76" y2="-68.58" width="0.1524" layer="91"/>
+<label x="-111.76" y="-68.58" size="1.778" layer="95" rot="R90" xref="yes"/>
+<pinref part="U$10" gate="G$1" pin="VCC"/>
 </segment>
 </net>
@@
 </segment>
 <segment>
-<pinref part="U$3" gate="G$1" pin="DI"/>
-<wire x1="-144.78" y1="-88.9" x2="-147.32" y2="-88.9" width="0.1524" layer="91"/>
-<label x="-147.32" y="-88.9" size="1.778" layer="95" rot="R180" xref="yes"/>
+<label x="-142.24" y="-88.9" size="1.778" layer="95" rot="R180" xref="yes"/>
+<pinref part="U$10" gate="G$1" pin="DI"/>
+<wire x1="-142.24" y1="-88.9" x2="-137.16" y2="-88.9" width="0.1524" layer="91"/>
 </segment>
 </net>
@@
 </segment>
 <segment>
-<pinref part="U$3" gate="G$1" pin="RO"/>
-<wire x1="-144.78" y1="-83.82" x2="-147.32" y2="-83.82" width="0.1524" layer="91"/>
-<label x="-147.32" y="-83.82" size="1.778" layer="95" rot="R180" xref="yes"/>
+<label x="-142.24" y="-73.66" size="1.778" layer="95" rot="R180" xref="yes"/>
+<pinref part="U$10" gate="G$1" pin="RO"/>
+<wire x1="-142.24" y1="-73.66" x2="-137.16" y2="-73.66" width="0.1524" layer="91"/>
 </segment>
 </net>
@@
 <net name="N$34" class="0">
 <segment>
-<pinref part="U$3" gate="G$1" pin="B"/>
-<pinref part="U$3" gate="G$1" pin="Z"/>
-<wire x1="-116.84" y1="-83.82" x2="-116.84" y2="-88.9" width="0.1524" layer="91"/>
+<pinref part="U$10" gate="G$1" pin="A"/>
 <pinref part="U$4" gate="G$1" pin="2"/>
-<wire x1="-116.84" y1="-83.82" x2="-96.52" y2="-83.82" width="0.1524" layer="91"/>
-<junction x="-116.84" y="-83.82"/>
+<wire x1="-114.3" y1="-83.82" x2="-96.52" y2="-83.82" width="0.1524" layer="91"/>
 <pinref part="R30" gate="G$1" pin="2"/>
 <wire x1="-96.52" y1="-83.82" x2="-88.9" y2="-83.82" width="0.1524" layer="91"/>
@@
 <net name="N$36" class="0">
 <segment>
-<pinref part="U$3" gate="G$1" pin="A"/>
-<wire x1="-116.84" y1="-78.74" x2="-114.3" y2="-78.74" width="0.1524" layer="91"/>
-<wire x1="-114.3" y1="-78.74" x2="-114.3" y2="-93.98" width="0.1524" layer="91"/>
-<pinref part="U$3" gate="G$1" pin="Y"/>
-<wire x1="-114.3" y1="-93.98" x2="-116.84" y2="-93.98" width="0.1524" layer="91"/>
+<pinref part="U$10" gate="G$1" pin="B"/>
 <pinref part="U$4" gate="G$1" pin="1"/>
 <wire x1="-114.3" y1="-78.74" x2="-106.68" y2="-78.74" width="0.1524" layer="91"/>
-<junction x="-114.3" y="-78.74"/>
 <pinref part="R30" gate="G$1" pin="1"/>
 <wire x1="-106.68" y1="-78.74" x2="-88.9" y2="-78.74" width="0.1524" layer="91"/>
@@
 </segment>
 </net>
+<net name="NRE" class="0">
+<segment>
+<pinref part="U$10" gate="G$1" pin="NRE"/>
+<wire x1="-137.16" y1="-78.74" x2="-142.24" y2="-78.74" width="0.1524" layer="91"/>
+<label x="-142.24" y="-78.74" size="1.778" layer="95" rot="R180" xref="yes"/>
+</segment>
+<segment>
+<pinref part="U$2" gate="G$1" pin="PC7"/>
+<wire x1="246.38" y1="15.24" x2="238.76" y2="15.24" width="0.1524" layer="91"/>
+<label x="238.76" y="15.24" size="1.778" layer="95" rot="R180" xref="yes"/>
+</segment>
+</net>
+<net name="DE" class="0">
+<segment>
+<pinref part="U$10" gate="G$1" pin="DE"/>
+<wire x1="-137.16" y1="-83.82" x2="-142.24" y2="-83.82" width="0.1524" layer="91"/>
+<label x="-142.24" y="-83.82" size="1.778" layer="95" rot="R180" xref="yes"/>
+</segment>
+<segment>
+<pinref part="U$2" gate="G$1" pin="PD6"/>
+<wire x1="276.86" y1="7.62" x2="284.48" y2="7.62" width="0.1524" layer="91"/>
+<label x="284.48" y="7.62" size="1.778" layer="95" xref="yes"/>
+</segment>
+</net>

Commit message: Added signature
Parts:
- removed U$10: MAX3078E, MRDT-ICs:MAX3078E
- added U$3: MAX3077, MRDT-2015-General:MAX3077
Connections:
- removed net DE: U$10.DE, U$2.PD6
- removed net NRE: U$10.NRE, U$2.PC7
- net GND: now also U$3.GND
- net HALL_A: now also U$13.OUT4
- net N$34: now also U$3.B, U$3.Z; no longer U$10.A
- net N$36: now also U$3.A, U$3.Y; no longer U$10.B
- net RX: now also U$3.RO; no longer U$10.RO
- net TX: now also U$3.DI; no longer U$10.DI
- net VCC: now also U$3.VCC; no longer U$10.VCC
Changed lines of the file:
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@@
 <?xml version="1.0" encoding="utf-8"?>
 <!DOCTYPE eagle SYSTEM "eagle.dtd">
-<eagle version="7.4.0">
+<eagle version="7.3.0">
 <drawing>
 <settings>
@@
 <part name="J3" library="MRDT-Connectors" deviceset="APP_2POS_CONFIG" device="5V_HORIZ"/>
 <part name="C38" library="SparkFun-Passives" deviceset="CAP_POL" device="PTH4" value="220u"/>
+<part name="U$3" library="MRDT-2015-General" deviceset="MAX3077" device=""/>
 <part name="R30" library="SparkFun-Passives" deviceset="RESISTOR" device="0805-RES" value="120"/>
 <part name="U$4" library="Molex-SL" deviceset="5PIN" device=""/>
@@
 <part name="SH1" library="shorts-old" deviceset="SHORT-H" device="T5"/>
 <part name="SH2" library="shorts-old" deviceset="SHORT-H" device="T5"/>
-<part name="U$10" library="MRDT-ICs" deviceset="MAX3078E" device=""/>
 </parts>
 <sheets>
@@
 <instance part="J3" gate="VCC" x="256.54" y="-45.72"/>
 <instance part="C38" gate="G$1" x="-73.66" y="-121.92"/>
+<instance part="U$3" gate="G$1" x="-121.92" y="-96.52"/>
 <instance part="R30" gate="G$1" x="-101.6" y="-81.28"/>
 <instance part="U$4" gate="G$1" x="-81.28" y="-91.44"/>
 <instance part="GND36" gate="1" x="-93.98" y="-88.9" rot="R270"/>
-<instance part="GND37" gate="1" x="-111.76" y="-93.98"/>
+<instance part="GND37" gate="1" x="-147.32" y="-101.6"/>
 <instance part="C39" gate="G$1" x="-83.82" y="-121.92"/>
 <instance part="SH1" gate="G$1" x="93.98" y="-73.66"/>
 <instance part="SH2" gate="G$1" x="93.98" y="7.62"/>
-<instance part="U$10" gate="G$1" x="-124.46" y="-81.28"/>
 </instances>
 <busses>
@@
 </segment>
 <segment>
+<pinref part="U$3" gate="G$1" pin="GND"/>
 <pinref part="GND37" gate="1" pin="GND"/>
-<wire x1="-114.3" y1="-88.9" x2="-111.76" y2="-88.9" width="0.1524" layer="91"/>
-<wire x1="-111.76" y1="-88.9" x2="-111.76" y2="-91.44" width="0.1524" layer="91"/>
+<wire x1="-144.78" y1="-93.98" x2="-147.32" y2="-93.98" width="0.1524" layer="91"/>
+<wire x1="-147.32" y1="-93.98" x2="-147.32" y2="-99.06" width="0.1524" layer="91"/>
 </segment>
 <segment>
@@
 </segment>
 <segment>
-<wire x1="-114.3" y1="-73.66" x2="-111.76" y2="-73.66" width="0.1524" layer="91"/>
-<wire x1="-111.76" y1="-73.66" x2="-111.76" y2="-68.58" width="0.1524" layer="91"/>
-<label x="-111.76" y="-68.58" size="1.778" layer="95" rot="R90" xref="yes"/>
-<pinref part="U$10" gate="G$1" pin="VCC"/>
+<pinref part="U$3" gate="G$1" pin="VCC"/>
+<wire x1="-144.78" y1="-78.74" x2="-147.32" y2="-78.74" width="0.1524" layer="91"/>
+<wire x1="-147.32" y1="-78.74" x2="-147.32" y2="-73.66" width="0.1524" layer="91"/>
+<label x="-147.32" y="-73.66" size="1.778" layer="95" rot="R90" xref="yes"/>
 </segment>
 </net>
@@
 <wire x1="223.52" y1="-142.24" x2="218.44" y2="-142.24" width="0.1524" layer="91"/>
 <label x="218.44" y="-142.24" size="1.778" layer="95" rot="R180" xref="yes"/>
+<pinref part="U$13" gate="G$1" pin="OUT4"/>
 </segment>
 <segment>
@@
 </segment>
 <segment>
-<label x="-142.24" y="-88.9" size="1.778" layer="95" rot="R180" xref="yes"/>
-<pinref part="U$10" gate="G$1" pin="DI"/>
-<wire x1="-142.24" y1="-88.9" x2="-137.16" y2="-88.9" width="0.1524" layer="91"/>
+<pinref part="U$3" gate="G$1" pin="DI"/>
+<wire x1="-144.78" y1="-88.9" x2="-147.32" y2="-88.9" width="0.1524" layer="91"/>
+<label x="-147.32" y="-88.9" size="1.778" layer="95" rot="R180" xref="yes"/>
 </segment>
 </net>
@@
 </segment>
 <segment>
-<label x="-142.24" y="-73.66" size="1.778" layer="95" rot="R180" xref="yes"/>
-<pinref part="U$10" gate="G$1" pin="RO"/>
-<wire x1="-142.24" y1="-73.66" x2="-137.16" y2="-73.66" width="0.1524" layer="91"/>
+<pinref part="U$3" gate="G$1" pin="RO"/>
+<wire x1="-144.78" y1="-83.82" x2="-147.32" y2="-83.82" width="0.1524" layer="91"/>
+<label x="-147.32" y="-83.82" size="1.778" layer="95" rot="R180" xref="yes"/>
 </segment>
 </net>
@@
 <net name="N$34" class="0">
 <segment>
-<pinref part="U$10" gate="G$1" pin="A"/>
+<pinref part="U$3" gate="G$1" pin="B"/>
+<pinref part="U$3" gate="G$1" pin="Z"/>
+<wire x1="-116.84" y1="-83.82" x2="-116.84" y2="-88.9" width="0.1524" layer="91"/>
 <pinref part="U$4" gate="G$1" pin="2"/>
-<wire x1="-114.3" y1="-83.82" x2="-96.52" y2="-83.82" width="0.1524" layer="91"/>
+<wire x1="-116.84" y1="-83.82" x2="-96.52" y2="-83.82" width="0.1524" layer="91"/>
+<junction x="-116.84" y="-83.82"/>
 <pinref part="R30" gate="G$1" pin="2"/>
 <wire x1="-96.52" y1="-83.82" x2="-88.9" y2="-83.82" width="0.1524" layer="91"/>
@@
 <net name="N$36" class="0">
 <segment>
-<pinref part="U$10" gate="G$1" pin="B"/>
+<pinref part="U$3" gate="G$1" pin="A"/>
+<wire x1="-116.84" y1="-78.74" x2="-114.3" y2="-78.74" width="0.1524" layer="91"/>
+<wire x1="-114.3" y1="-78.74" x2="-114.3" y2="-93.98" width="0.1524" layer="91"/>
+<pinref part="U$3" gate="G$1" pin="Y"/>
+<wire x1="-114.3" y1="-93.98" x2="-116.84" y2="-93.98" width="0.1524" layer="91"/>
 <pinref part="U$4" gate="G$1" pin="1"/>
 <wire x1="-114.3" y1="-78.74" x2="-106.68" y2="-78.74" width="0.1524" layer="91"/>
+<junction x="-114.3" y="-78.74"/>
 <pinref part="R30" gate="G$1" pin="1"/>
 <wire x1="-106.68" y1="-78.74" x2="-88.9" y2="-78.74" width="0.1524" layer="91"/>
@@
 </segment>
 </net>
-<net name="NRE" class="0">
-<segment>
-<pinref part="U$10" gate="G$1" pin="NRE"/>
-<wire x1="-137.16" y1="-78.74" x2="-142.24" y2="-78.74" width="0.1524" layer="91"/>
-<label x="-142.24" y="-78.74" size="1.778" layer="95" rot="R180" xref="yes"/>
-</segment>
-<segment>
-<pinref part="U$2" gate="G$1" pin="PC7"/>
-<wire x1="246.38" y1="15.24" x2="238.76" y2="15.24" width="0.1524" layer="91"/>
-<label x="238.76" y="15.24" size="1.778" layer="95" rot="R180" xref="yes"/>
-</segment>
-</net>
-<net name="DE" class="0">
-<segment>
-<pinref part="U$10" gate="G$1" pin="DE"/>
-<wire x1="-137.16" y1="-83.82" x2="-142.24" y2="-83.82" width="0.1524" layer="91"/>
-<label x="-142.24" y="-83.82" size="1.778" layer="95" rot="R180" xref="yes"/>
-</segment>
-<segment>
-<pinref part="U$2" gate="G$1" pin="PD6"/>
-<wire x1="276.86" y1="7.62" x2="284.48" y2="7.62" width="0.1524" layer="91"/>
-<label x="284.48" y="7.62" size="1.778" layer="95" xref="yes"/>
-</segment>
-</net>
