File: BLDC_Motor_Controller_2016_Rev1.sch (EAGLE design)
At the start: 141 parts, among them J3 APP_2POS_CONFIG5V_HORIZ, Q1 MOSFET-NCHANNELFQP30N06L, Q2 MOSFET-NCHANNELFQP30N06L, Q3 MOSFET-NCHANNELFQP30N06L, Q4 MOSFET-NCHANNELFQP30N06L, Q5 MOSFET-NCHANNELFQP30N06L, Q6 MOSFET-NCHANNELFQP30N06L, Q7 MOSFET-PCHANNEL, Q8 MOSFET-PCHANNEL, Q9 MOSFET-NCHANNELAO3404A

Commit message: Swapped zeners for NUP4201MR6, rerouted a lot
Parts:
- removed D2, D3, D4, D5: 3.3V, SparkFun-DiscreteSemi:DIODE-ZENER3.3V
- added U1: NUP4201MR6, MRDT-ICs:NUP4201MR6
Connections:
- net ASENSE: now also U1.I/O_1; no longer D2.A
- net BSENSE: now also U1.I/O_4; no longer D3.A
- net CSENSE: now also U$2.PD3, U1.I/O_3; no longer D4.A
- net GND: now also U1.VN
- net PVDDSENSE: now also U1.I/O_2; no longer D5.A
- net VCC: now also U1.VP; no longer D2.C, D3.C, D4.C, D5.C
Changed lines of the file:
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@@
 <part name="C20" library="SparkFun-Passives" deviceset="CAP" device="0805" value="0.1u"/>
 <part name="GND15" library="SparkFun-Aesthetics" deviceset="GND" device=""/>
-<part name="D2" library="SparkFun-DiscreteSemi" deviceset="DIODE-ZENER" device="3.3V" value="3.3V"/>
-<part name="SUPPLY4" library="SparkFun-Aesthetics" deviceset="VCC" device=""/>
 <part name="C21" library="SparkFun-Passives" deviceset="CAP" device="0805" value="1000p"/>
 <part name="Q3" library="SparkFun-DiscreteSemi" deviceset="MOSFET-NCHANNEL" device="FQP30N06L" value="MOSFET-NCHANNELFQP30N06L"/>
@@
 <part name="C23" library="SparkFun-Passives" deviceset="CAP" device="0805" value="0.1u"/>
 <part name="GND18" library="SparkFun-Aesthetics" deviceset="GND" device=""/>
-<part name="D3" library="SparkFun-DiscreteSemi" deviceset="DIODE-ZENER" device="3.3V" value="3.3V"/>
-<part name="SUPPLY5" library="SparkFun-Aesthetics" deviceset="VCC" device=""/>
 <part name="C24" library="SparkFun-Passives" deviceset="CAP" device="0805" value="1000p"/>
 <part name="Q5" library="SparkFun-DiscreteSemi" deviceset="MOSFET-NCHANNEL" device="FQP30N06L" value="MOSFET-NCHANNELFQP30N06L"/>
@@
 <part name="C26" library="SparkFun-Passives" deviceset="CAP" device="0805" value="0.1u"/>
 <part name="GND21" library="SparkFun-Aesthetics" deviceset="GND" device=""/>
-<part name="D4" library="SparkFun-DiscreteSemi" deviceset="DIODE-ZENER" device="3.3V" value="3.3V"/>
-<part name="SUPPLY6" library="SparkFun-Aesthetics" deviceset="VCC" device=""/>
 <part name="C29" library="SparkFun-Passives" deviceset="CAP" device="0805" value="0.1u"/>
 <part name="C30" library="SparkFun-Passives" deviceset="CAP" device="0805" value="0.01u"/>
@@
 <part name="GND22" library="SparkFun-Aesthetics" deviceset="GND" device=""/>
 <part name="GND23" library="SparkFun-Aesthetics" deviceset="GND" device=""/>
-<part name="D5" library="SparkFun-DiscreteSemi" deviceset="DIODE-ZENER" device="3.3V" value="3.3V"/>
-<part name="SUPPLY7" library="SparkFun-Aesthetics" deviceset="VCC" device=""/>
 <part name="U$2" library="MRDT-2015-General" deviceset="TIVA-C" device=""/>
 <part name="R28" library="SparkFun-Passives" deviceset="RESISTOR" device="0805-RES" value="1k"/>
@@
 <part name="D16" library="SparkFun-DiscreteSemi" deviceset="DIODE-ZENER" device="3.3V" value="3.3V"/>
 <part name="U$13" library="MRDT-ICs" deviceset="MAX3078E" device=""/>
+<part name="U1" library="MRDT-ICs" deviceset="NUP4201MR6" device=""/>
+<part name="GND42" library="SparkFun-Aesthetics" deviceset="GND" device=""/>
+<part name="SUPPLY9" library="SparkFun-Aesthetics" deviceset="VCC" device=""/>
 </parts>
 <sheets>
@@
 <instance part="C20" gate="G$1" x="180.34" y="12.7"/>
 <instance part="GND15" gate="1" x="175.26" y="2.54"/>
-<instance part="D2" gate="G$1" x="180.34" y="30.48" rot="R90"/>
-<instance part="SUPPLY4" gate="G$1" x="180.34" y="40.64"/>
 <instance part="C21" gate="G$1" x="129.54" y="12.7"/>
 <instance part="Q3" gate="G$1" x="142.24" y="-30.48"/>
@@
 <instance part="C23" gate="G$1" x="180.34" y="-68.58"/>
 <instance part="GND18" gate="1" x="175.26" y="-78.74"/>
-<instance part="D3" gate="G$1" x="180.34" y="-50.8" rot="R90"/>
-<instance part="SUPPLY5" gate="G$1" x="180.34" y="-40.64"/>
 <instance part="C24" gate="G$1" x="129.54" y="-68.58"/>
 <instance part="Q5" gate="G$1" x="142.24" y="-111.76"/>
@@
 <instance part="C26" gate="G$1" x="180.34" y="-149.86"/>
 <instance part="GND21" gate="1" x="175.26" y="-160.02"/>
-<instance part="D4" gate="G$1" x="180.34" y="-132.08" rot="R90"/>
-<instance part="SUPPLY6" gate="G$1" x="180.34" y="-121.92"/>
 <instance part="C29" gate="G$1" x="0" y="-124.46"/>
 <instance part="C30" gate="G$1" x="12.7" y="-119.38"/>
@@
 <instance part="GND22" gate="1" x="-5.08" y="-139.7"/>
 <instance part="GND23" gate="1" x="33.02" y="-142.24"/>
-<instance part="D5" gate="G$1" x="40.64" y="-119.38" rot="R90"/>
-<instance part="SUPPLY7" gate="G$1" x="40.64" y="-114.3"/>
 <instance part="U$2" gate="G$1" x="261.62" y="7.62"/>
 <instance part="R28" gate="G$1" x="-50.8" y="-17.78" rot="R270"/>
@@
 <instance part="D16" gate="G$1" x="-172.72" y="-17.78" rot="R90"/>
 <instance part="U$13" gate="G$1" x="-127" y="-81.28"/>
+<instance part="U1" gate="G$1" x="-154.94" y="38.1"/>
+<instance part="GND42" gate="1" x="-170.18" y="35.56"/>
+<instance part="SUPPLY9" gate="G$1" x="-137.16" y="38.1"/>
 </instances>
 <busses>
@@
 <wire x1="-116.84" y1="-91.44" x2="-116.84" y2="-88.9" width="0.1524" layer="91"/>
 </segment>
+<segment>
+<pinref part="U1" gate="G$1" pin="VN"/>
+<pinref part="GND42" gate="1" pin="GND"/>
+<wire x1="-170.18" y1="38.1" x2="-167.64" y2="38.1" width="0.1524" layer="91"/>
+</segment>
 </net>
 <net name="N$3" class="0">
@@
 </segment>
 <segment>
-<pinref part="D2" gate="G$1" pin="C"/>
-<wire x1="180.34" y1="33.02" x2="180.34" y2="40.64" width="0.1524" layer="91"/>
-<pinref part="SUPPLY4" gate="G$1" pin="VCC"/>
-</segment>
-<segment>
-<pinref part="D3" gate="G$1" pin="C"/>
-<wire x1="180.34" y1="-48.26" x2="180.34" y2="-40.64" width="0.1524" layer="91"/>
-<pinref part="SUPPLY5" gate="G$1" pin="VCC"/>
-</segment>
-<segment>
-<pinref part="D4" gate="G$1" pin="C"/>
-<wire x1="180.34" y1="-129.54" x2="180.34" y2="-121.92" width="0.1524" layer="91"/>
-<pinref part="SUPPLY6" gate="G$1" pin="VCC"/>
-</segment>
-<segment>
-<pinref part="D5" gate="G$1" pin="C"/>
-<wire x1="40.64" y1="-116.84" x2="40.64" y2="-114.3" width="0.1524" layer="91"/>
-<pinref part="SUPPLY7" gate="G$1" pin="VCC"/>
-</segment>
-<segment>
 <pinref part="U$2" gate="G$1" pin="+3V3"/>
 <wire x1="246.38" y1="-15.24" x2="238.76" y2="-15.24" width="0.1524" layer="91"/>
@@
 <wire x1="-165.1" y1="-7.62" x2="-165.1" y2="-5.08" width="0.1524" layer="91"/>
 <label x="-165.1" y="-5.08" size="1.778" layer="95" rot="R90" xref="yes"/>
+</segment>
+<segment>
+<pinref part="U1" gate="G$1" pin="VP"/>
+<pinref part="SUPPLY9" gate="G$1" pin="VCC"/>
+<wire x1="-137.16" y1="38.1" x2="-139.7" y2="38.1" width="0.1524" layer="91"/>
 </segment>
 </net>
@@
 <wire x1="180.34" y1="22.86" x2="185.42" y2="22.86" width="0.1524" layer="91"/>
 <junction x="180.34" y="22.86"/>
-<pinref part="D2" gate="G$1" pin="A"/>
-<wire x1="180.34" y1="22.86" x2="180.34" y2="27.94" width="0.1524" layer="91"/>
 <label x="185.42" y="22.86" size="1.778" layer="95" xref="yes"/>
 </segment>
@@
 <wire x1="276.86" y1="15.24" x2="284.48" y2="15.24" width="0.1524" layer="91"/>
 <label x="284.48" y="15.24" size="1.27" layer="95" xref="yes"/>
+</segment>
+<segment>
+<pinref part="U1" gate="G$1" pin="I/O_1"/>
+<wire x1="-167.64" y1="43.18" x2="-175.26" y2="43.18" width="0.1524" layer="91"/>
+<label x="-175.26" y="43.18" size="1.27" layer="95" rot="R180" xref="yes"/>
 </segment>
 </net>
@@
 <pinref part="R20" gate="G$1" pin="1"/>
 <wire x1="170.18" y1="-55.88" x2="170.18" y2="-58.42" width="0.1524" layer="91"/>
-<pinref part="D3" gate="G$1" pin="A"/>
 <pinref part="C23" gate="G$1" pin="1"/>
 <wire x1="170.18" y1="-58.42" x2="170.18" y2="-63.5" width="0.1524" layer="91"/>
-<wire x1="180.34" y1="-53.34" x2="180.34" y2="-58.42" width="0.1524" layer="91"/>
 <wire x1="180.34" y1="-58.42" x2="180.34" y2="-63.5" width="0.1524" layer="91"/>
 <wire x1="170.18" y1="-58.42" x2="180.34" y2="-58.42" width="0.1524" layer="91"/>
@@
 <label x="284.48" y="12.7" size="1.27" layer="95" xref="yes"/>
 </segment>
+<segment>
+<pinref part="U1" gate="G$1" pin="I/O_4"/>
+<wire x1="-139.7" y1="43.18" x2="-132.08" y2="43.18" width="0.1524" layer="91"/>
+<label x="-132.08" y="43.18" size="1.27" layer="95" xref="yes"/>
+</segment>
 </net>
 <net name="N$22" class="0">
@@
 <segment>
 <pinref part="C31" gate="G$1" pin="1"/>
-<pinref part="D5" gate="G$1" pin="A"/>
-<wire x1="40.64" y1="-127" x2="40.64" y2="-121.92" width="0.1524" layer="91"/>
 <wire x1="40.64" y1="-129.54" x2="40.64" y2="-127" width="0.1524" layer="91"/>
 <wire x1="40.64" y1="-127" x2="48.26" y2="-127" width="0.1524" layer="91"/>
@@
 <label x="284.48" y="17.78" size="1.27" layer="95" xref="yes"/>
 </segment>
+<segment>
+<pinref part="U1" gate="G$1" pin="I/O_2"/>
+<wire x1="-167.64" y1="33.02" x2="-175.26" y2="33.02" width="0.1524" layer="91"/>
+<label x="-175.26" y="33.02" size="1.27" layer="95" rot="R180" xref="yes"/>
+</segment>
 </net>
 <net name="CSENSE" class="0">
@@
 <pinref part="R25" gate="G$1" pin="1"/>
 <wire x1="170.18" y1="-137.16" x2="170.18" y2="-139.7" width="0.1524" layer="91"/>
-<pinref part="D4" gate="G$1" pin="A"/>
 <pinref part="C26" gate="G$1" pin="1"/>
 <wire x1="170.18" y1="-139.7" x2="170.18" y2="-144.78" width="0.1524" layer="91"/>
-<wire x1="180.34" y1="-134.62" x2="180.34" y2="-139.7" width="0.1524" layer="91"/>
 <wire x1="180.34" y1="-139.7" x2="180.34" y2="-144.78" width="0.1524" layer="91"/>
 <wire x1="170.18" y1="-139.7" x2="180.34" y2="-139.7" width="0.1524" layer="91"/>
@@
 <label x="185.42" y="-139.7" size="1.778" layer="95" xref="yes"/>
 </segment>
-</net>
+<segment>
+<pinref part="U$2" gate="G$1" pin="PD3"/>
+<wire x1="276.86" y1="10.16" x2="284.48" y2="10.16" width="0.1524" layer="91"/>
+<label x="284.48" y="10.16" size="1.27" layer="95" xref="yes"/>
+</segment>
+<segment>
+<pinref part="U1" gate="G$1" pin="I/O_3"/>
+<wire x1="-139.7" y1="33.02" x2="-132.08" y2="33.02" width="0.1524" layer="91"/>
+<label x="-132.08" y="33.02" size="1.27" layer="95" xref="yes"/>
+</segment>
+</net>

Commit message: Minor routing changes
Parts:
- SH1, SH2: device shorts-old:SHORT-HT5 -> BLDC_Motor_Controller_2016_Rev1:SHORT-HT5
Changed lines of the file:
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@@
 <part name="GND37" library="SparkFun-Aesthetics" deviceset="GND" device=""/>
 <part name="C39" library="SparkFun-Passives" deviceset="CAP_POL" device="PTH4" value="220u"/>
-<part name="SH1" library="shorts-old" deviceset="SHORT-H" device="T5"/>
-<part name="SH2" library="shorts-old" deviceset="SHORT-H" device="T5"/>
+<part name="SH1" library="BLDC_Motor_Controller_2016_Rev1" deviceset="SHORT-H" device="T5"/>
+<part name="SH2" library="BLDC_Motor_Controller_2016_Rev1" deviceset="SHORT-H" device="T5"/>
 <part name="R31" library="SparkFun-Passives" deviceset="RESISTOR" device="0805-RES" value="100"/>
 <part name="C40" library="SparkFun-Passives" deviceset="CAP" device="0805" value=".015u"/>

Commit message: Switched to MAX232
Parts:
- removed R30: 120, SparkFun-Passives:RESISTOR0805-RES
- removed U$13: MAX3078E, MRDT-ICs:MAX3078E
- added C44, C45, C46, C47, C48: 1u, SparkFun-Passives:CAP0805
- added U2: MAX232, MRDT-ICs:MAX232
- D16: value 3.3V -> 15V
- R3: value 31.6k -> 53.3k
Connections:
- removed net N$36: R30.1, U$13.B, U$4.1
- removed net N$37: R31.2, U$4.5
- removed net RX: U$13.RO, U$2.PB0
- removed net TX: U$13.DI, U$2.PB1
- new net 232_RX: U$4.4, U2.R2OUT
- new net 232_TX: U$4.5, U2.T2OUT
- new net N$40: C44.1, U2.C1+
- new net N$42: C44.2, U2.C1-
- new net N$43: C45.1, U2.C2+
- new net N$44: C45.2, U2.C2-
- new net N$45: C48.1, U2.VS-
- new net N$46: C47.1, U2.VS+
- new net UART_RX: U$2.PB0, U2.T2IN
- new net UART_TX: U$2.PB1, U2.R2IN
- net DE: no longer U$13.DE
- net GND: now also C46.2, C47.2, C48.2, U2.GND; no longer U$13.GND
- net N$34: now also R31.2, U$4.1; no longer R30.2, U$13.A, U$4.2
- net NRE: no longer U$13.!RE
- net VCC: now also C46.1, U2.VCC; no longer U$13.VCC
Other:
- moved on the sheet: C15, C19, C20, C21, C22, C23, C24, C27, C28, C29, C30, C31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
