File: BLDC_Motor_Controller_2018_Rev1.sch (EAGLE design)
At the start: 142 parts, among them J3 APP_2POS_CONFIG5V_HORIZ, Q1 MOSFET-NCHANNELFQP30N06L, Q2 MOSFET-NCHANNELFQP30N06L, Q3 MOSFET-NCHANNELFQP30N06L, Q4 MOSFET-NCHANNELFQP30N06L, Q5 MOSFET-NCHANNELFQP30N06L, Q6 MOSFET-NCHANNELFQP30N06L, Q7 MOSFET-PCHANNEL, Q8 MOSFET-PCHANNEL, Q9 MOSFET-NCHANNELAO3404A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

Commit message: Deleted hall effect hardware, four 220uF caps
Reusing board for 2018 rover but deleting hall effect hardware, deleted four 220uF power conditioning caps and changed remaining caps to 470uF. Added 3pin SL to carry PWM signal to control card without passing through a filter. Changed names of the files to include 2018.
Parts:
- removed C27, C28, C37, C39: 220u, SparkFun-Passives:CAP_POLPTH4
- removed C41, C42, C43: .015u, SparkFun-Passives:CAP0805
- removed R36, R37, R38: 10k, SparkFun-Passives:RESISTOR0805-RES
- removed R39, R40, R41: 10, SparkFun-Passives:RESISTOR0805-RES
- removed U$21, U$22, U$23: TEST_POINT_0.1INDIAM, MRDT-Connectors:TEST_POINT_0.1INDIAM
- removed U$8: 5PIN, Molex-SL:5PIN
- added J1: SL03THROUGH_HOLE, MRDT-Connectors:SL03THROUGH_HOLE
- C15, C34, C35, C38: value 220u -> 470u
Connections:
- removed net HALL_A: C41.1, R41.1, U$2.PA5, U$22.P$1
- removed net HALL_B: C42.1, R40.1, U$2.PE5, U$21.P$1
- removed net HALL_C: C43.1, R39.1, U$2.PB5, U$23.P$1
- removed net N$20: R37.2, R39.2, U$8.2
- removed net N$33: R36.2, R40.2, U$8.3
- removed net N$39: R38.2, R41.2, U$8.4
- new net PWM_IN_NO_FILTER: J1.3, U$2.PF4
- net GND: now also J1.1; no longer C27.-, C28.-, C37.-, C39.-, C41.2, C42.2, C43.2, U$8.5
- net PVDD: no longer C27.+, C28.+, C37.+, C39.+
- net VCC: no longer R36.1, R37.1, R38.1, U$8.1
Other:
- moved on the sheet: C34, C35, C38
