File: Motor_Controller_2019_Rev1.sch (KiCad schematic (older format))
At the start: 124 parts, among them Q1 Q_NMOS_DGS, Q2 Q_PMOS_SGD, Q3 Q_PMOS_SGD, Q4 Q_NMOS_DGS, Q5 Q_NMOS_DGS, Q6 Q_NMOS_DGS, Q7 Q_NMOS_DGS, Q8 Q_NMOS_DGS, Q9 Q_NMOS_DGS, U1 DRV8301, U2 NUP4201MR6, U3 MAX3232

Commit message: Start of TIVA Header section
Other:
- note added: "TIVA Header"
Changed lines of the file:
@@
 LIBS:MRDT_ICs
 LIBS:MRDT_Passives
-LIBS:MRDT_Sensors
 LIBS:MRDT_Shields
 LIBS:MRDT_Silkscreens
@@
 	7900 1900 7950 1900
 Wire Notes Line
-	550  550  10800 550
+	550  550  18100 550
 Wire Notes Line
 	550  3050 10100 3050
@@
 Connection ~ 8700 12000
 Wire Notes Line
-	550  12800 18100 12800
+	18100 12800 550  12800
 Wire Wire Line
 	1850 10600 1850 10800
@@
 SH_C
 Wire Notes Line
-	18100 12800 18100 6150
+	18100 550  18100 12800
+Text Notes 10900 900  0    197  ~ 0
+TIVA Header
 $EndSCHEMATC

Commit message: Changed NSCS and serial receive flag locations, started development on second motor controller circuit
Parts:
- removed C41: 0.015u, Capacitors_SMD:C_0805_HandSoldering, symbol C
- removed Conn1: Molex_SL_03, MRDT_Connectors.pretty:MOLEX_SL_03_Horizontal, symbol Molex_SL_03
- removed Conn2: Molex_SL_05, MRDT_Connectors.pretty:MOLEX_SL_05_Horizontal, symbol Molex_SL_05
- removed R36: 100, symbol R
- added C? (x9): 0.1u, Capacitors_SMD:C_0805_HandSoldering, symbol C
- added C? (x2): 4.7u, Capacitors_SMD:C_0805_HandSoldering, symbol C
- added C? (x3): 1u, Capacitors_SMD:C_0805_HandSoldering, symbol C
- added C?: 47u, Capacitors_SMD:C_0805_HandSoldering, symbol CP1
- added C? (x3): 2.2u, Capacitors_SMD:C_0805_HandSoldering, symbol C
- added C?: 0.015u, Capacitors_SMD:C_0805_HandSoldering, symbol C
- added C? (x2): 2200p, Capacitors_SMD:C_0805_HandSoldering, symbol C
- added C?: .022u, Capacitors_SMD:C_0805_HandSoldering, symbol C
- added C?: 6800p, Capacitors_SMD:C_0805_HandSoldering, symbol C
- added C?: 120p, Capacitors_SMD:C_0805_HandSoldering, symbol C
- added C? (x2): 1000p, Capacitors_SMD:C_0805_HandSoldering, symbol C
- added C? (x4): 470u, Capacitors_THT:CP_Radial_D12.5mm_P5.00mm, symbol CP1
- added Conn?: Molex_SL_04, symbol Molex_SL_04
- added D? (x5): D_Zener, Diodes_SMD:D_SOD-123, symbol D_Zener
- added L?: 33u, MRDT_Passives.pretty:DR74_330_R, symbol L
- added Q? (x4): Q_NMOS_DGS, symbol Q_NMOS_DGS
- added R?: 150k, symbol R
- added R? (x4): 10k, symbol R
- added R?: 31.6k, symbol R
- added R? (x2): 1k, symbol R
- added R? (x2): 56, symbol R
- added R?: 205k, symbol R
- added R?: 16.2k, symbol R
- added R? (x4): 10, symbol R
- added R? (x2): 46.4k, symbol R
- added R? (x2): 4.99k, symbol R
- added R? (x2): .001, symbol R
- added TP? (x7): TEST, symbol TEST
- added U? (x8): LAUNCHXL_F28069M_Launchpad, symbol LAUNCHXL_F28069M_Launchpad
- added U?: NUP4201MR6, symbol NUP4201MR6
- added U? (x5): DRV8301, symbol DRV8301
Connections:
- net labels added: ASENSE_A1, ASENSE_A2, BSENSE_A1, BSENSE_A2, CSENSE_A1, CSENSE_A2, DC_CAL_A1, DC_CAL_A2, EN_GATE_A1, EN_GATE_A2, GH_A_A1, GH_B_A1, GH_C_A1, GL_A_A1, GL_B_A1, GL_C_A1, INH_A_A1, INH_A_A2, INH_B_A1, INH_B_A2, INH_C_A1, INH_C_A2, INL_A_A1, INL_A_A2, INL_B_A1, INL_B_A2, INL_C_A1, INL_C_A2, NFAULT_A1, NFAULT_A2, NOCTW_A1, NOCTW_A2, NSCS_A1, NSCS_M2, PVDDSENSE_A1, PVDDSENSE_A2, PWM_IN_A1, PWM_IN_A2, PWRGD_A1, SCLK_A1, SCLK_A2, SD1_A2, SDI_A1, SDO_A1, SDO_A2, SH_A_A1, SH_B_A1, SH_C_A1, SL_A_A1, SL_B_A1, SO1_A1, SO1_A2, SO2_A1, SO2_A2, UART_RX_A1, UART_RX_A2, UART_RX_M1
- net labels removed: 232_TX, PWM_IN, PWM_IN_NO_FILTER, UART_TX
- wire segments 250 -> 425
Other:
- note added: "A1"
- note added: "A2"
- note added: "Analogue out from ACS711 \ngoes to S01 (A_A0) and \nS02 (A_B0) on F28069 headers"
- note added: "Motor Driver_A1"
- note added: "Motor Header 1"
- note added: "Motor Header 2"
- note added: "New current sensing technique in \nGimbal VFD schematic, uses ACS711 in \nPhase A and B instead of current \nsensing using DRV8301"
- note added: "Phase A_A1"
- note added: "Phase B_A1"
- note added: "Phase C_A1"
- note added: "Transient Protection_A1"
- note added: "Transient Protection_A2"
- note added: "change a1 to m1 in all the flags have fun"
- note added: "update to mrdt library"
- note added: "use ground andersons for all these connections"
- note removed: "Phase C"
- note removed: "TIVA Header"
- note removed: "Transient Protection"

Commit message: Duplicated and added appropriate naming for motor 2 phases, driver, and transient protection. Swapped out max3232 device for MRDT version. Replaced phase a and b wiring to drv with buses for neatness and clarity.
Parts:
- removed C36, C37, C38, C39, C40: 0.1u, Capacitors_SMD:C_0805_HandSoldering, symbol C
- removed Conn3, Conn4, Conn5, Conn6, Conn7: AndersonPP, MRDT_Connectors.pretty:Anderson_1_Horisontal, symbol AndersonPP
- removed U3: MAX3232, symbol MAX3232
- added C?: 2.2u, Capacitors_SMD:C_0805_HandSoldering, symbol C
- added C? (x11): 0.1u, Capacitors_SMD:C_0805_HandSoldering, symbol C
- added Conn? (x10): AndersonPP, symbol AndersonPP
- added Conn?: Molex_SL_04, symbol Molex_SL_04
- added D? (x2): LED, LEDs:LED_1206_HandSoldering, symbol LED
- added D? (x2): D_Zener, Diodes_SMD:D_SOD-123, symbol D_Zener
- added Q? (x2): Q_PMOS_SGD, symbol Q_PMOS_SGD
- added Q? (x2): Q_NMOS_DGS, symbol Q_NMOS_DGS
- added R? (x2): 330, symbol R
- added R? (x2): 10, symbol R
- added R?: 46.4k, symbol R
- added R?: 4.99k, symbol R
- added TP? (x7): TEST, symbol TEST
- added U? (x2): MAX_3232, symbol MAX_3232
Connections:
- net labels added: 232_RX_M1, 232_RX_M2, ASENSE_M1, ASENSE_M2, BSENSE_M1, BSENSE_M2, CSENSE_M1, CSENSE_M2, DC_CAL_M1, DC_CAL_M2, EN_GATE_M1, EN_GATE_M2, GH_A_M1, GH_A_M2, GH_B_M1, GH_B_M2, GH_C_M1, GH_C_M2, GL_A_M1, GL_A_M2, GL_B_M1, GL_B_M2, GL_C_M1, GL_C_M2, INH_A_M1, INH_A_M2, INH_B_M1, INH_B_M2, INH_C_M1, INH_C_M2, INL_A_M1, INL_A_M2, INL_B_M1, INL_B_M2, INL_C_M1, INL_C_M2, NFAULT_M1, NFAULT_M2, NOCTW_M1, NOCTW_M2, NSCS_M1, PWM_IN_M1, PWM_IN_M2, PWRGD_M1, PWRGD_M2, SCLK_M1, SCLK_M2, SD1_M2, SDI_M1, SDI_M2, SDO_M1, SDO_M2, SH_A_M1, SH_A_M2, SH_B_M1, SH_B_M2, SH_C_M1, SH_C_M2, SL_A_M1, SL_A_M2, SL_B_M1, SL_B_M2, SN1_M1, SN1_M2, SN2_M1, SN2_M2, SO1_M1, SO1_M2, SO2_M1, SO2_M2, SP1_M1, SP1_M2, SP2_M1, SP2_M2, UART_RX_M2
- net labels removed: 232_RX, ASENSE, ASENSE_A1, ASENSE_A2, BSENSE, BSENSE_A1, BSENSE_A2, CSENSE, CSENSE_A1, CSENSE_A2, DC_CAL, DC_CAL_A1, DC_CAL_A2, EN_GATE, EN_GATE_A1, EN_GATE_A2, GH_A, GH_A_A1, GH_B, GH_B_A1, GH_C, GH_C_A1, GL_A, GL_A_A1, GL_B, GL_B_A1, GL_C, GL_C_A1, INH_A, INH_A_A1, INH_A_A2, INH_B, INH_B_A1, INH_B_A2, INH_C, INH_C_A1, INH_C_A2, INL_A, INL_A_A1, INL_A_A2, INL_B, INL_B_A1, INL_B_A2, INL_C, INL_C_A1, INL_C_A2, NFAULT, NFAULT_A1, NFAULT_A2, NOCTW, NOCTW_A1, NOCTW_A2, NSCS, NSCS_A1, PVDDSENSE_A1, PVDDSENSE_A2, PWM_IN_A1, PWM_IN_A2, PWRGD, PWRGD_A1, SCLK, SCLK_A1, SCLK_A2, SD1_A2, SDI, SDI_A1, SDO, SDO_A1, SDO_A2, SH_A, SH_A_A1, SH_B, SH_B_A1, SH_C, SH_C_A1, SL_A, SL_A_A1, SL_B, SL_B_A1, SO1, SO1_A1, SO1_A2, SO2, SO2_A1, SO2_A2, UART_RX, UART_RX_A1, UART_RX_A2
- wire segments 425 -> 458
Other:
- note added: "M1"
- note added: "M2"
- note added: "Motor Driver_M1"
- note added: "Motor Driver_M2"
- note added: "Phase A_M1"
- note added: "Phase A_M2"
- note added: "Phase B_M1"
- note added: "Phase B_M2"
- note added: "Phase C_M1"
- note added: "Phase C_M2"
- note added: "Transient Protection_M1"
- note added: "Transient Protection_M2"
- note removed: "A1"
- note removed: "A2"
- note removed: "Motor Driver"
- note removed: "Motor Driver_A1"
- note removed: "Phase A"
- note removed: "Phase A_A1"
- note removed: "Phase B"
- note removed: "Phase B_A1"
- note removed: "Phase C_A1"
- note removed: "Transient Protection_A1"
- note removed: "Transient Protection_A2"
- note removed: "change a1 to m1 in all the flags have fun"
- note removed: "update to mrdt library"
- note removed: "use ground andersons for all these connections"

Commit message: Re-annotated schematic
Parts:
- gave numbers to parts that had none: 119
