File: Motor_Controller_2019_Rev1.sch (KiCad schematic (older format))
At the start: 222 parts, among them Q1 Q_NMOS_DGS, Q10 Q_PMOS_SGD, Q11 Q_PMOS_SGD, Q12 Q_NMOS_DGS, Q13 Q_NMOS_DGS, Q14 Q_NMOS_DGS, Q15 Q_NMOS_DGS, Q16 Q_NMOS_DGS, Q17 Q_NMOS_DGS, Q2 Q_PMOS_SGD, Q3 Q_PMOS_SGD, Q4 Q_NMOS_DGS, Q5 Q_NMOS_DGS, Q6 Q_NMOS_DGS, Q7 Q_NMOS_DGS, Q8 Q_NMOS_DGS, Q9 Q_NMOS_DGS, U1 DRV8301, U2 NUP4201MR6, U3 LAUNCHXL_F28069M_Launchpad, U4 MAX_3232, U6 NUP4201MR6, U7 DRV8301

Commit message: Cleaned up ground connections, fixed an issue with the device library directory paths
Parts:
- removed Conn1, Conn11, Conn12, Conn2, Conn3, Conn5, Conn6, Conn7, Conn8, Conn9: AndersonPP, symbol Motor_Controller_2019_Rev1-rescue:AndersonPP
- removed Conn10, Conn4: Molex_SL_04, symbol Motor_Controller_2019_Rev1-rescue:Molex_SL_04
- removed U1, U7: DRV8301, symbol Motor_Controller_2019_Rev1-rescue:DRV8301
- removed U2, U6: NUP4201MR6, symbol Motor_Controller_2019_Rev1-rescue:NUP4201MR6
- removed U3: LAUNCHXL_F28069M_Launchpad, symbol Motor_Controller_2019_Rev1-rescue:LAUNCHXL_F28069M_Launchpad
- removed U4: MAX_3232, symbol Motor_Controller_2019_Rev1-rescue:MAX_3232
- added Conn? (x10): AndersonPP, symbol MRDT_Connectors:AndersonPP
- added Conn? (x2): Molex_SL_04, symbol MRDT_Connectors:Molex_SL_04
- added U? (x10): DRV8301, symbol MRDT_ICs:DRV8301
- added U? (x2): NUP4201MR6, symbol MRDT_ICs:NUP4201MR6
- added U?: MAX_3232, symbol MRDT_ICs:MAX_3232
Connections:
- wire segments 599 -> 575

Commit message: Reorganized schematic structure, fixed the TIVA headers, added dual serial TX and RX for both motors to the MAX3232 and the headers
Parts:
- removed Conn? (x2): Molex_SL_04, symbol MRDT_Connectors:Molex_SL_04
- added Conn?: Molex_SL_05, symbol MRDT_Connectors:Molex_SL_05
- added U? (x8): TM4C123G_Launchpad, symbol MRDT_Shields:TM4C123G_Launchpad
Connections:
- net labels added: 232_RX_M2, 232_TX_M1, 232_TX_M2, UART_TX_M1, UART_TX_M2
- wire segments 575 -> 571
Other:
- note added: "Analog out from ACS711 \ngoes to S01 (A_A0) and \nS02 (A_B0) on F28069 headers"
- note added: "Motor 1"
- note added: "Motor 2"
- note added: "Motor Driver"
- note added: "Phase A"
- note added: "Phase B"
- note added: "Phase C"
- note added: "Transient Protection"
- note removed: "Analogue out from ACS711 \ngoes to S01 (A_A0) and \nS02 (A_B0) on F28069 headers"
- note removed: "Motor Driver_M1"
- note removed: "Motor Driver_M2"
- note removed: "Phase A_M1"
- note removed: "Phase A_M2"
- note removed: "Phase B_M1"
- note removed: "Phase B_M2"
- note removed: "Phase C_M1"
- note removed: "Phase C_M2"
- note removed: "Transient Protection_M1"
- note removed: "Transient Protection_M2"

Commit message: Fixed flag connection spacing across the schematic, fixed the serial connections by adding them to the molex sl5 in place of the uart connections previously there, added indiactors for serial and phase GH,GL connections, replaced the header device with the f28069m device, restructered external connections into max_3232 and anderson sections, fixed labeling on andersonPP connections for context and clarity, other minor fixes
Parts:
- removed D2: D_Zener, Diodes_SMD:D_SOD-123, symbol Device:D_Zener
- removed Q1: Q_NMOS_DGS, symbol Device:Q_NMOS_DGS
- removed Q10, Q11, Q2, Q3: Q_PMOS_SGD, symbol Device:Q_PMOS_SGD
- removed R13, R17, R21, R36, R37: 330, symbol Device:R
- removed R7: 3M, symbol Device:R
- removed R9: 1M, symbol Device:R
- removed TP12, TP13, TP14, TP15, TP16, TP17, TP18, TP19: TEST, symbol Connector:TestPoint
- removed U? (x8): TM4C123G_Launchpad, symbol MRDT_Shields:TM4C123G_Launchpad
- added D? (x16): LED, LEDs:LED_1206_HandSoldering, symbol Device:LED
- added R? (x9): 500, symbol Device:R
- added R? (x12): 1k, symbol Device:R
- added U? (x8): LAUNCHXL_F28069M_Launchpad, symbol MRDT_Shields:LAUNCHXL_F28069M_Launchpad
- Conn?: value AndersonPP -> SH_A_M1_PP
- Conn?: value AndersonPP -> SH_B_M1_PP
- Conn?: value AndersonPP -> SH_C_M1_PP
- Conn? (x2): value AndersonPP -> GND_PP
- Conn? (x2): value AndersonPP -> PVDD_PP
- Conn?: value AndersonPP -> SH_A_M2_PP
- Conn?: value AndersonPP -> SH_B_M2_PP
- Conn?: value AndersonPP -> SH_C_M2_PP
- R10: value 330 -> 500
Connections:
- wire segments 571 -> 739
Other:
- note added: "Andersons"
- note added: "Double check with Jacob on\nif we need to double up on these\nor not"
- note added: "MAX_3232"
- note added: "confirm pack voltage to \ncalculate this value"
- note removed: "External Connections"

Commit message: Added resistor value for pack voltage LED, fixed some formatting for wiring, removed bus connections and replaced with flags (we're going to move to bus connections after PDR)
Parts:
- R10: value 500 -> 1.7k
Connections:
- wire segments 739 -> 725
Other:
- note removed: "confirm pack voltage to \ncalculate this value"
Changed lines of the file:
@@
 Text GLabel 3050 6550 0    39   Input ~ 0
 SCLK_M1
-Text GLabel 1500 6800 0    39   Input ~ 0
+Text GLabel 1500 6650 0    39   Input ~ 0
 DC_CAL_M1
 $Comp
@@
 	1    0    0    -1
 $EndComp
-Text GLabel 2050 6900 0    39   Input ~ 0
+Text GLabel 2050 6750 0    39   Input ~ 0
 EN_GATE_M1
 $Comp
@@
 P 11250 8300
 F 0 "R10" V 11330 8300 50  0000 C CNN
-F 1 "500" V 11250 8300 50  0000 C CNN
+F 1 "1.7k" V 11250 8300 50  0000 C CNN
 F 2 "" V 11180 8300 50  0001 C CNN
 F 3 "" H 11250 8300 50  0001 C CNN
@@
 Text GLabel 20900 6550 0    39   Input ~ 0
 SCLK_M2
-Text GLabel 19300 6800 0    39   Input ~ 0
+Text GLabel 19300 6650 0    39   Input ~ 0
 DC_CAL_M2
 $Comp
@@
 	1    0    0    -1
 $EndComp
-Text GLabel 19850 6900 0    39   Input ~ 0
+Text GLabel 19850 6750 0    39   Input ~ 0
 EN_GATE_M2
 $Comp
@@
 	0    -1   -1   0
 $EndComp
-Wire Wire Line
-	20000 6850 20000 6750
-Wire Wire Line
-	19950 6850 20000 6850
-Wire Wire Line
-	19300 6800 19350 6800
-Wire Wire Line
-	19950 6800 19950 6650
 Connection ~ 26250 9750
 Wire Wire Line
@@
 Wire Wire Line
 	12450 7750 12450 7650
-Connection ~ 1550 6800
-Wire Wire Line
-	1550 6850 1550 6800
 Wire Wire Line
 	2600 6850 2750 6850
-Connection ~ 25900 7150
-Connection ~ 25900 6850
 Connection ~ 26250 6550
 Connection ~ 25900 6550
@@
 Wire Wire Line
 	25500 5200 25350 5200
-Connection ~ 25900 3900
-Connection ~ 25900 3600
 Connection ~ 26250 3300
 Connection ~ 25900 3300
@@
 	20350 6850 20600 6850
 Wire Wire Line
-	20000 6750 20950 6750
-Connection ~ 19350 6800
-Wire Wire Line
-	19350 6850 19350 6800
-Connection ~ 19950 6900
-Wire Wire Line
-	19950 6950 19950 6900
-Wire Wire Line
-	19950 6650 20950 6650
-Wire Wire Line
 	20350 5650 20350 5600
 Connection ~ 19950 4950
@@
 Wire Wire Line
 	7800 8500 7650 8500
-Connection ~ 8200 7100
-Connection ~ 8200 6800
 Connection ~ 8550 6500
 Connection ~ 8200 6500
@@
 Wire Wire Line
 	7800 5150 7650 5150
-Connection ~ 8200 3950
-Connection ~ 8200 3650
 Connection ~ 8550 3350
 Connection ~ 8200 3350
@@
 	2500 6950 2550 6950
 Wire Wire Line
-	2300 6750 3100 6750
-Wire Wire Line
-	2300 6850 2300 6750
-Wire Wire Line
-	2100 6850 2300 6850
-Wire Wire Line
-	2200 6800 1550 6800
-Connection ~ 2100 6900
-Wire Wire Line
-	2050 6900 2100 6900
-Wire Wire Line
-	2100 6950 2100 6900
-Wire Wire Line
-	2200 6650 2200 6800
-Wire Wire Line
-	3100 6650 2200 6650
-Wire Wire Line
 	2500 5650 2500 5600
 Connection ~ 2100 4950
@@
 Text GLabel 16650 6350 0    39   Input ~ 0
 SH_C_M2
-Wire Wire Line
-	24650 6850 25900 6850
-Wire Wire Line
-	24650 7150 25900 7150
 Connection ~ 26250 6850
-Entry Wire Line
-	24550 6750 24650 6850
-Entry Wire Line
-	24550 7050 24650 7150
-Text Label 24650 6850 0    39   ~ 0
-SN2_M2
-Text Label 24650 7150 0    39   ~ 0
-SP2_M2
-Entry Wire Line
-	22300 6250 22400 6150
-Wire Wire Line
-	22050 6250 22300 6250
-Text Label 22050 6250 0    39   ~ 0
-SP2_M2
-Wire Wire Line
-	22050 6150 22300 6150
-Entry Wire Line
-	22300 6150 22400 6050
-Text Label 22050 6150 0    39   ~ 0
-SN2_M2
-Wire Wire Line
-	24650 3600 25900 3600
 Connection ~ 26250 3600
-Entry Wire Line
-	24550 3700 24650 3600
-Wire Wire Line
-	24650 3900 25900 3900
-Entry Wire Line
-	24550 4000 24650 3900
-Text Label 24650 3600 0    39   ~ 0
-SN1_M2
-Text Label 24650 3900 0    39   ~ 0
-SP1_M2
-Entry Wire Line
-	22300 5950 22400 5850
-Wire Wire Line
-	22050 5950 22300 5950
-Wire Wire Line
-	22050 6050 22300 6050
-Entry Wire Line
-	22300 6050 22400 5950
-Text Label 22050 5950 0    39   ~ 0
-SN1_M2
-Text Label 22050 6050 0    39   ~ 0
-SP1_M2
-Wire Wire Line
-	6950 6800 8200 6800
 Connection ~ 8550 6800
-Wire Wire Line
-	6950 7100 8200 7100
-Entry Wire Line
-	4450 6250 4550 6150
-Wire Wire Line
-	4200 6250 4450 6250
-Entry Wire Line
-	4450 6150 4550 6050
-Wire Wire Line
-	4200 6150 4450 6150
-Entry Wire Line
-	4450 6050 4550 5950
-Wire Wire Line
-	4200 6050 4450 6050
-Entry Wire Line
-	4450 5950 4550 5850
-Wire Wire Line
-	4200 5950 4450 5950
-Text Label 4200 5950 0    39   ~ 0
-SN1_M1
-Text Label 4200 6050 0    39   ~ 0
-SP1_M1
-Text Label 4200 6150 0    39   ~ 0
-SN2_M1
-Text Label 4200 6250 0    39   ~ 0
-SP2_M1
-Entry Wire Line
-	6850 7000 6950 7100
-Text Label 6950 7100 0    39   ~ 0
-SP2_M1
-Entry Wire Line
-	6850 6700 6950 6800
-Text Label 6950 6800 0    39   ~ 0
-SN2_M1
-Entry Wire Line
-	6850 3750 6950 3650
-Wire Wire Line
-	6950 3650 8200 3650
 Connection ~ 8550 3650
 Wire Wire Line
-	6950 3950 8200 3950
-Entry Wire Line
-	6850 4050 6950 3950
-Text Label 6950 3650 0    39   ~ 0
-SN1_M1
-Text Label 6950 3950 0    39   ~ 0
-SP1_M1
-Wire Wire Line
 	25900 9400 25900 9450
 Wire Wire Line
@@
 	25900 8550 25950 8550
 Wire Wire Line
-	1550 6800 1500 6800
-Wire Wire Line
 	25900 7150 26250 7150
 Wire Wire Line
@@
 	20400 6950 20650 6950
 Wire Wire Line
-	19350 6800 19950 6800
-Wire Wire Line
-	19950 6900 19950 6850
-Wire Wire Line
 	19950 4950 20150 4950
 Wire Wire Line
@@
 	2550 6950 2800 6950
 Wire Wire Line
-	2100 6900 2100 6850
-Wire Wire Line
 	2100 4950 2300 4950
 Wire Wire Line
@@
 Connection ~ 27000 8550
 Connection ~ 15150 9650
-Entry Bus Bus
-	6750 5750 6850 5650
-Entry Bus Bus
-	22400 5850 22500 5750
-Entry Bus Bus
-	4550 5850 4650 5750
-Wire Bus Line
-	4650 5750 6750 5750
-Entry Bus Bus
-	24450 5750 24550 5650
 Wire Wire Line
 	2100 2000 2400 2000
@@
 Connection ~ 9600 8900
 Connection ~ 19350 1700
-Wire Bus Line
-	22500 5750 24450 5750
 Connection ~ 27300 8950
 Text Notes 4650 950  0    276  ~ 55
@@
 Wire Wire Line
 	19350 7350 19950 7350
-Wire Wire Line
-	19850 6900 19950 6900
 Connection ~ 19950 7350
 Connection ~ 27300 2350
@@
 Wire Wire Line
 	11250 7650 11250 7750
-Text Notes 11200 7250 0    31   ~ 0
-confirm pack voltage to \ncalculate this value
 Connection ~ 16350 8550
 $Comp
@@
 	17250 8550 17550 8550
 Connection ~ 17250 8550
-Wire Bus Line
-	22400 5850 22400 6150
-Wire Bus Line
-	4550 5850 4550 6150
-Wire Bus Line
-	6850 3750 6850 7000
-Wire Bus Line
-	24550 3700 24550 7050
+Text GLabel 4250 5950 2    39   Input ~ 0
+SN1_M1
+Text GLabel 4250 6050 2    39   Input ~ 0
+SP1_M1
+Text GLabel 4250 6150 2    39   Input ~ 0
+SN2_M1
+Text GLabel 4250 6250 2    39   Input ~ 0
+SP2_M1
+Wire Wire Line
+	4250 6250 4200 6250
+Wire Wire Line
+	4200 6150 4250 6150
+Wire Wire Line
+	4200 6050 4250 6050
+Wire Wire Line
+	4200 5950 4250 5950
+Wire Wire Line
+	8200 7100 8100 7100
+Connection ~ 8200 7100
+Wire Wire Line
+	8200 6800 8100 6800
+Connection ~ 8200 6800
+Text GLabel 8100 6800 0    39   Input ~ 0
+SN2_M1
+Text GLabel 8100 7100 0    39   Input ~ 0
+SP2_M1
+Wire Wire Line
+	8200 3950 8100 3950
+Connection ~ 8200 3950
+Wire Wire Line
+	8200 3650 8100 3650
+Connection ~ 8200 3650
+Text GLabel 8100 3650 0    39   Input ~ 0
+SN1_M1
+Text GLabel 8100 3950 0    39   Input ~ 0
+SN2_M2
+Text GLabel 22050 5950 2    39   Input ~ 0
+SN1_M2
+Text GLabel 22050 6050 2    39   Input ~ 0
+SP1_M2
+Text GLabel 22050 6150 2    39   Input ~ 0
+SN2_M2
+Text GLabel 22050 6250 2    39   Input ~ 0
+SP2_M2
+Wire Wire Line
+	25900 3900 25800 3900
+Connection ~ 25900 3900
+Wire Wire Line
+	25900 3600 25800 3600
+Connection ~ 25900 3600
+Text GLabel 25800 3600 0    39   Input ~ 0
+SN1_M2
+Text GLabel 25800 3900 0    39   Input ~ 0
+SP1_M2
+Wire Wire Line
+	25900 7150 25800 7150
+Connection ~ 25900 7150
+Wire Wire Line
+	25900 6850 25800 6850
+Connection ~ 25900 6850
+Text GLabel 25800 6850 0    39   Input ~ 0
+SN2_M2
+Text GLabel 25800 7150 0    39   Input ~ 0
+SP2_M2
+Wire Wire Line
+	19300 6650 19350 6650
+Wire Wire Line
+	19350 6850 19350 6650
+Connection ~ 19350 6650
+Wire Wire Line
+	19350 6650 20950 6650
+Wire Wire Line
+	19950 6750 20950 6750
+Wire Wire Line
+	19950 6750 19950 6950
+Wire Wire Line
+	19850 6750 19950 6750
+Connection ~ 19950 6750
+Wire Wire Line
+	1500 6650 1550 6650
+Wire Wire Line
+	1550 6850 1550 6650
+Connection ~ 1550 6650
+Wire Wire Line
+	1550 6650 3100 6650
+Wire Wire Line
+	2050 6750 2100 6750
+Wire Wire Line
+	2100 6950 2100 6750
+Connection ~ 2100 6750
+Wire Wire Line
+	2100 6750 3100 6750
 $EndSCHEMATC

Commit message: Started draft of high level layout, fixed capacitor values in schematic
Parts:
- removed C11: 470u, Capacitors_THT:CP_Radial_D12.5mm_P5.00mm, symbol Device:CP1
- added C45: 470u, Capacitors_THT:CP_Radial_D12.5mm_P5.00mm, symbol Device:CP1
- added C47, C49: 0.1u, Capacitors_SMD:C_0603_HandSoldering, symbol Device:C
- added C48: 0.01u, Capacitors_SMD:C_0603_HandSoldering, symbol Device:C
- added R78: 3.3, Resistors_SMD:R_0603_HandSoldering, symbol Device:R
- added R79: 46.4k, Resistors_SMD:R_0603_HandSoldering, symbol Device:R
- added R80: 4.99k, Resistors_SMD:R_0603_HandSoldering, symbol Device:R
- added TP12: TEST, Wire_Pads:SolderWirePad_single_1mmDrill, symbol Connector:TestPoint
- C1, C10, C12, C13, C14, C15, C16, C17, C18, C19, C2, C20, C21, C22, C23, C24, C25, C26, C27, C28, C29, C3, C30, C31, C32, C33, C34, C35, C4, C40, C41, C42, C43, C44, C50, C51, C52, C53, C54, C55, C56, C57, C58, C59, C6, C60, C61, C62, C63, C64, C65, C66, C67, C68, C69, C70, C71, C72, C73, C74, C75, C76, C77, C8: footprint Capacitors_SMD:C_0805_HandSoldering -> Capacitors_SMD:C_0603_HandSoldering
- C36, C37, C38, C39, C5, C7: value 470u -> 220u; footprint Capacitors_THT:CP_Radial_D12.5mm_P5.00mm -> Capacitors_THT:CP_Radial_D10.0mm_P5.00mm
- Conn1: renamed from Conn?; footprint (none) -> MRDT_Connectors:MOLEX_SL_05_Horizontal
- Conn10, Conn11, Conn4, Conn5, Conn6, Conn9: renamed from Conn?; footprint (none) -> MRDT_Connectors:Anderson_1_Horisontal
- Conn2: renamed from Conn?; value PVDD_PP -> PVDD_M1_PP; footprint (none) -> MRDT_Connectors:Anderson_1_Horisontal
- Conn3: renamed from Conn?; value GND_PP -> GND_M1_PP; footprint (none) -> MRDT_Connectors:Anderson_1_Horisontal
- Conn7: renamed from Conn?; value PVDD_PP -> PVDD_M2_PP; footprint (none) -> MRDT_Connectors:Anderson_1_Horisontal
- Conn8: renamed from Conn?; value GND_PP -> GND_M2_PP; footprint (none) -> MRDT_Connectors:Anderson_1_Horisontal
- L1, L2: footprint MRDT_Passives.pretty:DR74_330_R -> MRDT_Passives:DR74_330_R
- Q12, Q13, Q14, Q15, Q16, Q17, Q4, Q5, Q6, Q7, Q8, Q9: footprint (none) -> MotorController_Hardware:TO-220-3_Horizontal_Reversed_NoHole
- R1, R11, R12, R14, R15, R16, R18, R19, R2, R20, R22, R23, R24, R25, R26, R27, R28, R29, R3, R30, R31, R32, R33, R34, R35, R38, R39, R4, R40, R41, R42, R43, R44, R45, R46, R47, R48, R49, R5, R50, R51, R52, R53, R54, R55, R56, R57, R58, R59, R6, R60, R61, R62, R63, R8: footprint (none) -> Resistors_SMD:R_0603_HandSoldering
- R10: value 1.7k -> 2k; footprint (none) -> Resistors_SMD:R_0603_HandSoldering
- R13, R17, R21, R36, R37, R64, R65, R66, R67, R68, R69, R7, R70, R71, R72, R73, R74, R75, R76, R77, R9: renamed from R?; footprint (none) -> Resistors_SMD:R_0603_HandSoldering
- TP1, TP10, TP11, TP20, TP21, TP22, TP23, TP24, TP25, TP26, TP27, TP28, TP29, TP3, TP4, TP5, TP6, TP7, TP8, TP9: footprint (none) -> Wire_Pads:SolderWirePad_single_1mmDrill
- TP2: renamed from TP?; value TestPoint -> TEST; footprint (none) -> Wire_Pads:SolderWirePad_single_1mmDrill
- U1, U5: renamed from U?; footprint (none) -> MRDT_ICs:DRV8301
- U2, U6: renamed from U?; footprint (none) -> MRDT_ICs:NUP4201MR6
- U3: renamed from U?; footprint (none) -> MotorController_Hardware:LAUNCHXL_F28069M_Launchpad_FULL_Booster_SMD_Bottom
- U4: renamed from U?; footprint (none) -> MRDT_ICs:SOIC_16_3.9x9.9mm_Pitch1.27mm
- gave numbers to parts that had none: 16
Connections:
- net labels added: PVDDSENSE_M1, PVDDSENSE_M2, PVDD_M1, PVDD_M2
- wire segments 725 -> 745
Other:
- note removed: "Double check with Jacob on\nif we need to double up on these\nor not"
