File: _saved_CameraBoard.sch (KiCad schematic (older format))
At the start: 32 parts, among them J1 BNC_75_OHM_HORIZ, J2 BNC_75_OHM_HORIZ, U1 TM4C129E_Launchpad, U2 AP1509-33SG-13, U3 MAX4314ESD+, U4 MAX4314ESD+

Commit message: Rev 1 Layout for first round board review
Parts:
- Conn1: renamed from Conn?; footprint (none) -> MRDT_Connectors:Anderson_1_Horisontal
Changed lines of the file:
@@
 +12V
 $Comp
-L MRDT_Connectors:AndersonPP Conn?
+L MRDT_Connectors:AndersonPP Conn1
 U 2 1 5C03B8AB
 P 3200 3000
-F 0 "Conn?" H 3000 3150 60  0000 C CNN
+F 0 "Conn1" H 3000 3150 60  0000 C CNN
 F 1 "AndersonPP_LOG" H 2800 3050 60  0000 C CNN
-F 2 "" H 3050 2450 60  0001 C CNN
+F 2 "MRDT_Connectors:Anderson_1_Horisontal" H 3050 2450 60  0001 C CNN
 F 3 "" H 3050 2450 60  0001 C CNN
 	2    3200 3000
