File: CameraBoard.sch (KiCad schematic (older format))
At the start: 32 parts, among them J1 BNC_75_OHM_HORIZ, J2 BNC_75_OHM_HORIZ, U1 TM4C129E_Launchpad, U2 AP1509-33SG-13, U3 MAX4314ESD+, U4 MAX4314ESD+

Commit message: Completed schematic changes from PDR, currently partway through layout changes. Uploading progress, details listed in the PDR Notes documentation with marks for each item completed
Parts:
- removed Conn2: AndersonPP_GND, MRDT_Connectors:Anderson_1_Horisontal, symbol MRDT_Connectors:AndersonPP
- removed L1: 47u, Inductors_SMD:L_0603_HandSoldering, symbol pspice:INDUCTOR
- removed U2: AP1509-33SG-13, AP150933SG13:AP1509-33SG-13, symbol AP150933SG13:AP1509-33SG-13
- added unit 1 of Conn1
- added D6: LED, LEDs:LED_0603_HandSoldering, symbol Device:LED
- added JP1, JP2: Jumper_NC_Dual, Pin_Headers:Pin_Header_Straight_1x03_Pitch2.54mm, symbol Device:Jumper_NC_Dual
- added L1: 47u, Inductors_SMD:L_0603_HandSoldering, symbol Device:L
- added R11, R13, R15: 500, Resistors_SMD:R_0603_HandSoldering, symbol Device:R
- added R12, R14: 100, Resistors_SMD:R_0603_HandSoldering, symbol Device:R
- added U2: AP1059, Housings_SOIC:HTSOP-8-1EP_3.9x4.9mm_Pitch1.27mm, symbol MRDT_ICs:AP1059
- C1: value 1u -> 10u
- Conn1: value AndersonPP_LOG -> AndersonPP; footprint MRDT_Connectors:Anderson_1_Horisontal -> MRDT_Connectors:Anderson_2_Horisontal_Side_by_Side
- D5: footprint Diodes_SMD:D_SOT-23_ANK -> Diodes_SMD:D_0603
Connections:
- net labels added: +5V, SW_ERR
- net labels removed: +3.3V
- wire segments 97 -> 117
