File: CameraBoard_Hardware.sch (KiCad schematic (older format))
At the start: 39 parts, among them J1 BNC_75_OHM_HORIZ, J2 BNC_75_OHM_HORIZ, U1 TM4C129E_Launchpad, U2 AP1059, U3 MAX4314ESD+, U4 MAX4314ESD+

Commit message: Finished changes discussed at PDR, added labels for jumpers and andersons
Parts:
- removed R14: 100, Resistors_SMD:R_0603_HandSoldering, symbol Device:R
- removed R15: 500, Resistors_SMD:R_0603_HandSoldering, symbol Device:R
- U1: footprint MRDT_Shields:TM4C129E_Launchpad_X9_SMD -> MRDT_Shields:TM4C129E_Launchpad_X9_THT
Connections:
- net labels added: +10V
- wire segments 117 -> 114
