File: 2018/PT_2018_PB_4lyr_Rev1.brd (EAGLE design)
At the start: 165.1 x 209.5 mm, 168 parts, among them J1 APP_2POS_CONFIG12V_VERT, J2 APP_2POS_CONFIG12V_VERT, J3 APP_2POS_CONFIG12V_VERT, J4 APP_2POS_CONFIG12V_VERT, Q1 Q_IRFS7437PbF, Q10 MOSFET-NCHANNELFDD8780, Q11 MOSFET-NCHANNELFDD8780, Q12 2N7002, Q13 2N7002PW, Q2 Q_IRFS7437PbF, Q3 Q_IRFS7437PbF, Q4 Q_IRFS7437PbF, Q5 Q_IRFS7437PbF, Q6 Q_IRFS7437PbF, Q7 Q_IRFS7437PbF, Q8 2N7002, Q9 2N7002, U1 LT1910, U10 ACS722LLCTR-40AU-T, U11 ACS722LLCTR-40AU-T, U12 ACS722LLCTR-40AU-T, U13 ACS722LLCTR-40AU-T, U14 ACS722LLCTR-40AU-T, U15 LT1910, U16 LT1910, U17 ACS722LLCTR-40AU-T, U18 ACS722LLCTR-40AU-T, U19 ACS722LLCTR-40AU-T, U2 LT1910, U20 ACS722LLCTR-40AU-T, U21 MAX3232D, U3 LT1910, U4 LT1910, U5 LT1910, U6 LT1910, U7 LT1910, U8 ACS722LLCTR-40AU-T, U9 ACS722LLCTR-40AU-T, X1 22-23-2021

Commit message: Integrated TIVA added, New Logic bus started
Parts:
- removed C.22: .1µF, SparkFun-Capacitors:0805
- removed C.32, C.33: 330µF, resistor:E5-8,5
- removed C.34: 2.2uF, SparkFun-Capacitors:1206
- removed C.38: 1nF, SparkFun-Capacitors:0805
- removed DORY-12V: UQW-12/20-T48NBS, MRDT-2015-PowerBoard:U-T48-QB-NO_TRIM
- removed J4: APP_2POS_CONFIG12V_VERT, MRDT-Connectors:APP45_12V_VERT_CONFIG
- removed LED-8: (no value), SparkFun-LED:LED-1206
- removed Q9: 2N7002, SparkFun-DiscreteSemi:SOT323
- removed R.20: 1k, resistor:R1206
- removed R.21: 100k, resistor:R1206
- removed R.8: 1kΩ, SparkFun-Passives:1206
- removed U$1: TIVA-C-CONNECTED, MRDT-2015-General:TIVA-C-CONNECTED
- removed U$14: ATC_FUSE_BLOCK, MRDT-Hardware:BLOCK_3557-2
- added C1, C10, C11, C12, C17, C2, C20, C21, C3, C4, C7, C8, C9: 0.1uF, resistor:C0603
- added C13: 1.0uF, resistor:C0603
- added C14, C22: 2.2uF, resistor:C0603
- added C15, C16, C18, C19: 12pF, resistor:C0603
- added C23, C24, C25, C26: 10uF, resistor:C1206
- added C27: 10pF, SparkFun-Capacitors:0603
- added C5: 1000pF, resistor:C0603
- added C6: 4700pF, resistor:C1206
- added J5: RJ45KEYSTONE-942, MRDT-Connectors:KEYSTONE-942
- added J6: JTAG_ARM_10PIN, MRDT-Connectors:CON_2X5_50MIL
- added J7: APP_2POS_CONFIG12V_HORIZ, MRDT-Connectors:APP45_12V_HORIZ_CONFIG
- added J8: APPPP45_PCB_HORIZ_RIGHT, MRDT-Connectors:APP45_PCB_HORIZ_RIGHT
- added LED1, LED2: GREEN, led:CHIP-LED0603
- added LED3: ORANGE, led:CHIP-LED0603
- added R1: 49.9, rcl:R0603
- added R10, R11, R19: 330, resistor:R0603
- added R12: 1M, resistor:R0603
- added R13: 51, resistor:R0603
- added R14: 4.87k 1%, resistor:R0603
- added R15: 2k, resistor:R0603
- added R16: 100, resistor:R0603
- added R17: 10k, resistor:R0603
- added R18: 100k, resistor:R0603
- added R2: 49.4, resistor:R0603
- added R3, R4: 49.9, resistor:R0603
- added R5, R6, R7, R8: 75, resistor:R0603
- added R9: 1M, resistor:R1206
- added S1: SWITCH_TACTILE, MRDT-UserInput:SWITCH_6MM_6MM_TE_CON_SMD
- added U$11, U$12, U$6: MOUNTING_HOLE#6, MRDT-Hardware:#6_SCREW
- added U$4: MRDT_LOGO, MRDT-Hardware:MRDT_LOGO
- added U22: TM4C1294NCPDT, MRDT-Microcontrollers:TQFP-128
- added U23: HX1198FNL, MRDT-ICs:HX1198FNL
- added U24: SLVU2.8-4, MRDT-ICs:SOIC8
- added U25, U27: OKI-78SR-5/1.5-W36HC, MRDT-ICs:OKI-78SR_HORIZ
- added U26: TPS73733DCQ, MRDT-ICs:SOT-223-6
- added Y1: NX3225GA, MRDT-Passives:NDK3.2X2.5
- added Y2: CRYATL_32K_SMD, MRDT-Passives:CRYSTAL_32K_SMD
- U17: value ACS722LLCTR-40AU-T -> LM2678S-3.3; device MRDT-2015-PowerBoard:SOIC8_ACS711 -> LM2678S-3.3:TO127P1435X457-8N
- moved Q13 746.0 mm to (384.8, -475.0)
- moved C.59 716.2 mm to (381.0, -473.7), turned to 0 degrees
- moved C.57 712.3 mm to (373.4, -473.7), turned to 0 degrees
- moved C.56 712.0 mm to (369.6, -473.7), turned to 0 degrees
- moved C.58 711.7 mm to (377.2, -473.7)
- moved X1 701.3 mm to (331.5, -449.6)
- moved Q12 696.3 mm to (396.2, -475.0), turned to 0 degrees
- moved C.55 696.0 mm to (365.8, -473.7), turned to 0 degrees
- moved C.48 693.2 mm to (354.3, -473.7), turned to 0 degrees
- moved U21 690.5 mm to (392.4, -448.3), turned to 0 degrees
- moved U$41 690.1 mm to (377.2, -453.4)
- moved C.42 690.0 mm to (342.9, -473.7), turned to 0 degrees
- moved Q8 687.2 mm to (388.6, -475.0), turned to 0 degrees
- moved C.49 687.0 mm to (358.1, -473.7), turned to 0 degrees
- moved C.43 683.9 mm to (346.7, -473.7), turned to 0 degrees
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Connections:
- removed net 12V-AUX-EXTRA: J4.VCC, R.8.1, U17.4
- removed net COM/LOGIC-CTL: R.15.2, U$1.PP2
- removed net EXTRA-CTL: R.20.2, U$1.PH3
- removed net IMEAS-EXTRA: U$1.PE3, U17.7
- removed net LOGIC-SIG: U$1.PH2, U15.4
- removed net N$10: C.38.1, U17.6
- removed net N$23: C.32.+, DORY-12V.8, U$14.IN_1, U$14.IN_2
- removed net N$27: Q9.1, R.20.1, R.21.1
- removed net N$46: LED-8.A, R.8.2
- new net !RESET: J6.P10, R16.2, S1.P$3, S1.P$4
- new net +12V_ACT: C25.1, J8.P$1, U27.1
- new net +12V_LOGIC: C23.1, J7.12V, U25.1
- new net +3V3: C1.1, C10.1, C11.1, C2.1, C22.1, C3.1, C4.1, C8.1, C9.1, J6.P1, LED3.A, R1.1, R12.2, R13.2, R17.1, R2.1, R3.1, R4.1, U22.P$101, U22.P$113, U22.P$122, U22.P$16, U22.P$26, U22.P$28, U22.P$39, U22.P$47, U22.P$51, U22.P$52, U22.P$69, U22.P$7, U22.P$79, U22.P$8, U22.P$9, U22.P$90, U23.P$2, U23.P$7, U26.2
- new net +5V_ACT: C26.1, U27.3
- new net +5V_LOGIC: C20.1, C24.1, R18.1, U25.3, U26.1
- new net ACT-SIG: U15.4, U22.P$31
- new net ACT/COM-CTL: R.15.2, U22.P$103
- new net EN0LED0: LED1.A, U22.P$42
- new net EN0LED1: LED2.A, U22.P$46
- new net EN0RXI_N: R4.2, U22.P$53, U23.P$8
- new net EN0RXI_P: R3.2, U22.P$54, U23.P$6
- new net EN0TXO_N: R2.2, U22.P$56, U23.P$3
- new net EN0TXO_P: R1.2, U22.P$57, U23.P$1
- new net N_$1: R5.2, U23.P$15
- new net N_$10: C7.1, R13.1, U22.P$68
- new net N_$11: J5.P$4, J5.P$5, R7.2
- new net N_$12: R12.1, U22.P$64
- new net N_$13: J5.P$1, J5.P$2, R8.2
- new net N_$14: C5.1, R5.1, R6.1, R7.1, R8.1
- new net N_$15: C5.2, C6.1, R9.2
- new net N_$16: C12.1, C13.1, C14.1, U22.P$115, U22.P$87
- new net N_$17: R15.2, U22.P$89
- new net N_$18: C16.1, U22.P$88, Y1.P$3
- new net N_$19: R14.2, U22.P$59
- new net N_$20: C17.1, R16.1, R17.2, U22.P$70
- new net N_$21: C15.1, R15.1, Y1.P$1
- new net N_$22: C18.1, U22.P$67, Y2.P$2
- new net N_$23: C19.1, U22.P$66, Y2.P$1
- new net N_$25: R18.2, U26.5
- new net N_$26: LED3.C, R19.1
- new net N_$27: C21.1, U26.4
- new net N_$3: R6.2, U23.P$10
- new net N_$4: J5.P$7, U23.P$14, U24.2, U24.7
- new net N_$5: J5.P$6, U23.P$11, U24.3, U24.6
- new net N_$6: J5.P$8, U23.P$16, U24.1, U24.8
- new net N_$7: J5.P$3, U23.P$9, U24.4, U24.5
- new net N_$8: LED2.C, R11.1
- new net N_$9: LED1.C, R10.1
- new net RX: J6.P7, U22.P$33
- new net TARGET_TCK/SWCLK: J6.P4, U22.P$100
- new net TARGET_TDI: J6.P8, U22.P$98
- new net TARGET_TDO/SWO: J6.P6, U22.P$97
- new net TARGET_TMS/SWDIO: J6.P2, U22.P$99
- new net TX: J6.P9, U22.P$34
- net 3.3V: no longer C.22.2, U$1.+3V3_1, U$1.+3V3_2, U17.8
- net 5V: no longer U$1.+5V_1, U$1.+5V_2
- net ACT-CTL: now also U22.P$109; no longer U$1.PN2
- net COM-SIG: now also U22.P$81; no longer U$1.PL0
- net FAN_CTL_1: now also U22.P$3; no longer U$1.PD2
- net GND: now also C1.2, C10.2, C11.2, C12.2, C13.2, C14.2, C15.2, C16.2, C17.2, C18.2, C19.2, C2.2, C20.2, C21.2, C22.2, C23.2, C24.2, C25.2, C26.2, C3.2, C4.2, C6.2, C7.2, C8.2, C9.2, J6.P3, J6.P5, J7.GND, R10.2, R11.2, R14.1, R19.2, R9.1, S1.P$1, S1.P$2, U17.8, U22.P$10, U22.P$114, U22.P$17, U22.P$48, U22.P$55, U22.P$58, U22.P$80, U25.2, U26.3, U26.6, U27.2; no longer C.22.1, C.32.-, C.33.-, C.34.2, C.38.2, DORY-12V.3, DORY-12V.4, J4.GND, LED-8.C, Q9.2, R.21.2, U$1.GND_1, U$1.GND_2, U$1.GND_3, U$1.GND_4, U17.5
- net IMEAS-ACT: now also U20.7, U22.P$13; no longer U$1.PE2, U18.7
- net IMEAS-COM: now also U22.P$15; no longer U$1.PE0
- net IMEAS-LOGIC: now also U18.7, U22.P$14; no longer U$1.PE1, U20.7
- net IMEAS-M1: now also U22.P$21; no longer U$1.PK3
- net IMEAS-M2: now also U22.P$20; no longer U$1.PK2
- net IMEAS-M3: now also U22.P$19; no longer U$1.PK1
- net IMEAS-M4: now also U22.P$125; no longer U$1.PD4
- net IMEAS-M5: now also U22.P$18; no longer U$1.PK0
- net IMEAS-M6: now also U22.P$120; no longer U$1.PB5
- net IMEAS-M7: now also U22.P$121; no longer U$1.PB4
- net N$2: now also C27.2, U17.3; no longer C.33.+, C.34.1, U$14.OUT_1, U$14.OUT_2, U17.1
- net N$5: now also C27.1, U17.1; no longer DORY-12V.2, Q9.3
- net SER_RX: now also U22.P$25; no longer U$1.PC4
- net SER_TX: now also U22.P$24; no longer U$1.PC5
- net SIG-M1: now also U22.P$106; no longer U$1.PP5
- net SIG-M2: now also U22.P$41; no longer U$1.PA7
- net SIG-M3: now also U22.P$29; no longer U$1.PH0
- net SIG-M4: now also U22.P$104; no longer U$1.PP3
- net SIG-M5: now also U22.P$30; no longer U$1.PH1
- net SIG-M6: now also U22.P$61; no longer U$1.PK6
- net SIG-M7: now also U22.P$60; no longer U$1.PK7
- net VMEAS-VBATT: now also U22.P$124; no longer U$1.PE5
- net V_BATT: now also U17.2; no longer DORY-12V.1
Routing:
- net GND: track 338.5 -> 0.00 mm, vias 46 -> 0
- net IMEAS-M1: track 216.4 -> 0.00 mm, vias 1 -> 0
- net IMEAS-M2: track 199.9 -> 0.00 mm, vias 1 -> 0
- net IMEAS-EXTRA: track 198.2 -> 0.00 mm, vias 1 -> 0
- net IMEAS-M3: track 183.0 -> 0.00 mm, vias 1 -> 0
- net 5V: track 177.5 -> 0.00 mm
- net IMEAS-M4: track 168.6 -> 0.00 mm, vias 1 -> 0
- net SIG-M1: track 161.3 -> 0.00 mm, vias 1 -> 0
- net IMEAS-ACT: track 156.5 -> 0.00 mm, vias 1 -> 0
- net IMEAS-M5: track 148.0 -> 0.00 mm, vias 1 -> 0
- net SIG-M2: track 141.9 -> 0.00 mm, vias 1 -> 0
- net 232_RX: track 141.1 -> 0.00 mm
- net 232_TX: track 136.6 -> 0.00 mm
- net IMEAS-M6: track 131.0 -> 0.00 mm, vias 1 -> 0
- net N$5: track 129.8 -> 0.00 mm, vias 1 -> 0
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- removed copper zone on layer 1, net 12V-AUX-ACT
- removed copper zone on layer 1, net 12V-AUX-COM
- removed copper zone on layer 1, net 12V-AUX-EXTRA
- removed copper zone on layer 1, net 12V-AUX-LOGIC
- removed copper zone on layer 1, net 3.3V
- removed copper zone on layer 2, net 3.3V
- removed copper zone on layer 1, net 5V
- removed copper zone on layer 2, net 5V
- removed copper zone on layer 1, net DRAIN-M1
- removed copper zone on layer 1, net DRAIN-M2
- removed copper zone on layer 1, net DRAIN-M3
- removed copper zone on layer 1, net DRAIN-M4
- removed copper zone on layer 1, net DRAIN-M5
- removed copper zone on layer 1, net DRAIN-M6
- removed copper zone on layer 1, net DRAIN-M7
- removed copper zone on layer 1, net GND
- removed copper zone on layer 16, net GND
- removed copper zone on layer 1, net N$1
- removed copper zone on layer 1, net N$18
- removed copper zone on layer 1, net N$19
- removed copper zone on layer 1, net N$2
- removed copper zone on layer 1, net N$20
- removed copper zone on layer 1, net N$21
- removed copper zone on layer 1, net N$22
- removed copper zone on layer 1, net N$23
- removed copper zone on layer 1, net N$9
- removed copper zone on layer 1, net SOURCE-M1
- removed copper zone on layer 1, net SOURCE-M2
- removed copper zone on layer 1, net SOURCE-M3
- removed copper zone on layer 1, net SOURCE-M4
- removed copper zone on layer 1, net SOURCE-M5
- removed copper zone on layer 1, net SOURCE-M6
- removed copper zone on layer 1, net SOURCE-M7
- removed copper zone on layer 1, net V_BATT
- removed copper zone on layer 2, net V_BATT
- removed copper zone on layer 1, net V_BATT_M1
- removed copper zone on layer 1, net V_BATT_M2
- removed copper zone on layer 1, net V_BATT_M3
- removed copper zone on layer 1, net V_BATT_M4
- removed copper zone on layer 1, net V_BATT_M5
- removed copper zone on layer 1, net V_BATT_M6
- removed copper zone on layer 1, net V_BATT_M7
Other:
- board size 165.1 x 209.5 mm -> 165.1 x 215.9 mm
- board text removed: "#R VE SOHARD"
- board text removed: "+"
- board text removed: "-"
- board text removed: "15A"
- board text removed: "3.3V-OKI"
- board text removed: "30A"
- board text removed: "5A"
- board text removed: "5V"
- board text removed: "5V-OKI"
- board text removed: "ACTUATION"
- board text removed: "C1"
- board text removed: "C10"
- board text removed: "C11"
- board text removed: "C12"
- board text removed: "C13"
- board text removed: "C14"
- board text removed: "C15"
- board text removed: "C16"
- board text removed: "C17"
- board text removed: "C18"
- board text removed: "C19"
- board text removed: "C2"
- board text removed: "C20"
- board text removed: "C21"
- board text removed: "C22"
- board text removed: "C23"
- board text removed: "C24"
- board text removed: "C25"
- board text removed: "C26"
- board text removed: "C27"
- board text removed: "C28"
- board text removed: "C29"
- board text removed: "C3"
- board text removed: "C30"
- board text removed: "C31"
- board text removed: "C32"
- board text removed: "C33"
- board text removed: "C34"
- board text removed: "C35"
- board text removed: "C36"
- board text removed: "C37"
- board text removed: "C38"
- board text removed: "C39"
- board text removed: "C4"
- board text removed: "C40"
- board text removed: "C41"
- board text removed: "C42"
- board text removed: "C43"
- board text removed: "C44"
- board text removed: "C45"
- board text removed: "C46"
- board text removed: "C47"
- board text removed: "C48"
- board text removed: "C49"
- board text removed: "C5"
- board text removed: "C50"
- board text removed: "C51"
- board text removed: "C52"
- board text removed: "C53"
- board text removed: "C54"
- board text removed: "C55"
- board text removed: "C56"
- board text removed: "C57"
- board text removed: "C58"
- board text removed: "C59"
- board text removed: "C6"
- board text removed: "C7"
- board text removed: "C8"
- board text removed: "C9"
- board text removed: "COM"
- board text removed: "D1"
- board text removed: "D2"
- board text removed: "EXTRA-12V"
- board text removed: "FAN_5V"
- board text removed: "FUSE_BLOCK"
- board text removed: "LED1"
- board text removed: "LED10"
- board text removed: "LED11"
- board text removed: "LED2"
- board text removed: "LED3"
- board text removed: "LED4"
- board text removed: "LED5"
- board text removed: "LED6"
- board text removed: "LED7"
- board text removed: "LED8"
- board text removed: "LED9"
- board text removed: "LOGIC"
- board text removed: "M1"
- board text removed: "M2"
- board text removed: "M3"
- board text removed: "M4"
- board text removed: "M5"
- board text removed: "M6"
- board text removed: "M7"
- board text removed: "Missouri S&T Mars Rover Design Team Power Board 2017 Rev2 Jacob Lipina"
- board text removed: "Q1"
- board text removed: "Q10"
- board text removed: "Q11"
- board text removed: "Q12"
- board text removed: "Q13"
- board text removed: "Q2"
- board text removed: "Q3"
- board text removed: "Q4"
- board text removed: "Q5"
- board text removed: "Q6"
- board text removed: "Q7"
- board text removed: "Q8"
- board text removed: "Q9"
- board text removed: "R1"
- board text removed: "R10"
- board text removed: "R11"
- board text removed: "R14"
- board text removed: "R15"
- board text removed: "R16"
- board text removed: "R17"
- board text removed: "R18"
- board text removed: "R19"
- board text removed: "R2"
- board text removed: "R20"
- board text removed: "R21"
- board text removed: "R3"
- board text removed: "R4"
- board text removed: "R5"
- board text removed: "R6"
- board text removed: "R7"
- board text removed: "R8"
- board text removed: "R9"
- board text removed: "U1"
- board text removed: "U10"
- board text removed: "U11"
- board text removed: "U12"
- board text removed: "U13"
- board text removed: "U14"
- board text removed: "U15"
- board text removed: "U16"
- board text removed: "U17"
- board text removed: "U18"
- board text removed: "U19"
- board text removed: "U2"
- board text removed: "U20"
- board text removed: "U21"
- board text removed: "U3"
- board text removed: "U4"
- board text removed: "U5"
- board text removed: "U6"
- board text removed: "U7"
- board text removed: "U8"
- board text removed: "U9"
- board text removed: "X1"
- board text removed: "|"
