File: PowerBoardHardware/PT_2018_PB_4lyr_Rev1.brd (EAGLE design)
At the start: 165.1 x 215.9 mm, 220 parts, among them J1 APP_2POS_CONFIG12V_VERT, J2 APP_2POS_CONFIG12V_VERT, J3 APP_2POS_CONFIG12V_VERT, J5 RJ45KEYSTONE-942, J6 JTAG_ARM_10PIN, J7 APP_2POS_CONFIG12V_HORIZ, J8 APPPP45_PCB_HORIZ_RIGHT, Q1 Q_IRFS7437PbF, Q10 MOSFET-NCHANNELFDD8780, Q11 MOSFET-NCHANNELFDD8780, Q12 2N7002, Q13 2N7002PW, Q2 Q_IRFS7437PbF, Q3 Q_IRFS7437PbF, Q4 Q_IRFS7437PbF, Q5 Q_IRFS7437PbF, Q6 Q_IRFS7437PbF, Q7 Q_IRFS7437PbF, Q8 2N7002, U1 LT1910, U10 ACS722LLCTR-40AU-T, U11 ACS722LLCTR-40AU-T, U12 ACS722LLCTR-40AU-T, U13 ACS722LLCTR-40AU-T, U14 ACS722LLCTR-40AU-T, U15 LT1910, U16 LT1910, U17 LM2678S-3.3, U18 ACS722LLCTR-40AU-T, U19 ACS722LLCTR-40AU-T, U2 LT1910, U20 ACS722LLCTR-40AU-T, U21 MAX3232D, U22 TM4C1294NCPDT, U23 HX1198FNL, U24 SLVU2.8-4, U25 OKI-78SR-5/1.5-W36HC, U26 TPS73733DCQ, U27 OKI-78SR-5/1.5-W36HC, U3 LT1910, U4 LT1910, U5 LT1910, U6 LT1910, U7 LT1910, U8 ACS722LLCTR-40AU-T, U9 ACS722LLCTR-40AU-T, X1 22-23-2021, Y1 NX3225GA, Y2 CRYATL_32K_SMD

Commit message: Midway push
Motor buses copied from last year, actuation bus copied, com/logic bus oriented to not take up as much room in +y direction to allow patch panel to be shorter and make room for buck converter board.  Tiva pins rearranged for more convenient trace paths
Parts:
- removed C20, C21: 0.1uF, resistor:C0603
- removed C22: 2.2uF, resistor:C0603
- removed C23, C24, C25, C26: 10uF, resistor:C1206
- removed C27: 10pF, SparkFun-Capacitors:0603
- removed J7: APP_2POS_CONFIG12V_HORIZ, MRDT-Connectors:APP45_12V_HORIZ_CONFIG
- removed J8: APPPP45_PCB_HORIZ_RIGHT, MRDT-Connectors:APP45_PCB_HORIZ_RIGHT
- removed R18: 100k, resistor:R0603
- removed U17: LM2678S-3.3, LM2678S-3.3:TO127P1435X457-8N
- removed U25, U27: OKI-78SR-5/1.5-W36HC, MRDT-ICs:OKI-78SR_HORIZ
- removed U26: TPS73733DCQ, MRDT-ICs:SOT-223-6
- added 3.3V-OKI1: Q_OKI-78SR, MRDT-2015-PowerBoard:OKI-78SR_HORIZ
- added C28: 22p, SparkFun-Passives:0603-CAP
- added C29: 22u, buckconverter:CAP_POL_22UF
- added CB: 0.1u, SparkFun-Passives:0603-CAP
- added CC1: 470p, SparkFun-Passives:0603-CAP
- added CC2, CIN2: 1000p, SparkFun-Passives:0603-CAP
- added CC3: 2200p, SparkFun-Passives:0603-CAP
- added CDRVCC: 10u, SparkFun-Passives:0603-CAP
- added CIN1: 100u, buckconverter:CAP_POL_220UF
- added COUT1, COUT2: 220u, buckconverter:CAP_POL_220UF
- added CSS: 0.1uF, SparkFun-Passives:0603-CAP
- added CVCC: 1uF, SparkFun-Passives:0603-CAP
- added D3: RBR3MM30ATR, buckconverter:DIODE_SCHOTTKY_30V_1A
- added DB: RF05VAM1STR, buckconverter:DIODE_STANDARD_100V
- added J4: APP_2POS_CONFIGMOCO_VERT, MRDT-Connectors:APP45_MOCO_VERT_CONFIG
- added L1: 3.3uH, buckconverter:PLANAR_INDUCTOR_3.3UH
- added LOGO1: MRDT_LOGO, MRDT-Hardware:MRDT_LOGO
- added R20: 113k, SparkFun-Passives:0603-RES
- added R21: 8.06k, SparkFun-Passives:0603-RES
- added RC1, RC2: 10k, SparkFun-Passives:0603-RES
- added RF: 10, SparkFun-Passives:0603-RES
- added RMAX: 16.5k, SparkFun-Passives:0603-RES
- added RSET: 19.1k, SparkFun-Passives:0603-RES
- added U$1: LTC3703-5, MRDT-ICs:SSOP-16
- added U$13, U$14: IPP052N06L3GXKSA1, buckconverter:TO-220
- added U$17, U$18: 530002B02500G, buckconverter:RADIAL_FIN_HEATSINK
- moved Q8 855.5 mm to (-24.1, 274.3), turned to 90 degrees
- moved Q13 850.3 mm to (-24.1, 270.5), turned to 90 degrees
- moved C.59 844.6 mm to (-25.4, 266.7), turned to 90 degrees
- moved C.58 839.4 mm to (-25.4, 262.9), turned to 90 degrees
- moved C.57 834.3 mm to (-25.4, 259.1), turned to 90 degrees
- moved C.56 829.1 mm to (-25.4, 255.3), turned to 90 degrees
- moved C.55 823.9 mm to (-25.4, 251.5), turned to 90 degrees
- moved C.50 818.8 mm to (-25.4, 247.7), turned to 90 degrees
- moved C.49 813.6 mm to (-25.4, 243.8), turned to 90 degrees
- moved C.48 808.5 mm to (-25.4, 240.0), turned to 90 degrees
- moved C.44 803.3 mm to (-25.4, 236.2), turned to 90 degrees
- moved C.43 798.2 mm to (-25.4, 232.4), turned to 90 degrees
- moved C.42 793.0 mm to (-25.4, 228.6), turned to 90 degrees
- moved C11 758.7 mm to (5.08, 180.3), turned to 90 degrees
- moved C10 753.4 mm to (7.62, 180.3), turned to 90 degrees
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Connections:
- removed net +12V_ACT: C25.1, J8.P$1, U27.1
- removed net +12V_LOGIC: C23.1, J7.12V, U25.1
- removed net +5V_ACT: C26.1, U27.3
- removed net +5V_LOGIC: C20.1, C24.1, R18.1, U25.3, U26.1
- removed net ACT-SIG: U15.4, U22.P$31
- removed net ACT/COM-CTL: R.15.2, U22.P$103
- removed net N$2: C27.2, U17.3
- removed net N$5: C27.1, U17.1
- removed net N_$25: R18.2, U26.5
- removed net N_$27: C21.1, U26.4
- new net LOGIC-SIG: U15.4, U22.P$120
- new net LOGIC/COM-CTL: R.15.2, U22.P$112
- new net N$10: RMAX.2, U$1.5
- new net N$14: CSS.1, U$1.7
- new net N$23: CC1.1, RC1.2, U$1.3
- new net N$24: CC2.1, RC1.1
- new net N$26: CC3.1, RC2.1
- new net N$27: CC1.2, CC2.2, R20.2, R21.1, RC2.2, U$1.4
- new net N$29: CVCC.1, RF.1, U$1.12
- new net N$30: U$1.10, U$14.1
- new net N$31: CB.2, D3.P$2, L1.P$2, U$1.13, U$13.3, U$14.2
- new net N$32: CB.1, DB.P$1, U$1.15
- new net N$33: U$1.14, U$13.1
- new net N$34: RSET.2, U$1.2
- new net VOUT12+: C28.1, CC3.2, COUT1.+, COUT2.+, J4.GND, L1.P$1, R20.1
- net +3V3: now also 3.3V-OKI1.3; no longer C22.1, U26.2
- net 5V: now also C29.+, CDRVCC.1, DB.P$2, RF.2, U$1.1, U$1.11
- net COM-SIG: now also U22.P$118; no longer U22.P$81
- net GND: now also 3.3V-OKI1.2, C28.2, C29.-, CDRVCC.2, CIN1.GND, CIN2.2, COUT1.GND, COUT2.GND, CSS.2, CVCC.2, D3.P$1, J4.VCC, R21.2, RMAX.1, RSET.1, U$1.6, U$1.8, U$1.9, U$14.3; no longer C20.2, C21.2, C22.2, C23.2, C24.2, C25.2, C26.2, J7.GND, U17.8, U25.2, U26.3, U26.6, U27.2
- net IMEAS-ACT: now also U18.7, U22.P$107; no longer U20.7, U22.P$13
- net IMEAS-COM: now also U22.P$119; no longer U22.P$15
- net IMEAS-LOGIC: now also U20.7, U22.P$121; no longer U18.7, U22.P$14
- net IMEAS-M1: now also U22.P$71; no longer U22.P$21
- net IMEAS-M2: now also U22.P$72; no longer U22.P$20
- net IMEAS-M3: now also U22.P$73; no longer U22.P$19
- net IMEAS-M4: now also U22.P$74; no longer U22.P$125
- net IMEAS-M5: now also U22.P$75; no longer U22.P$18
- net IMEAS-M6: now also U22.P$76; no longer U22.P$120
- net IMEAS-M7: now also U22.P$77; no longer U22.P$121
- net SIG-M1: now also U22.P$94; no longer U22.P$106
- net SIG-M2: now also U22.P$86; no longer U22.P$41
- net SIG-M3: now also U22.P$85; no longer U22.P$29
- net SIG-M4: now also U22.P$84; no longer U22.P$104
- net SIG-M5: now also U22.P$83; no longer U22.P$30
- net SIG-M6: now also U22.P$82; no longer U22.P$61
- net SIG-M7: now also U22.P$81; no longer U22.P$60
- net V_BATT: now also 3.3V-OKI1.1, CIN1.+, CIN2.1, U$1.16, U$13.2; no longer U17.2
Routing:
- net GND: track 0.00 -> 98.6 mm, vias 0 -> 50
- net N_$15: track 0.00 -> 35.4 mm, vias 0 -> 2
- net 3.3V: track 0.00 -> 32.9 mm, vias 0 -> 7
- net N_$13: track 0.00 -> 24.5 mm
- net N_$3: track 0.00 -> 22.3 mm, vias 0 -> 2
- net N_$11: track 0.00 -> 22.3 mm
- net N_$7: track 0.00 -> 19.3 mm
- net DRAIN-M1: track 0.00 -> 18.1 mm
- net N_$4: track 0.00 -> 16.6 mm
- net N_$5: track 0.00 -> 16.0 mm
- net DRAIN-M7: track 0.00 -> 15.8 mm
- net DRAIN-M3: track 0.00 -> 15.7 mm
- net DRAIN-M2: track 0.00 -> 15.6 mm
- net DRAIN-M6: track 0.00 -> 15.2 mm
- net DRAIN-M5: track 0.00 -> 15.2 mm
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- added copper zone on layer 1, net +3V3
- added copper zone on layer 1, net 12V-AUX-ACT
- added copper zone on layer 2, net 3.3V
- added copper zone on layer 1, net DRAIN-M1
- added copper zone on layer 1, net DRAIN-M2
- added copper zone on layer 1, net DRAIN-M3
- added copper zone on layer 1, net DRAIN-M4
- added copper zone on layer 1, net DRAIN-M5
- added copper zone on layer 1, net DRAIN-M6
- added copper zone on layer 1, net DRAIN-M7
- added copper zone on layer 16, net GND
- added copper zone on layer 1, net N$1
- added copper zone on layer 1, net N$18
- added copper zone on layer 1, net SOURCE-M1
- added copper zone on layer 1, net SOURCE-M2
- added copper zone on layer 1, net SOURCE-M3
- added copper zone on layer 1, net SOURCE-M4
- added copper zone on layer 1, net SOURCE-M5
- added copper zone on layer 1, net SOURCE-M6
- added copper zone on layer 1, net SOURCE-M7
- added copper zone on layer 1, net V_BATT
- added copper zone on layer 2, net V_BATT
- added copper zone on layer 1, net V_BATT_M1
- added copper zone on layer 1, net V_BATT_M2
- added copper zone on layer 1, net V_BATT_M3
- added copper zone on layer 1, net V_BATT_M4
- added copper zone on layer 1, net V_BATT_M5
- added copper zone on layer 1, net V_BATT_M6
- added copper zone on layer 1, net V_BATT_M7
Other:
- board size 165.1 x 215.9 mm -> 177.8 x 209.6 mm

Commit message: Custom buck converter finished
Left to do: via stitch buck converter, route rest of tiva signals, place rs232 comm unit
Parts:
- added C.22, C.32: .1µF, SparkFun-Capacitors:0805
- added LED-8: (no value), SparkFun-LED:LED-1206
- added Q9: Q_IRFS7437PbF, MRDT-2015-PowerBoard:D2PACK
- added R.8: 1kΩ, SparkFun-Passives:1206
- added U$21: MLX91210, buckconverter:SOIC8_ACS711
- added U17: LT1910, Jake:SO8
- moved U21 474.2 mm to (52.8, 195.6), turned to 180 degrees
- moved C.46 470.9 mm to (35.6, 249.9)
- moved X1 464.6 mm to (49.5, 250.4)
- moved TEMP_1 440.8 mm to (68.6, 256.5)
- moved C.50 276.4 mm to (109.5, 6.35), turned to 0 degrees
- moved C.44 268.1 mm to (109.5, 4.57), turned to 0 degrees
- moved U$13 237.6 mm to (138.7, 170.9), turned to 90 degrees
- moved RSET 212.2 mm to (167.1, 129.5)
- moved RC2 205.8 mm to (155.7, 133.1)
- moved RMAX 204.4 mm to (170.7, 128.5), turned to 90 degrees
- moved C.47 202.6 mm to (109.5, 8.38), turned to 0 degrees
- moved C28 201.1 mm to (79.8, 173.9), turned to 180 degrees
- moved RC1 196.0 mm to (161.0, 133.1), turned to 180 degrees
- moved RF 193.7 mm to (171.2, 140.7)
- moved L1 193.4 mm to (85.3, 185.4)
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Connections:
- removed net RX: J6.P7, U22.P$33
- removed net TX: J6.P9, U22.P$34
- new net ARM-BUS: J4.VCC, R.8.1, U$21.4
- new net IMEAS-ARM: U$21.7, U22.P$128
- new net N$2: LED-8.A, R.8.2
- new net N$36: Q9.1, U17.5
- new net SIG-ARM: U17.4, U22.P$127
- new net SOURCE-ARM: CIN1.+, CIN2.1, Q9.2, U$1.16, U$13.2
- net 5V: now also C.32.2, U$21.8
- net GND: now also C.22.1, C.32.1, J4.GND, LED-8.C, U$21.5, U$21.6, U17.1; no longer J4.VCC
- net SER_RX: now also J6.P7
- net SER_TX: now also J6.P9
- net VOUT12+: now also U$21.1; no longer J4.GND
- net V_BATT: now also C.22.2, Q9.TAB, U17.6, U17.8; no longer CIN1.+, CIN2.1, U$1.16, U$13.2
Routing:
- net IMEAS-M1: track 0.00 -> 189.2 mm, vias 0 -> 2
- net SIG-M1: track 0.00 -> 177.0 mm, vias 0 -> 2
- net IMEAS-M2: track 0.00 -> 174.6 mm, vias 0 -> 2
- net IMEAS-M3: track 0.00 -> 156.7 mm, vias 0 -> 2
- net SIG-M2: track 0.00 -> 156.5 mm, vias 0 -> 2
- net IMEAS-M4: track 0.00 -> 138.9 mm, vias 0 -> 2
- net SIG-M3: track 0.00 -> 137.2 mm, vias 0 -> 2
- net 5V: track 0.00 -> 128.8 mm, vias 0 -> 5
- net IMEAS-M5: track 0.00 -> 121.7 mm, vias 0 -> 2
- net SIG-M4: track 0.00 -> 117.7 mm, vias 0 -> 2
- net IMEAS-M6: track 0.00 -> 104.6 mm, vias 0 -> 2
- net SIG-M5: track 0.00 -> 98.3 mm, vias 0 -> 2
- net IMEAS-M7: track 0.00 -> 86.3 mm, vias 0 -> 2
- net SIG-M6: track 0.00 -> 80.5 mm, vias 0 -> 2
- net VOUT12+: track 0.00 -> 77.9 mm, vias 0 -> 2
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- added copper zone on layer 1, net 12V-AUX-COM
- added copper zone on layer 1, net 12V-AUX-LOGIC
- added copper zone on layer 1, net ARM-BUS
- added copper zone on layer 16, net ARM-BUS
- added copper zone on layer 1, net GND
- added copper zone on layer 1, net N$19
- added copper zone on layer 1, net N$20
- added copper zone on layer 1, net N$21
- added copper zone on layer 1, net N$22
- added copper zone on layer 1, net N$31
- added copper zone on layer 16, net N$31
- added copper zone on layer 1, net N$9
- added copper zone on layer 1, net SOURCE-ARM
- added copper zone on layer 16, net SOURCE-ARM
- added copper zone on layer 1, net VOUT12+
- added copper zone on layer 16, net VOUT12+
- removed copper zone on layer 2, net V_BATT

Commit message: REV 1 COMPLETE
Signal traces sloppy, probably should be redone.  Labeling, silkscreen etc still needs to be done.
Parts:
- added C.33: 1nF, SparkFun-Capacitors:0805
- added C.34: 10uF, SparkFun-Capacitors:1206
- added C.38: .1uF, SparkFun-Capacitors:0805
- moved U$4 400.2 mm to (124.5, 195.8)
- moved U$12 309.5 mm to (4.57, 205.2)
- moved U$35 308.2 mm to (80.8, 205.5)
- moved U$16 281.9 mm to (173.2, 205.2)
- moved C.48 188.6 mm to (131.8, 135.9)
- moved C.42 184.5 mm to (134.1, 135.9)
- moved Q8 170.5 mm to (83.3, 142.0), turned to 270 degrees
- moved C.45 164.9 mm to (129.3, 135.9)
- moved C.49 160.4 mm to (92.7, 135.4)
- moved C.43 151.1 mm to (90.4, 135.4)
- moved R.17 135.3 mm to (49.0, 129.8)
- moved R.16 129.3 mm to (51.6, 129.8), turned to 270 degrees
- moved C.46 126.0 mm to (88.1, 135.4), turned to 90 degrees
- moved U$10 118.6 mm to (172.2, 4.32)
- moved U$34 117.5 mm to (96.5, 4.83)
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Connections:
- net +3V3: now also C.33.1, C.34.1, C.38.1
- net GND: now also C.33.2, C.34.2, C.38.2
Routing:
- net IMEAS-ACT: track 0.00 -> 286.5 mm, vias 0 -> 2
- net IMEAS-LOGIC: track 0.00 -> 247.4 mm, vias 0 -> 2
- net LOGIC-SIG: track 0.00 -> 220.7 mm, vias 0 -> 2
- net COM-SIG: track 0.00 -> 196.9 mm, vias 0 -> 2
- net IMEAS-COM: track 0.00 -> 187.7 mm, vias 0 -> 2
- net SIG-ARM: track 0.00 -> 133.4 mm, vias 0 -> 2
- net IMEAS-ARM: track 0.00 -> 109.0 mm, vias 0 -> 2
- net 5V: track 128.8 -> 235.9 mm, vias 5 -> 6
- net N$8: track 0.00 -> 102.9 mm, vias 0 -> 1
- net LOGIC/COM-CTL: track 0.00 -> 98.7 mm, vias 0 -> 2
- net GND: track 160.1 -> 249.6 mm, vias 67 -> 114
- net ACT-CTL: track 0.00 -> 86.3 mm, vias 0 -> 2
- net !RESET: track 0.00 -> 82.4 mm, vias 0 -> 4
- net VMEAS-VBATT: track 0.00 -> 82.1 mm, vias 0 -> 2
- net N$3: track 0.00 -> 63.2 mm, vias 0 -> 1
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- added copper zone on layer 1, net 3.3V
- added copper zone on layer 1, net 5V

Commit message: Small tweaks
Rearranged logic bus components to line anderson up with the other buses.  Ethernet  jack rotated.  Mounting holes lined up, corners rounded.  Patch panel mounting holes added
Parts:
- removed X1: 22-23-2021, con-molex:22-23-2021
- added C.60: 10n, SparkFun-Capacitors:0805
- added J7: SL02, MRDT-Connectors:MOLEX-70543-0001
- added RC3: 10k, SparkFun-Passives:0603-RES
- moved U$5 283.1 mm to (171.2, 110.5)
- moved U$35 218.0 mm to (166.6, 5.08)
- moved U$11 197.9 mm to (98.6, 110.5)
- moved U$31 45.9 mm to (132.3, 106.9), turned to 0 degrees
- moved LED-11 31.4 mm to (169.9, 117.3), turned to 180 degrees
- moved R.11 28.4 mm to (169.9, 120.1), turned to 0 degrees
- moved Q11 27.2 mm to (136.7, 115.8), turned to 90 degrees
- moved C.22 19.7 mm to (97.3, 133.3), turned to 180 degrees
- moved C.40 19.4 mm to (161.3, 124.2), turned to 0 degrees
- moved U16 18.8 mm to (145.0, 109.7), turned to 90 degrees
- moved C.25 17.3 mm to (157.0, 124.2), turned to 0 degrees
- moved J2 16.7 mm to (149.9, 115.3)
- moved U19 9.76 mm to (159.8, 119.4), turned to 0 degrees
- moved J5 9.48 mm to (7.11, 144.8), turned to 270 degrees
- moved C.37 6.67 mm to (153.7, 99.6), turned to 270 degrees
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Connections:
- removed net N$66: Q13.3, X1.1
- new net N$5: J7.1, Q13.3
- net 5V: now also J7.2; no longer X1.2
- net GND: now also C.60.2, RC3.1
- net IMEAS-ARM: now also C.60.1, RC3.2
Routing:
- net N$17: track 17.0 -> 2.11 mm
- net N_$13: track 24.5 -> 13.4 mm, vias 0 -> 2
- net IMEAS-ARM: track 109.0 -> 119.7 mm
- net N_$6: track 19.1 -> 28.8 mm
- net N_$15: track 35.4 -> 43.9 mm, vias 2 -> 0
- net N_$4: track 21.9 -> 29.5 mm
- net COM-SIG: track 196.9 -> 202.7 mm
- net N_$5: track 21.2 -> 27.0 mm
- net 12V-AUX-LOGIC: track 0.00 -> 5.07 mm
- net IMEAS-COM: track 187.7 -> 184.1 mm
- net N$66: track 3.65 -> 0.00 mm
- net N$5: track 0.00 -> 3.65 mm
- net GND: track 249.6 -> 252.4 mm
- net N_$11: track 22.3 -> 24.8 mm, vias 0 -> 2
- net N$7: track 4.61 -> 2.84 mm
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Other:
- outline, holes or cut-outs redrawn
