File: PowerBoardHardware/PT_2018_PB_4lyr_Rev1.brd (EAGLE design)
At the start: 177.8 x 209.6 mm, 248 parts, among them J1 APP_2POS_CONFIG12V_VERT, J2 APP_2POS_CONFIG12V_VERT, J3 APP_2POS_CONFIG12V_VERT, J4 APP_2POS_CONFIGMOCO_VERT, J5 RJ45KEYSTONE-942, J6 JTAG_ARM_10PIN, J7 SL02, Q1 Q_IRFS7437PbF, Q10 MOSFET-NCHANNELFDD8780, Q11 MOSFET-NCHANNELFDD8780, Q12 2N7002, Q13 2N7002PW, Q2 Q_IRFS7437PbF, Q3 Q_IRFS7437PbF, Q4 Q_IRFS7437PbF, Q5 Q_IRFS7437PbF, Q6 Q_IRFS7437PbF, Q7 Q_IRFS7437PbF, Q8 2N7002, Q9 Q_IRFS7437PbF, U1 LT1910, U10 ACS722LLCTR-40AU-T, U11 ACS722LLCTR-40AU-T, U12 ACS722LLCTR-40AU-T, U13 ACS722LLCTR-40AU-T, U14 ACS722LLCTR-40AU-T, U15 LT1910, U16 LT1910, U17 LT1910, U18 ACS722LLCTR-40AU-T, U19 ACS722LLCTR-40AU-T, U2 LT1910, U20 ACS722LLCTR-40AU-T, U21 MAX3232D, U22 TM4C1294NCPDT, U23 HX1198FNL, U24 SLVU2.8-4, U3 LT1910, U4 LT1910, U5 LT1910, U6 LT1910, U7 LT1910, U8 ACS722LLCTR-40AU-T, U9 ACS722LLCTR-40AU-T, Y1 NX3225GA, Y2 CRYATL_32K_SMD

Commit message: Solidified patch panel holes, other changes
Removed planes from under ethernet circuitry. Adjusted custom converter planes to compensate for bolt holes for fan mount. Via stitched custom converter planes. Fixed naming sizes and location.  Still need to name components according to one scheme
Parts:
- added 5VFAN2: SL02, MRDT-Connectors:MOLEX-70543-0001
- added Q14: 2N7002PW, SparkFun-DiscreteSemi:SOT323
- moved U$41 446.9 mm to (58.2, 172.2)
- moved U$6 355.7 mm to (172.7, 196.8)
- moved U$8 348.6 mm to (172.2, 157.0)
- moved U$2 293.7 mm to (75.7, -18.5)
- moved LOGO1 230.6 mm to (72.9, 196.1)
- moved U$40 185.4 mm to (172.7, 90.4)
- moved U$39 138.8 mm to (172.7, 50.3)
- moved U$5 7.77 mm to (172.7, 118.1)
- moved U$11 7.66 mm to (97.8, 118.1)
- moved LED-11 6.86 mm to (169.9, 110.5)
- moved R.11 6.86 mm to (169.9, 113.3)
- moved U$35 1.52 mm to (165.1, 5.08)
- moved D3 0.76 mm to (150.1, 186.4)
- moved U$14 0.76 mm to (158.1, 186.7)
- moved U$17 0.76 mm to (154.6, 186.7)
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- renumbered J7 to 5VFAN1, TEMP_1 to RS232, U$1 to LTC3703-5, U22 to TM4C1294NCPDT
Connections:
- new net N$13: 5VFAN2.1, Q14.3
- net 5V: now also 5VFAN2.2
- net FAN_CTL_1: now also Q14.1
- net GND: now also Q14.2
Routing:
- net 5V: track 236.0 -> 250.8 mm
- net FAN_CTL_1: track 29.0 -> 41.2 mm
- net IMEAS-ACT: track 286.5 -> 279.8 mm
- net N$13: track 0.00 -> 3.14 mm
- net SOURCE-ARM: track 19.3 -> 21.2 mm, vias 2 -> 88
- net N$33: track 58.9 -> 57.1 mm
- net 12V-AUX-LOGIC: track 5.07 -> 3.43 mm
- net GND: track 252.4 -> 253.6 mm, vias 114 -> 157
- net VOUT12+: vias 2 -> 20
- net N$31: vias 2 -> 48
- net ARM-BUS: vias 0 -> 17
- added copper zone on layer 15, net ARM-BUS
- added copper zone on layer 2, net ARM-BUS
- added copper zone on layer 15, net N$31
- added copper zone on layer 2, net N$31
- added copper zone on layer 15, net SOURCE-ARM
- added copper zone on layer 2, net SOURCE-ARM
- added copper zone on layer 15, net VOUT12+
- added copper zone on layer 2, net VOUT12+
Other:
- board text added: "30A"
- board text added: "ACTUATION 12V"
- board text added: "ARM 12V 40A"
- board text added: "COMM 12V"
- board text added: "FUSE BLOCK"
- board text added: "LOGIC 12V"
- board text added: "M1"
- board text added: "M2"
- board text added: "M3"
- board text added: "M4"
- board text added: "M5"
- board text added: "M6"
- board text added: "M7"
- board text added: "Missouri S&T Mars Rover Design Team Power Board 2018 Rev1 Lucas Bonskowski"

Commit message: Changed silkscreen names
Could change still, this system isn't the best but could work
Parts:
- removed C28: 22p, SparkFun-Passives:0603-CAP
- removed C29: 22u, buckconverter:CAP_POL_22UF
- removed CB: 0.1u, SparkFun-Passives:0603-CAP
- removed CC1: 470p, SparkFun-Passives:0603-CAP
- removed CC2: 1000p, SparkFun-Passives:0603-CAP
- removed CC3: 2200p, SparkFun-Passives:0603-CAP
- removed CDRVCC: 10u, SparkFun-Passives:0603-CAP
- removed CSS: 0.1uF, SparkFun-Passives:0603-CAP
- removed CVCC: 1uF, SparkFun-Passives:0603-CAP
- removed DB: RF05VAM1STR, buckconverter:DIODE_STANDARD_100V
- removed R20: 113k, SparkFun-Passives:0603-RES
- removed R21: 8.06k, SparkFun-Passives:0603-RES
- removed RC1, RC2: 10k, SparkFun-Passives:0603-RES
- removed RF: 10, SparkFun-Passives:0603-RES
- removed RMAX: 16.5k, SparkFun-Passives:0603-RES
- removed U$38: ATC_FUSE_BLOCK, MRDT-Hardware:BLOCK_3557-2
- removed U$39, U$40: MOUNTING_HOLE#6, MRDT-Hardware:#6_SCREW
- removed U$41: MRDT_LOGO, MRDT-2015-General:MRDT_LOGO
- removed U24: SLVU2.8-4, MRDT-ICs:SOIC8
- added C.63: 10n, SparkFun-Capacitors:0805
- added C.65, C.83: 0.1uF, resistor:C0603
- added C.66: .1µF, SparkFun-Capacitors:0805
- added C.79, C.80, C.81, C.82, C.88: .1u, SparkFun-Passives:0805
- added D4: RBR3MM30ATR, buckconverter:DIODE_SCHOTTKY_30V_1A
- added R.13: 10kΩ 1%, resistor:R1206
- added R.20, R.22: 1k, resistor:R1206
- added R.21, R.23: 100k, resistor:R1206
- added R.28: 1kΩ, SparkFun-Passives:1206
- added U$1: MOUNTING_HOLE#6, MRDT-Hardware:#6_SCREW
- added U$24: ATC_FUSE_BLOCK, MRDT-Hardware:BLOCK_3557-2
- added U$25: APP_2POS_CONFIGMOCO_VERT, MRDT-Connectors:APP45_MOCO_VERT_CONFIG
- added U$33: IPP052N06L3GXKSA1, buckconverter:TO-220
- added U22: HX1198FNL, MRDT-ICs:HX1198FNL
- C.10, C.17, C.21, C.22: value .1µF -> 1nF
- C.11, C.20: value .1µF -> 1mF; device SparkFun-Capacitors:0805 -> MRDT-2014-All:C_12.5MM
- C.12, C.16: value .1µF -> 330µF; device SparkFun-Capacitors:0805 -> resistor:E5-8,5
- C.13: value .1µF -> 2.2uF; device SparkFun-Capacitors:0805 -> SparkFun-Capacitors:1206
- C.26: value 330µF -> 1nF; device resistor:E5-8,5 -> SparkFun-Capacitors:0805
- C.27: value 330µF -> 2.2uF; device resistor:E5-8,5 -> SparkFun-Capacitors:1206
- C.28: value 330µF -> .1µF; device resistor:E5-8,5 -> SparkFun-Capacitors:0805
- C.3, C.40, C.41, C.7: value 1nF -> .1µF
- C.31: value 330µF -> 1mF; device resistor:E5-8,5 -> MRDT-2014-All:C_12.5MM
- C.34: value 10uF -> 2.2uF
- C.35, C.36: value 2.2uF -> 330µF; device SparkFun-Capacitors:1206 -> resistor:E5-8,5
- C.37: value 2.2uF -> .1µF; device SparkFun-Capacitors:1206 -> SparkFun-Capacitors:0805
- C.38: value .1uF -> .1µF
- C.4: value 1nF -> .1uF
- C.43: value 1nF -> 1mF; device SparkFun-Capacitors:0805 -> MRDT-2014-All:C_12.5MM
- C.44: value 1nF -> 0.1uF; device SparkFun-Capacitors:0805 -> SparkFun-Passives:0603-CAP
- C.45: value 10uF -> 1000p; device SparkFun-Capacitors:1206 -> SparkFun-Passives:0603-CAP
- C.46: value 10uF -> .1µF; device SparkFun-Capacitors:1206 -> SparkFun-Capacitors:0805
- C.48: value .1uF -> 1nF
- C.5: value 1nF -> 10uF; device SparkFun-Capacitors:0805 -> SparkFun-Capacitors:1206
- C.50: value .1uF -> 10uF; device SparkFun-Capacitors:0805 -> SparkFun-Capacitors:1206
- C.51: value 1mF -> 1nF; device MRDT-2014-All:C_12.5MM -> SparkFun-Capacitors:0805
- C.52, C.54: value 1mF -> .1uF; device MRDT-2014-All:C_12.5MM -> SparkFun-Capacitors:0805
- C.53: value 1mF -> 10uF; device MRDT-2014-All:C_12.5MM -> SparkFun-Capacitors:1206
- C.55: value .1u -> 1nF; device SparkFun-Passives:0805 -> SparkFun-Capacitors:0805
- C.56: value .1u -> 470p; device SparkFun-Passives:0805 -> SparkFun-Passives:0603-CAP
- C.57: value .1u -> 2200p; device SparkFun-Passives:0805 -> SparkFun-Passives:0603-CAP
- C.58: value .1u -> 0.1uF; device SparkFun-Passives:0805 -> SparkFun-Passives:0603-CAP
- C.59: value .1u -> 1uF; device SparkFun-Passives:0805 -> SparkFun-Passives:0603-CAP
- C.60: value 10n -> 10u; device SparkFun-Capacitors:0805 -> SparkFun-Passives:0603-CAP
- C1: value 0.1uF -> 22u; device resistor:C0603 -> buckconverter:CAP_POL_22UF
- C2: value 0.1uF -> 22p; device resistor:C0603 -> SparkFun-Passives:0603-CAP
- CIN1: value 100u -> 1000p; device buckconverter:CAP_POL_220UF -> SparkFun-Passives:0603-CAP
- CIN2: value 1000p -> 100u; device SparkFun-Passives:0603-CAP -> buckconverter:CAP_POL_220UF
- D3: value RBR3MM30ATR -> RF05VAM1STR; device buckconverter:DIODE_SCHOTTKY_30V_1A -> buckconverter:DIODE_STANDARD_100V
- J4: value APP_2POS_CONFIGMOCO_VERT -> RJ45KEYSTONE-942; device MRDT-Connectors:APP45_MOCO_VERT_CONFIG -> MRDT-Connectors:KEYSTONE-942
- J5: value RJ45KEYSTONE-942 -> APP_2POS_CONFIGMOCO_VERT; device MRDT-Connectors:KEYSTONE-942 -> MRDT-Connectors:APP45_MOCO_VERT_CONFIG
- Q10: value MOSFET-NCHANNELFDD8780 -> Q_IRFS7437PbF; device SparkFun-DiscreteSemi:DPAK -> MRDT-2015-PowerBoard:D2PACK
- Q11: value MOSFET-NCHANNELFDD8780 -> 2N7002; device SparkFun-DiscreteSemi:DPAK -> SparkFun-DiscreteSemi:SOT323
- Q5: value Q_IRFS7437PbF -> MOSFET-NCHANNELFDD8780; device MRDT-2015-PowerBoard:D2PACK -> SparkFun-DiscreteSemi:DPAK
- Q8: value 2N7002 -> MOSFET-NCHANNELFDD8780; device SparkFun-DiscreteSemi:SOT323 -> SparkFun-DiscreteSemi:DPAK
- R.10, R.8: value 1kΩ -> 5kΩ
- R.11: value 1kΩ -> 16.5k; device SparkFun-Passives:1206 -> SparkFun-Passives:0603-RES
- R.14: value 100k -> 100k 1%
- R.15: value 1k -> 10k; device resistor:R1206 -> SparkFun-Passives:0603-RES
- R.16: value 100k 1% -> 10k; device resistor:R1206 -> SparkFun-Passives:0603-RES
- R.17: value 10kΩ 1% -> 113k; device resistor:R1206 -> SparkFun-Passives:0603-RES
- R.18: value 1k -> 8.06k; device resistor:R1206 -> SparkFun-Passives:0603-RES
- R.19: value 100k -> 10; device resistor:R1206 -> SparkFun-Passives:0603-RES
- R.2, R.5: value 5kΩ -> 1kΩ
- U$10, U$16, U$5, U$9: value MOUNTING_HOLE#6 -> ATC_FUSE_BLOCK; device MRDT-Hardware:#6_SCREW -> MRDT-Hardware:BLOCK_3557-2
- U$12, U$6, U$8: value MOUNTING_HOLE#6 -> APP_2POS_CONFIGMOCO_VERT; device MRDT-Hardware:#6_SCREW -> MRDT-Connectors:APP45_MOCO_VERT_CONFIG
- U$13: value IPP052N06L3GXKSA1 -> ATC_FUSE_BLOCK; device buckconverter:TO-220 -> MRDT-Hardware:BLOCK_3557-2
- U$14: value IPP052N06L3GXKSA1 -> APP_2POS_CONFIGMOCO_VERT; device buckconverter:TO-220 -> MRDT-Connectors:APP45_MOCO_VERT_CONFIG
- U$15, U$19, U$20, U$7: value APP_2POS_CONFIGMOCO_VERT -> ATC_FUSE_BLOCK; device MRDT-Connectors:APP45_MOCO_VERT_CONFIG -> MRDT-Hardware:BLOCK_3557-2
- U$17: value 530002B02500G -> MOUNTING_HOLE#6; device buckconverter:RADIAL_FIN_HEATSINK -> MRDT-Hardware:#6_SCREW
- U$18: value 530002B02500G -> APP_2POS_CONFIGMOCO_VERT; device buckconverter:RADIAL_FIN_HEATSINK -> MRDT-Connectors:APP45_MOCO_VERT_CONFIG
- U$2: value JACOB_SIG -> MOUNTING_HOLE#6; device Jacob Signature:JACOB_SIG -> MRDT-Hardware:#6_SCREW
- U$21: value MLX91210 -> APP_2POS_CONFIGMOCO_VERT; device buckconverter:SOIC8_ACS711 -> MRDT-Connectors:APP45_MOCO_VERT_CONFIG
- U$22, U$23, U$3: value APP_2POS_CONFIGMOCO_VERT -> MOUNTING_HOLE#6; device MRDT-Connectors:APP45_MOCO_VERT_CONFIG -> MRDT-Hardware:#6_SCREW
- U$26: value ATC_FUSE_BLOCK -> LUCAS_BONSKOWSKI_SIGNATURE; device MRDT-Hardware:BLOCK_3557-2 -> MRDT-Signatures:LUCAS_BONSKOWSKI_SIGNATURE
- U$27, U$36, U$37: value ATC_FUSE_BLOCK -> MOUNTING_HOLE#6; device MRDT-Hardware:BLOCK_3557-2 -> MRDT-Hardware:#6_SCREW
- U$28: value ATC_FUSE_BLOCK -> MLX91210; device MRDT-Hardware:BLOCK_3557-2 -> buckconverter:SOIC8_ACS711
- U$29, U$32: value ATC_FUSE_BLOCK -> 530002B02500G; device MRDT-Hardware:BLOCK_3557-2 -> buckconverter:RADIAL_FIN_HEATSINK
- U$30: value ATC_FUSE_BLOCK -> IPP052N06L3GXKSA1; device MRDT-Hardware:BLOCK_3557-2 -> buckconverter:TO-220
- U$31: value ATC_FUSE_BLOCK -> MRDT_LOGO; device MRDT-Hardware:BLOCK_3557-2 -> MRDT-2015-General:MRDT_LOGO
- U$34: value MOUNTING_HOLE#6 -> MRDT_LOGO; device MRDT-Hardware:#6_SCREW -> MRDT-Hardware:MRDT_LOGO
- U$4: value MRDT_LOGO -> MOUNTING_HOLE#6; device MRDT-Hardware:MRDT_LOGO -> MRDT-Hardware:#6_SCREW
- U1, U17, U2, U4, U6: value LT1910 -> ACS722LLCTR-40AU-T; device Jake:SO8 -> MRDT-2015-PowerBoard:SOIC8_ACS711
- U10, U11, U13, U19, U20: value ACS722LLCTR-40AU-T -> LT1910; device MRDT-2015-PowerBoard:SOIC8_ACS711 -> Jake:SO8
- U21: value MAX3232D -> SLVU2.8-4; device MRDT-ICs:SOIC16 -> MRDT-ICs:SOIC8
- U23: value HX1198FNL -> MAX3232D; device MRDT-ICs:HX1198FNL -> MRDT-ICs:SOIC16
- Y1: value NX3225GA -> CRYATL_32K_SMD; device MRDT-Passives:NDK3.2X2.5 -> MRDT-Passives:CRYSTAL_32K_SMD
- Y2: value CRYATL_32K_SMD -> NX3225GA; device MRDT-Passives:CRYSTAL_32K_SMD -> MRDT-Passives:NDK3.2X2.5
- moved U$6 245.2 mm to (1.91, 21.0), turned to 270 degrees
- moved U$8 207.3 mm to (1.91, 38.7), turned to 270 degrees
- moved U$4 196.8 mm to (172.7, 5.08)
- moved U$34 192.6 mm to (124.5, 195.8)
- moved U$14 192.4 mm to (1.91, 74.3), turned to 270 degrees
- moved U$35 191.9 mm to (172.7, 196.8)
- moved U$23 188.4 mm to (172.7, 118.1), turned to 0 degrees
- moved U$37 179.7 mm to (172.7, 204.5)
- moved U$15 174.7 mm to (176.5, 78.7), turned to 180 degrees
- moved U$16 172.4 mm to (49.5, 83.8)
- moved U$27 169.9 mm to (172.2, 157.0)
- moved U$7 169.7 mm to (168.9, 26.7), turned to 90 degrees
- moved R.10 167.9 mm to (11.4, 114.3), turned to 270 degrees
- moved LED-10 165.6 mm to (15.2, 114.3), turned to 90 degrees
- moved U$3 164.0 mm to (165.1, 5.08), turned to 0 degrees
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- renumbered C10 to C.75, C11 to C.74, C12 to C.86, C13 to C.87, C14 to C.85, C15 to C.77, C16 to C.73, C17 to C.64, C18 to C.69, C19 to C.68, C3 to C.84, C4 to C.72, C5 to C.61, C6 to C.62, C7 to C.71, C8 to C.76, C9 to C.70, COUT1 to C.67, COUT2 to C.78, LED1 to LED-14, LED2 to LED-13, LED3 to LED-12, LTC3703-5 to LTC3703-1, R1 to R.33, R10 to R.43, R11 to R.42, R12 to R.35, R13 to R.38, R14 to R.34, R15 to R.40, R16 to R.32, R17 to R.31, R19 to R.41, R2 to R.36, R3 to R.37, R4 to R.39, R5 to R.29, R6 to R.27, R7 to R.25, R8 to R.24, R9 to R.26, RC3 to R.30, RS232 to RS1, RSET to R.12
Connections:
- removed net N$7 (its old number): LED-11.A, R.11.2
- new net N$6: LED-2.A, R.2.2
- net +3V3: now also C.47.1, C.48.1, C.49.1, C.65.1, C.83.1, U22.P$2, U22.P$7; no longer C.33.1, C.34.1, C.38.1, C1.1, C2.1, U23.P$2, U23.P$7
- net 12V-AUX-ACT: now also J1.VCC, R.2.1, U2.4; no longer J3.VCC, R.9.1, U18.4
- net 12V-AUX-COM: now also J2.VCC, R.5.1, U9.4; no longer J1.VCC, R.10.1, U20.4
- net 12V-AUX-LOGIC: now also J3.VCC, R.9.1, U18.4; no longer J2.VCC, R.11.1, U19.4
- net 232_RX: now also U23.13; no longer U21.13
- net 232_TX: now also U23.14; no longer U21.14
- net 3.3V: now also C.18.2, C.28.2, C.3.2, C.37.2, C.41.2, C.50.1, C.51.1, C.52.1, C.7.2, C.80.1, U1.8, U17.8, U2.8, U23.16, U4.8, U6.8; no longer C.10.2, C.11.2, C.12.2, C.13.2, C.25.2, C.43.1, C.46.1, C.49.1, C.55.1, C.8.2, U10.8, U11.8, U13.8, U19.8, U20.8, U21.16
- net 5V: now also C.53.1, C.54.1, C.55.1, C.60.1, C.66.2, C1.+, D3.P$2, R.19.2, U$28.8; no longer C.32.2, C.42.1, C.45.1, C.48.1, C29.+, CDRVCC.1, DB.P$2, RF.2, U$21.8
- net ACT-CTL: now also R.20.2; no longer R.18.2
- net ARM-BUS: now also J5.VCC, R.28.1, U$28.4; no longer J4.VCC, R.8.1, U$21.4
- net COM-SIG: now also U15.4; no longer U16.4
- net DRAIN-M1: now also C.8.2, U1.4, U3.6, U3.8; no longer C.15.2, U1.6, U1.8, U8.4
- net DRAIN-M2: now also C.15.2, U4.4, U5.6, U5.8; no longer C.16.2, U2.6, U2.8, U9.4
- net DRAIN-M3: now also C.19.2, U6.4, U7.6, U7.8; no longer C.17.2, U10.4, U3.6, U3.8
- net DRAIN-M4: now also C.25.2, U11.6, U11.8, U8.4; no longer C.18.2, U11.4, U4.6, U4.8
- net DRAIN-M5: now also C.32.2, Q6.TAB, U13.6, U13.8; no longer C.19.2, Q5.TAB, U5.6, U5.8
- net DRAIN-M6: now also C.38.2, Q7.TAB, U14.4, U16.6, U16.8; no longer C.20.2, Q6.TAB, U13.4, U6.6, U6.8
- net DRAIN-M7: now also C.40.2, Q9.TAB, U17.4, U19.6, U19.8; no longer C.21.2, Q7.TAB, U14.4, U7.6, U7.8
- net EN0RXI_N: now also U22.P$8; no longer U23.P$8
- net EN0RXI_P: now also U22.P$6; no longer U23.P$6
- net EN0TXO_N: now also U22.P$3; no longer U23.P$3
- net EN0TXO_P: now also U22.P$1; no longer U23.P$1
- net FILTER-M1: now also C.2.1, U1.6; no longer C.1.1, U8.6
- net FILTER-M2: now also C.10.1, U4.6; no longer C.2.1, U9.6
- net FILTER-M3: now also C.17.1, U6.6; no longer C.3.1, U10.6
- net FILTER-M4: now also C.21.1, U8.6; no longer C.4.1, U11.6
- net FILTER-M5: now also C.26.1; no longer C.5.1
- net FILTER-M6: now also C.33.1, U14.6; no longer C.6.1, U13.6
- net FILTER-M7: now also C.39.1, U17.6; no longer C.7.1, U14.6
- net GATE-M1: now also U3.5; no longer U1.5
- net GATE-M2: now also U5.5; no longer U2.5
- net GATE-M3: now also U7.5; no longer U3.5
- net GATE-M4: now also U11.5; no longer U4.5
- net GATE-M5: now also Q6.1, U13.5; no longer Q5.1, U5.5
- net GATE-M6: now also Q7.1, U16.5; no longer Q6.1, U6.5
- net GATE-M7: now also Q9.1, U19.5; no longer Q7.1, U7.5
- net GND: now also C.10.2, C.11.-, C.12.-, C.13.2, C.16.-, C.17.2, C.20.-, C.21.2, C.22.2, C.26.2, C.27.2, C.28.1, C.3.1, C.35.-, C.36.-, C.37.1, C.38.1, C.40.1, C.41.1, C.43.-, C.46.1, C.51.2, C.52.2, C.53.2, C.54.2, C.63.2, C.65.2, C.66.1, C.7.1, C.79.2, C.80.2, C.83.2, C.88.2, C1.-, CIN1.2, CIN2.GND, D4.P$1, J5.GND, Q11.2, R.11.1, R.13.1, R.18.2, R.21.2, R.23.2, U$12.GND, U$14.GND, U$18.GND, U$21.GND, U$25.GND, U$28.5, U$28.6, U$33.3, U$6.GND, U$8.GND, U1.5, U10.1, U11.1, U13.1, U17.5, U19.1, U2.5, U20.1, U23.15, U4.5, U6.5; no longer C.10.1, C.11.1, C.12.1, C.13.1, C.16.1, C.17.1, C.20.1, C.21.1, C.22.1, C.26.-, C.27.-, C.28.-, C.3.2, C.35.2, C.36.2, C.37.2, C.38.2, C.40.2, C.41.2, C.43.2, C.45.2, C.46.2, C.51.-, C.52.-, C.53.-, C.54.-, C.58.2, C.7.2, C1.2, C28.2, C29.-, CDRVCC.2, CIN1.GND, CIN2.2, CSS.2, CVCC.2, D3.P$1, J4.GND, Q8.2, R.14.2, R.17.1, R.19.2, R21.2, RMAX.1, U$14.3, U$15.GND, U$19.GND, U$20.GND, U$21.5, U$21.6, U$22.GND, U$23.GND, U$3.GND, U$7.GND, U1.1, U10.5, U11.5, U13.5, U17.1, U19.5, U2.1, U20.5, U21.15, U4.1, U6.1
- net IMEAS-ACT: now also U2.7; no longer U18.7
- net IMEAS-ARM: now also C.63.1, U$28.7; no longer C.60.1, U$21.7
- net IMEAS-COM: now also U18.7; no longer U19.7
- net IMEAS-LOGIC: now also U9.7; no longer U20.7
- net IMEAS-M1: now also U1.7; no longer U8.7
- net IMEAS-M2: now also U4.7; no longer U9.7
- net IMEAS-M3: now also U6.7; no longer U10.7
- net IMEAS-M4: now also U8.7; no longer U11.7
- net IMEAS-M6: now also U14.7; no longer U13.7
- net IMEAS-M7: now also U17.7; no longer U14.7
- net LEDLINE-M2: now also LED-3.A, R.3.2; no longer LED-2.A, R.2.2
- net LEDLINE-M3: now also LED-4.A, R.4.2; no longer LED-3.A, R.3.2
- net LEDLINE-M4: now also LED-6.A, R.6.2; no longer LED-4.A, R.4.2
- net LEDLINE-M5: now also LED-7.A, R.7.2; no longer LED-5.A, R.5.2
- net LEDLINE-M6: now also LED-8.A, R.8.2; no longer LED-6.A, R.6.2
- net LEDLINE-M7: now also LED-10.A, R.10.2; no longer LED-7.A, R.7.2
- net LOGIC-SIG: now also U10.4; no longer U15.4
- net LOGIC/COM-CTL: now also R.22.2; no longer R.15.2
- net N$1: now also C.16.+, U$7.IN_1, U$7.IN_2; no longer C.26.+, U$30.IN_1, U$30.IN_2
- net N$10: now also R.11.2; no longer RMAX.2
- net N$11: now also C.79.1, U23.2; no longer C.58.1, U21.2
- net N$114: now also R.22.1, R.23.1; no longer R.14.1, R.15.1
- net N$12: now also C.6.1, U2.6; no longer C.39.1, U18.6
- net N$14: now also C.44.1; no longer CSS.1
- net N$15: now also C.42.1, U18.6; no longer C.40.1, U19.6
- net N$16: now also LED-5.A, R.5.2; no longer LED-10.A, R.10.2
- net N$17: now also Q8.1, U15.5; no longer Q11.1, U16.5
- net N$18: now also C.12.+, C.13.1, U$7.OUT_1, U$7.OUT_2, U2.1; no longer C.27.+, C.35.1, U$30.OUT_1, U$30.OUT_2, U18.1
- net N$19: now also Q8.3, U18.1; no longer Q11.3, U19.1
- net N$2: now also LED-11.A, R.28.2; no longer LED-8.A, R.8.2
- net N$20: now also Q8.4, U$19.OUT_1, U$19.OUT_2, U15.6, U15.8; no longer Q11.4, U$31.OUT_1, U$31.OUT_2, U16.6, U16.8
- net N$21: now also Q5.4, U$15.OUT_1, U$15.OUT_2, U10.6, U10.8; no longer Q10.4, U$32.OUT_1, U$32.OUT_2, U15.6, U15.8
- net N$22: now also Q5.3, U9.1; no longer Q10.3, U20.1
- net N$23: now also C.56.1, R.16.2; no longer CC1.1, RC1.2
- net N$24: now also C.45.1, R.16.1; no longer CC2.1, RC1.1
- net N$25: now also Q11.1, R.20.1, R.21.1; no longer Q8.1, R.18.1, R.19.1
- net N$26: now also C.57.1, R.15.1; no longer CC3.1, RC2.1
- net N$27: now also C.45.2, C.56.2, R.15.2, R.17.2, R.18.1; no longer CC1.2, CC2.2, R20.2, R21.1, RC2.2
- net N$28: now also Q5.1, U10.5; no longer Q10.1, U15.5
- net N$29: now also C.59.1, R.19.1; no longer CVCC.1, RF.1
- net N$30: now also U$33.1; no longer U$14.1
- net N$31: now also C.58.2, D4.P$2, U$30.3, U$33.2; no longer CB.2, D3.P$2, U$13.3, U$14.2
- net N$32: now also C.58.1, D3.P$1; no longer CB.1, DB.P$1
- net N$33: now also U$30.1; no longer U$13.1
- net N$36: now also Q10.1, U20.5; no longer Q9.1, U17.5
- net N$4: now also C.22.1, U9.6; no longer C.41.1, U20.6
- net N$40: now also C.81.1, U23.1; no longer C.56.1, U21.1
- net N$42: now also C.81.2, U23.3; no longer C.56.2, U21.3
- net N$43: now also C.82.1, U23.4; no longer C.57.1, U21.4
- net N$44: now also C.82.2, U23.5; no longer C.57.2, U21.5
- net N$45: now also C.88.1, U23.6; no longer C.59.1, U21.6
- net N$8: now also Q11.3; no longer Q8.3
- net N$9: now also C.27.1, C.34.1, C.35.+, C.36.+, U$15.IN_1, U$15.IN_2, U$19.IN_1, U$19.IN_2; no longer C.28.+, C.31.+, C.36.1, C.37.1, U$31.IN_1, U$31.IN_2, U$32.IN_1, U$32.IN_2
- net N_$1: now also U22.P$15; no longer U23.P$15
- net N_$11: now also J4.P$4, J4.P$5; no longer J5.P$4, J5.P$5
- net N_$13: now also J4.P$1, J4.P$2; no longer J5.P$1, J5.P$2
- net N_$18: now also Y2.P$3; no longer Y1.P$3
- net N_$21: now also Y2.P$1; no longer Y1.P$1
- net N_$22: now also Y1.P$2; no longer Y2.P$2
- net N_$23: now also Y1.P$1; no longer Y2.P$1
- net N_$3: now also U22.P$10; no longer U23.P$10
- net N_$4: now also J4.P$7, U21.2, U21.7, U22.P$14; no longer J5.P$7, U23.P$14, U24.2, U24.7
- net N_$5: now also J4.P$6, U21.3, U21.6, U22.P$11; no longer J5.P$6, U23.P$11, U24.3, U24.6
- net N_$6: now also J4.P$8, U21.1, U21.8, U22.P$16; no longer J5.P$8, U23.P$16, U24.1, U24.8
- net N_$7: now also J4.P$3, U21.4, U21.5, U22.P$9; no longer J5.P$3, U23.P$9, U24.4, U24.5
- net SER_RX: now also U23.12; no longer U21.12
- net SER_TX: now also U23.11; no longer U21.11
- net SIG-ARM: now also U20.4; no longer U17.4
- net SIG-M1: now also U3.4; no longer U1.4
- net SIG-M2: now also U5.4; no longer U2.4
- net SIG-M3: now also U7.4; no longer U3.4
- net SIG-M4: now also U11.4; no longer U4.4
- net SIG-M5: now also U13.4; no longer U5.4
- net SIG-M6: now also U16.4; no longer U6.4
- net SIG-M7: now also U19.4; no longer U7.4
- net SOURCE-ARM: now also CIN1.1, CIN2.+, Q10.2, U$30.2; no longer CIN1.+, CIN2.1, Q9.2, U$13.2
- net SOURCE-M1: now also U$6.VCC; no longer U$3.VCC
- net SOURCE-M2: now also R.3.1, U$8.VCC; no longer R.2.1, U$23.VCC
- net SOURCE-M3: now also R.4.1, U$12.VCC; no longer R.3.1, U$7.VCC
- net SOURCE-M4: now also R.6.1, U$14.VCC; no longer R.4.1, U$15.VCC
- net SOURCE-M5: now also Q6.2, R.7.1, U$18.VCC; no longer Q5.2, R.5.1, U$19.VCC
- net SOURCE-M6: now also Q7.2, R.8.1, U$21.VCC; no longer Q6.2, R.6.1, U$20.VCC
- net SOURCE-M7: now also Q9.2, R.10.1, U$25.VCC; no longer Q7.2, R.7.1, U$22.VCC
- net VMEAS-VBATT: now also R.13.2, R.14.1; no longer R.16.1, R.17.2
- net VOUT12+: now also C.57.2, C2.1, R.17.1, U$28.1; no longer C28.1, CC3.2, R20.1, U$21.1
- net V_BATT: now also C.1.1, C.11.+, C.20.+, C.31.+, C.4.1, C.43.+, C.46.2, C.5.1, Q10.TAB, R.14.2, U$10.IN_1, U$10.IN_2, U$13.IN_1, U$13.IN_2, U$16.IN_1, U$16.IN_2, U$20.IN_1, U$20.IN_2, U$24.IN_1, U$24.IN_2, U$5.IN_1, U$5.IN_2, U$9.IN_1, U$9.IN_2, U20.6, U20.8; no longer C.22.2, C.44.1, C.47.1, C.50.1, C.51.+, C.52.+, C.53.+, C.54.+, Q9.TAB, R.16.2, U$26.IN_1, U$26.IN_2, U$27.IN_1, U$27.IN_2, U$28.IN_1, U$28.IN_2, U$29.IN_1, U$29.IN_2, U$36.IN_1, U$36.IN_2, U$37.IN_1, U$37.IN_2, U$38.IN_1, U$38.IN_2, U17.6, U17.8
- net V_BATT_M1: now also U$5.OUT_1, U$5.OUT_2, U1.1; no longer U$26.OUT_1, U$26.OUT_2, U8.1
- net V_BATT_M2: now also U$9.OUT_1, U$9.OUT_2, U4.1; no longer U$27.OUT_1, U$27.OUT_2, U9.1
- net V_BATT_M3: now also U$10.OUT_1, U$10.OUT_2, U6.1; no longer U$36.OUT_1, U$36.OUT_2, U10.1
- net V_BATT_M4: now also U$13.OUT_1, U$13.OUT_2, U8.1; no longer U$37.OUT_1, U$37.OUT_2, U11.1
- net V_BATT_M5: now also U$16.OUT_1, U$16.OUT_2; no longer U$38.OUT_1, U$38.OUT_2
- net V_BATT_M6: now also U$20.OUT_1, U$20.OUT_2, U14.1; no longer U$29.OUT_1, U$29.OUT_2, U13.1
- net V_BATT_M7: now also U$24.OUT_1, U$24.OUT_2, U17.1; no longer U$28.OUT_1, U$28.OUT_2, U14.1
Routing:
- net N$6: track 0.00 -> 3.85 mm
- net N$7 (its old number): track 2.84 -> 0.00 mm
- net N$7: track 3.85 -> 2.84 mm
