File: PowerBoardHardware/PT_2018_PB_4lyr_Rev1.sch (EAGLE design)
At the start: 250 parts, among them J1 APP_2POS_CONFIG12V_VERT, J2 APP_2POS_CONFIG12V_VERT, J3 APP_2POS_CONFIG12V_VERT, J4 RJ45KEYSTONE-942, J5 APP_2POS_CONFIGMOCO_VERT, J6 JTAG_ARM_10PIN, Q1 Q_IRFS7437PbF, Q10 Q_IRFS7437PbF, Q11 2N7002, Q12 2N7002, Q13 2N7002PW, Q14 2N7002PW, Q2 Q_IRFS7437PbF, Q3 Q_IRFS7437PbF, Q4 Q_IRFS7437PbF, Q5 MOSFET-NCHANNELFDD8780, Q6 Q_IRFS7437PbF, Q7 Q_IRFS7437PbF, Q8 MOSFET-NCHANNELFDD8780, Q9 Q_IRFS7437PbF, U1 ACS722LLCTR-40AU-T, U10 LT1910, U11 LT1910, U12 ACS722LLCTR-40AU-T, U13 LT1910, U14 ACS722LLCTR-40AU-T, U15 LT1910, U16 LT1910, U17 ACS722LLCTR-40AU-T, U18 ACS722LLCTR-40AU-T, U19 LT1910, U2 ACS722LLCTR-40AU-T, U20 LT1910, U21 SLVU2.8-4, U22 HX1198FNL, U23 MAX3232D, U3 LT1910, U4 ACS722LLCTR-40AU-T, U5 LT1910, U6 ACS722LLCTR-40AU-T, U7 LT1910, U8 ACS722LLCTR-40AU-T, U9 ACS722LLCTR-40AU-T, Y1 CRYATL_32K_SMD, Y2 NX3225GA

Commit message: FINAL REV 1 TO BE ORDERED
Made ground plane around buck converter 4 layers. Adjusted via stitch to allow 3.3v plane to have a larger bottleneck.  Flipped logic and comm bus locations.  Added + and - near battery terminals. Renumbered components since we missed a few before.
Parts:
- removed C1: 22u, buckconverter:UCZ1K220MCL1GS
- removed C2: 22p, SparkFun-Passives:CAP0603-CAP
- removed CIN1: 1000p, SparkFun-Passives:CAP0603-CAP
- removed CIN2: 100u, buckconverter:B41858C9107M000
- removed Q14: 2N7002PW, SparkFun-DiscreteSemi:MOSFET-NCHANNEL2N7002PW
- added C.89: 2.2uF, resistor:C-USC0603
- added C.90: 0.1uF, resistor:C-USC0603
- added C.91: 1.0uF, resistor:C-USC0603
- added C.92: .1u, SparkFun-Passives:CAP0805
- C.44: value 0.1uF -> 22u; device SparkFun-Passives:CAP0603-CAP -> buckconverter:UCZ1K220MCL1GS
- C.45: value 1000p -> 0.1uF
- C.46: value .1µF -> 1000p; device SparkFun-Capacitors:CAP0805 -> SparkFun-Passives:CAP0603-CAP
- C.47: value 10uF -> .1µF; device SparkFun-Capacitors:CAP1206 -> SparkFun-Capacitors:CAP0805
- C.48, C.51: value 1nF -> 10uF; device SparkFun-Capacitors:CAP0805 -> SparkFun-Capacitors:CAP1206
- C.49, C.52: value .1uF -> 1nF
- C.50, C.53: value 10uF -> .1uF; device SparkFun-Capacitors:CAP1206 -> SparkFun-Capacitors:CAP0805
- C.54: value .1uF -> 10uF; device SparkFun-Capacitors:CAP0805 -> SparkFun-Capacitors:CAP1206
- C.55: value 1nF -> .1uF
- C.56: value 470p -> 1nF; device SparkFun-Passives:CAP0603-CAP -> SparkFun-Capacitors:CAP0805
- C.57: value 2200p -> 470p
- C.58: value 0.1uF -> 2200p
- C.59: value 1uF -> 0.1uF
- C.60: value 10u -> 1uF
- C.61: value 1000pF -> 10u; device resistor:C-USC0603 -> SparkFun-Passives:CAP0603-CAP
- C.62: value 4700pF -> 1000pF; device resistor:C-USC1206 -> resistor:C-USC0603
- C.63: value 10n -> 4700pF; device SparkFun-Capacitors:CAP0805 -> resistor:C-USC1206
- C.64: value 0.1uF -> 1000p; device resistor:C-USC0603 -> SparkFun-Passives:CAP0603-CAP
- C.65: value 0.1uF -> 100u; device resistor:C-USC0603 -> buckconverter:B41858C9107M000
- C.66: value .1µF -> 10n
- C.67, C.78: value 220u -> 0.1uF; device buckconverter:EGPD101ELL221MK25H -> resistor:C-USC0603
- C.68, C.73: value 12pF -> 0.1uF
- C.69: value 12pF -> .1µF; device resistor:C-USC0603 -> SparkFun-Capacitors:CAP0805
- C.70: value 0.1uF -> 220u; device resistor:C-USC0603 -> buckconverter:EGPD101ELL221MK25H
- C.71, C.72: value 0.1uF -> 12pF
- C.76: value 0.1uF -> 22p; device resistor:C-USC0603 -> SparkFun-Passives:CAP0603-CAP
- C.79, C.80, C.88: value .1u -> 0.1uF; device SparkFun-Passives:CAP0805 -> resistor:C-USC0603
- C.81: value .1u -> 12pF; device SparkFun-Passives:CAP0805 -> resistor:C-USC0603
- C.82: value .1u -> 220u; device SparkFun-Passives:CAP0805 -> buckconverter:EGPD101ELL221MK25H
- C.83, C.84, C.86: value 0.1uF -> .1u; device resistor:C-USC0603 -> SparkFun-Passives:CAP0805
- C.85: value 2.2uF -> .1u; device resistor:C-USC0603 -> SparkFun-Passives:CAP0805
- C.87: value 1.0uF -> 0.1uF
- U$11, U$17: value MOUNTING_HOLE#6 -> ATC_FUSE_BLOCK; device MRDT-Hardware:MOUNTING_HOLE#6 -> MRDT-Hardware:ATC_FUSE_BLOCK
- U$12, U$18: value APP_2POS_CONFIGMOCO_VERT -> MOUNTING_HOLE#6; device MRDT-Connectors:APP_2POS_CONFIGMOCO_VERT -> MRDT-Hardware:MOUNTING_HOLE#6
- U$13, U$15, U$19, U$9: value ATC_FUSE_BLOCK -> APP_2POS_CONFIGMOCO_VERT; device MRDT-Hardware:ATC_FUSE_BLOCK -> MRDT-Connectors:APP_2POS_CONFIGMOCO_VERT
- U$14, U$21, U$25: value APP_2POS_CONFIGMOCO_VERT -> ATC_FUSE_BLOCK; device MRDT-Connectors:APP_2POS_CONFIGMOCO_VERT -> MRDT-Hardware:ATC_FUSE_BLOCK
- U$22: value MOUNTING_HOLE#6 -> APP_2POS_CONFIGMOCO_VERT; device MRDT-Hardware:MOUNTING_HOLE#6 -> MRDT-Connectors:APP_2POS_CONFIGMOCO_VERT
- U$24: value ATC_FUSE_BLOCK -> MOUNTING_HOLE#6; device MRDT-Hardware:ATC_FUSE_BLOCK -> MRDT-Hardware:MOUNTING_HOLE#6
- U$26: value LUCAS_BONSKOWSKI_SIGNATURE -> APP_2POS_CONFIGMOCO_VERT; device MRDT-Signatures:LUCAS_BONSKOWSKI_SIGNATURE -> MRDT-Connectors:APP_2POS_CONFIGMOCO_VERT
- U$27: value MOUNTING_HOLE#6 -> LUCAS_BONSKOWSKI_SIGNATURE; device MRDT-Hardware:MOUNTING_HOLE#6 -> MRDT-Signatures:LUCAS_BONSKOWSKI_SIGNATURE
- U$28: value MLX91210 -> MOUNTING_HOLE#6; device buckconverter:MLX91210 -> MRDT-Hardware:MOUNTING_HOLE#6
- U$29: value 530002B02500G -> MLX91210; device buckconverter:530002B02500G -> buckconverter:MLX91210
- U$30: value IPP052N06L3GXKSA1 -> 530002B02500G; device buckconverter:IPP052N06L3GXKSA1 -> buckconverter:530002B02500G
- U$31: value MRDT_LOGO -> IPP052N06L3GXKSA1; device MRDT-2015-General:MRDT_LOGO -> buckconverter:IPP052N06L3GXKSA1
- U$8: value APP_2POS_CONFIGMOCO_VERT -> MRDT_LOGO; device MRDT-Connectors:APP_2POS_CONFIGMOCO_VERT -> MRDT-2015-General:MRDT_LOGO
- renumbered MARLIN-12V to RICK-12V, NEMO-12V to MORTY-12V, RS1 to BMS_SERIAL
Connections:
- removed net N$13: 5VFAN2.1, Q14.D
- net +3V3: now also C.50.1, C.68.1, C.73.1, C.78.1, C.79.1, C.80.1, C.87.1, C.88.1; no longer C.47.1, C.65.1, C.70.1, C.72.1, C.74.1, C.76.1, C.83.1, C.84.1
- net 3.3V: now also C.53.1, C.84.1; no longer C.50.1, C.80.1
- net 5V: now also C.44.+, C.56.1, C.61.1, C.69.2, U$29.VCC; no longer C.53.1, C.60.1, C.66.2, C1.+, U$28.VCC
- net ARM-BUS: now also U$29.IP-; no longer U$28.IP-
- net FAN_CTL_1: no longer Q14.G
- net GND: now also C.44.-, C.45.2, C.47.1, C.56.2, C.61.2, C.65.-, C.66.2, C.67.2, C.69.1, C.70.-, C.78.2, C.81.2, C.82.-, C.89.2, C.90.2, C.91.2, C.92.2, U$13GND.P$1, U$15GND.P$1, U$19GND.P$1, U$22GND.P$1, U$26GND.P$1, U$29.MUST, U$29.VSS, U$9GND.P$1; no longer C.44.2, C.46.1, C.47.2, C.59.2, C.62.2, C.65.2, C.66.1, C.67.-, C.69.2, C.70.2, C.78.-, C.85.2, C.86.2, C1.-, C2.2, CIN1.2, CIN2.-, Q14.S, U$12GND.P$1, U$14GND.P$1, U$18GND.P$1, U$21GND.P$1, U$25GND.P$1, U$28.MUST, U$28.VSS, U$8GND.P$1
- net IMEAS-ARM: now also C.66.1, U$29.VOUT; no longer C.63.1, U$28.VOUT
- net N$11: now also C.83.1; no longer C.79.1
- net N$14: now also C.45.1; no longer C.44.1
- net N$20: now also U$20.OUT; no longer U$19.OUT
- net N$21: now also U$16.OUT; no longer U$15.OUT
- net N$23: now also C.57.1; no longer C.56.1
- net N$24: now also C.46.1; no longer C.45.1
- net N$26: now also C.58.1; no longer C.57.1
- net N$27: now also C.46.2, C.57.2; no longer C.45.2, C.56.2
- net N$29: now also C.60.1; no longer C.59.1
- net N$31: now also C.59.2, U$31.S; no longer C.58.2, U$30.S
- net N$32: now also C.59.1; no longer C.58.1
- net N$33: now also U$31.G; no longer U$30.G
- net N$40: now also C.85.1; no longer C.81.1
- net N$42: now also C.85.2; no longer C.81.2
- net N$43: now also C.86.1; no longer C.82.1
- net N$44: now also C.86.2; no longer C.82.2
- net N$45: now also C.92.1; no longer C.88.1
- net N$5: now also 5VFAN2.1
- net N$9: now also U$16.IN, U$20.IN; no longer U$15.IN, U$19.IN
- net N_$10: now also C.74.1; no longer C.71.1
- net N_$14: now also C.62.1; no longer C.61.1
- net N_$15: now also C.62.2, C.63.1; no longer C.61.2, C.62.1
- net N_$16: now also C.89.1, C.90.1, C.91.1; no longer C.85.1, C.86.1, C.87.1
- net N_$18: now also C.77.1; no longer C.73.1
- net N_$20: now also C.67.1; no longer C.64.1
- net N_$21: now also C.81.1; no longer C.77.1
- net N_$22: now also C.72.1; no longer C.69.1
- net N_$23: now also C.71.1; no longer C.68.1
- net SOURCE-ARM: now also C.64.1, C.65.+, U$31.D; no longer CIN1.1, CIN2.+, U$30.D
- net SOURCE-M2: now also U$9VCC.P$1; no longer U$8VCC.P$1
- net SOURCE-M3: now also U$13VCC.P$1; no longer U$12VCC.P$1
- net SOURCE-M4: now also U$15VCC.P$1; no longer U$14VCC.P$1
- net SOURCE-M5: now also U$19VCC.P$1; no longer U$18VCC.P$1
- net SOURCE-M6: now also U$22VCC.P$1; no longer U$21VCC.P$1
- net SOURCE-M7: now also U$26VCC.P$1; no longer U$25VCC.P$1
- net VOUT12+: now also C.58.2, C.70.+, C.76.1, C.82.+, U$29.IP+; no longer C.57.2, C.67.+, C.78.+, C2.1, U$28.IP+
- net V_BATT: now also C.47.2, U$11.IN, U$14.IN, U$17.IN, U$21.IN, U$25.IN; no longer C.46.2, U$13.IN, U$16.IN, U$20.IN, U$24.IN, U$9.IN
- net V_BATT_M2: now also U$10.OUT; no longer U$9.OUT
- net V_BATT_M3: now also U$11.OUT; no longer U$10.OUT
- net V_BATT_M4: now also U$14.OUT; no longer U$13.OUT
- net V_BATT_M5: now also U$17.OUT; no longer U$16.OUT
- net V_BATT_M6: now also U$21.OUT; no longer U$20.OUT
- net V_BATT_M7: now also U$25.OUT; no longer U$24.OUT
Other:
- moved on the sheet: C.45, C.46, C.47, C.48, C.49, C.50, C.51, C.52, C.53, C.54, C.55, C.56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

Commit message: Rev 2 2018
Integrated tiva/ buck converter removed.  Pack voltage arm bus added. Positive and negative terminals flipped.  Could add pin receptacles to muratas still
Parts:
- removed 3.3V-OKI1: Q_OKI-78SR, MRDT-2015-PowerBoard:Q_OKI-78SR
- removed 5VFAN2: SL02, MRDT-Connectors:SL02
- removed C.47, C.69: .1µF, SparkFun-Capacitors:CAP0805
- removed C.48: 10uF, SparkFun-Capacitors:CAP1206
- removed C.49: 1nF, SparkFun-Capacitors:CAP0805
- removed C.50: .1uF, SparkFun-Capacitors:CAP0805
- removed C.57: 470p, SparkFun-Passives:CAP0603-CAP
- removed C.58: 2200p, SparkFun-Passives:CAP0603-CAP
- removed C.59: 0.1uF, SparkFun-Passives:CAP0603-CAP
- removed C.60: 1uF, SparkFun-Passives:CAP0603-CAP
- removed C.61: 10u, SparkFun-Passives:CAP0603-CAP
- removed C.62: 1000pF, resistor:C-USC0603
- removed C.63: 4700pF, resistor:C-USC1206
- removed C.64: 1000p, SparkFun-Passives:CAP0603-CAP
- removed C.65: 100u, buckconverter:B41858C9107M000
- removed C.66: 10n, SparkFun-Capacitors:CAP0805
- removed C.67, C.68, C.73, C.74, C.75, C.78, C.79, C.80, C.87, C.88, C.90: 0.1uF, resistor:C-USC0603
- removed C.70, C.82: 220u, buckconverter:EGPD101ELL221MK25H
- removed C.71, C.72, C.77, C.81: 12pF, resistor:C-USC0603
- removed C.76: 22p, SparkFun-Passives:CAP0603-CAP
- removed C.89: 2.2uF, resistor:C-USC0603
- removed C.91: 1.0uF, resistor:C-USC0603
- removed D3: RF05VAM1STR, buckconverter:RF05VAM1STR
- removed D4: RBR3MM30ATR, buckconverter:RBR3MM30ATR
- removed J4: RJ45KEYSTONE-942, MRDT-Connectors:RJ45KEYSTONE-942
- removed J5: APP_2POS_CONFIGMOCO_VERT, MRDT-Connectors:APP_2POS_CONFIGMOCO_VERT
- removed J6: JTAG_ARM_10PIN, MRDT-Connectors:JTAG_ARM_10PIN
- removed L1: 3.3uH, buckconverter:PQ3218-3R3-70-T
- removed LED-12: ORANGE, led:LEDCHIP-LED0603
- removed LED-13, LED-14: GREEN, led:LEDCHIP-LED0603
- removed LOGO1, U$34: MRDT_LOGO, MRDT-Hardware:MRDT_LOGO
- removed LTC3703-1: LTC3703-5, MRDT-ICs:LTC3703-5
- removed R.12: 19.1k, SparkFun-Passives:RESISTOR0603-RES
- removed R.15, R.16, R.30: 10k, SparkFun-Passives:RESISTOR0603-RES
- removed R.17: 113k, SparkFun-Passives:RESISTOR0603-RES
- removed R.18: 8.06k, SparkFun-Passives:RESISTOR0603-RES
- removed R.19: 10, SparkFun-Passives:RESISTOR0603-RES
- removed R.24, R.25, R.27, R.29: 75, resistor:R-US_R0603
- removed R.26: 1M, resistor:R-US_R1206
- removed R.28: 1kΩ, SparkFun-Passives:RESISTOR1206
- removed R.31: 10k, resistor:R-US_R0603
- removed R.32: 100, resistor:R-US_R0603
- removed R.33: 49.9, rcl:R-US_R0603
- removed R.34: 4.87k 1%, resistor:R-US_R0603
- removed R.35: 1M, resistor:R-US_R0603
- removed R.36: 49.4, resistor:R-US_R0603
- removed R.37, R.39: 49.9, resistor:R-US_R0603
- removed R.38: 51, resistor:R-US_R0603
- removed R.40: 2k, resistor:R-US_R0603
- removed R.41, R.42, R.43: 330, resistor:R-US_R0603
- removed S1: SWITCH_TACTILE, MRDT-UserInput:SWITCH_TACTILE
- removed TM4C1294NCPDT: TM4C1294NCPDT, MRDT-Microcontrollers:TM4C1294NCPDT
- removed U$32: 530002B02500G, buckconverter:530002B02500G
- removed U$33: IPP052N06L3GXKSA1, buckconverter:IPP052N06L3GXKSA1
- removed U$35, U$36, U$37: MOUNTING_HOLE#6, MRDT-Hardware:MOUNTING_HOLE#6
- removed Y1: CRYATL_32K_SMD, MRDT-Passives:CRYATL_32K_SMD
- removed Y2: NX3225GA, MRDT-Passives:NX3225GA
- C.44: value 22u -> .1µF; device buckconverter:UCZ1K220MCL1GS -> SparkFun-Capacitors:CAP0805
- C.45: value 0.1uF -> .1µF; device SparkFun-Passives:CAP0603-CAP -> SparkFun-Capacitors:CAP0805
- C.46: value 1000p -> 1nF; device SparkFun-Passives:CAP0603-CAP -> SparkFun-Capacitors:CAP0805
- R.11: value 16.5k -> 5kΩ; device SparkFun-Passives:RESISTOR0603-RES -> SparkFun-Passives:RESISTOR1206
- U$23: value MOUNTING_HOLE#6 -> APP_2POS_CONFIGMOCO_VERT; device MRDT-Hardware:MOUNTING_HOLE#6 -> MRDT-Connectors:APP_2POS_CONFIGMOCO_VERT
- U$29: value MLX91210 -> ATC_FUSE_BLOCK; device buckconverter:MLX91210 -> MRDT-Hardware:ATC_FUSE_BLOCK
- U$30: value 530002B02500G -> MOUNTING_HOLE#6; device buckconverter:530002B02500G -> MRDT-Hardware:MOUNTING_HOLE#6
- U$31: value IPP052N06L3GXKSA1 -> MOUNTING_HOLE#6; device buckconverter:IPP052N06L3GXKSA1 -> MRDT-Hardware:MOUNTING_HOLE#6
- U20: value LT1910 -> TIVA-1294; device Jake:LT1910 -> MRDT-Microcontrollers:TIVA-1294
- U21: value SLVU2.8-4 -> LT1910; device MRDT-ICs:SLVU2.8-4 -> Jake:LT1910
- U22: value HX1198FNL -> ACS722LLCTR-40AU-T; device MRDT-ICs:HX1198FNL -> MRDT-2015-PowerBoard:Q_ACS714
Connections:
- removed net !RESET: J6.!RESET, R.32.2, S1.1@A, S1.1@B
- removed net +3V3: 3.3V-OKI1.VO, C.48.1, C.49.1, C.50.1, C.68.1, C.73.1, C.75.1, C.78.1, C.79.1, C.80.1, C.87.1, C.88.1, J6.VTARGET, LED-12.A, R.31.1, R.33.1, R.35.2, R.36.1, R.37.1, R.38.2, R.39.1, TM4C1294NCPDTG$2.VDD@101, TM4C1294NCPDTG$2.VDD@113, TM4C1294NCPDTG$2.VDD@122, TM4C1294NCPDTG$2.VDD@16, TM4C1294NCPDTG$2.VDD@26, TM4C1294NCPDTG$2.VDD@28, TM4C1294NCPDTG$2.VDD@39, TM4C1294NCPDTG$2.VDD@47, TM4C1294NCPDTG$2.VDD@51, TM4C1294NCPDTG$2.VDD@52, TM4C1294NCPDTG$2.VDD@69, TM4C1294NCPDTG$2.VDD@7, TM4C1294NCPDTG$2.VDD@79, TM4C1294NCPDTG$2.VDD@90, TM4C1294NCPDTG$2.VDDA@8, TM4C1294NCPDTG$2.VREFA+@9, U22.P$2, U22.P$7
- removed net ARM-BUS: J5VCC.P$1, R.28.1, U$29.IP-
- removed net EN0LED0: LED-14.A, TM4C1294NCPDTG$1.PF0@42
- removed net EN0LED1: LED-13.A, TM4C1294NCPDTG$1.PF4@46
- removed net EN0RXI_N: R.39.2, TM4C1294NCPDTG$2.EN0RXIN@53, U22.P$8
- removed net EN0RXI_P: R.37.2, TM4C1294NCPDTG$2.EN0RXIP@54, U22.P$6
- removed net EN0TXO_N: R.36.2, TM4C1294NCPDTG$2.EN0TXON@56, U22.P$3
- removed net EN0TXO_P: R.33.2, TM4C1294NCPDTG$2.EN0TXOP@57, U22.P$1
- removed net FAN_CTL_1: Q13.G, TM4C1294NCPDTG$1.PD2@3
- removed net N$10: LTC3703-1.IMAX, R.11.2
- removed net N$14: C.45.1, LTC3703-1.RUN/SS
- removed net N$2: LED-11.A, R.28.2
- removed net N$23: C.57.1, LTC3703-1.COMP, R.16.2
- removed net N$24: C.46.1, R.16.1
- removed net N$26: C.58.1, R.15.1
- removed net N$27: C.46.2, C.57.2, LTC3703-1.FB, R.15.2, R.17.2, R.18.1
- removed net N$29: C.60.1, LTC3703-1.VCC, R.19.1
- removed net N$30: LTC3703-1.BG, U$33.G
- removed net N$31: C.59.2, D4.C, L1.2, LTC3703-1.SW, U$31.S, U$33.D
- removed net N$32: C.59.1, D3.K, LTC3703-1.BOOST
- removed net N$33: LTC3703-1.TG, U$31.G
- removed net N$34: LTC3703-1.FSET, R.12.2
- removed net N$36: Q10.G, U20.GATE
- removed net N_$1: R.29.2, U22.P$15
- removed net N_$10: C.74.1, R.38.1, TM4C1294NCPDTG$2.VBAT@68
- removed net N_$11: J4.4, J4.5, R.25.2
- removed net N_$12: R.35.1, TM4C1294NCPDTG$2.!WAKE@64
- removed net N_$13: J4.7, J4.8, R.24.2
- removed net N_$14: C.62.1, R.24.1, R.25.1, R.27.1, R.29.1
- removed net N_$15: C.62.2, C.63.1, R.26.2
- removed net N_$16: C.89.1, C.90.1, C.91.1, TM4C1294NCPDTG$2.VDDC@115, TM4C1294NCPDTG$2.VDDC@87
- removed net N_$17: R.40.2, TM4C1294NCPDTG$2.OSC1@89
- removed net N_$18: C.77.1, TM4C1294NCPDTG$2.OSC0@88, Y2.OSC1
- removed net N_$19: R.34.2, TM4C1294NCPDTG$2.RBIAS@59
- removed net N_$20: C.67.1, R.31.2, R.32.1, TM4C1294NCPDTG$2.!RESET@70
- removed net N_$21: C.81.1, R.40.1, Y2.OSC0
- removed net N_$22: C.72.1, TM4C1294NCPDTG$2.XOSC1@67, Y1.P$2
- removed net N_$23: C.71.1, TM4C1294NCPDTG$2.XOSC0@66, Y1.P$1
- removed net N_$26: LED-12.C, R.41.1
- removed net N_$3: R.27.2, U22.P$10
- removed net N_$4: J4.2, U21.P$2, U21.P$7, U22.P$14
- removed net N_$5: J4.3, U21.P$3, U21.P$6, U22.P$11
- removed net N_$6: J4.1, U21.P$1, U21.P$8, U22.P$16
- removed net N_$7: J4.6, U21.P$4, U21.P$5, U22.P$9
- removed net N_$8: LED-13.C, R.42.1
- removed net N_$9: LED-14.C, R.43.1
- removed net TARGET_TCK/SWCLK: J6.TCK, TM4C1294NCPDTG$1.PC0@100
- removed net TARGET_TDI: J6.TDI, TM4C1294NCPDTG$1.PC2@98
- removed net TARGET_TDO/SWO: J6.TDO, TM4C1294NCPDTG$1.PC3@97
- removed net TARGET_TMS/SWDIO: J6.TMS, TM4C1294NCPDTG$1.PC1@99
- removed net VOUT12+: C.58.2, C.70.+, C.76.1, C.82.+, L1.1, R.17.1, U$29.IP+
- new net DRAIN-ARM: C.44.2, Q10.D, U21.SENSE, U21.V+, U22.IP-
- new net FAN-CTL: Q13.G, U20.PM3
- new net FILTER-ARM: C.46.1, U22.FILTER
- new net GATE-ARM: Q10.G, U21.GATE
- new net LEDLINE-ARM: LED-11.A, R.11.2
- new net SIG-LOGIC: U20.PH2
- new net V_BATT_ARM: U$29.OUT, U22.IP+
- net 12V-AUX-COM: now also J3VCC.P$1, R.9.1, U18.IP-; no longer J2VCC.P$1, R.5.1, U9.IP-
- net 12V-AUX-LOGIC: now also J2VCC.P$1, R.5.1, U9.IP-; no longer J3VCC.P$1, R.9.1, U18.IP-
- net 3.3V: now also C.45.2, U20.+3V3, U22.VCC
- net 5V: now also U20.+5V; no longer 5VFAN2.2, C.44.+, C.61.1, C.69.2, D3.A, LTC3703-1.DRVCC, LTC3703-1.MODE, R.19.2, U$29.VCC
- net ACT-CTL: now also U20.PN3; no longer TM4C1294NCPDTG$1.PN2@109
- net COM-SIG: no longer TM4C1294NCPDTG$1.PP0@118
- net GND: now also C.44.1, C.45.1, C.46.2, U$23GND.P$1, U21.GND, U22.GND; no longer 3.3V-OKI1.GND, C.44.-, C.45.2, C.47.1, C.48.2, C.49.2, C.50.2, C.60.2, C.61.2, C.63.2, C.64.2, C.65.-, C.66.2, C.67.2, C.68.2, C.69.1, C.70.-, C.71.2, C.72.2, C.73.2, C.74.2, C.75.2, C.76.2, C.77.2, C.78.2, C.79.2, C.80.2, C.81.2, C.82.-, C.87.2, C.88.2, C.89.2, C.90.2, C.91.2, D4.A, J5GND.P$1, J6.!EXTDBG, J6.GND, LTC3703-1.BGRTN, LTC3703-1.GND, LTC3703-1.INV, R.11.1, R.12.1, R.18.2, R.26.1, R.30.1, R.34.1, R.41.2, R.42.2, R.43.2, S1.0@A, S1.0@B, TM4C1294NCPDTG$2.GND@114, TM4C1294NCPDTG$2.GND@17, TM4C1294NCPDTG$2.GND@48, TM4C1294NCPDTG$2.GND@55, TM4C1294NCPDTG$2.GND@58, TM4C1294NCPDTG$2.GND@80, TM4C1294NCPDTG$2.GNDA@10, U$29.MUST, U$29.VSS, U$33.S
- net IMEAS-ACT: now also U20.PE2; no longer TM4C1294NCPDTG$1.PN0@107
- net IMEAS-ARM: now also U20.PD0, U22.VIOUT; no longer C.66.1, R.30.2, TM4C1294NCPDTG$1.PD7@128, U$29.VOUT
- net IMEAS-COM: now also U20.PE1; no longer TM4C1294NCPDTG$1.PP1@119
- net IMEAS-LOGIC: now also U20.PE0; no longer TM4C1294NCPDTG$1.PB4@121
- net IMEAS-M1: now also U20.PK3; no longer TM4C1294NCPDTG$1.PM7@71
- net IMEAS-M2: now also U20.PK2; no longer TM4C1294NCPDTG$1.PM6@72
- net IMEAS-M3: now also U20.PK1; no longer TM4C1294NCPDTG$1.PM5@73
- net IMEAS-M4: now also U20.PK0; no longer TM4C1294NCPDTG$1.PM4@74
- net IMEAS-M5: now also U20.PB5; no longer TM4C1294NCPDTG$1.PM3@75
- net IMEAS-M6: now also U20.PB4; no longer TM4C1294NCPDTG$1.PM2@76
- net IMEAS-M7: now also U20.PE3; no longer TM4C1294NCPDTG$1.PM1@77
- net LOGIC-SIG: no longer TM4C1294NCPDTG$1.PB5@120
- net LOGIC/COM-CTL: now also U20.PP2; no longer TM4C1294NCPDTG$1.PN5@112
- net N$5: no longer 5VFAN2.1
- net SER_RX: now also U20.PC4; no longer J6.P$7, TM4C1294NCPDTG$1.PC4@25
- net SER_TX: now also U20.PC5; no longer J6.GND1, TM4C1294NCPDTG$1.PC5@24
- net SIG-ARM: now also U20.PK5, U21.IN; no longer TM4C1294NCPDTG$1.PD6@127, U20.IN
- net SIG-M1: now also U20.PK7; no longer TM4C1294NCPDTG$1.PL6@94
- net SIG-M2: now also U20.PK6; no longer TM4C1294NCPDTG$1.PL5@86
- net SIG-M3: now also U20.PH1; no longer TM4C1294NCPDTG$1.PL4@85
- net SIG-M4: now also U20.PH0; no longer TM4C1294NCPDTG$1.PL3@84
- net SIG-M5: now also U20.PM2; no longer TM4C1294NCPDTG$1.PL2@83
- net SIG-M6: now also U20.PM1; no longer TM4C1294NCPDTG$1.PL1@82
- net SIG-M7: now also U20.PM0; no longer TM4C1294NCPDTG$1.PL0@81
- net SOURCE-ARM: now also R.11.1, U$23VCC.P$1; no longer C.64.1, C.65.+, LTC3703-1.VIN, U$31.D
- net VMEAS-VBATT: now also U20.PE5; no longer TM4C1294NCPDTG$1.PE5@124
- net V_BATT: now also U$29.IN; no longer 3.3V-OKI1.VI, C.47.2, Q10.D, U20.SENSE, U20.V+
Other:
- note added: "ARM"
- note added: "TIVA"
- note removed: "12V 40A converter"
- note removed: "Ethernet"
- note removed: "Ethernet Activity LED"
- note removed: "Ethernet Link LED"
- note removed: "GPIO"
- note removed: "HEATSINKS"
- note removed: "Hardware"
- note removed: "Integrated Tiva"
- note removed: "JTAG"
- note removed: "JTAG Signals"
- note removed: "MCU Power"
- note removed: "Main Power"
- note removed: "Serial0 back to programmer"
- moved on the sheet: C.45, C.46, LED-11, Q10, R.11
