File: Motor_Controller/Motor_Controller_2019_Rev1.sch (KiCad schematic (older format))
At the start: 244 parts, among them Q12 Q_NMOS_DGS, Q13 Q_NMOS_DGS, Q14 Q_NMOS_DGS, Q15 Q_NMOS_DGS, Q16 Q_NMOS_DGS, Q17 Q_NMOS_DGS, Q4 Q_NMOS_DGS, Q5 Q_NMOS_DGS, Q6 Q_NMOS_DGS, Q7 Q_NMOS_DGS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

Commit message: Fixed netlist naming for GND
Parts:
- removed Conn2: PVDD_M1_PP, MRDT_Connectors:Anderson_1_Horisontal, symbol MRDT_Connectors:AndersonPP
- removed Conn7: PVDD_M2_PP, MRDT_Connectors:Anderson_1_Horisontal, symbol MRDT_Connectors:AndersonPP
- added unit 2 of Conn3
- added unit 2 of Conn8
- Conn3: value GND_M1_PP -> AndersonPP; footprint MRDT_Connectors:Anderson_1_Horisontal -> MRDT_Connectors:Anderson_2_Vertical
- Conn8: value GND_M2_PP -> AndersonPP; footprint MRDT_Connectors:Anderson_1_Horisontal -> MRDT_Connectors:Anderson_2_Vertical
Connections:
- net labels added: SN2_M2_
- net labels removed: SN2_M2, SP1_M1, SP1_M2, SP2_M1, SP2_M2
- wire segments 745 -> 741

Commit message: moved dimension to F.fab layer
Parts:
- C15, C16, C30, C31, C32, C47, C48, C72, C73, C74: footprint Capacitors_SMD:C_0603_HandSoldering -> Capacitors_SMD:C_1206_HandSoldering
- Conn3, Conn8: footprint (none) -> MRDT_Connectors:Anderson_2_Vertical
- R28, R29, R56, R57: footprint Resistors_SMD:R_0603_HandSoldering -> Resistors_SMD:R_1206_HandSoldering
- U3: footprint MotorController_Hardware:LAUNCHXL_F28069M_Launchpad_FULL_Booster_SMD_Bottom -> MotorController_Hardware:LAUNCHXL_F28069M_Launchpad_FULL_Booster_SMD_Top
Changed lines of the file:
@@
 F 0 "C15" H 3975 14800 50  0000 L CNN
 F 1 "0.1u" H 3975 14600 50  0000 L CNN
-F 2 "Capacitors_SMD:C_0603_HandSoldering" H 3988 14550 50  0001 C CNN
+F 2 "Capacitors_SMD:C_1206_HandSoldering" H 3988 14550 50  0001 C CNN
 F 3 "" H 3950 14700 50  0001 C CNN
 	1    3950 14700
@@
 F 0 "C16" H 4475 14650 50  0000 L CNN
 F 1 "0.01u" H 4475 14450 50  0000 L CNN
-F 2 "Capacitors_SMD:C_0603_HandSoldering" H 4488 14400 50  0001 C CNN
+F 2 "Capacitors_SMD:C_1206_HandSoldering" H 4488 14400 50  0001 C CNN
 F 3 "" H 4450 14550 50  0001 C CNN
 	1    4450 14550
@@
 F 0 "C30" H 11375 7750 50  0000 L CNN
 F 1 "2.2u" H 11375 7550 50  0000 L CNN
-F 2 "Capacitors_SMD:C_0603_HandSoldering" H 11388 7500 50  0001 C CNN
+F 2 "Capacitors_SMD:C_1206_HandSoldering" H 11388 7500 50  0001 C CNN
 F 3 "" H 11350 7650 50  0001 C CNN
 	1    11350 7650
@@
 SL_A_M1
 $Comp
-L Device:R R28
-U 1 1 5BA9263F
-P 10600 9600
-F 0 "R28" V 10680 9600 50  0000 C CNN
-F 1 ".001" V 10600 9600 50  0000 C CNN
-F 2 "Resistors_SMD:R_0603_HandSoldering" V 10530 9600 50  0001 C CNN
-F 3 "" H 10600 9600 50  0001 C CNN
-	1    10600 9600
-	1    0    0    -1
-$EndComp
-$Comp
 L Device:C C28
 U 1 1 5BA928E0
@@
 F 0 "C31" H 11375 10900 50  0000 L CNN
 F 1 "2.2u" H 11375 10700 50  0000 L CNN
-F 2 "Capacitors_SMD:C_0603_HandSoldering" H 11388 10650 50  0001 C CNN
+F 2 "Capacitors_SMD:C_1206_HandSoldering" H 11388 10650 50  0001 C CNN
 F 3 "" H 11350 10800 50  0001 C CNN
 	1    11350 10800
@@
 F 0 "R29" V 10680 12750 50  0000 C CNN
 F 1 ".001" V 10600 12750 50  0000 C CNN
-F 2 "Resistors_SMD:R_0603_HandSoldering" V 10530 12750 50  0001 C CNN
+F 2 "Resistors_SMD:R_1206_HandSoldering" V 10530 12750 50  0001 C CNN
 F 3 "" H 10600 12750 50  0001 C CNN
 	1    10600 12750
@@
 F 0 "C32" H 11375 14250 50  0000 L CNN
 F 1 "2.2u" H 11375 14050 50  0000 L CNN
-F 2 "Capacitors_SMD:C_0603_HandSoldering" H 11388 14000 50  0001 C CNN
+F 2 "Capacitors_SMD:C_1206_HandSoldering" H 11388 14000 50  0001 C CNN
 F 3 "" H 11350 14150 50  0001 C CNN
 	1    11350 14150
@@
 F 0 "C72" H 29075 7700 50  0000 L CNN
 F 1 "2.2u" H 29075 7500 50  0000 L CNN
-F 2 "Capacitors_SMD:C_0603_HandSoldering" H 29088 7450 50  0001 C CNN
+F 2 "Capacitors_SMD:C_1206_HandSoldering" H 29088 7450 50  0001 C CNN
 F 3 "" H 29050 7600 50  0001 C CNN
 	1    29050 7600
@@
 F 0 "R56" V 28380 9550 50  0000 C CNN
 F 1 ".001" V 28300 9550 50  0000 C CNN
-F 2 "Resistors_SMD:R_0603_HandSoldering" V 28230 9550 50  0001 C CNN
+F 2 "Resistors_SMD:R_1206_HandSoldering" V 28230 9550 50  0001 C CNN
 F 3 "" H 28300 9550 50  0001 C CNN
 	1    28300 9550
@@
 F 0 "C73" H 29075 10950 50  0000 L CNN
 F 1 "2.2u" H 29075 10750 50  0000 L CNN
-F 2 "Capacitors_SMD:C_0603_HandSoldering" H 29088 10700 50  0001 C CNN
+F 2 "Capacitors_SMD:C_1206_HandSoldering" H 29088 10700 50  0001 C CNN
 F 3 "" H 29050 10850 50  0001 C CNN
 	1    29050 10850
@@
 F 0 "R57" V 28380 12800 50  0000 C CNN
 F 1 ".001" V 28300 12800 50  0000 C CNN
-F 2 "Resistors_SMD:R_0603_HandSoldering" V 28230 12800 50  0001 C CNN
+F 2 "Resistors_SMD:R_1206_HandSoldering" V 28230 12800 50  0001 C CNN
 F 3 "" H 28300 12800 50  0001 C CNN
 	1    28300 12800
@@
 F 0 "C74" H 29075 14300 50  0000 L CNN
 F 1 "2.2u" H 29075 14100 50  0000 L CNN
-F 2 "Capacitors_SMD:C_0603_HandSoldering" H 29088 14050 50  0001 C CNN
+F 2 "Capacitors_SMD:C_1206_HandSoldering" H 29088 14050 50  0001 C CNN
 F 3 "" H 29050 14200 50  0001 C CNN
 	1    29050 14200
@@
 Connection ~ 28300 9400
 Connection ~ 10600 12600
-Connection ~ 10600 9450
 Wire Wire Line
 	27950 15200 27950 15250
@@
 F 0 "U3" H 13850 8200 60  0000 L CNN
 F 1 "LAUNCHXL_F28069M_Launchpad" H 13300 9400 60  0000 L CNN
-F 2 "MotorController_Hardware:LAUNCHXL_F28069M_Launchpad_FULL_Booster_SMD_Bottom" H 13850 8250 60  0001 C CNN
+F 2 "MotorController_Hardware:LAUNCHXL_F28069M_Launchpad_FULL_Booster_SMD_Top" H 13850 8250 60  0001 C CNN
 F 3 "" H 13850 8250 60  0001 C CNN
 	1    13850 8250
@@
 F 0 "U3" H 15350 8200 60  0000 L CNN
 F 1 "LAUNCHXL_F28069M_Launchpad" H 14800 9400 60  0000 L CNN
-F 2 "MotorController_Hardware:LAUNCHXL_F28069M_Launchpad_FULL_Booster_SMD_Bottom" H 15350 8250 60  0001 C CNN
+F 2 "MotorController_Hardware:LAUNCHXL_F28069M_Launchpad_FULL_Booster_SMD_Top" H 15350 8250 60  0001 C CNN
 F 3 "" H 15350 8250 60  0001 C CNN
 	3    15350 8250
@@
 F 0 "U3" H 15350 9650 60  0000 L CNN
 F 1 "LAUNCHXL_F28069M_Launchpad" H 14800 10850 60  0000 L CNN
-F 2 "MotorController_Hardware:LAUNCHXL_F28069M_Launchpad_FULL_Booster_SMD_Bottom" H 15350 9700 60  0001 C CNN
+F 2 "MotorController_Hardware:LAUNCHXL_F28069M_Launchpad_FULL_Booster_SMD_Top" H 15350 9700 60  0001 C CNN
 F 3 "" H 15350 9700 60  0001 C CNN
 	2    15350 9700
@@
 F 0 "U3" H 13850 9650 60  0000 L CNN
 F 1 "LAUNCHXL_F28069M_Launchpad" H 13300 10850 60  0000 L CNN
-F 2 "MotorController_Hardware:LAUNCHXL_F28069M_Launchpad_FULL_Booster_SMD_Bottom" H 13850 9700 60  0001 C CNN
+F 2 "MotorController_Hardware:LAUNCHXL_F28069M_Launchpad_FULL_Booster_SMD_Top" H 13850 9700 60  0001 C CNN
 F 3 "" H 13850 9700 60  0001 C CNN
 	4    13850 9700
@@
 F 0 "U3" H 17300 8200 60  0000 L CNN
 F 1 "LAUNCHXL_F28069M_Launchpad" H 16750 9400 60  0000 L CNN
-F 2 "MotorController_Hardware:LAUNCHXL_F28069M_Launchpad_FULL_Booster_SMD_Bottom" H 17300 8250 60  0001 C CNN
+F 2 "MotorController_Hardware:LAUNCHXL_F28069M_Launchpad_FULL_Booster_SMD_Top" H 17300 8250 60  0001 C CNN
 F 3 "" H 17300 8250 60  0001 C CNN
 	5    17300 8250
@@
 F 0 "U3" H 18900 8250 60  0000 L CNN
 F 1 "LAUNCHXL_F28069M_Launchpad" H 18350 9450 60  0000 L CNN
-F 2 "MotorController_Hardware:LAUNCHXL_F28069M_Launchpad_FULL_Booster_SMD_Bottom" H 18900 8300 60  0001 C CNN
+F 2 "MotorController_Hardware:LAUNCHXL_F28069M_Launchpad_FULL_Booster_SMD_Top" H 18900 8300 60  0001 C CNN
 F 3 "" H 18900 8300 60  0001 C CNN
 	7    18900 8300
@@
 F 0 "U3" H 18900 9650 60  0000 L CNN
 F 1 "LAUNCHXL_F28069M_Launchpad" H 18350 10850 60  0000 L CNN
-F 2 "MotorController_Hardware:LAUNCHXL_F28069M_Launchpad_FULL_Booster_SMD_Bottom" H 18900 9700 60  0001 C CNN
+F 2 "MotorController_Hardware:LAUNCHXL_F28069M_Launchpad_FULL_Booster_SMD_Top" H 18900 9700 60  0001 C CNN
 F 3 "" H 18900 9700 60  0001 C CNN
 	6    18900 9700
@@
 F 0 "U3" H 17300 9650 60  0000 L CNN
 F 1 "LAUNCHXL_F28069M_Launchpad" H 16750 10850 60  0000 L CNN
-F 2 "MotorController_Hardware:LAUNCHXL_F28069M_Launchpad_FULL_Booster_SMD_Bottom" H 17300 9700 60  0001 C CNN
+F 2 "MotorController_Hardware:LAUNCHXL_F28069M_Launchpad_FULL_Booster_SMD_Top" H 17300 9700 60  0001 C CNN
 F 3 "" H 17300 9700 60  0001 C CNN
 	8    17300 9700
@@
 	1    0    0    -1
 $EndComp
-Connection ~ 10600 9750
 $Comp
 L power:GND #PWR0108
@@
 F 0 "C47" H 21675 14800 50  0000 L CNN
 F 1 "0.1u" H 21675 14600 50  0000 L CNN
-F 2 "Capacitors_SMD:C_0603_HandSoldering" H 21688 14550 50  0001 C CNN
+F 2 "Capacitors_SMD:C_1206_HandSoldering" H 21688 14550 50  0001 C CNN
 F 3 "" H 21650 14700 50  0001 C CNN
 	1    21650 14700
@@
 F 0 "C48" H 22175 14650 50  0000 L CNN
 F 1 "0.01u" H 22175 14450 50  0000 L CNN
-F 2 "Capacitors_SMD:C_0603_HandSoldering" H 22188 14400 50  0001 C CNN
+F 2 "Capacitors_SMD:C_1206_HandSoldering" H 22188 14400 50  0001 C CNN
 F 3 "" H 22150 14550 50  0001 C CNN
 	1    22150 14550
@@
 F 0 "Conn8" H 19123 10397 60  0000 R CNN
 F 1 "AndersonPP" H 19123 10503 60  0000 R CNN
-F 2 "" H 19000 9800 60  0001 C CNN
+F 2 "MRDT_Connectors:Anderson_2_Vertical" H 19000 9800 60  0001 C CNN
 F 3 "" H 19000 9800 60  0001 C CNN
 	2    19150 10350
@@
 F 0 "Conn3" H 17773 10397 60  0000 R CNN
 F 1 "AndersonPP" H 17773 10503 60  0000 R CNN
-F 2 "" H 17650 9800 60  0001 C CNN
+F 2 "MRDT_Connectors:Anderson_2_Vertical" H 17650 9800 60  0001 C CNN
 F 3 "" H 17650 9800 60  0001 C CNN
 	2    17800 10350
@@
 Text GLabel 24100 12050 2    39   UnSpc ~ 0
 GND
+Connection ~ 10600 9750
+Connection ~ 10600 9450
+$Comp
+L Device:R R28
+U 1 1 5BA9263F
+P 10600 9600
+F 0 "R28" V 10680 9600 50  0000 C CNN
+F 1 ".001" V 10600 9600 50  0000 C CNN
+F 2 "Resistors_SMD:R_1206_HandSoldering" V 10530 9600 50  0001 C CNN
+F 3 "" H 10600 9600 50  0001 C CNN
+	1    10600 9600
+	1    0    0    -1
+$EndComp
 $EndSCHEMATC
