File: Motor_Controller/Motor_Controller_2019_Rev1.sch (KiCad schematic (older format))
At the start: 242 parts, among them Q12 Q_NMOS_DGS, Q13 Q_NMOS_DGS, Q14 Q_NMOS_DGS, Q15 Q_NMOS_DGS, Q16 Q_NMOS_DGS, Q17 Q_NMOS_DGS, Q4 Q_NMOS_DGS, Q5 Q_NMOS_DGS, Q6 Q_NMOS_DGS, Q7 Q_NMOS_DGS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

Commit message: routed primary control traces
Parts:
- C54, C6: footprint Capacitors_SMD:C_0603_HandSoldering -> Capacitor_THT:CP_Radial_D6.3mm_P2.50mm
Changed lines of the file:
@@
 F 0 "C6" H 3825 8400 50  0000 L CNN
 F 1 "47u" H 3825 8200 50  0000 L CNN
-F 2 "Capacitors_SMD:C_0603_HandSoldering" H 3800 8300 50  0001 C CNN
+F 2 "Capacitor_THT:CP_Radial_D6.3mm_P2.50mm" H 3800 8300 50  0001 C CNN
 F 3 "" H 3800 8300 50  0001 C CNN
 	1    3800 8300
@@
 F 0 "C54" H 21675 8400 50  0000 L CNN
 F 1 "47u" H 21675 8200 50  0000 L CNN
-F 2 "Capacitors_SMD:C_0603_HandSoldering" H 21650 8300 50  0001 C CNN
+F 2 "Capacitor_THT:CP_Radial_D6.3mm_P2.50mm" H 21650 8300 50  0001 C CNN
 F 3 "" H 21650 8300 50  0001 C CNN
 	1    21650 8300

Commit message: Almost done with half of the board
Connections:
- net labels added: +3V3
- net labels removed: PVDDSENSE
- wire segments 741 -> 742
Changed lines of the file:
@@
 NOCTW_M1
 Text GLabel 15100 7500 0    39   Input ~ 0
-PVDDSENSE
+PVDDSENSE_M1
 Text GLabel 15100 7600 0    39   Input ~ 0
 ASENSE_M1
@@
 PWM_IN_M2
 Text GLabel 18650 7550 0    39   Input ~ 0
-PVDDSENSE
+PVDDSENSE_M2
 Text GLabel 18650 7650 0    39   Input ~ 0
 ASENSE_M2
@@
 	4450 8350 4500 8350
 Wire Wire Line
-	4350 8150 4500 8150
+	4350 8150 4400 8150
 Wire Wire Line
 	4500 8150 4500 8250
@@
 	1    0    0    -1
 $EndComp
+$Comp
+L power:+3V3 #PWR0112
+U 1 1 5C04F94E
+P 4500 8150
+F 0 "#PWR0112" H 4500 8000 50  0001 C CNN
+F 1 "+3V3" H 4515 8323 50  0000 C CNN
+F 2 "" H 4500 8150 50  0001 C CNN
+F 3 "" H 4500 8150 50  0001 C CNN
+	1    4500 8150
+	1    0    0    -1
+$EndComp
+$Comp
+L power:+3V3 #PWR0113
+U 1 1 5C04FE6F
+P 22350 8150
+F 0 "#PWR0113" H 22350 8000 50  0001 C CNN
+F 1 "+3V3" H 22365 8323 50  0000 C CNN
+F 2 "" H 22350 8150 50  0001 C CNN
+F 3 "" H 22350 8150 50  0001 C CNN
+	1    22350 8150
+	1    0    0    -1
+$EndComp
+$Comp
+L power:VCC #PWR0114
+U 1 1 5C059F99
+P 4400 8150
+F 0 "#PWR0114" H 4400 8000 50  0001 C CNN
+F 1 "VCC" H 4400 8300 50  0000 C CNN
+F 2 "" H 4400 8150 50  0001 C CNN
+F 3 "" H 4400 8150 50  0001 C CNN
+	1    4400 8150
+	1    0    0    -1
+$EndComp
+Connection ~ 4400 8150
+Wire Wire Line
+	4400 8150 4500 8150
 $EndSCHEMATC

Commit message: Added MAX 3232
Parts:
- removed D2, D22, D23, D24, D25, D26, D27, D28, D29, D30, D31, D32: LED, LEDs:LED_1206_HandSoldering, symbol Device:LED
- removed R36, R37, R64, R65, R66, R67, R68, R69, R70, R71, R72, R73: 1k, Resistors_SMD:R_0603_HandSoldering, symbol Device:R
Connections:
- net labels added: SL_RX_M1, SL_RX_M2, SL_TX_M1, SL_TX_M2
- net labels removed: 232_RX_M1, 232_RX_M2, 232_TX_M1, 232_TX_M2
- wire segments 742 -> 695

Commit message: finished all routing
Parts:
- added D2, D22, D23, D24, D25, D26, D27, D28, D29, D30, D31, D32: LED, LEDs:LED_0603_HandSoldering, symbol Device:LED
- added R36, R37, R64, R65, R66, R67, R68, R69, R70, R71, R72, R73: 500, Resistors_SMD:R_0603_HandSoldering, symbol Device:R
- D13, D14, D3, D33, D34, D35, D36, D4, D5, D6: footprint LEDs:LED_1206_HandSoldering -> LEDs:LED_0603_HandSoldering
Connections:
- net labels removed: SD1_M2
- wire segments 695 -> 742
- no-connect marks 0 -> 27

Commit message: final touches
Parts:
- removed TP20: TEST, Wire_Pads:SolderWirePad_single_1mmDrill, symbol Connector:TestPoint
- added D37: LED, LEDs:LED_0603_HandSoldering, symbol Device:LED
- added R81: 2k, Resistors_SMD:R_0603_HandSoldering, symbol Device:R
Connections:
- net labels added: MGH_A_M1, MGH_A_M2, MGH_B_M1, MGH_B_M2, MGH_C_M1, MGH_C_M2, MGL_A_M1, MGL_A_M2, MGL_B_M1, MGL_B_M2, MGL_C_M1, MGL_C_M2
- net labels removed: PVDD
- wire segments 742 -> 746
- no-connect marks 27 -> 28
Changed lines of the file:
@@
 Text Notes 15850 12800 0    157  ~ 31
 Indicators
-Text GLabel 13300 13250 1    39   Input ~ 0
-PVDD
 $Comp
 L Device:LED D3
@@
 Wire Notes Line
 	30750 16250 20150 16250
-Wire Notes Line
-	12750 12800 20100 12800
 Wire Wire Line
 	3950 15100 4450 15100
@@
 	16300 14150 16600 14150
 Text GLabel 19250 13250 1    39   Input ~ 0
-UART_TX_M2
+SL_TX_M2
 Text GLabel 19550 13250 1    39   Input ~ 0
-UART_RX_M2
+SL_RX_M2
 Text GLabel 18650 13250 1    39   Input ~ 0
-UART_TX_M1
+SL_TX_M1
 Text GLabel 18950 13250 1    39   Input ~ 0
-UART_RX_M1
+SL_RX_M1
 Text GLabel 15400 11600 2    39   Output ~ 0
 SL_TX_M1
@@
 	1    0    0    -1
 $EndComp
-$Comp
-L Connector:TestPoint TP20
-U 1 1 5BB180D3
-P 22000 10750
-F 0 "TP20" H 22000 11050 50  0000 C BNN
-F 1 "TEST" H 22000 11000 50  0000 C CNN
-F 2 "Wire_Pads:SolderWirePad_single_1mmDrill" H 22000 10750 50  0001 C CNN
-F 3 "" H 22000 10750 50  0001 C CNN
-	1    22000 10750
-	1    0    0    -1
-$EndComp
 NoConn ~ 15150 7400
 $Comp
@@
 	18950 14150 19250 14150
 Text GLabel 15100 13250 1    39   Input ~ 0
-GH_A_M1
+MGH_A_M1
 Text GLabel 15400 13250 1    39   Input ~ 0
-SL_A_M1
+MGL_A_M1
 Text GLabel 15700 13250 1    39   Input ~ 0
-GH_B_M1
+MGH_B_M1
 Text GLabel 16000 13250 1    39   Input ~ 0
-GL_B_M1
+MGL_B_M1
 Text GLabel 16300 13250 1    39   Input ~ 0
-GH_C_M1
+MGH_C_M1
 Text GLabel 16600 13250 1    39   Input ~ 0
-GL_C_M1
+MGL_C_M1
 Text GLabel 16900 13250 1    39   Input ~ 0
-GH_A_M2
+MGH_A_M2
 Text GLabel 17200 13250 1    39   Input ~ 0
-GL_A_M2
-Text GLabel 17500 13250 1    39   Input ~ 0
-SH_B_M2
+MGL_A_M2
 Text GLabel 17800 13250 1    39   Input ~ 0
-GL_B_M2
+MGL_B_M2
 Text GLabel 18050 13250 1    39   Input ~ 0
-GH_C_M2
+MGH_C_M2
 Text GLabel 18350 13250 1    39   Input ~ 0
-GL_C_M2
+MGL_C_M2
+Text GLabel 13300 13250 1    39   Input ~ 0
+PVDD_M1
+$Comp
+L Device:LED D37
+U 1 1 5E0B3DA6
+P 13050 13500
+F 0 "D37" H 13050 13600 50  0000 C CNN
+F 1 "LED" H 13050 13400 50  0000 C CNN
+F 2 "LEDs:LED_0603_HandSoldering" H 13050 13500 50  0001 C CNN
+F 3 "" H 13050 13500 50  0001 C CNN
+	1    13050 13500
+	0    -1   -1   0
+$EndComp
+$Comp
+L Device:R R81
+U 1 1 5E0B3DAC
+P 13050 13900
+F 0 "R81" V 13130 13900 50  0000 C CNN
+F 1 "2k" V 13050 13900 50  0000 C CNN
+F 2 "Resistors_SMD:R_0603_HandSoldering" V 12980 13900 50  0001 C CNN
+F 3 "" H 13050 13900 50  0001 C CNN
+	1    13050 13900
+	-1   0    0    1
+$EndComp
+Wire Wire Line
+	13050 13650 13050 13750
+Wire Wire Line
+	13050 13250 13050 13350
+Text GLabel 13050 13250 1    39   Input ~ 0
+PVDD_M2
+Wire Wire Line
+	13050 14150 13050 14050
+Connection ~ 13300 14150
+Wire Wire Line
+	13300 14150 13050 14150
+Wire Notes Line
+	12800 12850 20150 12850
+Text GLabel 17500 13250 1    39   Input ~ 0
+MGH_B_M2
+Text Label 10250 7800 0    50   ~ 0
+MGH_A_M1
+Text Label 10250 8650 0    50   ~ 0
+MGL_A_M1
+Text Label 10250 10950 0    50   ~ 0
+MGH_B_M1
+Text Label 10250 11800 0    50   ~ 0
+MGL_B_M1
+Text Label 10250 14300 0    50   ~ 0
+MGH_C_M1
+Text Label 10250 15150 0    50   ~ 0
+MGL_C_M1
+Text Label 27950 7750 0    50   ~ 0
+MGH_A_M2
+Text Label 27950 8600 0    50   ~ 0
+MGL_A_M2
+Text Label 27950 11000 0    50   ~ 0
+MGH_B_M2
+Text Label 27950 11850 0    50   ~ 0
+MGL_B_M2
+Text Label 27950 14350 0    50   ~ 0
+MGH_C_M2
+Text Label 27950 15200 0    50   ~ 0
+MGL_C_M2
+NoConn ~ 22850 8000
 $EndSCHEMATC

Commit message: Schematic changes
Connections:
- net labels added: +BATT
- wire segments 746 -> 745
Changed lines of the file:
@@
 	4450 8350 4500 8350
-Wire Wire Line
-	4350 8150 4400 8150
 Wire Wire Line
 	4500 8150 4500 8250
@@
 Text GLabel 14700 11950 0    39   Input ~ 0
 SL_TX_M1
-Text GLabel 14700 12050 0    39   Input ~ 0
+Text GLabel 14700 12050 0    39   Output ~ 0
 SL_RX_M1
-Text GLabel 14700 12150 0    39   Input ~ 0
-SL_TX_M2
-Text GLabel 14700 12250 0    39   Input ~ 0
-SL_RX_M2
 Wire Wire Line
 	14700 11950 14750 11950
 Wire Wire Line
 	14700 12050 14750 12050
-Wire Wire Line
-	14700 12150 14750 12150
-Wire Wire Line
-	14700 12250 14750 12250
 $Comp
 L Device:R R9
@@
 	1    0    0    -1
 $EndComp
-$Comp
-L power:VCC #PWR0114
-U 1 1 5C059F99
-P 4400 8150
-F 0 "#PWR0114" H 4400 8000 50  0001 C CNN
-F 1 "VCC" H 4400 8300 50  0000 C CNN
-F 2 "" H 4400 8150 50  0001 C CNN
-F 3 "" H 4400 8150 50  0001 C CNN
-	1    4400 8150
-	1    0    0    -1
-$EndComp
-Connection ~ 4400 8150
-Wire Wire Line
-	4400 8150 4500 8150
 Wire Wire Line
 	14800 14150 15100 14150
@@
 MGL_C_M2
 NoConn ~ 22850 8000
+Wire Wire Line
+	14700 12250 14750 12250
+Wire Wire Line
+	14700 12150 14750 12150
+Text GLabel 14700 12250 0    39   Output ~ 0
+SL_RX_M2
+Text GLabel 14700 12150 0    39   Input ~ 0
+SL_TX_M2
+$Comp
+L power:+BATT #PWR?
+U 1 1 5C113B51
+P 4400 7150
+F 0 "#PWR?" H 4400 7000 50  0001 C CNN
+F 1 "+BATT" H 4415 7323 50  0000 C CNN
+F 2 "" H 4400 7150 50  0001 C CNN
+F 3 "" H 4400 7150 50  0001 C CNN
+	1    4400 7150
+	1    0    0    -1
+$EndComp
+Wire Wire Line
+	4350 8150 4500 8150
 $EndSCHEMATC

Commit message: saved sch
Parts:
- D7: value D_Zener -> 15V
Other:
- note added: "Look at these"
- note added: "MAX 3232"
- note added: "MUX Sel (7=1, 6=1)"
- note added: "Why here?"
- note removed: "Analog out from ACS711 \ngoes to S01 (A_A0) and \nS02 (A_B0) on F28069 headers"
- note removed: "MAX_3232"
- note removed: "New current sensing technique in \nGimbal VFD schematic, uses ACS711 in \nPhase A and B instead of current \nsensing using DRV8301"
Changed lines of the file:
@@
 P 10250 8050
 F 0 "D7" H 10250 8150 50  0000 C CNN
-F 1 "D_Zener" H 10250 7950 50  0000 C CNN
+F 1 "15V" H 10250 7950 50  0000 C CNN
 F 2 "Diodes_SMD:D_SOD-123" H 10250 8050 50  0001 C CNN
 F 3 "" H 10250 8050 50  0001 C CNN
@@
 $EndComp
 Text Notes 14100 10200 0    157  ~ 31
-MAX_3232
+MAX 3232
 Text GLabel 18700 10450 0    39   Input ~ 0
 PVDD_M2
@@
 Text Notes 17250 7000 0    157  ~ 31
 Motor Header 2
-Text Notes 2700 10000 0    60   ~ 0
-New current sensing technique in \nGimbal VFD schematic, uses ACS711 in \nPhase A and B instead of current \nsensing using DRV8301
-Text Notes 2700 10350 0    60   ~ 0
-Analog out from ACS711 \ngoes to S01 (A_A0) and \nS02 (A_B0) on F28069 headers
 $Comp
 L power:VCC #PWR044
@@
 	1    0    0    -1
 $EndComp
-Text Notes 20450 10000 0    60   ~ 0
-New current sensing technique in \nGimbal VFD schematic, uses ACS711 in \nPhase A and B instead of current \nsensing using DRV8301
-Text Notes 20450 10350 0    60   ~ 0
-Analog out from ACS711 \ngoes to S01 (A_A0) and \nS02 (A_B0) on F28069 headers
 $Comp
 L Device:CP1 C39
@@
 Wire Wire Line
 	4350 8150 4500 8150
+Text Notes 12900 7550 0    50   ~ 0
+Look at these
+Text Notes 12900 7750 0    50   ~ 0
+Why here?
+Text Notes 14300 7300 0    50   ~ 0
+MUX Sel (7=1, 6=1)
 $EndSCHEMATC
