File: Motor_Controller/Motor_Controller_2019_Rev1.kicad_pcb (KiCad board)
At the start: 2 copper layers, 124.4 x 86.1 mm, 242 parts, among them Q12 Q_NMOS_DGS, Q13 Q_NMOS_DGS, Q14 Q_NMOS_DGS, Q15 Q_NMOS_DGS, Q16 Q_NMOS_DGS, Q17 Q_NMOS_DGS, Q4 Q_NMOS_DGS, Q5 Q_NMOS_DGS, Q6 Q_NMOS_DGS, Q7 Q_NMOS_DGS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

Commit message: Almost done with half of the board
Parts:
- C54: footprint Capacitors_SMD:C_0603_HandSoldering -> Capacitor_THT:CP_Radial_D6.3mm_P2.50mm
- U1: value DCA56_6P35X3P61 -> DRV8301
- U2: moved to B.Cu
- moved R33 187.4 mm to (96.6, 45.5), turned to 270 degrees
- moved R15 179.8 mm to (104.1, 45.5), turned to 90 degrees
- moved C33 171.1 mm to (100.9, 50.0), turned to 270 degrees
- moved R32 170.8 mm to (98.2, 45.5), turned to 90 degrees
- moved R34 170.2 mm to (98.2, 50.1), turned to 90 degrees
- moved L1 157.1 mm to (120.9, 80.1), turned to 270 degrees
- moved U2 152.6 mm to (95.5, 35.2), turned to 270 degrees
- moved C3 150.8 mm to (115.6, 76.1), turned to 90 degrees
- moved C34 148.4 mm to (95.0, 45.3), turned to 270 degrees
- moved C21 148.1 mm to (100.9, 45.3), turned to 270 degrees
- moved C1 148.0 mm to (113.8, 76.1), turned to 90 degrees
- moved R35 147.3 mm to (96.6, 50.1), turned to 270 degrees
- moved C35 145.9 mm to (95.0, 50.0), turned to 270 degrees
- moved R31 140.4 mm to (102.5, 50.1), turned to 270 degrees
- moved R16 138.6 mm to (102.5, 45.5), turned to 270 degrees
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Connections:
- C13 pad 1: Net-(C13-Pad1) -> +3V3
- C42 pad 1: VCC -> +3V3
- C58 pad 1: Net-(C58-Pad1) -> +3V3
- D1 pad 1: Net-(C13-Pad1) -> +3V3
- D15 pad 1: Net-(C58-Pad1) -> +3V3
- D4 pad 2: VCC -> +3V3
- L1 pad 2: Net-(C13-Pad1) -> +3V3
- L2 pad 2: Net-(C58-Pad1) -> +3V3
- R1 pad 1: VCC -> +3V3
- R2 pad 1: VCC -> +3V3
- R3 pad 1: VCC -> +3V3
- R38 pad 1: VCC -> +3V3
- R39 pad 1: VCC -> +3V3
- R4 pad 1: VCC -> +3V3
- R40 pad 1: VCC -> +3V3
- R42 pad 1: VCC -> +3V3
- TP1 pad 1: VCC -> +3V3
- TP20 pad 1: VCC -> +3V3
- U1 pad 24: VCC -> +3V3
- U1 pad 49: VCC -> +3V3
- U1 pad 50: Net-(C13-Pad1) -> +3V3
- U1 pad 51: Net-(C13-Pad1) -> +3V3
- U2 pad 2: VCC -> +3V3
- U3 pad +3V3: VCC -> +3V3
- U3 pad A_A7: PVDDSENSE -> PVDDSENSE_M1
- U3 pad A_B7: PVDDSENSE -> PVDDSENSE_M2
- U4 pad 16: VCC -> +3V3
- U5 pad 24: VCC -> +3V3
- U5 pad 49: VCC -> +3V3
- U5 pad 50: Net-(C58-Pad1) -> +3V3
- U5 pad 51: Net-(C58-Pad1) -> +3V3
- U6 pad 2: VCC -> +3V3
Routing:
- net +3V3: track 0.00 -> 142.3 mm
- net SDI_M1: track 9.20 -> 71.2 mm, vias 0 -> 2
- net SO1_M1: track 0.00 -> 61.6 mm, vias 0 -> 2
- net SO2_M1: track 0.00 -> 61.2 mm, vias 0 -> 2
- net EN_GATE_M1: track 0.00 -> 60.1 mm, vias 0 -> 2
- net INH_A_M1: track 0.00 -> 58.1 mm, vias 0 -> 2
- net SDO_M1: track 9.08 -> 65.6 mm, vias 0 -> 2
- net INL_A_M1: track 0.00 -> 54.4 mm, vias 0 -> 2
- net INH_B_M1: track 0.00 -> 50.8 mm, vias 0 -> 2
- net DC_CAL_M1: track 6.02 -> 55.5 mm, vias 0 -> 2
- net NSCS_M1: track 9.20 -> 58.3 mm, vias 0 -> 2
- net INL_B_M1: track 0.00 -> 47.0 mm, vias 0 -> 2
- net SCLK_M1: track 9.33 -> 56.3 mm, vias 0 -> 2
- net INH_C_M1: track 0.00 -> 44.9 mm, vias 0 -> 2
- net INL_C_M1: track 0.00 -> 40.3 mm, vias 0 -> 2
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- added copper zone on B.Cu, net (none)
