File: Motor_Controller/_saved_Motor_Controller_2019_Rev1.sch (KiCad schematic (older format))
At the start: 218 parts, among them Q12 Q_NMOS_DGS, Q13 Q_NMOS_DGS, Q14 Q_NMOS_DGS, Q15 Q_NMOS_DGS, Q16 Q_NMOS_DGS, Q17 Q_NMOS_DGS, Q4 Q_NMOS_DGS, Q5 Q_NMOS_DGS, Q6 Q_NMOS_DGS, Q7 Q_NMOS_DGS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

Commit message: finished all routing
Parts:
- removed TP20: TEST, Wire_Pads:SolderWirePad_single_1mmDrill, symbol Connector:TestPoint
- added D2, D22, D23, D24, D25, D26, D27, D28, D29, D30, D31, D32, D37: LED, LEDs:LED_0603_HandSoldering, symbol Device:LED
- added R36, R37, R64, R65, R66, R67, R68, R69, R70, R71, R72, R73: 500, Resistors_SMD:R_0603_HandSoldering, symbol Device:R
- added R81: 2k, Resistors_SMD:R_0603_HandSoldering, symbol Device:R
- D13, D14, D3, D33, D34, D35, D36, D4, D5, D6: footprint LEDs:LED_1206_HandSoldering -> LEDs:LED_0603_HandSoldering
Connections:
- net labels added: MGH_A_M1, MGH_A_M2, MGH_B_M1, MGH_B_M2, MGH_C_M1, MGH_C_M2, MGL_A_M1, MGL_A_M2, MGL_B_M1, MGL_B_M2, MGL_C_M1, MGL_C_M2
- net labels removed: PVDD
- wire segments 695 -> 746
- no-connect marks 0 -> 28
