File: PowerBoardHardware/PowerBoard-Hardware(Evan Hite)/PowerBoard-Hardware(Evan Hite).sch (KiCad schematic (older format))
At the start: 38 parts

Commit message: Added Tiva Headers
I added Tiva Headers, a full booster and finished the Logic/Communication/Actuation circuit from direct battery power.
Parts:
- added 0.1nF, 1nF, 2.2uF: C_Small, symbol Device:C_Small
- added 100k, 1k (x2): R_US, symbol Device:R_US
- added 330uF: CP1, symbol Device:CP1
- added ATC_FUSE_BLOCK (x4): Fuse_Polarized, symbol Device:Fuse_Polarized
- added CONV?: DC-DC_Converter, symbol DC-DC~Converter:DC-DC_Converter
- added Conn?, VCC: AndersonPP, symbol MRDT_Connectors:AndersonPP
- added D?: LED, symbol Device:LED
- added Q?: IPT020N10N3, Package_TO_SOT_SMD:Infineon_PG-HSOF-8-1, symbol Transistor_FET:IPT020N10N3
- added U?: ACS714xLCTR-05B, Package_SO:SOIC-8_3.9x4.9mm_P1.27mm, symbol Sensor_Current:ACS714xLCTR-05B
- added U? (x8): TM4C129E_Launchpad, symbol MRDT_Shields:TM4C129E_Launchpad
Connections:
- net labels added: 5V, ACT-CTL, FAN-CTL, IMEAS-ACT, IMEAS-ARM, IMEAS-M1, IMEAS-M2, IMEAS-M3, IMEAS-M4, IMEAS-M5, IMEAS-M6, IMEAS-M7, LOGIC-SIG, SER_RX, SER_TX, SIG-ARM, SIG-M1, SIG-M2, SIG-M3, SIG-M4, SIG-M5, SIG-M6, SIG-M7
- wire segments 122 -> 204
Other:
- note added: "Actuation 12V"
- note added: "TIVA Headers"
- moved on the sheet: Q?, U?

Commit message: Finished Schematic and added new library
The ATC_FUSE_BLOCK Library was added for this project. The Murata library was now moved to the project folder. It was in the project earlier, but now is present. MRDT Libraries were updated as well. The schematic is now finished and is now complete. The netlist is yet to be generated.
Parts:
- removed ATC_FUSE_BLOCK (x6): Fuse_Polarized, symbol Device:Fuse_Polarized
- added 0.1uF (x23), 10uF (x2), 1nF (x10): C_Small, symbol Device:C_Small
- added 3V3FAN: Molex_SL_02, symbol MRDT_Connectors:Molex_SL_02
- added 5k (x8): R_US, symbol Device:R_US
- added Conn?: Molex_SL_03, symbol MRDT_Connectors:Molex_SL_03
- added Conn? (x8), VCC (x8): AndersonPP, symbol MRDT_Connectors:AndersonPP
- added D? (x8): LED, symbol Device:LED
- added Q?: IPT020N10N3, Package_TO_SOT_SMD:Infineon_PG-HSOF-8-1, symbol Transistor_FET:IPT020N10N3
- added Q? (x8): Q_NMOS_DGS, symbol Device:Q_NMOS_DGS
- added U?: OKI, symbol MRDT_Devices:OKI
- added U?: MAX3232, symbol Interface_UART:MAX3232
- added U? (x11): ATC_FUSE_BLOCK, symbol Fuse_Block:ATC_FUSE_BLOCK
- added U? (x8): ACS714xLCTR-05B, Package_SO:SOIC-8_3.9x4.9mm_P1.27mm, symbol Sensor_Current:ACS714xLCTR-05B
- added U? (x8): LT1910, symbol MRDT_ICs:LT1910
- renumbered 0.1nF to 0.1uF
Connections:
- wire segments 204 -> 601
Other:
- note added: "ARM"
- note added: "DATA"
- note added: "Decoupling Capacitors"
- note added: "M1"
- note added: "M2"
- note added: "M3"
- note added: "M4"
- note added: "M5"
- note added: "M6"
- note added: "M7"
- note added: "MOTORS 1-7 AND ARM"
- note added: "On-Board Power"

Commit message: Updated labelings on Schematic
Got rid of data section of schematic. Made labels bigger and prettier for the schematic for ease of viewing.
Parts:
- removed 0.1uF (x5): C_Small, symbol Device:C_Small
- removed Conn?: Molex_SL_03, symbol MRDT_Connectors:Molex_SL_03
- removed U?: MAX3232, symbol Interface_UART:MAX3232
Connections:
- wire segments 601 -> 566
Other:
- note added: "Arm Motor"
- note added: "Fan Power/Control"
- note added: "Motor 1"
- note added: "Motor 2"
- note added: "Motor 3"
- note added: "Motor 4"
- note added: "Motor 5"
- note added: "Motor 6"
- note added: "Motor 7"
- note added: "Primary Voltage Measuring\n<---------------"
- note removed: "ARM"
- note removed: "DATA"
- note removed: "M1"
- note removed: "M2"
- note removed: "M3"
- note removed: "M4"
- note removed: "M5"
- note removed: "M6"
- note removed: "M7"
- note removed: "Primary Voltage Measuring"
- moved on the sheet: U?

Commit message: Completed Netlist
Netlist is complete, possible errors to be fixed in next commit. The schematic is finalized, only flags need correction. Updated Schematic FIles for DC-DC Buck Converter. Created obsolete Fuse Block. DO NOT ADD. Layout is generated but no work has begun.
Parts:
- 0.1uF1, 0.1uF10, 0.1uF11, 0.1uF12, 0.1uF13, 0.1uF14, 0.1uF15, 0.1uF16, 0.1uF17, 0.1uF18, 0.1uF19, 0.1uF2, 0.1uF20, 0.1uF21, 0.1uF3, 0.1uF4, 0.1uF5, 0.1uF6, 0.1uF7, 0.1uF8, 0.1uF9: renamed from 0.1uF; footprint (none) -> Capacitors_SMD:C_0603_HandSoldering
- 1.5KE36A1, 1.5KE36A2: renamed from 1.5KE36A; footprint (none) -> Diodes_THT:D_DO-201AD_P5.08mm_Vertical_KathodeUp
- 100k1, 100k2, 100k3: renamed from 100k; footprint (none) -> Resistors_SMD:R_0603_HandSoldering
- 10k1: renamed from 10k; footprint (none) -> Resistors_SMD:R_0603_HandSoldering
- 10uF1, 10uF2: renamed from 10uF; footprint (none) -> Capacitors_SMD:C_0603_HandSoldering
- 1k1, 1k2, 1k3, 1k4, 1k5: renamed from 1k; footprint (none) -> Resistors_SMD:R_0603_HandSoldering
- 1mF1: renamed from 1mF; footprint (none) -> Capacitors_THT:CP_Radial_D12.5mm_P5.00mm
- 1mF2, 1mF3, 1mF4: renamed from 1mF?; footprint (none) -> Capacitors_THT:CP_Radial_D12.5mm_P5.00mm
- 1nF1, 1nF10, 1nF11, 1nF12, 1nF13, 1nF2, 1nF3, 1nF4, 1nF5, 1nF6, 1nF7, 1nF8, 1nF9: renamed from 1nF; footprint (none) -> Capacitors_SMD:C_0603_HandSoldering
- 2.2uF1, 2.2uF2, 2.2uF3: renamed from 2.2uF; footprint (none) -> Capacitors_SMD:C_0603_HandSoldering
- 330uF1, 330uF2, 330uF3, 330uF4, 330uF5: renamed from 330uF; footprint (none) -> Capacitors_THT:CP_Radial_D6.3mm_P2.50mm
- 3V3FAN1: renamed from 3V3FAN; footprint (none) -> MRDT-Connectors:MOLEX_SL_02_Horizontal
- 5k1, 5k2, 5k3, 5k4, 5k5, 5k6, 5k7, 5k8: renamed from 5k; footprint (none) -> Resistors_SMD:R_0603_HandSoldering
- CONV1, CONV2: renamed from CONV?; footprint (none) -> DC-DC_Converter_Quarter_Brick:DC-DC Converter (Murata)
- Conn1, Conn10, Conn11, Conn2, Conn3, Conn4, Conn5, Conn6, Conn7, Conn8, Conn9: renamed from Conn?; footprint (none) -> MRDT-Connectors:Anderson_2_Vertical
- D1, D10, D11, D2, D3, D4, D5, D6, D7, D8, D9: renamed from D?; footprint (none) -> LEDs:LED_0603_HandSoldering
- Q1, Q2, Q3, Q4, Q5: renamed from Q?; footprint Package_TO_SOT_SMD:Infineon_PG-HSOF-8-1 -> TO_SOT_Packages_SMD:SOT-323_SC-70_Handsoldering
- Q10, Q11, Q12, Q13, Q6, Q7, Q8, Q9: renamed from Q?; footprint (none) -> TO_SOT_Packages_SMD:TO-263-2
- U1: renamed from U?; footprint (none) -> MRDT-SHIELDS:TM4C129E_Launchpad_FULL
- U10: renamed from U?; footprint (none) -> MRDT-Devices:OKI_Horizontal
- U11, U12, U13, U14, U23, U24, U25, U26, U5, U6: renamed from U?; footprint (none) -> Housings_SOIC:SOIC-8_3.9x4.9mm_Pitch1.27mm
- U15, U16, U17, U18, U2, U27, U28, U29, U3, U30, U4: renamed from U?; footprint (none) -> MRDT-Passives:ATC_Fuse_Block
- gave numbers to parts that had none: 11
- renumbered VCC to VCC1, VCC to VCC10, VCC to VCC11, VCC to VCC2, VCC to VCC3, VCC to VCC4, VCC to VCC5, VCC to VCC6, VCC to VCC7, VCC to VCC8, VCC to VCC9
Connections:
- net labels added: IMEAS-AUX, SIG-AUX
- net labels removed: IMEAS-ARM, SIG-ARM
- wire segments 566 -> 574
Other:
- note added: "Auxillary"
- note added: "MOTORS 1-7 AND AUX"
- note removed: "Arm Motor"
- note removed: "MOTORS 1-7 AND ARM"

Commit message: Reassigned Libraries
Reassigned Libraries to make sure everything works after file organization.
Parts:
- CONV1, CONV2: footprint DC-DC_Converter_Quarter_Brick:DC-DC Converter (Murata) -> DC-DC_Converter_Quarter_Brick:DC-DC_Converter_Quarter_Brick; symbol DC-DC~Converter:DC-DC_Converter -> DC-DC_Converter:DC-DC_Converter
Connections:
- wire segments 574 -> 572
Changed lines of the file:
@@
 	4350 2400 4350 2650
 $Comp
-L DC-DC~Converter:DC-DC_Converter CONV1
+L DC-DC_Converter:DC-DC_Converter CONV1
 U 1 1 5BB35538
 P 2450 2350
 F 0 "CONV1" H 3100 2500 50  0000 C CNN
 F 1 "DC-DC_Converter" H 3100 2400 50  0000 C CNN
-F 2 "DC-DC_Converter_Quarter_Brick:DC-DC Converter (Murata)" H 3000 2650 50  0001 C CNN
+F 2 "DC-DC_Converter_Quarter_Brick:DC-DC_Converter_Quarter_Brick" H 3000 2650 50  0001 C CNN
 F 3 "" H 3000 2650 50  0001 C CNN
 	1    2450 2350
@@
 $EndComp
 $Comp
-L DC-DC~Converter:DC-DC_Converter CONV2
+L DC-DC_Converter:DC-DC_Converter CONV2
 U 1 1 5BBF2506
 P 3050 7200
 F 0 "CONV2" H 3818 7775 50  0000 C CNN
 F 1 "DC-DC_Converter" H 3818 7684 50  0000 C CNN
-F 2 "DC-DC_Converter_Quarter_Brick:DC-DC Converter (Murata)" H 3600 7500 50  0001 C CNN
+F 2 "DC-DC_Converter_Quarter_Brick:DC-DC_Converter_Quarter_Brick" H 3600 7500 50  0001 C CNN
 F 3 "" H 3600 7500 50  0001 C CNN
 	1    3050 7200
@@
 Connection ~ 3800 2400
 Wire Wire Line
-	3700 2800 3700 2950
-Wire Wire Line
 	3700 2950 3500 2950
 Wire Wire Line
@@
 	3750 2400 3700 2400
 Wire Wire Line
-	3700 2700 3700 2800
-Connection ~ 3700 2800
-Wire Wire Line
 	4600 7150 4600 7250
 Wire Wire Line
@@
 	4600 7250 4600 7400
 Wire Wire Line
-	4300 7550 4300 7650
-Wire Wire Line
-	4300 7650 4300 7750
-Connection ~ 4300 7650
-Wire Wire Line
 	4300 7350 4300 7250
-Connection ~ 4300 7250
 Wire Wire Line
 	3100 7250 3050 7250
@@
 Wire Wire Line
 	2650 7400 2650 7550
+Wire Wire Line
+	3700 2700 3700 2950
+Wire Wire Line
+	4300 7550 4300 7750
 $EndSCHEMATC

Commit message: Updated Layout
Basic Layout Positioning has begun. DC-DC converters placed. Logic, Actuation, and Communication are placed. One motor has been placed. The rest will be placed at a later time.
Parts:
- U19, U20, U21, U22, U31, U32, U33, U34, U7, U8, U9: footprint Package_SO:SOIC-8_3.9x4.9mm_P1.27mm -> Housings_SOIC:SOIC-8_3.9x4.9mm_Pitch1.27mm
- VCC1, VCC10, VCC11, VCC2, VCC3, VCC4, VCC5, VCC6, VCC7, VCC8, VCC9: footprint (none) -> MRDT-Connectors:Anderson_2_Vertical
Connections:
- net labels added: PVDD
- net labels removed: +BATT, -BATT, V_BATT
- wire segments 572 -> 570

Commit message: 1st Placement is complete
The first placement is now complete, traces still need to be added. The schematic was updated with the placement of Andersons. Certain andersons were in the wrong areas on the schematic. Silkscreen of each motor needs to be added. Outline of board is now in edge cuts.
Connections:
- wire segments 570 -> 572

Commit message: Added Signal Lines
Most of the traces for all signals have been made. Added a pin map file.
Connections:
- net labels removed: LOGIC_SIG
Changed lines of the file:
@@
 $EndComp
 Text GLabel 5100 3000 0    50   Input ~ 0
-LOGIC_SIG
+LOGIC-SIG
 Wire Wire Line
 	5850 3450 5850 3600
