File: PowerBoardHardware/PowerBoard-Hardware(Evan Hite)/PowerBoard-Hardware(Evan Hite).kicad_pcb (KiCad board)
At the start: 4 copper layers, 279.4 x 127 mm, 141 parts, among them Q1 IPT020N10N3, Q10 Q_NMOS_DGS, Q11 Q_NMOS_DGS, Q12 Q_NMOS_DGS, Q13 Q_NMOS_DGS, Q2 IPT020N10N3, Q3 IPT020N10N3, Q4 IPT020N10N3, Q5 IPT020N10N3, Q6 Q_NMOS_DGS, Q7 Q_NMOS_DGS, Q8 Q_NMOS_DGS, Q9 Q_NMOS_DGS, U1 TM4C129E_Launchpad, U10 OKI, U11 LT1910, U12 LT1910, U13 LT1910, U14 LT1910, U15 ATC_FUSE_BLOCK, U16 ATC_FUSE_BLOCK, U17 ATC_FUSE_BLOCK, U18 ATC_FUSE_BLOCK, U19 ACS714xLCTR-05B, U2 ATC_FUSE_BLOCK, U20 ACS714xLCTR-05B, U21 ACS714xLCTR-05B, U22 ACS714xLCTR-05B, U23 LT1910, U24 LT1910, U25 LT1910, U26 LT1910, U27 ATC_FUSE_BLOCK, U28 ATC_FUSE_BLOCK, U29 ATC_FUSE_BLOCK, U3 ATC_FUSE_BLOCK, U30 ATC_FUSE_BLOCK, U31 ACS714xLCTR-05B, U32 ACS714xLCTR-05B, U33 ACS714xLCTR-05B, U34 ACS714xLCTR-05B, U4 ATC_FUSE_BLOCK, U5 LT1910, U6 LT1910, U7 ACS714xLCTR-05B, U8 ACS714xLCTR-05B, U9 ACS714xLCTR-05B

Commit message: Completed Motor Bus 5,6,7, and acutuation traces
Motor Busses 5,6,7, and Actuation traces are complete. Analog traces were rerouted around the Buck converters.
Parts:
- moved 2.2uF2 26.6 mm to (188.6, 49.5)
- moved 0.1uF19 9.94 mm to (83.2, 128.3), turned to 90 degrees
- moved 1nF10 8.13 mm to (81.3, 128.3), turned to 90 degrees
- moved 0.1uF17 3.70 mm to (99.7, 78.1)
- moved 2.2uF1 2.22 mm to (188.3, 53.3)
- moved Q3 1.80 mm to (35.6, 43.2), turned to 90 degrees
- moved 0.1uF16 1.27 mm to (86.4, 85.1), turned to 0 degrees
Routing:
- net 3.3V: track 27.2 -> 367.2 mm, vias 0 -> 9
- net IMEAS-M7: track 0.00 -> 145.6 mm, vias 0 -> 3
- net FAN-CTL: track 0.00 -> 131.0 mm, vias 0 -> 3
- net VMEAS-VBATT: track 0.00 -> 96.5 mm, vias 0 -> 2
- net GND: track 9.54 -> 98.8 mm, vias 3 -> 36
- net Net-(0.1uF14-Pad1): track 0.00 -> 77.5 mm, vias 0 -> 2
- net 5V: track 0.00 -> 70.0 mm, vias 0 -> 2
- net Net-(0.1uF17-Pad1): track 0.00 -> 66.5 mm
- net Net-(0.1uF15-Pad1): track 0.00 -> 62.0 mm
- net Net-(0.1uF16-Pad1): track 0.00 -> 61.3 mm
- net Net-(Q11-Pad2): track 0.00 -> 21.4 mm
- net Net-(Q13-Pad2): track 0.00 -> 21.4 mm
- net Net-(5k7-Pad1): track 0.00 -> 19.6 mm
- net Net-(5k6-Pad1): track 0.00 -> 19.6 mm
- net Net-(5k8-Pad1): track 0.00 -> 19.4 mm
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- added copper zone on F.Cu, net GND

Commit message: Routing Finished
Routing is now complete for the entire board. Board has passed DRC. Adjusted Silkscreen on board, and removed 5V signal from schematic because it was not contributing anything.
Parts:
- moved Q6 26.4 mm to (266.7, 52.1), turned to 90 degrees
- moved 5k3 26.1 mm to (278.1, 52.1)
- moved Q9 24.3 mm to (277.9, 76.2)
- moved Conn6 23.5 mm to (273.1, 87.6)
- moved Conn5 23.5 mm to (273.7, 64.1)
- moved D7 22.1 mm to (290.2, 80.0), turned to 90 degrees
- moved D6 21.4 mm to (288.9, 58.4), turned to 180 degrees
- moved 5k4 19.5 mm to (288.9, 73.7)
- moved Conn1 14.7 mm to (236.9, 16.5), turned to 90 degrees
- moved Conn3 14.0 mm to (192.4, 16.5), turned to 90 degrees
- moved Conn2 13.2 mm to (143.5, 17.1), turned to 90 degrees
- moved D11 3.98 mm to (19.1, 76.2)
- moved Q8 3.87 mm to (267.0, 28.2), turned to 90 degrees
- moved D10 3.81 mm to (19.1, 92.7)
- moved D8 3.81 mm to (19.1, 123.2)
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Connections:
- net 5V renamed Net-(U1-Pad+5V)
Routing:
- net 3.3V: track 367.2 -> 695.5 mm, vias 9 -> 25
- net GND: track 98.8 -> 248.1 mm, vias 36 -> 70
- net Net-(0.1uF9-Pad1): track 5.17 -> 101.7 mm
- net Net-(Q7-Pad2): track 0.00 -> 74.2 mm, vias 0 -> 2
- net Net-(U1-PadRese): track 0.00 -> 66.1 mm, vias 0 -> 1
- net Net-(0.1uF6-Pad1): track 5.14 -> 52.3 mm
- net IMEAS-COM: track 26.5 -> 69.8 mm
- net Net-(Q8-Pad2): track 0.00 -> 36.4 mm
- net Net-(Q9-Pad2): track 0.00 -> 26.8 mm
- net Net-(0.1uF8-Pad1): track 69.0 -> 88.9 mm
- net Net-(Q6-Pad2): track 0.00 -> 17.3 mm
- net Net-(5k3-Pad1): track 5.24 -> 16.4 mm
- net Net-(0.1uF7-Pad1): track 9.58 -> 20.4 mm
- net Net-(1nF5-Pad1): track 0.00 -> 7.78 mm
- net Net-(1nF6-Pad2): track 0.00 -> 5.20 mm
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
Commit message: Polished Tracing
Polished some ugly tracing. Adjusted Polygon distance. Added a ground to one of the buck converters that was not showing up.
Parts:
- moved 0.1uF3 2.84 mm to (166.4, 15.9)
- moved 0.1uF4 0.90 mm to (172.1, 22.2), turned to 90 degrees
Connections:
- CONV2 pad 4: Net-(CONV2-Pad4) -> GND
Routing:
- net LOGIC-SIG: track 81.7 -> 86.7 mm
- net 3.3V: track 695.5 -> 700.0 mm, vias 25 -> 24
- net Net-(0.1uF8-Pad1): track 88.9 -> 92.1 mm
- net GND: track 248.1 -> 250.3 mm
- net IMEAS-LOGIC: track 65.6 -> 63.5 mm
- net COM-SIG: track 115.7 -> 117.4 mm
- net IMEAS-COM: track 69.8 -> 71.3 mm
- net IMEAS-M4: track 296.9 -> 298.1 mm
- net Net-(0.1uF9-Pad1): track 101.7 -> 101.0 mm
