File: MotorController_Hardware/MotorController_Hardware.kicad_pcb (KiCad board)
At the start: 2 copper layers, 124.5 x 150.9 mm, 246 parts, among them Q12 FQP30N06L, Q13 FQP30N06L, Q14 FQP30N06L, Q15 FQP30N06L, Q16 FQP30N06L, Q17 FQP30N06L, Q4 FQP30N06L, Q5 FQP30N06L, Q6 FQP30N06L, Q7 FQP30N06L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

Commit message: Updated to Rev 2
Parts:
- Conn10, Conn11, Conn4, Conn5, Conn6, Conn9: footprint MRDT_Connectors:Anderson_1_Horisontal -> MRDT_Connectors:Anderson_1_Horizontal
- Conn3, Conn8: footprint MRDT_Connectors:Anderson_2_Vertical -> MRDT_Connectors:Anderson_2_Horizontal_Stacked
- D1: value D_Zener -> D_Shottky
- D10, D11, D12, D16, D17, D18, D19, D20, D21, D7, D8, D9: value 15V -> 3.3V
- D15: value D_Zener -> D_Schottky
- Q12, Q13, Q14, Q15, Q16, Q17, Q4, Q5, Q6, Q7, Q8, Q9: footprint MotorController_Hardware:TO-220-3_Horizontal_Reversed_NoHole -> MRDT_Actives:TO-220-3_Horizontal_Reversed_NoHole
- U3: footprint MRDT_Shields:LAUNCHXL_F28069M_Launchpad_FULL_Booster_SMD_Bottom -> MRDT_Shields:LAUNCHXL_F28069M_FULL_SMD_BOTTOM
Connections:
- U1 pad 14: Net-(C17-Pad1) -> Net-(C17-Pad2)
- U1 pad 15: Net-(C17-Pad2) -> Net-(C17-Pad1)
- U5 pad 14: Net-(C60-Pad1) -> Net-(C60-Pad2)
- U5 pad 15: Net-(C60-Pad2) -> Net-(C60-Pad1)
