File: MotorController_Hardware/MotorController_Hardware.sch (KiCad schematic (older format))
At the start: 243 parts, among them Q12 Q_NMOS_DGS, Q13 Q_NMOS_DGS, Q14 Q_NMOS_DGS, Q15 Q_NMOS_DGS, Q16 Q_NMOS_DGS, Q17 Q_NMOS_DGS, Q4 Q_NMOS_DGS, Q5 Q_NMOS_DGS, Q6 Q_NMOS_DGS, Q7 Q_NMOS_DGS, Q8 Q_NMOS_DGS, Q9 Q_NMOS_DGS, U1 DRV8301, U2 NUP4201MR6, U3 LAUNCHXL_F28069M_Launchpad, U4 MAX_3232, U5 DRV8301, U6 NUP4201MR6

Commit message: CDR Schemati Changes
Parts:
- C17, C18, C19, C22, C25, C26, C27, C40, C41, C42, C43, C44, C60, C61, C62, C63, C64, C67, C68, C69: symbol Device:C -> Device:C_Small
- D10, D11, D12, D16, D17, D18, D19, D20, D21, D8, D9: value D_Zener -> 15V
- Q12, Q13, Q14, Q15, Q16, Q17, Q4, Q5, Q6, Q7, Q8, Q9: value Q_NMOS_DGS -> FQP30N06L; symbol Device:Q_NMOS_DGS -> Device:Q_NMOS_GDS
- R10, R81: value 2k -> 1.5K
Connections:
- net labels added: SL_RX, SL_TX, UART_RX, UART_TX
- net labels removed: +BATT, UART_RX_M1, UART_RX_M2, UART_TX_M1, UART_TX_M2
- wire segments 745 -> 771
- no-connect marks 28 -> 33
Other:
- note added: "Green"
- note added: "Orng"
- note added: "Red"
- note added: "Yellow"
- note removed: "Look at these"
- note removed: "Why here?"

Commit message: silkscreen touchups
Parts:
- removed D35, D36: LED, LEDs:LED_0603_HandSoldering, symbol Device:LED
- removed R76, R77: 500, Resistors_SMD:R_0603_HandSoldering, symbol Device:R
- GHA_M1: renamed from TP3; value TEST -> tp
- R14, R78: footprint Resistors_SMD:R_0603_HandSoldering -> Resistors_SMD:R_1206_HandSoldering
- U3: footprint MotorController_Hardware:LAUNCHXL_F28069M_Launchpad_FULL_Booster_SMD_Top -> (none)
- renumbered TP1 to +3V3, TP21 to GHA_M2, TP5 to GHB_M1, TP23 to GHB_M2, TP7 to GHC_M1, TP25 to GHC_M2, TP4 to GLA_M1, TP22 to GLA_M2, TP6 to GLB_M1, TP24 to GLB_M2, TP8 to GLC_M1, TP26 to GLC_M2, TP2 to PVDD_M1, TP12 to PVDD_M2, TP9 to SHA_M1, TP27 to SHA_M2, TP10 to SHB_M1, TP28 to SHB_M2, TP11 to SHC_M1, TP29 to SHC_M2
Connections:
- net labels removed: SL_RX_M1, SL_RX_M2, SL_TX_M1, SL_TX_M2, VCC
- wire segments 771 -> 765

Commit message: Added Pinout text
Connections:
- wire segments 765 -> 759
Other:
- note added: "AA2"
- note added: "AA7"
- note added: "AB1"
- note added: "AB2"
- note added: "EPWM1A"
- note added: "EPWM1B"
- note added: "EPWM2A"
- note added: "EPWM2B"
- note added: "EPWM3A"
- note added: "EPWM3B"
- note added: "EPWM4A"
- note added: "EPWM4B"
- note added: "EPWM5A"
- note added: "EPWM5B"
- note added: "EPWM6A"
- note added: "EPWM6B"
- note added: "SCI A"
- note added: "SCI B"
- note added: "SPI A"
- note added: "SPI B"
Changed lines of the file:
@@
 EESchema Schematic File Version 4
+LIBS:MotorController_Hardware-cache
 EELAYER 26 0
 EELAYER END
@@
 L Device:C_Small C17
 U 1 1 5BA76504
-P 6350 12250
-F 0 "C17" H 6350 12300 50  0000 L CNN
-F 1 ".022u" H 6400 12200 50  0000 L CNN
-F 2 "Capacitors_SMD:C_0603_HandSoldering" H 6388 12100 50  0001 C CNN
-F 3 "" H 6350 12250 50  0001 C CNN
-	1    6350 12250
-	1    0    0    -1
+P 6400 12200
+F 0 "C17" V 6350 12000 50  0000 L CNN
+F 1 ".022u" V 6350 12250 50  0000 L CNN
+F 2 "Capacitors_SMD:C_0603_HandSoldering" H 6438 12050 50  0001 C CNN
+F 3 "" H 6400 12200 50  0001 C CNN
+	1    6400 12200
+	0    1    1    0
 $EndComp
 $Comp
@@
 L Device:C_Small C60
 U 1 1 5BB18126
-P 24200 12250
-F 0 "C60" H 24225 12350 50  0000 L CNN
-F 1 ".022u" H 24225 12150 50  0000 L CNN
-F 2 "Capacitors_SMD:C_0603_HandSoldering" H 24238 12100 50  0001 C CNN
-F 3 "" H 24200 12250 50  0001 C CNN
-	1    24200 12250
-	1    0    0    -1
+P 24250 12200
+F 0 "C60" V 24200 12000 50  0000 L CNN
+F 1 ".022u" V 24200 12250 50  0000 L CNN
+F 2 "Capacitors_SMD:C_0603_HandSoldering" H 24288 12050 50  0001 C CNN
+F 3 "" H 24250 12200 50  0001 C CNN
+	1    24250 12200
+	0    1    1    0
 $EndComp
 $Comp
@@
 	6800 12450 6800 12500
 Wire Wire Line
-	24100 12300 24150 12300
-Wire Wire Line
-	24150 12300 24150 12350
-Wire Wire Line
-	24150 12350 24200 12350
-Wire Wire Line
-	24100 12200 24150 12200
-Wire Wire Line
-	24150 12200 24150 12150
-Wire Wire Line
-	24150 12150 24200 12150
-Wire Wire Line
 	24700 12450 24700 12050
 Wire Wire Line
@@
 Connection ~ 6800 12450
 Wire Wire Line
-	6350 12150 6300 12150
-Wire Wire Line
-	6300 12150 6300 12200
-Wire Wire Line
-	6300 12200 6250 12200
-Wire Wire Line
-	6250 12300 6300 12300
-Wire Wire Line
-	6300 12300 6300 12350
-Wire Wire Line
-	6300 12350 6350 12350
-Wire Wire Line
 	24150 11750 24100 11750
 Wire Wire Line
@@
 	1    0    0    -1
 $EndComp
+Wire Wire Line
+	6250 12200 6300 12200
+Wire Wire Line
+	6250 12300 6500 12300
+Wire Wire Line
+	6500 12300 6500 12200
+Wire Wire Line
+	24100 12200 24150 12200
+Wire Wire Line
+	24100 12300 24350 12300
+Wire Wire Line
+	24350 12300 24350 12200
+Text Notes 13050 7600 0    50   ~ 0
+SCI A
+Text Notes 16500 7600 0    50   ~ 0
+SCI B
+Text Notes 14600 9350 0    50   ~ 0
+SPI A
+Text Notes 18100 9350 0    50   ~ 0
+SPI B
+Text Notes 14450 7550 0    50   ~ 0
+AA7
+Text Notes 14450 7650 0    50   ~ 0
+AB1
+Text Notes 14450 7750 0    50   ~ 0
+AA2
+Text Notes 14450 7850 0    50   ~ 0
+AB2
+Text Notes 12950 8800 0    50   ~ 0
+EPWM1A
+Text Notes 12950 8900 0    50   ~ 0
+EPWM1B
+Text Notes 12950 9000 0    50   ~ 0
+EPWM2A
+Text Notes 12950 9100 0    50   ~ 0
+EPWM2B
+Text Notes 12950 9200 0    50   ~ 0
+EPWM3A
+Text Notes 12950 9300 0    50   ~ 0
+EPWM3B
+Text Notes 16400 8800 0    50   ~ 0
+EPWM4A
+Text Notes 16400 8900 0    50   ~ 0
+EPWM4B
+Text Notes 16400 9000 0    50   ~ 0
+EPWM5A
+Text Notes 16400 9100 0    50   ~ 0
+EPWM5B
+Text Notes 16400 9200 0    50   ~ 0
+EPWM6A
+Text Notes 16400 9300 0    50   ~ 0
+EPWM6B
 $EndSCHEMATC

Commit message: Schematic changes
Parts:
- C20: symbol Device:C -> Device:C_Small
Connections:
- wire segments 759 -> 757
- no-connect marks 33 -> 35
Changed lines of the file:
@@
 SL_B_M1
 $Comp
-L Device:C C20
+L Device:C_Small C20
 U 1 1 5BA7FAC1
-P 6600 10650
-F 0 "C20" H 6625 10750 50  0000 L CNN
-F 1 "0.1u" V 6650 10400 50  0000 L CNN
-F 2 "Capacitors_SMD:C_0603_HandSoldering" H 6638 10500 50  0001 C CNN
-F 3 "" H 6600 10650 50  0001 C CNN
-	1    6600 10650
-	0    -1   -1   0
+P 6650 10750
+F 0 "C20" H 6675 10850 50  0000 L CNN
+F 1 "0.1u" H 6700 10700 50  0000 L CNN
+F 2 "Capacitors_SMD:C_0603_HandSoldering" H 6688 10600 50  0001 C CNN
+F 3 "" H 6650 10750 50  0001 C CNN
+	1    6650 10750
+	1    0    0    -1
 $EndComp
 Text GLabel 6950 10850 2    39   Input ~ 0
@@
 Wire Wire Line
 	9850 7800 9700 7800
-Connection ~ 6850 10850
-Wire Wire Line
-	6150 10850 6850 10850
-Wire Wire Line
-	6850 10650 6850 10850
-Wire Wire Line
-	6750 10650 6850 10650
-Wire Wire Line
-	6450 10650 6150 10650
 Wire Wire Line
 	6150 9950 6650 9950
@@
 	11650 8750 11650 8600
 Wire Wire Line
-	6850 10850 6950 10850
-Wire Wire Line
 	4350 11650 3750 11650
 Wire Wire Line
@@
 U 1 1 5BC8BD99
 P 5450 9300
-F 0 "U1" H 5700 10076 59  0000 C CNN
+F 0 "U1" H 5550 9250 59  0000 C CNN
 F 1 "DRV8301" H 5700 9250 69  0001 C CNN
 F 2 "MRDT_ICs:DRV8301" H 6050 11250 394 0001 C CNN
@@
 U 2 1 5BC922E9
 P 5450 10200
-F 0 "U1" H 5700 10976 59  0000 C CNN
+F 0 "U1" H 5550 10150 59  0000 C CNN
 F 1 "DRV8301" H 5700 10150 69  0001 C CNN
 F 2 "MRDT_ICs:DRV8301" H 6050 12150 394 0001 C CNN
@@
 U 3 1 5BC924DA
 P 5450 11100
-F 0 "U1" H 5700 11876 59  0000 C CNN
+F 0 "U1" H 5550 11050 59  0000 C CNN
 F 1 "DRV8301" H 5700 11050 69  0001 C CNN
 F 2 "MRDT_ICs:DRV8301" H 6050 13050 394 0001 C CNN
@@
 U 4 1 5BC930B8
 P 5200 8450
-F 0 "U1" H 5700 9826 59  0000 C CNN
+F 0 "U1" H 5300 8400 59  0000 C CNN
 F 1 "DRV8301" H 5450 8400 69  0001 C CNN
 F 2 "MRDT_ICs:DRV8301" H 5800 10400 394 0001 C CNN
@@
 U 5 1 5BCFAC02
 P 5350 12800
-F 0 "U1" H 5700 14376 59  0000 C CNN
+F 0 "U1" H 5450 12750 59  0000 C CNN
 F 1 "DRV8301" H 5600 12750 69  0001 C CNN
 F 2 "MRDT_ICs:DRV8301" H 5950 14750 394 0001 C CNN
@@
 U 4 1 5BD00408
 P 23050 8450
-F 0 "U5" H 23550 9826 59  0000 C CNN
+F 0 "U5" H 23150 8400 59  0000 C CNN
 F 1 "DRV8301" H 23300 8400 69  0001 C CNN
 F 2 "MRDT_ICs:DRV8301" H 23650 10400 394 0001 C CNN
@@
 U 1 1 5BD69058
 P 23300 9300
-F 0 "U5" H 23550 10076 59  0000 C CNN
+F 0 "U5" H 23400 9250 59  0000 C CNN
 F 1 "DRV8301" H 23550 9250 69  0001 C CNN
 F 2 "MRDT_ICs:DRV8301" H 23900 11250 394 0001 C CNN
@@
 U 2 1 5BD6A297
 P 23300 10200
-F 0 "U5" H 23550 10976 59  0000 C CNN
+F 0 "U5" H 23400 10150 59  0000 C CNN
 F 1 "DRV8301" H 23550 10150 69  0001 C CNN
 F 2 "MRDT_ICs:DRV8301" H 23900 12150 394 0001 C CNN
@@
 U 3 1 5BD6A477
 P 23300 11100
-F 0 "U5" H 23550 11876 59  0000 C CNN
+F 0 "U5" H 23400 11050 59  0000 C CNN
 F 1 "DRV8301" H 23550 11050 69  0001 C CNN
 F 2 "MRDT_ICs:DRV8301" H 23900 13050 394 0001 C CNN
@@
 U 5 1 5BD6A66D
 P 23200 12800
-F 0 "U5" H 23550 14376 59  0000 C CNN
+F 0 "U5" H 23300 12750 59  0000 C CNN
 F 1 "DRV8301" H 23450 12750 69  0001 C CNN
 F 2 "MRDT_ICs:DRV8301" H 23800 14750 394 0001 C CNN
@@
 Text Notes 16400 9300 0    50   ~ 0
 EPWM6B
+NoConn ~ 17100 9550
+NoConn ~ 17100 9650
+Wire Wire Line
+	6150 10850 6650 10850
+Connection ~ 6650 10850
+Wire Wire Line
+	6650 10850 6950 10850
+Wire Wire Line
+	6150 10650 6650 10650
 $EndSCHEMATC

Commit message: Created BOM
Parts:
- C2, C51, C55, C8: footprint Capacitors_SMD:C_0603_HandSoldering -> Capacitors_SMD:C_0805_HandSoldering
- D1: value D_Zener -> D_Shottky; symbol Device:D_Zener -> Device:D_Schottky
- D15: value D_Zener -> D_Schottky; symbol Device:D_Zener -> Device:D_Schottky
Changed lines of the file:
@@
 F 0 "C8" H 4175 7750 50  0000 L CNN
 F 1 "4.7u" H 4175 7550 50  0000 L CNN
-F 2 "Capacitors_SMD:C_0603_HandSoldering" H 4188 7500 50  0001 C CNN
+F 2 "Capacitors_SMD:C_0805_HandSoldering" H 4188 7500 50  0001 C CNN
 F 3 "" H 4150 7650 50  0001 C CNN
 	1    4150 7650
@@
 F 0 "C2" H 3275 7750 50  0000 L CNN
 F 1 "4.7u" H 3275 7550 50  0000 L CNN
-F 2 "Capacitors_SMD:C_0603_HandSoldering" H 3288 7500 50  0001 C CNN
+F 2 "Capacitors_SMD:C_0805_HandSoldering" H 3288 7500 50  0001 C CNN
 F 3 "" H 3250 7650 50  0001 C CNN
 	1    3250 7650
@@
 F 0 "C55" H 22025 7750 50  0000 L CNN
 F 1 "4.7u" H 22025 7550 50  0000 L CNN
-F 2 "Capacitors_SMD:C_0603_HandSoldering" H 22038 7500 50  0001 C CNN
+F 2 "Capacitors_SMD:C_0805_HandSoldering" H 22038 7500 50  0001 C CNN
 F 3 "" H 22000 7650 50  0001 C CNN
 	1    22000 7650
@@
 F 0 "C51" H 21125 7750 50  0000 L CNN
 F 1 "4.7u" H 21125 7550 50  0000 L CNN
-F 2 "Capacitors_SMD:C_0603_HandSoldering" H 21138 7500 50  0001 C CNN
+F 2 "Capacitors_SMD:C_0805_HandSoldering" H 21138 7500 50  0001 C CNN
 F 3 "" H 21100 7650 50  0001 C CNN
 	1    21100 7650
@@
 $EndComp
 $Comp
-L Device:D_Zener D15
+L Device:D_Schottky D15
 U 1 1 5BB1804F
 P 22150 8350
 F 0 "D15" H 22150 8450 50  0000 C CNN
-F 1 "D_Zener" H 22150 8250 50  0000 C CNN
+F 1 "D_Schottky" H 22150 8250 50  0000 C CNN
 F 2 "Diodes_SMD:D_SOD-123" H 22150 8350 50  0001 C CNN
 F 3 "" H 22150 8350 50  0001 C CNN
@@
 $EndComp
 $Comp
-L Device:D_Zener D1
+L Device:D_Schottky D1
 U 1 1 5BA6C283
 P 4300 8350
 F 0 "D1" H 4300 8450 50  0000 C CNN
-F 1 "D_Zener" H 4300 8250 50  0000 C CNN
+F 1 "D_Shottky" H 4300 8250 50  0000 C CNN
 F 2 "Diodes_SMD:D_SOD-123" H 4300 8350 50  0001 C CNN
 F 3 "" H 4300 8350 50  0001 C CNN

Commit message: Created Gerbs
Parts:
- D10, D11, D12, D16, D17, D18, D19, D20, D21, D7, D8, D9: value 15V -> 3.3V
Other:
- note added: "AA5"
- note added: "AB4"
- note added: "AB5"
Changed lines of the file:
@@
 	1    0    0    -1
 $EndComp
-Text GLabel 5600 14750 2    39   Input ~ 0
+Text GLabel 5600 14750 2    39   Output ~ 0
 PVDDSENSE_M1
 $Comp
@@
 U 1 1 5BA6E8A2
 P 6700 8150
-F 0 "C22" H 6725 8250 50  0000 L CNN
+F 0 "C22" H 6750 8200 50  0000 L CNN
 F 1 "0.015u" H 6750 8100 50  0000 L CNN
 F 2 "Capacitors_SMD:C_0603_HandSoldering" H 6738 8000 50  0001 C CNN
@@
 P 10250 8000
 F 0 "D7" H 10250 8100 50  0000 C CNN
-F 1 "15V" H 10250 7900 50  0000 C CNN
+F 1 "3.3V" H 10250 7900 50  0000 C CNN
 F 2 "Diodes_SMD:D_SOD-123" H 10250 8000 50  0001 C CNN
 F 3 "" H 10250 8000 50  0001 C CNN
@@
 	1    0    0    -1
 $EndComp
-Text GLabel 12250 8750 2    39   Input ~ 0
+Text GLabel 12250 8750 2    39   Output ~ 0
 ASENSE_M1
 Text GLabel 9700 8650 0    39   Input ~ 0
@@
 P 10250 8850
 F 0 "D8" H 10250 8950 50  0000 C CNN
-F 1 "15V" H 10250 8750 50  0000 C CNN
+F 1 "3.3V" H 10250 8750 50  0000 C CNN
 F 2 "Diodes_SMD:D_SOD-123" H 10250 8850 50  0001 C CNN
 F 3 "" H 10250 8850 50  0001 C CNN
@@
 P 10250 11150
 F 0 "D9" H 10250 11250 50  0000 C CNN
-F 1 "15V" H 10250 11050 50  0000 C CNN
+F 1 "3.3V" H 10250 11050 50  0000 C CNN
 F 2 "Diodes_SMD:D_SOD-123" H 10250 11150 50  0001 C CNN
 F 3 "" H 10250 11150 50  0001 C CNN
@@
 	1    0    0    -1
 $EndComp
-Text GLabel 12250 11900 2    39   Input ~ 0
+Text GLabel 12250 11900 2    39   Output ~ 0
 BSENSE_M1
 Text GLabel 9700 11800 0    39   Input ~ 0
@@
 P 10250 12000
 F 0 "D10" H 10250 12100 50  0000 C CNN
-F 1 "15V" H 10250 11900 50  0000 C CNN
+F 1 "3.3V" H 10250 11900 50  0000 C CNN
 F 2 "Diodes_SMD:D_SOD-123" H 10250 12000 50  0001 C CNN
 F 3 "" H 10250 12000 50  0001 C CNN
@@
 P 10250 14500
 F 0 "D11" H 10250 14600 50  0000 C CNN
-F 1 "15V" H 10250 14400 50  0000 C CNN
+F 1 "3.3V" H 10250 14400 50  0000 C CNN
 F 2 "Diodes_SMD:D_SOD-123" H 10250 14500 50  0001 C CNN
 F 3 "" H 10250 14500 50  0001 C CNN
@@
 	1    0    0    -1
 $EndComp
-Text GLabel 12250 15250 2    39   Input ~ 0
+Text GLabel 12250 15250 2    39   Output ~ 0
 CSENSE_M1
 Text GLabel 9700 15150 0    39   Input ~ 0
@@
 P 10250 15350
 F 0 "D12" H 10250 15450 50  0000 C CNN
-F 1 "15V" H 10250 15250 50  0000 C CNN
+F 1 "3.3V" H 10250 15250 50  0000 C CNN
 F 2 "Diodes_SMD:D_SOD-123" H 10250 15350 50  0001 C CNN
 F 3 "" H 10250 15350 50  0001 C CNN
@@
 U 1 1 5BB18079
 P 25450 8150
-F 0 "C69" H 25475 8250 50  0000 L CNN
+F 0 "C69" H 25500 8200 50  0000 L CNN
 F 1 "1u" H 25475 8050 50  0000 L CNN
 F 2 "Capacitors_SMD:C_0603_HandSoldering" H 25488 8000 50  0001 C CNN
@@
 U 1 1 5BB1808B
 P 25150 8150
-F 0 "C68" H 25175 8250 50  0000 L CNN
+F 0 "C68" H 25200 8200 50  0000 L CNN
 F 1 "1u" H 25175 8050 50  0000 L CNN
 F 2 "Capacitors_SMD:C_0603_HandSoldering" H 25188 8000 50  0001 C CNN
@@
 U 1 1 5BB18091
 P 24850 8150
-F 0 "C67" H 24875 8250 50  0000 L CNN
+F 0 "C67" H 24900 8200 50  0000 L CNN
 F 1 "2.2u" H 24875 8050 50  0000 L CNN
 F 2 "Capacitors_SMD:C_0603_HandSoldering" H 24888 8000 50  0001 C CNN
@@
 U 1 1 5BB1809D
 P 24550 8150
-F 0 "C64" H 24575 8250 50  0000 L CNN
+F 0 "C64" H 24600 8200 50  0000 L CNN
 F 1 "0.015u" H 24600 8100 50  0000 L CNN
 F 2 "Capacitors_SMD:C_0603_HandSoldering" H 24588 8000 50  0001 C CNN
@@
 P 27950 7950
 F 0 "D16" H 27950 8050 50  0000 C CNN
-F 1 "15V" H 27950 7850 50  0000 C CNN
+F 1 "3.3V" H 27950 7850 50  0000 C CNN
 F 2 "Diodes_SMD:D_SOD-123" H 27950 7950 50  0001 C CNN
 F 3 "" H 27950 7950 50  0001 C CNN
@@
 	1    0    0    -1
 $EndComp
-Text GLabel 29950 8700 2    39   Input ~ 0
+Text GLabel 29950 8700 2    39   Output ~ 0
 ASENSE_M2
 Text GLabel 27400 8600 0    39   Input ~ 0
@@
 P 27950 8800
 F 0 "D17" H 27950 8900 50  0000 C CNN
-F 1 "15V" H 27950 8700 50  0000 C CNN
+F 1 "3.3V" H 27950 8700 50  0000 C CNN
 F 2 "Diodes_SMD:D_SOD-123" H 27950 8800 50  0001 C CNN
 F 3 "" H 27950 8800 50  0001 C CNN
@@
 P 27950 11200
 F 0 "D18" H 27950 11300 50  0000 C CNN
-F 1 "15V" H 27950 11100 50  0000 C CNN
+F 1 "3.3V" H 27950 11100 50  0000 C CNN
 F 2 "Diodes_SMD:D_SOD-123" H 27950 11200 50  0001 C CNN
 F 3 "" H 27950 11200 50  0001 C CNN
@@
 	1    0    0    -1
 $EndComp
-Text GLabel 29950 11950 2    39   Input ~ 0
+Text GLabel 29950 11950 2    39   Output ~ 0
 BSENSE_M2
 Text GLabel 27400 11850 0    39   Input ~ 0
@@
 P 27950 12050
 F 0 "D19" H 27950 12150 50  0000 C CNN
-F 1 "15V" H 27950 11950 50  0000 C CNN
+F 1 "3.3V" H 27950 11950 50  0000 C CNN
 F 2 "Diodes_SMD:D_SOD-123" H 27950 12050 50  0001 C CNN
 F 3 "" H 27950 12050 50  0001 C CNN
@@
 P 27950 14600
 F 0 "D20" H 27950 14700 50  0000 C CNN
-F 1 "15V" H 27950 14500 50  0000 C CNN
+F 1 "3.3V" H 27950 14500 50  0000 C CNN
 F 2 "Diodes_SMD:D_SOD-123" H 27950 14600 50  0001 C CNN
 F 3 "" H 27950 14600 50  0001 C CNN
@@
 	1    0    0    -1
 $EndComp
-Text GLabel 29950 15300 2    39   Input ~ 0
+Text GLabel 29950 15300 2    39   Output ~ 0
 CSENSE_M2
 Text GLabel 27400 15200 0    39   Input ~ 0
@@
 P 27950 15400
 F 0 "D21" H 27950 15500 50  0000 C CNN
-F 1 "15V" H 27950 15300 50  0000 C CNN
+F 1 "3.3V" H 27950 15300 50  0000 C CNN
 F 2 "Diodes_SMD:D_SOD-123" H 27950 15400 50  0001 C CNN
 F 3 "" H 27950 15400 50  0001 C CNN
@@
 	1    0    0    -1
 $EndComp
-Text GLabel 23300 14750 2    39   Input ~ 0
+Text GLabel 23300 14750 2    39   Output ~ 0
 PVDDSENSE_M2
 $Comp
@@
 Wire Wire Line
 	6150 10650 6650 10650
+Text Notes 18000 7600 0    50   ~ 0
+AB4
+Text Notes 18000 7700 0    50   ~ 0
+AB4
+Text Notes 18000 7800 0    50   ~ 0
+AA5
+Text Notes 18000 7900 0    50   ~ 0
+AB5
 $EndSCHEMATC
