File: MotorController_Hardware/MotorController_Hardware.sch (KiCad schematic (older format))
At the start: 239 parts, among them Q12 FQP30N06L, Q13 FQP30N06L, Q14 FQP30N06L, Q15 FQP30N06L, Q16 FQP30N06L, Q17 FQP30N06L, Q4 FQP30N06L, Q5 FQP30N06L, Q6 FQP30N06L, Q7 FQP30N06L, Q8 FQP30N06L, Q9 FQP30N06L, U1 DRV8301, U2 NUP4201MR6, U3 LAUNCHXL_F28069M_Launchpad, U4 MAX_3232, U5 DRV8301, U6 NUP4201MR6

Commit message: Updated to Rev 2
Parts:
- Conn10, Conn11, Conn4, Conn5, Conn6, Conn9: footprint MRDT_Connectors:Anderson_1_Horisontal -> MRDT_Connectors:Anderson_1_Horizontal
- Conn3, Conn8: footprint MRDT_Connectors:Anderson_2_Vertical -> MRDT_Connectors:Anderson_2_Horizontal_Stacked
- Q12, Q13, Q14, Q15, Q16, Q17, Q4, Q5, Q6, Q7, Q8, Q9: footprint MotorController_Hardware:TO-220-3_Horizontal_Reversed_NoHole -> MRDT_Actives:TO-220-3_Horizontal_Reversed_NoHole
- U3: footprint MotorController_Hardware:LAUNCHXL_F28069M_Launchpad_FULL_Booster_SMD_Top -> MRDT_Shields:LAUNCHXL_F28069M_FULL_SMD_BOTTOM
- U3: footprint (none) -> MRDT_Shields:LAUNCHXL_F28069M_FULL_SMD_BOTTOM
Changed lines of the file:
@@
 F 0 "Q4" H 10900 7850 50  0000 L CNN
 F 1 "FQP30N06L" H 10850 7700 50  0000 L CNN
-F 2 "MotorController_Hardware:TO-220-3_Horizontal_Reversed_NoHole" H 10900 7900 50  0001 C CNN
+F 2 "MRDT_Actives:TO-220-3_Horizontal_Reversed_NoHole" H 10900 7900 50  0001 C CNN
 F 3 "" H 10700 7800 50  0001 C CNN
 	1    10700 7800
@@
 F 0 "Q5" H 10900 8700 50  0000 L CNN
 F 1 "FQP30N06L" H 10850 8550 50  0000 L CNN
-F 2 "MotorController_Hardware:TO-220-3_Horizontal_Reversed_NoHole" H 10900 8750 50  0001 C CNN
+F 2 "MRDT_Actives:TO-220-3_Horizontal_Reversed_NoHole" H 10900 8750 50  0001 C CNN
 F 3 "" H 10700 8650 50  0001 C CNN
 	1    10700 8650
@@
 F 0 "Q6" H 10900 11000 50  0000 L CNN
 F 1 "FQP30N06L" H 10850 10850 50  0000 L CNN
-F 2 "MotorController_Hardware:TO-220-3_Horizontal_Reversed_NoHole" H 10900 11050 50  0001 C CNN
+F 2 "MRDT_Actives:TO-220-3_Horizontal_Reversed_NoHole" H 10900 11050 50  0001 C CNN
 F 3 "" H 10700 10950 50  0001 C CNN
 	1    10700 10950
@@
 F 0 "Q7" H 10900 11850 50  0000 L CNN
 F 1 "FQP30N06L" H 10850 11700 50  0000 L CNN
-F 2 "MotorController_Hardware:TO-220-3_Horizontal_Reversed_NoHole" H 10900 11900 50  0001 C CNN
+F 2 "MRDT_Actives:TO-220-3_Horizontal_Reversed_NoHole" H 10900 11900 50  0001 C CNN
 F 3 "" H 10700 11800 50  0001 C CNN
 	1    10700 11800
@@
 F 0 "Q8" H 10900 14350 50  0000 L CNN
 F 1 "FQP30N06L" H 10850 14200 50  0000 L CNN
-F 2 "MotorController_Hardware:TO-220-3_Horizontal_Reversed_NoHole" H 10900 14400 50  0001 C CNN
+F 2 "MRDT_Actives:TO-220-3_Horizontal_Reversed_NoHole" H 10900 14400 50  0001 C CNN
 F 3 "" H 10700 14300 50  0001 C CNN
 	1    10700 14300
@@
 F 0 "Q9" H 10900 15200 50  0000 L CNN
 F 1 "FQP30N06L" H 10850 15050 50  0000 L CNN
-F 2 "MotorController_Hardware:TO-220-3_Horizontal_Reversed_NoHole" H 10900 15250 50  0001 C CNN
+F 2 "MRDT_Actives:TO-220-3_Horizontal_Reversed_NoHole" H 10900 15250 50  0001 C CNN
 F 3 "" H 10700 15150 50  0001 C CNN
 	1    10700 15150
@@
 F 0 "Q12" H 28600 7800 50  0000 L CNN
 F 1 "FQP30N06L" H 28550 7650 50  0000 L CNN
-F 2 "MotorController_Hardware:TO-220-3_Horizontal_Reversed_NoHole" H 28600 7850 50  0001 C CNN
+F 2 "MRDT_Actives:TO-220-3_Horizontal_Reversed_NoHole" H 28600 7850 50  0001 C CNN
 F 3 "" H 28400 7750 50  0001 C CNN
 	1    28400 7750
@@
 F 0 "Q13" H 28600 8650 50  0000 L CNN
 F 1 "FQP30N06L" H 28550 8500 50  0000 L CNN
-F 2 "MotorController_Hardware:TO-220-3_Horizontal_Reversed_NoHole" H 28600 8700 50  0001 C CNN
+F 2 "MRDT_Actives:TO-220-3_Horizontal_Reversed_NoHole" H 28600 8700 50  0001 C CNN
 F 3 "" H 28400 8600 50  0001 C CNN
 	1    28400 8600
@@
 F 0 "Q14" H 28600 11050 50  0000 L CNN
 F 1 "FQP30N06L" H 28550 10900 50  0000 L CNN
-F 2 "MotorController_Hardware:TO-220-3_Horizontal_Reversed_NoHole" H 28600 11100 50  0001 C CNN
+F 2 "MRDT_Actives:TO-220-3_Horizontal_Reversed_NoHole" H 28600 11100 50  0001 C CNN
 F 3 "" H 28400 11000 50  0001 C CNN
 	1    28400 11000
@@
 F 0 "Q15" H 28600 11900 50  0000 L CNN
 F 1 "FQP30N06L" H 28550 11750 50  0000 L CNN
-F 2 "MotorController_Hardware:TO-220-3_Horizontal_Reversed_NoHole" H 28600 11950 50  0001 C CNN
+F 2 "MRDT_Actives:TO-220-3_Horizontal_Reversed_NoHole" H 28600 11950 50  0001 C CNN
 F 3 "" H 28400 11850 50  0001 C CNN
 	1    28400 11850
@@
 F 0 "Q16" H 28600 14400 50  0000 L CNN
 F 1 "FQP30N06L" H 28550 14250 50  0000 L CNN
-F 2 "MotorController_Hardware:TO-220-3_Horizontal_Reversed_NoHole" H 28600 14450 50  0001 C CNN
+F 2 "MRDT_Actives:TO-220-3_Horizontal_Reversed_NoHole" H 28600 14450 50  0001 C CNN
 F 3 "" H 28400 14350 50  0001 C CNN
 	1    28400 14350
@@
 F 0 "Q17" H 28600 15250 50  0000 L CNN
 F 1 "FQP30N06L" H 28550 15100 50  0000 L CNN
-F 2 "MotorController_Hardware:TO-220-3_Horizontal_Reversed_NoHole" H 28600 15300 50  0001 C CNN
+F 2 "MRDT_Actives:TO-220-3_Horizontal_Reversed_NoHole" H 28600 15300 50  0001 C CNN
 F 3 "" H 28400 15200 50  0001 C CNN
 	1    28400 15200
@@
 F 0 "U3" H 13850 8200 60  0000 L CNN
 F 1 "LAUNCHXL_F28069M_Launchpad" H 14000 9450 60  0000 L CNN
-F 2 "MotorController_Hardware:LAUNCHXL_F28069M_Launchpad_FULL_Booster_SMD_Top" H 13850 8250 60  0001 C CNN
+F 2 "MRDT_Shields:LAUNCHXL_F28069M_FULL_SMD_BOTTOM" H 13850 8250 60  0001 C CNN
 F 3 "" H 13850 8250 60  0001 C CNN
 	1    13850 8250
@@
 F 0 "U3" H 15350 8200 60  0000 L CNN
 F 1 "LAUNCHXL_F28069M_Launchpad" H 14800 9400 60  0001 L CNN
-F 2 "MotorController_Hardware:LAUNCHXL_F28069M_Launchpad_FULL_Booster_SMD_Top" H 15350 8250 60  0001 C CNN
+F 2 "MRDT_Shields:LAUNCHXL_F28069M_FULL_SMD_BOTTOM" H 15350 8250 60  0001 C CNN
 F 3 "" H 15350 8250 60  0001 C CNN
 	3    15350 8250
@@
 F 0 "U3" H 15350 9650 60  0000 L CNN
 F 1 "LAUNCHXL_F28069M_Launchpad" H 14800 10850 60  0001 L CNN
-F 2 "MotorController_Hardware:LAUNCHXL_F28069M_Launchpad_FULL_Booster_SMD_Top" H 15350 9700 60  0001 C CNN
+F 2 "MRDT_Shields:LAUNCHXL_F28069M_FULL_SMD_BOTTOM" H 15350 9700 60  0001 C CNN
 F 3 "" H 15350 9700 60  0001 C CNN
 	2    15350 9700
@@
 F 0 "U3" H 13850 9650 60  0000 L CNN
 F 1 "LAUNCHXL_F28069M_Launchpad" H 13300 10850 60  0001 L CNN
-F 2 "MotorController_Hardware:LAUNCHXL_F28069M_Launchpad_FULL_Booster_SMD_Top" H 13850 9700 60  0001 C CNN
+F 2 "MRDT_Shields:LAUNCHXL_F28069M_FULL_SMD_BOTTOM" H 13850 9700 60  0001 C CNN
 F 3 "" H 13850 9700 60  0001 C CNN
 	4    13850 9700
@@
 F 0 "U3" H 17300 8200 60  0000 L CNN
 F 1 "LAUNCHXL_F28069M_Launchpad" H 16750 9400 60  0001 L CNN
-F 2 "MotorController_Hardware:LAUNCHXL_F28069M_Launchpad_FULL_Booster_SMD_Top" H 17300 8250 60  0001 C CNN
+F 2 "MRDT_Shields:LAUNCHXL_F28069M_FULL_SMD_BOTTOM" H 17300 8250 60  0001 C CNN
 F 3 "" H 17300 8250 60  0001 C CNN
 	5    17300 8250
@@
 F 0 "U3" H 18900 9650 60  0000 L CNN
 F 1 "LAUNCHXL_F28069M_Launchpad" H 18350 10850 60  0001 L CNN
-F 2 "MotorController_Hardware:LAUNCHXL_F28069M_Launchpad_FULL_Booster_SMD_Top" H 18900 9700 60  0001 C CNN
+F 2 "MRDT_Shields:LAUNCHXL_F28069M_FULL_SMD_BOTTOM" H 18900 9700 60  0001 C CNN
 F 3 "" H 18900 9700 60  0001 C CNN
 	6    18900 9700
@@
 F 0 "Conn9" H 19123 11297 60  0000 R CNN
 F 1 "SH_A_M2_PP" H 19123 11403 60  0000 R CNN
-F 2 "MRDT_Connectors:Anderson_1_Horisontal" H 19000 10700 60  0001 C CNN
+F 2 "MRDT_Connectors:Anderson_1_Horizontal" H 19000 10700 60  0001 C CNN
 F 3 "" H 19000 10700 60  0001 C CNN
 	1    19150 11250
@@
 F 0 "Conn10" H 19123 11697 60  0000 R CNN
 F 1 "SH_B_M2_PP" H 19123 11803 60  0000 R CNN
-F 2 "MRDT_Connectors:Anderson_1_Horisontal" H 19000 11100 60  0001 C CNN
+F 2 "MRDT_Connectors:Anderson_1_Horizontal" H 19000 11100 60  0001 C CNN
 F 3 "" H 19000 11100 60  0001 C CNN
 	1    19150 11650
@@
 F 0 "Conn11" H 19123 12097 60  0000 R CNN
 F 1 "SH_C_M2_PP" H 19123 12203 60  0000 R CNN
-F 2 "MRDT_Connectors:Anderson_1_Horisontal" H 19000 11500 60  0001 C CNN
+F 2 "MRDT_Connectors:Anderson_1_Horizontal" H 19000 11500 60  0001 C CNN
 F 3 "" H 19000 11500 60  0001 C CNN
 	1    19150 12050
@@
 F 0 "Conn6" H 17773 12097 60  0000 R CNN
 F 1 "SH_C_M1_PP" H 17773 12203 60  0000 R CNN
-F 2 "MRDT_Connectors:Anderson_1_Horisontal" H 17650 11500 60  0001 C CNN
+F 2 "MRDT_Connectors:Anderson_1_Horizontal" H 17650 11500 60  0001 C CNN
 F 3 "" H 17650 11500 60  0001 C CNN
 	1    17800 12050
@@
 F 0 "Conn5" H 17773 11697 60  0000 R CNN
 F 1 "SH_B_M1_PP" H 17773 11803 60  0000 R CNN
-F 2 "MRDT_Connectors:Anderson_1_Horisontal" H 17650 11100 60  0001 C CNN
+F 2 "MRDT_Connectors:Anderson_1_Horizontal" H 17650 11100 60  0001 C CNN
 F 3 "" H 17650 11100 60  0001 C CNN
 	1    17800 11650
@@
 F 0 "Conn4" H 17773 11297 60  0000 R CNN
 F 1 "SH_A_M1_PP" H 17773 11403 60  0000 R CNN
-F 2 "MRDT_Connectors:Anderson_1_Horisontal" H 17650 10700 60  0001 C CNN
+F 2 "MRDT_Connectors:Anderson_1_Horizontal" H 17650 10700 60  0001 C CNN
 F 3 "" H 17650 10700 60  0001 C CNN
 	1    17800 11250
@@
 F 0 "Conn8" H 19123 10597 60  0000 R CNN
 F 1 "AndersonPP" H 19123 10703 60  0000 R CNN
-F 2 "MRDT_Connectors:Anderson_2_Vertical" H 19000 10000 60  0001 C CNN
+F 2 "MRDT_Connectors:Anderson_2_Horizontal_Stacked" H 19000 10000 60  0001 C CNN
 F 3 "" H 19000 10000 60  0001 C CNN
 	1    19150 10550
@@
 F 0 "Conn3" H 17773 10597 60  0000 R CNN
 F 1 "AndersonPP" H 17773 10703 60  0000 R CNN
-F 2 "MRDT_Connectors:Anderson_2_Vertical" H 17650 10000 60  0001 C CNN
+F 2 "MRDT_Connectors:Anderson_2_Horizontal_Stacked" H 17650 10000 60  0001 C CNN
 F 3 "" H 17650 10000 60  0001 C CNN
 	1    17800 10550
@@
 $Comp
 L MRDT_Connectors:AndersonPP Conn8
-U 2 1 5BF99F47
+U 4 1 5BF99F47
 P 19150 10350
 F 0 "Conn8" H 19123 10397 60  0000 R CNN
 F 1 "AndersonPP" H 19123 10503 60  0000 R CNN
-F 2 "MRDT_Connectors:Anderson_2_Vertical" H 19000 9800 60  0001 C CNN
+F 2 "MRDT_Connectors:Anderson_2_Horizontal_Stacked" H 19000 9800 60  0001 C CNN
 F 3 "" H 19000 9800 60  0001 C CNN
-	2    19150 10350
+	4    19150 10350
 	-1   0    0    1
 $EndComp
 $Comp
 L MRDT_Connectors:AndersonPP Conn3
-U 2 1 5BF9A381
+U 4 1 5BF9A381
 P 17800 10350
 F 0 "Conn3" H 17773 10397 60  0000 R CNN
 F 1 "AndersonPP" H 17773 10503 60  0000 R CNN
-F 2 "MRDT_Connectors:Anderson_2_Vertical" H 17650 9800 60  0001 C CNN
+F 2 "MRDT_Connectors:Anderson_2_Horizontal_Stacked" H 17650 9800 60  0001 C CNN
 F 3 "" H 17650 9800 60  0001 C CNN
-	2    17800 10350
+	4    17800 10350
 	-1   0    0    1
 $EndComp
@@
 F 0 "U3" H 18900 8250 60  0000 L CNN
 F 1 "LAUNCHXL_F28069M_Launchpad" H 17500 9550 60  0000 L CNN
-F 2 "MotorController_Hardware:LAUNCHXL_F28069M_Launchpad_FULL_Booster_SMD_Top" H 18900 8300 60  0001 C CNN
+F 2 "MRDT_Shields:LAUNCHXL_F28069M_FULL_SMD_BOTTOM" H 18900 8300 60  0001 C CNN
 F 3 "" H 18900 8300 60  0001 C CNN
 	7    18900 8300
@@
 F 0 "U3" H 17300 9650 60  0000 L CNN
 F 1 "LAUNCHXL_F28069M_Launchpad" H 17599 10192 60  0001 L CNN
-F 2 "" H 17300 9700 60  0001 C CNN
+F 2 "MRDT_Shields:LAUNCHXL_F28069M_FULL_SMD_BOTTOM" H 17300 9700 60  0001 C CNN
 F 3 "" H 17300 9700 60  0001 C CNN
 	8    17300 9700
