File: PowerBoard_Hardware/PowerBoard_Hardware.kicad_pcb (KiCad board)
At the start: 4 copper layers, 279.4 x 126.9 mm, 153 parts, among them Q1 BSS138PW.115, Q10 Q_NMOS_GDS, Q11 Q_NMOS_GDS, Q12 Q_NMOS_GDS, Q13 Q_NMOS_GDS, Q2 BSS138PW.115, Q3 IPT020N10N3, Q4 IPT020N10N3, Q5 IPT020N10N3, Q6 Q_NMOS_GDS, Q7 Q_NMOS_GDS, Q8 Q_NMOS_GDS, Q9 Q_NMOS_GDS, U1 TM4C129E_Launchpad, U10 OKI, U11 LT1910, U12 LT1910, U13 LT1910, U14 LT1910, U15 ATC_FUSE_BLOCK, U16 ATC_FUSE_BLOCK, U17 ATC_FUSE_BLOCK, U18 ATC_FUSE_BLOCK, U19 ACS722xLCTR-40AU, U2 ATC_FUSE_BLOCK, U20 ACS722xLCTR-40AU, U21 ACS722xLCTR-40AU, U22 ACS722xLCTR-40AU, U23 LT1910, U24 LT1910, U25 LT1910, U26 LT1910, U27 ATC_FUSE_BLOCK, U28 ATC_FUSE_BLOCK, U29 ATC_FUSE_BLOCK, U3 ATC_FUSE_BLOCK, U30 ATC_FUSE_BLOCK, U31 ACS722xLCTR-40AU, U32 ACS722xLCTR-40AU, U33 ACS722xLCTR-40AU, U34 ACS722xLCTR-40AU, U4 ATC_FUSE_BLOCK, U5 LT1910, U6 LT1910, U7 ACS722xLCTR-40AU, U8 ACS722xLCTR-40AU, U9 ACS722xLCTR-40AU

Commit message: Updated to KiCAD libraries Rev 2
Parts:
- CONV1, CONV2: footprint PowerBoard_Hardware2:DC_DC_Converter_Quarter_Brick -> MRDT_Devices:Q36SR12020NRFA
- Conn1, Conn2, Conn3: footprint PowerBoard_Hardware:Vertical_Anderson_Double_SidebySide -> MRDT_Connectors:Anderson_2_Vertical_Sidy_by_Side
- Conn10, Conn11, Conn4, Conn5, Conn6, Conn7, Conn8, Conn9: footprint MRDT-Connectors:Anderson_2_Vertical -> MRDT_Connectors:Anderson_2_Horizontal_Stacked
- Q3: value IPT020N10N3 -> N_Fet
- Q4, Q5: value IPT020N10N3 -> FDD8780
- U1: footprint MRDT-SHIELDS:TM4C129E_Launchpad_FULL -> MRDT_Shields:TM4C129E_Launchpad_FULL_THT_TOP
- U10: footprint MRDT-Devices:OKI_Horizontal -> MRDT_Devices:OKI_Horizontal
- U15, U16, U17, U18, U27, U28, U29, U30, U4: footprint MRDT-Passives:ATC_Fuse_Block -> MRDT_Passives:ATC_Fuse_Block
- moved CONV2 60.6 mm to (223.3, 110.0)
- moved CONV1 59.6 mm to (170.9, 110.0)
Connections:
- CONV1 pad 6: Net-(CONV1-Pad6) -> (no net)
- CONV2 pad 6: Net-(CONV2-Pad6) -> (no net)
- Q10 pad 3: Net-(Conn11-Pad2) -> Net-(Conn11-Pad4)
- Q11 pad 3: Net-(Conn10-Pad2) -> Net-(Conn10-Pad4)
- Q12 pad 3: Net-(Conn8-Pad2) -> Net-(Conn8-Pad4)
- Q13 pad 3: Net-(Conn9-Pad2) -> Net-(Conn9-Pad4)
- Q6 pad 3: Net-(Conn5-Pad2) -> Net-(Conn5-Pad4)
- Q7 pad 3: Net-(Conn7-Pad2) -> Net-(Conn7-Pad4)
- Q8 pad 3: Net-(Conn4-Pad2) -> Net-(Conn4-Pad4)
- Q9 pad 3: Net-(Conn6-Pad2) -> Net-(Conn6-Pad4)
- R10 pad 2: Net-(Conn7-Pad2) -> Net-(Conn7-Pad4)
- R11 pad 2: Net-(Conn4-Pad2) -> Net-(Conn4-Pad4)
- R12 pad 2: Net-(Conn5-Pad2) -> Net-(Conn5-Pad4)
- R13 pad 2: Net-(Conn6-Pad2) -> Net-(Conn6-Pad4)
- R14 pad 2: Net-(Conn11-Pad2) -> Net-(Conn11-Pad4)
- R15 pad 2: Net-(Conn10-Pad2) -> Net-(Conn10-Pad4)
- R16 pad 2: Net-(Conn9-Pad2) -> Net-(Conn9-Pad4)
- R17 pad 2: Net-(Conn8-Pad2) -> Net-(Conn8-Pad4)
- U1 pad +5V: Net-(U1-Pad+5V) -> (no net)
- U1 pad PA4: Net-(U1-PadPA4) -> (no net)
- U1 pad PA5: Net-(U1-PadPA5) -> (no net)
- U1 pad PA6: Net-(U1-PadPA6) -> (no net)
- U1 pad PA7: Net-(U1-PadPA7) -> (no net)
- U1 pad PB2: Net-(U1-PadPB2) -> (no net)
- U1 pad PB3: Net-(U1-PadPB3) -> (no net)
- U1 pad PC4: Net-(U1-PadPC4) -> (no net)
- U1 pad PC5: Net-(U1-PadPC5) -> (no net)
- U1 pad PC6: Net-(U1-PadPC6) -> (no net)
- U1 pad PC7: Net-(U1-PadPC7) -> (no net)
- U1 pad PD2: Net-(U1-PadPD2) -> (no net)
- U1 pad PD3: Net-(U1-PadPD3) -> (no net)
- U1 pad PD4: Net-(U1-PadPD4) -> (no net)
- U1 pad PD5: Net-(U1-PadPD5) -> (no net)
- U1 pad PD7: Net-(U1-PadPD7) -> (no net)
- U1 pad PE4: Net-(U1-PadPE4) -> (no net)
- U1 pad PF1: Net-(U1-PadPF1) -> (no net)
- U1 pad PF2: Net-(U1-PadPF2) -> (no net)
- U1 pad PF3: Net-(U1-PadPF3) -> (no net)
- U1 pad PG0: Net-(U1-PadPG0) -> (no net)
- U1 pad PG1: Net-(U1-PadPG1) -> (no net)
- U1 pad PH3: Net-(U1-PadPH3) -> (no net)
- U1 pad PK4: Net-(U1-PadPK4) -> (no net)
- U1 pad PL0: Net-(U1-PadPL0) -> (no net)
- U1 pad PL1: Net-(U1-PadPL1) -> (no net)
- U1 pad PL2: Net-(U1-PadPL2) -> (no net)
- U1 pad PL3: Net-(U1-PadPL3) -> (no net)
- U1 pad PL4: Net-(U1-PadPL4) -> (no net)
- U1 pad PL5: Net-(U1-PadPL5) -> (no net)
- U1 pad PM4: Net-(U1-PadPM4) -> (no net)
- U1 pad PM5: Net-(U1-PadPM5) -> (no net)
- U1 pad PM6: Net-(U1-PadPM6) -> (no net)
- U1 pad PM7: Net-(U1-PadPM7) -> (no net)
- U1 pad PN2: Net-(U1-PadPN2) -> (no net)
- U1 pad PN4: Net-(U1-PadPN4) -> (no net)
- U1 pad PN5: Net-(U1-PadPN5) -> (no net)
- U1 pad PP0: Net-(U1-PadPP0) -> (no net)
- U1 pad PP1: Net-(U1-PadPP1) -> (no net)
- U1 pad PP3: Net-(U1-PadPP3) -> (no net)
- U1 pad PP4: Net-(U1-PadPP4) -> (no net)
- U1 pad PP5: Net-(U1-PadPP5) -> (no net)
- U1 pad PQ0: Net-(U1-PadPQ0) -> (no net)
- U1 pad PQ1: Net-(U1-PadPQ1) -> (no net)
- U1 pad PQ2: Net-(U1-PadPQ2) -> (no net)
- U1 pad PQ3: Net-(U1-PadPQ3) -> (no net)
- U1 pad Rese: Net-(U1-PadRese) -> (no net)
- U11 pad 2: Net-(U11-Pad2) -> (no net)
- U11 pad 3: Net-(U11-Pad3) -> (no net)
- U12 pad 2: Net-(U12-Pad2) -> (no net)
- U12 pad 3: Net-(U12-Pad3) -> (no net)
- U13 pad 2: Net-(U13-Pad2) -> (no net)
- U13 pad 3: Net-(U13-Pad3) -> (no net)
- U14 pad 2: Net-(U14-Pad2) -> (no net)
- U14 pad 3: Net-(U14-Pad3) -> (no net)
- U23 pad 2: Net-(U23-Pad2) -> (no net)
- U23 pad 3: Net-(U23-Pad3) -> (no net)
- U24 pad 2: Net-(U24-Pad2) -> (no net)
- U24 pad 3: Net-(U24-Pad3) -> (no net)
- U25 pad 2: Net-(U25-Pad2) -> (no net)
- U25 pad 3: Net-(U25-Pad3) -> (no net)
- U26 pad 2: Net-(U26-Pad2) -> (no net)
- U26 pad 3: Net-(U26-Pad3) -> (no net)
- U5 pad 2: Net-(U5-Pad2) -> (no net)
- U5 pad 3: Net-(U5-Pad3) -> (no net)
- U6 pad 2: Net-(U6-Pad2) -> (no net)
- U6 pad 3: Net-(U6-Pad3) -> (no net)
Routing:
- net Net-(Conn4-Pad4): track 0.00 -> 4.56 mm
- net Net-(Conn4-Pad2): track 4.56 -> 0.00 mm
- added copper zone on F.Cu, net (none)
- added copper zone on F.Cu, net Net-(Conn10-Pad4)
- added copper zone on F.Cu, net Net-(Conn11-Pad4)
- added copper zone on F.Cu, net Net-(Conn8-Pad4)
- added copper zone on F.Cu, net Net-(Conn9-Pad4)
- removed copper zone on F.Cu, net Net-(Conn10-Pad2)
- removed copper zone on F.Cu, net Net-(Conn11-Pad2)
- removed copper zone on F.Cu, net Net-(Conn4-Pad2)
- removed copper zone on F.Cu, net Net-(Conn5-Pad2)
- removed copper zone on F.Cu, net Net-(Conn6-Pad2)
- removed copper zone on F.Cu, net Net-(Conn7-Pad2)
- removed copper zone on F.Cu, net Net-(Conn8-Pad2)
- removed copper zone on F.Cu, net Net-(Conn9-Pad2)
Other:
- board size 279.4 x 126.9 mm -> 279.4 x 127 mm
