File: PowerBoard_Hardware/PowerBoard_Hardware.sch (KiCad schematic (older format))
At the start: 140 parts, among them Q1 BSS138PW.115, Q10 Q_NMOS_GDS, Q11 Q_NMOS_GDS, Q12 Q_NMOS_GDS, Q13 Q_NMOS_GDS, Q2 BSS138PW.115, Q3 IPT020N10N3, Q4 IPT020N10N3, Q5 IPT020N10N3, Q6 Q_NMOS_GDS, Q7 Q_NMOS_GDS, Q8 Q_NMOS_GDS, Q9 Q_NMOS_GDS, U1 TM4C129E_Launchpad, U10 OKI, U11 LT1910, U12 LT1910, U13 LT1910, U14 LT1910, U15 ATC_FUSE_BLOCK, U16 ATC_FUSE_BLOCK, U17 ATC_FUSE_BLOCK, U18 ATC_FUSE_BLOCK, U19 ACS722xLCTR-40AU, U2 ATC_FUSE_BLOCK, U20 ACS722xLCTR-40AU, U21 ACS722xLCTR-40AU, U22 ACS722xLCTR-40AU, U23 LT1910, U24 LT1910, U25 LT1910, U26 LT1910, U27 ATC_FUSE_BLOCK, U28 ATC_FUSE_BLOCK, U29 ATC_FUSE_BLOCK, U3 ATC_FUSE_BLOCK, U30 ATC_FUSE_BLOCK, U31 ACS722xLCTR-40AU, U32 ACS722xLCTR-40AU, U33 ACS722xLCTR-40AU, U34 ACS722xLCTR-40AU, U4 ATC_FUSE_BLOCK, U5 LT1910, U6 LT1910, U7 ACS722xLCTR-40AU, U8 ACS722xLCTR-40AU, U9 ACS722xLCTR-40AU

Commit message: Added Extra Documentation and Finished Layout and ready for final review
Documentation of the libraries required for this project were added. The layout is now finished and updtated from the last review. It is now ready for another review. After next review a BOM will be added.
Connections:
- net labels removed: LOGIC-SIG
Changed lines of the file:
@@
 LIBS:MRDT_Silkscreens
 LIBS:MRDT_Switches
+LIBS:PowerBoard_Hardware-cache
 EELAYER 26 0
 EELAYER END
@@
 $EndComp
 Text GLabel 5200 3000 0    50   Input ~ 0
-LOGIC-SIG
+LOGIC_CTL
 Wire Wire Line
 	6450 2400 6450 2850
@@
 	3300 14350 3450 14350
 $Comp
-L power:+3.3VA #PWR?
+L power:+3.3VA #PWR0102
 U 1 1 5D01A417
 P 2050 10900
-F 0 "#PWR?" H 2050 10750 50  0001 C CNN
+F 0 "#PWR0102" H 2050 10750 50  0001 C CNN
 F 1 "+3.3VA" H 2065 11073 50  0000 C CNN
 F 2 "" H 2050 10900 50  0001 C CNN
@@
 $EndComp
 $Comp
-L power:+3.3VA #PWR?
+L power:+3.3VA #PWR0103
 U 1 1 5D01AD6C
 P 3350 10900
-F 0 "#PWR?" H 3350 10750 50  0001 C CNN
+F 0 "#PWR0103" H 3350 10750 50  0001 C CNN
 F 1 "+3.3VA" H 3365 11073 50  0000 C CNN
 F 2 "" H 3350 10900 50  0001 C CNN
@@
 	8300 10500 8300 10550
 $Comp
-L power:+3.3VA #PWR?
+L power:+3.3VA #PWR0143
 U 1 1 5D180712
 P 8750 10200
-F 0 "#PWR?" H 8750 10050 50  0001 C CNN
+F 0 "#PWR0143" H 8750 10050 50  0001 C CNN
 F 1 "+3.3VA" H 8765 10373 50  0000 C CNN
 F 2 "" H 8750 10200 50  0001 C CNN
@@
 	7950 2600 8000 2600
 $Comp
-L power:+3.3VA #PWR?
+L power:+3.3VA #PWR0144
 U 1 1 5D694E20
 P 8000 2150
-F 0 "#PWR?" H 8000 2000 50  0001 C CNN
+F 0 "#PWR0144" H 8000 2000 50  0001 C CNN
 F 1 "+3.3VA" H 8015 2323 50  0000 C CNN
 F 2 "" H 8000 2150 50  0001 C CNN
@@
 	8200 5200 8250 5200
 $Comp
-L power:+3.3VA #PWR?
+L power:+3.3VA #PWR0145
 U 1 1 5D9DEEDD
 P 8300 4800
-F 0 "#PWR?" H 8300 4650 50  0001 C CNN
+F 0 "#PWR0145" H 8300 4650 50  0001 C CNN
 F 1 "+3.3VA" H 8315 4973 50  0000 C CNN
 F 2 "" H 8300 4800 50  0001 C CNN
@@
 	8150 7450 8200 7450
 $Comp
-L power:+3.3VA #PWR?
+L power:+3.3VA #PWR0146
 U 1 1 5DB72D3B
 P 8300 7050
-F 0 "#PWR?" H 8300 6900 50  0001 C CNN
+F 0 "#PWR0146" H 8300 6900 50  0001 C CNN
 F 1 "+3.3VA" H 8315 7223 50  0000 C CNN
 F 2 "" H 8300 7050 50  0001 C CNN
@@
 	8800 7350 8800 7400
 $Comp
-L power:+3.3VA #PWR?
+L power:+3.3VA #PWR0147
 U 1 1 5DBFAD18
 P 5800 10200
-F 0 "#PWR?" H 5800 10050 50  0001 C CNN
+F 0 "#PWR0147" H 5800 10050 50  0001 C CNN
 F 1 "+3.3VA" H 5815 10373 50  0000 C CNN
 F 2 "" H 5800 10200 50  0001 C CNN
@@
 	13000 2300 13050 2300
 $Comp
-L power:+3.3VA #PWR?
+L power:+3.3VA #PWR0197
 U 1 1 5DD0FE22
 P 13100 1900
-F 0 "#PWR?" H 13100 1750 50  0001 C CNN
+F 0 "#PWR0197" H 13100 1750 50  0001 C CNN
 F 1 "+3.3VA" H 13115 2073 50  0000 C CNN
 F 2 "" H 13100 1900 50  0001 C CNN
@@
 	13050 5450 13550 5450
 $Comp
-L power:+3.3VA #PWR?
+L power:+3.3VA #PWR0198
 U 1 1 5E04EFB8
 P 13550 5450
-F 0 "#PWR?" H 13550 5300 50  0001 C CNN
+F 0 "#PWR0198" H 13550 5300 50  0001 C CNN
 F 1 "+3.3VA" H 13565 5623 50  0000 C CNN
 F 2 "" H 13550 5450 50  0001 C CNN
@@
 	10700 9900 10650 9900
 $Comp
-L power:+3.3VA #PWR?
+L power:+3.3VA #PWR0199
 U 1 1 5E1F7246
 P 13500 9150
-F 0 "#PWR?" H 13500 9000 50  0001 C CNN
+F 0 "#PWR0199" H 13500 9000 50  0001 C CNN
 F 1 "+3.3VA" H 13515 9323 50  0000 C CNN
 F 2 "" H 13500 9150 50  0001 C CNN
@@
 	12150 12600 12150 13300
 $Comp
-L power:+3.3VA #PWR?
+L power:+3.3VA #PWR0200
 U 1 1 5E4331EF
 P 13300 13100
-F 0 "#PWR?" H 13300 12950 50  0001 C CNN
+F 0 "#PWR0200" H 13300 12950 50  0001 C CNN
 F 1 "+3.3VA" H 13315 13273 50  0000 C CNN
 F 2 "" H 13300 13100 50  0001 C CNN
@@
 	13800 13300 13800 13350
 $Comp
-L power:+3.3VA #PWR?
+L power:+3.3VA #PWR0201
 U 1 1 5E4C2DFE
 P 5600 15900
-F 0 "#PWR?" H 5600 15750 50  0001 C CNN
+F 0 "#PWR0201" H 5600 15750 50  0001 C CNN
 F 1 "+3.3VA" H 5615 16073 50  0000 C CNN
 F 2 "" H 5600 15900 50  0001 C CNN
@@
 	20900 2250 20900 2300
 $Comp
-L power:+3.3VA #PWR?
+L power:+3.3VA #PWR0202
 U 1 1 5E79D8E9
 P 20400 2000
-F 0 "#PWR?" H 20400 1850 50  0001 C CNN
+F 0 "#PWR0202" H 20400 1850 50  0001 C CNN
 F 1 "+3.3VA" H 20415 2173 50  0000 C CNN
 F 2 "" H 20400 2000 50  0001 C CNN
@@
 	19600 6100 19650 6100
 $Comp
-L power:+3.3VA #PWR?
+L power:+3.3VA #PWR0203
 U 1 1 5E8C4FB9
 P 19700 5700
-F 0 "#PWR?" H 19700 5550 50  0001 C CNN
+F 0 "#PWR0203" H 19700 5550 50  0001 C CNN
 F 1 "+3.3VA" H 19715 5873 50  0000 C CNN
 F 2 "" H 19700 5700 50  0001 C CNN
@@
 	20750 9400 20750 9550
 $Comp
-L power:+3.3VA #PWR?
+L power:+3.3VA #PWR0204
 U 1 1 5EBADC4C
 P 20300 9200
-F 0 "#PWR?" H 20300 9050 50  0001 C CNN
+F 0 "#PWR0204" H 20300 9050 50  0001 C CNN
 F 1 "+3.3VA" H 20315 9373 50  0000 C CNN
 F 2 "" H 20300 9200 50  0001 C CNN
@@
 	20800 12650 20800 12750
 $Comp
-L power:+3.3VA #PWR?
+L power:+3.3VA #PWR0205
 U 1 1 5EE02C07
 P 20300 12450
-F 0 "#PWR?" H 20300 12300 50  0001 C CNN
+F 0 "#PWR0205" H 20300 12300 50  0001 C CNN
 F 1 "+3.3VA" H 20315 12623 50  0000 C CNN
 F 2 "" H 20300 12450 50  0001 C CNN

Commit message: Moved Packages and Devices. Performed Basic Touch ups
Fixed some silkscreen and bad routing for a cleaner look. Moved the Packages and Devices to their own folder.
Parts:
- added D14: D_Schottky, Diodes_SMD:D_0603, symbol Device:D_Schottky
- CONV1, CONV2: footprint DC-DC_Converter_Quarter_Brick:DC-DC_Converter_Quarter_Brick -> DC_DC_Converter_Quarter_Brick:DC_DC_Converter_Quarter_Brick; symbol DC-DC_Converter:DC-DC_Converter -> DC_DC_Converter:DC-DC_Converter
- Conn1, Conn2, Conn3: footprint Vertical Anderson Double:Vertical Anderson Double -> Vertical Anderson Double:Vertical_Anderson_Double
Connections:
- wire segments 543 -> 547
Changed lines of the file:
@@
 	5350 1000 5350 1050
 Wire Wire Line
-	5350 1000 5850 1000
+	5350 1000 5700 1000
 Text GLabel 5850 1000 2    50   Output ~ 0
 VMEAS_VBATT
@@
 F 0 "Conn2" H 7250 4650 60  0000 R CNN
 F 1 "AndersonPP" H 7450 4750 60  0000 R CNN
-F 2 "Vertical Anderson Double:Vertical Anderson Double" H 6850 3850 60  0001 C CNN
+F 2 "Vertical Anderson Double:Vertical_Anderson_Double" H 6850 3850 60  0001 C CNN
 F 3 "" H 6850 3850 60  0001 C CNN
 	1    7000 4400
@@
 F 0 "Conn2" V 7510 4372 60  0000 R CNN
 F 1 "AndersonPP" V 7404 4372 60  0000 R CNN
-F 2 "Vertical Anderson Double:Vertical Anderson Double" H 7100 3850 60  0001 C CNN
+F 2 "Vertical Anderson Double:Vertical_Anderson_Double" H 7100 3850 60  0001 C CNN
 F 3 "" H 7100 3850 60  0001 C CNN
 	2    7250 4400
@@
 	4600 2400 4600 2650
 $Comp
-L DC-DC_Converter:DC-DC_Converter CONV1
+L DC_DC_Converter:DC-DC_Converter CONV1
 U 1 1 5BB35538
 P 2450 2350
 F 0 "CONV1" H 3100 2500 50  0000 C CNN
 F 1 "DC-DC_Converter" H 3100 2400 50  0000 C CNN
-F 2 "DC-DC_Converter_Quarter_Brick:DC-DC_Converter_Quarter_Brick" H 3000 2650 50  0001 C CNN
+F 2 "DC_DC_Converter_Quarter_Brick:DC_DC_Converter_Quarter_Brick" H 3000 2650 50  0001 C CNN
 F 3 "" H 3000 2650 50  0001 C CNN
 	1    2450 2350
@@
 F 0 "Conn3" H 7350 7100 60  0000 R CNN
 F 1 "AndersonPP" H 7550 7200 60  0000 R CNN
-F 2 "Vertical Anderson Double:Vertical Anderson Double" H 6950 6300 60  0001 C CNN
+F 2 "Vertical Anderson Double:Vertical_Anderson_Double" H 6950 6300 60  0001 C CNN
 F 3 "" H 6950 6300 60  0001 C CNN
 	1    7100 6850
@@
 F 0 "Conn3" V 7610 6822 60  0000 R CNN
 F 1 "AndersonPP" V 7504 6822 60  0000 R CNN
-F 2 "Vertical Anderson Double:Vertical Anderson Double" H 7200 6300 60  0001 C CNN
+F 2 "Vertical Anderson Double:Vertical_Anderson_Double" H 7200 6300 60  0001 C CNN
 F 3 "" H 7200 6300 60  0001 C CNN
 	2    7350 6850
@@
 $EndComp
 $Comp
-L DC-DC_Converter:DC-DC_Converter CONV2
+L DC_DC_Converter:DC-DC_Converter CONV2
 U 1 1 5BBF2506
 P 3050 7200
-F 0 "CONV2" H 3818 7775 50  0000 C CNN
-F 1 "DC-DC_Converter" H 3818 7684 50  0000 C CNN
-F 2 "DC-DC_Converter_Quarter_Brick:DC-DC_Converter_Quarter_Brick" H 3600 7500 50  0001 C CNN
+F 0 "CONV2" H 3650 7350 50  0000 C CNN
+F 1 "DC-DC_Converter" H 3700 7250 50  0000 C CNN
+F 2 "DC_DC_Converter_Quarter_Brick:DC_DC_Converter_Quarter_Brick" H 3600 7500 50  0001 C CNN
 F 3 "" H 3600 7500 50  0001 C CNN
 	1    3050 7200
@@
 F 0 "Conn1" V 6460 9272 60  0000 R CNN
 F 1 "AndersonPP" V 6354 9272 60  0000 R CNN
-F 2 "Vertical Anderson Double:Vertical Anderson Double" H 6050 8750 60  0001 C CNN
+F 2 "Vertical Anderson Double:Vertical_Anderson_Double" H 6050 8750 60  0001 C CNN
 F 3 "" H 6050 8750 60  0001 C CNN
 	2    6200 9300
@@
 F 0 "Conn1" H 6200 9550 60  0000 R CNN
 F 1 "AndersonPP" H 6400 9650 60  0000 R CNN
-F 2 "Vertical Anderson Double:Vertical Anderson Double" H 5800 8750 60  0001 C CNN
+F 2 "Vertical Anderson Double:Vertical_Anderson_Double" H 5800 8750 60  0001 C CNN
 F 3 "" H 5800 8750 60  0001 C CNN
 	1    5950 9300
@@
 Wire Notes Line
 	14250 1000 14250 16500
+$Comp
+L Device:D_Schottky D14
+U 1 1 5C0CE66D
+P 5700 850
+F 0 "D14" V 5654 929 50  0000 L CNN
+F 1 "D_Schottky" V 5745 929 50  0000 L CNN
+F 2 "Diodes_SMD:D_0603" H 5700 850 50  0001 C CNN
+F 3 "~" H 5700 850 50  0001 C CNN
+	1    5700 850
+	0    1    1    0
+$EndComp
+Connection ~ 5700 1000
+Wire Wire Line
+	5700 1000 5850 1000
+$Comp
+L power:+3.3VA #PWR0206
+U 1 1 5C0CEA57
+P 6000 750
+F 0 "#PWR0206" H 6000 600 50  0001 C CNN
+F 1 "+3.3VA" H 6015 923 50  0000 C CNN
+F 2 "" H 6000 750 50  0001 C CNN
+F 3 "" H 6000 750 50  0001 C CNN
+	1    6000 750
+	1    0    0    -1
+$EndComp
+Wire Wire Line
+	6000 750  5800 750
+Wire Wire Line
+	5800 750  5800 700
+Wire Wire Line
+	5800 700  5700 700
 $EndSCHEMATC

Commit message: Corrected Vertical Anderson Package
Parts:
- CONV1, CONV2: footprint DC_DC_Converter_Quarter_Brick:DC_DC_Converter_Quarter_Brick -> PowerBoard_Hardware:DC_DC_Converter_Quarter_Brick
- Conn1, Conn2, Conn3: footprint Vertical Anderson Double:Vertical_Anderson_Double -> PowerBoard_Hardware:Vertical_Anderson_Double_SidebySide
Changed lines of the file:
@@
 LIBS:power
 LIBS:device
+LIBS:switches
+LIBS:relays
+LIBS:motors
+LIBS:transistors
+LIBS:conn
+LIBS:linear
+LIBS:regul
 LIBS:74xx
+LIBS:cmos4000
+LIBS:adc-dac
+LIBS:memory
+LIBS:xilinx
+LIBS:microcontrollers
+LIBS:dsp
+LIBS:microchip
+LIBS:analog_switches
+LIBS:motorola
+LIBS:texas
+LIBS:intel
 LIBS:audio
 LIBS:interface
-LIBS:MRDT_Actives
-LIBS:MRDT_Connectors
-LIBS:MRDT_Devices
-LIBS:MRDT_Drill_Holes
-LIBS:MRDT_Headers
-LIBS:MRDT_ICs
-LIBS:MRDT_Passives
-LIBS:MRDT_Sensors
-LIBS:MRDT_Shields
-LIBS:MRDT_Silkscreens
-LIBS:MRDT_Switches
+LIBS:digital-audio
+LIBS:philips
+LIBS:display
+LIBS:cypress
+LIBS:siliconi
+LIBS:opto
+LIBS:atmel
+LIBS:contrib
+LIBS:valves
 LIBS:PowerBoard_Hardware-cache
 EELAYER 26 0
@@
 F 0 "Conn2" H 7250 4650 60  0000 R CNN
 F 1 "AndersonPP" H 7450 4750 60  0000 R CNN
-F 2 "Vertical Anderson Double:Vertical_Anderson_Double" H 6850 3850 60  0001 C CNN
+F 2 "PowerBoard_Hardware:Vertical_Anderson_Double_SidebySide" H 6850 3850 60  0001 C CNN
 F 3 "" H 6850 3850 60  0001 C CNN
 	1    7000 4400
@@
 F 0 "Conn2" V 7510 4372 60  0000 R CNN
 F 1 "AndersonPP" V 7404 4372 60  0000 R CNN
-F 2 "Vertical Anderson Double:Vertical_Anderson_Double" H 7100 3850 60  0001 C CNN
+F 2 "PowerBoard_Hardware:Vertical_Anderson_Double_SidebySide" H 7100 3850 60  0001 C CNN
 F 3 "" H 7100 3850 60  0001 C CNN
 	2    7250 4400
@@
 F 0 "CONV1" H 3100 2500 50  0000 C CNN
 F 1 "DC-DC_Converter" H 3100 2400 50  0000 C CNN
-F 2 "DC_DC_Converter_Quarter_Brick:DC_DC_Converter_Quarter_Brick" H 3000 2650 50  0001 C CNN
+F 2 "PowerBoard_Hardware:DC_DC_Converter_Quarter_Brick" H 3000 2650 50  0001 C CNN
 F 3 "" H 3000 2650 50  0001 C CNN
 	1    2450 2350
@@
 F 0 "Conn3" H 7350 7100 60  0000 R CNN
 F 1 "AndersonPP" H 7550 7200 60  0000 R CNN
-F 2 "Vertical Anderson Double:Vertical_Anderson_Double" H 6950 6300 60  0001 C CNN
+F 2 "PowerBoard_Hardware:Vertical_Anderson_Double_SidebySide" H 6950 6300 60  0001 C CNN
 F 3 "" H 6950 6300 60  0001 C CNN
 	1    7100 6850
@@
 F 0 "Conn3" V 7610 6822 60  0000 R CNN
 F 1 "AndersonPP" V 7504 6822 60  0000 R CNN
-F 2 "Vertical Anderson Double:Vertical_Anderson_Double" H 7200 6300 60  0001 C CNN
+F 2 "PowerBoard_Hardware:Vertical_Anderson_Double_SidebySide" H 7200 6300 60  0001 C CNN
 F 3 "" H 7200 6300 60  0001 C CNN
 	2    7350 6850
@@
 F 0 "CONV2" H 3650 7350 50  0000 C CNN
 F 1 "DC-DC_Converter" H 3700 7250 50  0000 C CNN
-F 2 "DC_DC_Converter_Quarter_Brick:DC_DC_Converter_Quarter_Brick" H 3600 7500 50  0001 C CNN
+F 2 "PowerBoard_Hardware:DC_DC_Converter_Quarter_Brick" H 3600 7500 50  0001 C CNN
 F 3 "" H 3600 7500 50  0001 C CNN
 	1    3050 7200
@@
 F 0 "Conn1" V 6460 9272 60  0000 R CNN
 F 1 "AndersonPP" V 6354 9272 60  0000 R CNN
-F 2 "Vertical Anderson Double:Vertical_Anderson_Double" H 6050 8750 60  0001 C CNN
+F 2 "PowerBoard_Hardware:Vertical_Anderson_Double_SidebySide" H 6050 8750 60  0001 C CNN
 F 3 "" H 6050 8750 60  0001 C CNN
 	2    6200 9300
@@
 F 0 "Conn1" H 6200 9550 60  0000 R CNN
 F 1 "AndersonPP" H 6400 9650 60  0000 R CNN
-F 2 "Vertical Anderson Double:Vertical_Anderson_Double" H 5800 8750 60  0001 C CNN
+F 2 "PowerBoard_Hardware:Vertical_Anderson_Double_SidebySide" H 5800 8750 60  0001 C CNN
 F 3 "" H 5800 8750 60  0001 C CNN
 	1    5950 9300

Commit message: Swapped Placment of Comm & Logic Busses
Connections:
- wire segments 547 -> 550
- no-connect marks 0 -> 55

Commit message: Added a BOM and Updated Capacitor Size
Added a BOM file in the Documentation file. Currently has 2 placeholder values in it due to unknown anderson powerpole colors. Updated the 330u capacitor package to fit a real capacitor.
Parts:
- C10, C11, C16, C6, C8, C9: footprint Capacitors_THT:CP_Radial_D6.3mm_P2.50mm -> Capacitors_THT:CP_Radial_D8.0mm_P3.50mm
- C26: value 0.1 -> 0.1u
Changed lines of the file:
@@
 LIBS:power
 LIBS:device
-LIBS:switches
-LIBS:relays
-LIBS:motors
-LIBS:transistors
-LIBS:conn
-LIBS:linear
-LIBS:regul
 LIBS:74xx
-LIBS:cmos4000
-LIBS:adc-dac
-LIBS:memory
-LIBS:xilinx
-LIBS:microcontrollers
-LIBS:dsp
-LIBS:microchip
-LIBS:analog_switches
-LIBS:motorola
-LIBS:texas
-LIBS:intel
 LIBS:audio
 LIBS:interface
-LIBS:digital-audio
-LIBS:philips
-LIBS:display
-LIBS:cypress
-LIBS:siliconi
-LIBS:opto
-LIBS:atmel
-LIBS:contrib
-LIBS:valves
+LIBS:MRDT_Actives
+LIBS:MRDT_Connectors
+LIBS:MRDT_Devices
+LIBS:MRDT_Drill_Holes
+LIBS:MRDT_Headers
+LIBS:MRDT_ICs
+LIBS:MRDT_Passives
+LIBS:MRDT_Sensors
+LIBS:MRDT_Shields
+LIBS:MRDT_Silkscreens
+LIBS:MRDT_Switches
 LIBS:PowerBoard_Hardware-cache
 EELAYER 26 0
@@
 F 0 "C9" H 4715 2896 50  0000 L CNN
 F 1 "330u" H 4715 2805 50  0000 L CNN
-F 2 "Capacitors_THT:CP_Radial_D6.3mm_P2.50mm" H 4600 2850 50  0001 C CNN
+F 2 "Capacitors_THT:CP_Radial_D8.0mm_P3.50mm" H 4600 2850 50  0001 C CNN
 F 3 "~" H 4600 2850 50  0001 C CNN
 	1    4600 2850
@@
 F 0 "C6" H 4200 2900 50  0000 L CNN
 F 1 "330u" H 4150 2800 50  0000 L CNN
-F 2 "Capacitors_THT:CP_Radial_D6.3mm_P2.50mm" H 4400 2850 50  0001 C CNN
+F 2 "Capacitors_THT:CP_Radial_D8.0mm_P3.50mm" H 4400 2850 50  0001 C CNN
 F 3 "~" H 4400 2850 50  0001 C CNN
 	1    4400 2850
@@
 F 0 "C8" H 3950 4500 50  0000 L CNN
 F 1 "330u" H 4000 4400 50  0000 L CNN
-F 2 "Capacitors_THT:CP_Radial_D6.3mm_P2.50mm" H 4250 4450 50  0001 C CNN
+F 2 "Capacitors_THT:CP_Radial_D8.0mm_P3.50mm" H 4250 4450 50  0001 C CNN
 F 3 "~" H 4250 4450 50  0001 C CNN
 	1    4250 4450
@@
 F 0 "C10" H 4565 4496 50  0000 L CNN
 F 1 "330u" H 4565 4405 50  0000 L CNN
-F 2 "Capacitors_THT:CP_Radial_D6.3mm_P2.50mm" H 4450 4450 50  0001 C CNN
+F 2 "Capacitors_THT:CP_Radial_D8.0mm_P3.50mm" H 4450 4450 50  0001 C CNN
 F 3 "~" H 4450 4450 50  0001 C CNN
 	1    4450 4450
@@
 F 0 "C11" H 4750 7600 50  0000 L CNN
 F 1 "330u" H 4750 7500 50  0000 L CNN
-F 2 "Capacitors_THT:CP_Radial_D6.3mm_P2.50mm" H 4600 7550 50  0001 C CNN
+F 2 "Capacitors_THT:CP_Radial_D8.0mm_P3.50mm" H 4600 7550 50  0001 C CNN
 F 3 "~" H 4600 7550 50  0001 C CNN
 	1    4600 7550
@@
 P 18800 9450
 F 0 "C26" V 18571 9450 50  0000 C CNN
-F 1 "0.1" V 18662 9450 50  0000 C CNN
+F 1 "0.1u" V 18662 9450 50  0000 C CNN
 F 2 "Capacitors_SMD:C_0603_HandSoldering" H 18800 9450 50  0001 C CNN
 F 3 "~" H 18800 9450 50  0001 C CNN
@@
 F 0 "C16" H 5865 7546 50  0000 L CNN
 F 1 "330u" H 5865 7455 50  0000 L CNN
-F 2 "Capacitors_THT:CP_Radial_D6.3mm_P2.50mm" H 5750 7500 50  0001 C CNN
+F 2 "Capacitors_THT:CP_Radial_D8.0mm_P3.50mm" H 5750 7500 50  0001 C CNN
 F 3 "~" H 5750 7500 50  0001 C CNN
 	1    5750 7500

Commit message: Updated Gerbs and Updated BOM
Basic Updates to make the BOM more legible. Also the Layout and Schematic were updated for easier reading and a new Gerbs was generated to reflect this.
Parts:
- Q3: value IPT020N10N3 -> N_Fet
- Q4, Q5: value IPT020N10N3 -> FDD8780
Other:
- note added: "20A"
- note added: "20A\n"
- note added: "30A"
- note added: "30A\n"
- note added: "5A"
- note added: "5A\n"
- note added: "A0"
- note added: "A10\n"
- note added: "A11"
- note added: "A12"
- note added: "A13"
- note added: "A14"
- note added: "A15"
- note added: "A1\n"
- note added: "A2"
- note added: "A3\n"
- note added: "A8"
- note added: "Green"
- note added: "IRFS7437TRLPDF"
- note added: "Orange"
- note added: "Orange\n"
- note added: "Q36SR12020NRFA"

Commit message: Updated to KiCAD libraries Rev 2
Parts:
- CONV1, CONV2: footprint PowerBoard_Hardware:DC_DC_Converter_Quarter_Brick -> MRDT_Devices:Q36SR12020NRFA; symbol DC_DC_Converter:DC-DC_Converter -> MRDT_Devices:Q36SR12020NRFA
- Conn1, Conn2, Conn3: footprint PowerBoard_Hardware:Vertical_Anderson_Double_SidebySide -> MRDT_Connectors:Anderson_2_Vertical_Sidy_by_Side
- U1: footprint MRDT-SHIELDS:TM4C129E_Launchpad_FULL -> MRDT_Shields:TM4C129E_Launchpad_FULL_THT_TOP
- U15, U16, U17, U18: footprint MRDT-Passives:ATC_Fuse_Block -> MRDT_Passives:ATC_Fuse_Block
Connections:
- wire segments 550 -> 551
