File: CameraBoard_Hardware/CameraBoard_Hardware.sch (KiCad schematic (older format))
At the start: 38 parts, among them J1 BNC_75_OHM_HORIZ, J2 BNC_75_OHM_HORIZ, U1 TM4C129E_Launchpad, U2 AP1059, U3 MAX4314ESD+, U4 MAX4314ESD+

Commit message: Updates Power Conversion
Parts:
- removed D5: D_Schottky, Diodes_SMD:D_0603, symbol Device:D_Schottky
- removed L1: 47u, MRDT_Passives:DR74_330_R, symbol Device:L
- removed U2: AP1059, Housings_SOIC:HTSOP-8-1EP_3.9x4.9mm_Pitch1.27mm, symbol MRDT_ICs:AP1059
- added U2: OKI, MRDT_Devices:OKI_Horizontal, symbol MRDT_Devices:OKI
- C1, C2: value 10u -> 10uF
Connections:
- wire segments 122 -> 108
Other:
- note added: "5V"
Changed lines of the file:
@@
 	1050 700  1050 7400
-$Comp
-L MRDT_ICs:AP1059 U2
-U 1 1 5C126042
-P 3000 1800
-F 0 "U2" H 3225 2397 60  0000 C CNN
-F 1 "AP1059" H 3225 2291 60  0000 C CNN
-F 2 "Housings_SOIC:HTSOP-8-1EP_3.9x4.9mm_Pitch1.27mm" H 2750 1700 60  0001 C CNN
-F 3 "" H 2750 1700 60  0001 C CNN
-	1    3000 1800
-	1    0    0    -1
-$EndComp
-$Comp
-L power:+12V #PWR0114
-U 1 1 5C12665D
-P 2200 1450
-F 0 "#PWR0114" H 2200 1300 50  0001 C CNN
-F 1 "+12V" H 2215 1623 50  0000 C CNN
-F 2 "" H 2200 1450 50  0001 C CNN
-F 3 "" H 2200 1450 50  0001 C CNN
-	1    2200 1450
-	1    0    0    -1
-$EndComp
-$Comp
-L Device:C C1
-U 1 1 5C1266C4
-P 2350 1600
-F 0 "C1" H 2465 1646 50  0000 L CNN
-F 1 "10u" H 2465 1555 50  0000 L CNN
-F 2 "Capacitors_SMD:C_0603_HandSoldering" H 2388 1450 50  0001 C CNN
-F 3 "~" H 2350 1600 50  0001 C CNN
-	1    2350 1600
-	1    0    0    -1
-$EndComp
-Wire Wire Line
-	2200 1450 2350 1450
-Wire Wire Line
-	2350 1450 2800 1450
-Connection ~ 2350 1450
-$Comp
-L Device:D_Schottky D5
-U 1 1 5C12891B
-P 2350 2000
-F 0 "D5" V 2400 2150 50  0000 R CNN
-F 1 "D_Schottky" V 2300 2500 50  0000 R CNN
-F 2 "Diodes_SMD:D_0603" H 2350 2000 50  0001 C CNN
-F 3 "~" H 2350 2000 50  0001 C CNN
-	1    2350 2000
-	0    -1   -1   0
-$EndComp
-Wire Wire Line
-	2350 1750 2350 1850
-$Comp
-L Device:L L1
-U 1 1 5C12AD0A
-P 2750 2150
-F 0 "L1" V 2800 2150 50  0000 C CNN
-F 1 "47u" V 2700 2150 50  0000 C CNN
-F 2 "MRDT_Passives:DR74_330_R" H 2750 2150 50  0001 C CNN
-F 3 "~" H 2750 2150 50  0001 C CNN
-	1    2750 2150
-	0    -1   -1   0
-$EndComp
-Wire Wire Line
-	2350 2150 2600 2150
-Wire Wire Line
-	2350 1850 2800 1850
-Wire Wire Line
-	3650 1850 3650 1750
-Connection ~ 2350 1850
-Wire Wire Line
-	3650 1550 3650 1450
-Connection ~ 3650 1550
-Wire Wire Line
-	3650 1650 3650 1550
-Connection ~ 3650 1650
-Wire Wire Line
-	3650 1750 3650 1650
-Connection ~ 3650 1750
-Wire Wire Line
-	2800 1750 2800 1850
-Wire Wire Line
-	2800 1850 3150 1850
-Connection ~ 2800 1850
-Wire Wire Line
-	2800 1650 2700 1650
-Wire Wire Line
-	2700 1650 2700 2000
-Wire Wire Line
-	2700 2000 2900 2000
-Wire Wire Line
-	2900 2000 2900 2150
-$Comp
-L Device:C C2
-U 1 1 5C13507C
-P 3150 2000
-F 0 "C2" H 3265 2046 50  0000 L CNN
-F 1 "10u" H 3265 1955 50  0000 L CNN
-F 2 "Capacitors_SMD:C_0603_HandSoldering" H 3188 1850 50  0001 C CNN
-F 3 "~" H 3150 2000 50  0001 C CNN
-	1    3150 2000
-	1    0    0    -1
-$EndComp
-Wire Wire Line
-	3150 1850 3650 1850
-Connection ~ 3150 1850
-Wire Wire Line
-	2900 2150 3150 2150
-Connection ~ 2900 2150
-Wire Wire Line
-	3150 2150 3850 2150
-Connection ~ 3150 2150
-Wire Wire Line
-	2800 1550 2600 1550
-Wire Wire Line
-	2600 1550 2600 2150
-Connection ~ 2600 2150
-$Comp
-L power:GND #PWR0116
-U 1 1 5C13EC2E
-P 3950 1450
-F 0 "#PWR0116" H 3950 1200 50  0001 C CNN
-F 1 "GND" H 3955 1277 50  0000 C CNN
-F 2 "" H 3950 1450 50  0001 C CNN
-F 3 "" H 3950 1450 50  0001 C CNN
-	1    3950 1450
-	1    0    0    -1
-$EndComp
-Wire Wire Line
-	3650 1450 3950 1450
-Connection ~ 3650 1450
-$Comp
-L power:+5V #PWR0117
-U 1 1 5C149AEC
-P 3850 2150
-F 0 "#PWR0117" H 3850 2000 50  0001 C CNN
-F 1 "+5V" H 3865 2323 50  0000 C CNN
-F 2 "" H 3850 2150 50  0001 C CNN
-F 3 "" H 3850 2150 50  0001 C CNN
-	1    3850 2150
-	1    0    0    -1
-$EndComp
 $Comp
 L power:+5V #PWR0118
@@
 L MRDT_Connectors:AndersonPP Conn1
 U 1 1 5C21D58C
-P 3400 3250
-F 0 "Conn1" H 3200 3400 60  0000 C CNN
-F 1 "AndersonPP" H 3100 3300 60  0000 C CNN
-F 2 "MRDT_Connectors:Anderson_2_Horisontal_Side_by_Side" H 3250 2700 60  0001 C CNN
-F 3 "" H 3250 2700 60  0001 C CNN
-	1    3400 3250
+P 1750 2000
+F 0 "Conn1" H 1550 2150 60  0000 C CNN
+F 1 "AndersonPP" H 1450 2050 60  0000 C CNN
+F 2 "MRDT_Connectors:Anderson_2_Horisontal_Side_by_Side" H 1600 1450 60  0001 C CNN
+F 3 "" H 1600 1450 60  0001 C CNN
+	1    1750 2000
 	1    0    0    -1
 $EndComp
@@
 L MRDT_Connectors:AndersonPP Conn1
 U 2 1 5C21D625
-P 3400 2950
-F 0 "Conn1" H 3200 3100 60  0000 C CNN
-F 1 "AndersonPP" H 3100 3000 60  0000 C CNN
-F 2 "MRDT_Connectors:Anderson_2_Horisontal_Side_by_Side" H 3250 2400 60  0001 C CNN
-F 3 "" H 3250 2400 60  0001 C CNN
-	2    3400 2950
+P 1750 1700
+F 0 "Conn1" H 1550 1850 60  0000 C CNN
+F 1 "AndersonPP" H 1450 1750 60  0000 C CNN
+F 2 "MRDT_Connectors:Anderson_2_Horisontal_Side_by_Side" H 1600 1150 60  0001 C CNN
+F 3 "" H 1600 1150 60  0001 C CNN
+	2    1750 1700
 	1    0    0    -1
 $EndComp
@@
 L power:+12V #PWR0111
 U 1 1 5C21D84B
-P 3850 2800
-F 0 "#PWR0111" H 3850 2650 50  0001 C CNN
-F 1 "+12V" H 3865 2973 50  0000 C CNN
-F 2 "" H 3850 2800 50  0001 C CNN
-F 3 "" H 3850 2800 50  0001 C CNN
-	1    3850 2800
+P 2200 1550
+F 0 "#PWR0111" H 2200 1400 50  0001 C CNN
+F 1 "+12V" H 2215 1723 50  0000 C CNN
+F 2 "" H 2200 1550 50  0001 C CNN
+F 3 "" H 2200 1550 50  0001 C CNN
+	1    2200 1550
 	1    0    0    -1
 $EndComp
@@
 L power:GND #PWR0119
 U 1 1 5C221CE3
-P 3850 3200
-F 0 "#PWR0119" H 3850 2950 50  0001 C CNN
-F 1 "GND" H 3855 3027 50  0000 C CNN
-F 2 "" H 3850 3200 50  0001 C CNN
-F 3 "" H 3850 3200 50  0001 C CNN
-	1    3850 3200
-	1    0    0    -1
-$EndComp
-Wire Wire Line
-	3800 3150 3850 3150
-Wire Wire Line
-	3850 3150 3850 3200
-Wire Wire Line
-	3800 2850 3850 2850
-Wire Wire Line
-	3850 2850 3850 2800
+P 2200 1950
+F 0 "#PWR0119" H 2200 1700 50  0001 C CNN
+F 1 "GND" H 2205 1777 50  0000 C CNN
+F 2 "" H 2200 1950 50  0001 C CNN
+F 3 "" H 2200 1950 50  0001 C CNN
+	1    2200 1950
+	1    0    0    -1
+$EndComp
+Wire Wire Line
+	2150 1900 2200 1900
+Wire Wire Line
+	2200 1900 2200 1950
+Wire Wire Line
+	2150 1600 2200 1600
+Wire Wire Line
+	2200 1600 2200 1550
 $Comp
 L Device:R R12
@@
 NoConn ~ 3750 5050
 NoConn ~ 4800 5150
+$Comp
+L MRDT_Devices:OKI U2
+U 1 1 5C1669E7
+P 2650 1700
+F 0 "U2" H 2700 1650 60  0001 C CNN
+F 1 "OKI" H 2850 1981 60  0000 C CNN
+F 2 "MRDT_Devices:OKI_Horizontal" H 2450 1600 60  0001 C CNN
+F 3 "" H 2450 1600 60  0001 C CNN
+	1    2650 1700
+	1    0    0    -1
+$EndComp
+$Comp
+L Device:C C1
+U 1 1 5C166A5A
+P 2350 1750
+F 0 "C1" H 2400 1850 50  0000 L CNN
+F 1 "10uF" H 2400 1650 50  0000 L CNN
+F 2 "Capacitors_SMD:C_0603_HandSoldering" H 2388 1600 50  0001 C CNN
+F 3 "~" H 2350 1750 50  0001 C CNN
+	1    2350 1750
+	1    0    0    -1
+$EndComp
+$Comp
+L Device:C C2
+U 1 1 5C166B56
+P 3350 1750
+F 0 "C2" H 3400 1850 50  0000 L CNN
+F 1 "10uF" H 3150 1650 50  0000 L CNN
+F 2 "Capacitors_SMD:C_0603_HandSoldering" H 3388 1600 50  0001 C CNN
+F 3 "~" H 3350 1750 50  0001 C CNN
+	1    3350 1750
+	1    0    0    -1
+$EndComp
+$Comp
+L power:+5V #PWR0114
+U 1 1 5C167097
+P 3350 1550
+F 0 "#PWR0114" H 3350 1400 50  0001 C CNN
+F 1 "+5V" H 3365 1723 50  0000 C CNN
+F 2 "" H 3350 1550 50  0001 C CNN
+F 3 "" H 3350 1550 50  0001 C CNN
+	1    3350 1550
+	1    0    0    -1
+$EndComp
+Connection ~ 2200 1900
+Connection ~ 2350 1900
+Wire Wire Line
+	2350 1900 2200 1900
+Connection ~ 2850 1900
+Wire Wire Line
+	2850 1900 2350 1900
+Wire Wire Line
+	3350 1900 2850 1900
+Wire Wire Line
+	2200 1600 2350 1600
+Connection ~ 2200 1600
+Connection ~ 2350 1600
+Wire Wire Line
+	2350 1600 2450 1600
+Wire Wire Line
+	3250 1600 3350 1600
+Text Notes 2950 1800 0    50   ~ 0
+5V
+Wire Wire Line
+	3350 1550 3350 1600
+Connection ~ 3350 1600
 $EndSCHEMATC

Commit message: fixed 5V via issue
Other:
- note removed: "Power Input"
Changed lines of the file:
@@
 encoding utf-8
 Sheet 1 1
-Title ""
-Date ""
-Rev ""
-Comp ""
-Comment1 ""
+Title "CameraBoard"
+Date "2018-12-16"
+Rev "1"
+Comp "Mars Rover Design Team"
+Comment1 "Shaun McManus"
 Comment2 ""
 Comment3 ""
@@
 	1    0    0    -1
 $EndComp
-Text Notes 1050 2750 0    157  ~ 31
-Power Input
 Text GLabel 3700 4750 0    50   Output ~ 0
 MUXB0
@@
 	3950 6350 3950 6400
 Wire Notes Line
-	1050 2500 5700 2500
-Wire Notes Line
 	5700 700  5700 7400
 Wire Notes Line
@@
 L MRDT_Connectors:AndersonPP Conn1
 U 1 1 5C21D58C
-P 1750 2000
-F 0 "Conn1" H 1550 2150 60  0000 C CNN
-F 1 "AndersonPP" H 1450 2050 60  0000 C CNN
-F 2 "MRDT_Connectors:Anderson_2_Horisontal_Side_by_Side" H 1600 1450 60  0001 C CNN
-F 3 "" H 1600 1450 60  0001 C CNN
-	1    1750 2000
+P 1700 2600
+F 0 "Conn1" H 1500 2750 60  0000 C CNN
+F 1 "AndersonPP" H 1400 2650 60  0000 C CNN
+F 2 "MRDT_Connectors:Anderson_2_Horisontal_Side_by_Side" H 1550 2050 60  0001 C CNN
+F 3 "" H 1550 2050 60  0001 C CNN
+	1    1700 2600
 	1    0    0    -1
 $EndComp
@@
 L MRDT_Connectors:AndersonPP Conn1
 U 2 1 5C21D625
-P 1750 1700
-F 0 "Conn1" H 1550 1850 60  0000 C CNN
-F 1 "AndersonPP" H 1450 1750 60  0000 C CNN
-F 2 "MRDT_Connectors:Anderson_2_Horisontal_Side_by_Side" H 1600 1150 60  0001 C CNN
-F 3 "" H 1600 1150 60  0001 C CNN
-	2    1750 1700
+P 1700 2300
+F 0 "Conn1" H 1500 2450 60  0000 C CNN
+F 1 "AndersonPP" H 1400 2350 60  0000 C CNN
+F 2 "MRDT_Connectors:Anderson_2_Horisontal_Side_by_Side" H 1550 1750 60  0001 C CNN
+F 3 "" H 1550 1750 60  0001 C CNN
+	2    1700 2300
 	1    0    0    -1
 $EndComp
@@
 L power:+12V #PWR0111
 U 1 1 5C21D84B
-P 2200 1550
-F 0 "#PWR0111" H 2200 1400 50  0001 C CNN
-F 1 "+12V" H 2215 1723 50  0000 C CNN
-F 2 "" H 2200 1550 50  0001 C CNN
-F 3 "" H 2200 1550 50  0001 C CNN
-	1    2200 1550
+P 2150 2150
+F 0 "#PWR0111" H 2150 2000 50  0001 C CNN
+F 1 "+12V" H 2165 2323 50  0000 C CNN
+F 2 "" H 2150 2150 50  0001 C CNN
+F 3 "" H 2150 2150 50  0001 C CNN
+	1    2150 2150
 	1    0    0    -1
 $EndComp
@@
 L power:GND #PWR0119
 U 1 1 5C221CE3
-P 2200 1950
-F 0 "#PWR0119" H 2200 1700 50  0001 C CNN
-F 1 "GND" H 2205 1777 50  0000 C CNN
-F 2 "" H 2200 1950 50  0001 C CNN
-F 3 "" H 2200 1950 50  0001 C CNN
-	1    2200 1950
-	1    0    0    -1
-$EndComp
-Wire Wire Line
-	2150 1900 2200 1900
-Wire Wire Line
-	2200 1900 2200 1950
-Wire Wire Line
-	2150 1600 2200 1600
-Wire Wire Line
-	2200 1600 2200 1550
+P 2150 2550
+F 0 "#PWR0119" H 2150 2300 50  0001 C CNN
+F 1 "GND" H 2155 2377 50  0000 C CNN
+F 2 "" H 2150 2550 50  0001 C CNN
+F 3 "" H 2150 2550 50  0001 C CNN
+	1    2150 2550
+	1    0    0    -1
+$EndComp
+Wire Wire Line
+	2100 2500 2150 2500
+Wire Wire Line
+	2150 2500 2150 2550
+Wire Wire Line
+	2100 2200 2150 2200
+Wire Wire Line
+	2150 2200 2150 2150
 $Comp
 L Device:R R12
 U 1 1 5C2363E3
-P 4650 1450
-F 0 "R12" H 4720 1496 50  0000 L CNN
-F 1 "100" H 4720 1405 50  0000 L CNN
-F 2 "Resistors_SMD:R_0603_HandSoldering" V 4580 1450 50  0001 C CNN
-F 3 "~" H 4650 1450 50  0001 C CNN
-	1    4650 1450
+P 4600 2050
+F 0 "R12" H 4670 2096 50  0000 L CNN
+F 1 "100" H 4670 2005 50  0000 L CNN
+F 2 "Resistors_SMD:R_0603_HandSoldering" V 4530 2050 50  0001 C CNN
+F 3 "~" H 4600 2050 50  0001 C CNN
+	1    4600 2050
 	1    0    0    -1
 $EndComp
@@
 L Device:R R13
 U 1 1 5C2363EA
-P 4650 1850
-F 0 "R13" H 4720 1896 50  0000 L CNN
-F 1 "500" H 4720 1805 50  0000 L CNN
-F 2 "Resistors_SMD:R_0603_HandSoldering" V 4580 1850 50  0001 C CNN
-F 3 "~" H 4650 1850 50  0001 C CNN
-	1    4650 1850
+P 4600 2450
+F 0 "R13" H 4670 2496 50  0000 L CNN
+F 1 "500" H 4670 2405 50  0000 L CNN
+F 2 "Resistors_SMD:R_0603_HandSoldering" V 4530 2450 50  0001 C CNN
+F 3 "~" H 4600 2450 50  0001 C CNN
+	1    4600 2450
 	1    0    0    -1
 $EndComp
@@
 L power:GND #PWR0121
 U 1 1 5C2363F1
-P 4650 2050
-F 0 "#PWR0121" H 4650 1800 50  0001 C CNN
-F 1 "GND" V 4655 1922 50  0000 R CNN
-F 2 "" H 4650 2050 50  0001 C CNN
-F 3 "" H 4650 2050 50  0001 C CNN
-	1    4650 2050
-	1    0    0    -1
-$EndComp
-Wire Wire Line
-	4650 2000 4650 2050
+P 4600 2650
+F 0 "#PWR0121" H 4600 2400 50  0001 C CNN
+F 1 "GND" V 4605 2522 50  0000 R CNN
+F 2 "" H 4600 2650 50  0001 C CNN
+F 3 "" H 4600 2650 50  0001 C CNN
+	1    4600 2650
+	1    0    0    -1
+$EndComp
+Wire Wire Line
+	4600 2600 4600 2650
 $Comp
 L power:+12V #PWR0122
 U 1 1 5C2363F8
-P 4650 1250
-F 0 "#PWR0122" H 4650 1100 50  0001 C CNN
-F 1 "+12V" H 4665 1423 50  0000 C CNN
-F 2 "" H 4650 1250 50  0001 C CNN
-F 3 "" H 4650 1250 50  0001 C CNN
-	1    4650 1250
-	1    0    0    -1
-$EndComp
-Wire Wire Line
-	4650 1300 4650 1250
+P 4600 1850
+F 0 "#PWR0122" H 4600 1700 50  0001 C CNN
+F 1 "+12V" H 4615 2023 50  0000 C CNN
+F 2 "" H 4600 1850 50  0001 C CNN
+F 3 "" H 4600 1850 50  0001 C CNN
+	1    4600 1850
+	1    0    0    -1
+$EndComp
+Wire Wire Line
+	4600 1900 4600 1850
 $Comp
 L power:+10V #PWR0124
 U 1 1 5C23ABD5
-P 5000 1650
-F 0 "#PWR0124" H 5000 1500 50  0001 C CNN
-F 1 "+10V" H 5015 1823 50  0000 C CNN
-F 2 "" H 5000 1650 50  0001 C CNN
-F 3 "" H 5000 1650 50  0001 C CNN
-	1    5000 1650
-	1    0    0    -1
-$EndComp
-Wire Wire Line
-	4650 1600 4650 1650
-Wire Wire Line
-	4650 1650 5000 1650
-Connection ~ 4650 1650
-Wire Wire Line
-	4650 1650 4650 1700
+P 4950 2250
+F 0 "#PWR0124" H 4950 2100 50  0001 C CNN
+F 1 "+10V" H 4965 2423 50  0000 C CNN
+F 2 "" H 4950 2250 50  0001 C CNN
+F 3 "" H 4950 2250 50  0001 C CNN
+	1    4950 2250
+	1    0    0    -1
+$EndComp
+Wire Wire Line
+	4600 2200 4600 2250
+Wire Wire Line
+	4600 2250 4950 2250
+Connection ~ 4600 2250
+Wire Wire Line
+	4600 2250 4600 2300
 $Comp
 L power:+10V #PWR0125
@@
 L MRDT_Devices:OKI U2
 U 1 1 5C1669E7
-P 2650 1700
-F 0 "U2" H 2700 1650 60  0001 C CNN
-F 1 "OKI" H 2850 1981 60  0000 C CNN
-F 2 "MRDT_Devices:OKI_Horizontal" H 2450 1600 60  0001 C CNN
-F 3 "" H 2450 1600 60  0001 C CNN
-	1    2650 1700
+P 2600 2300
+F 0 "U2" H 2650 2250 60  0001 C CNN
+F 1 "OKI" H 2800 2581 60  0000 C CNN
+F 2 "MRDT_Devices:OKI_Horizontal" H 2400 2200 60  0001 C CNN
+F 3 "" H 2400 2200 60  0001 C CNN
+	1    2600 2300
 	1    0    0    -1
 $EndComp
@@
 L Device:C C1
 U 1 1 5C166A5A
-P 2350 1750
-F 0 "C1" H 2400 1850 50  0000 L CNN
-F 1 "10uF" H 2400 1650 50  0000 L CNN
-F 2 "Capacitors_SMD:C_0603_HandSoldering" H 2388 1600 50  0001 C CNN
-F 3 "~" H 2350 1750 50  0001 C CNN
-	1    2350 1750
+P 2300 2350
+F 0 "C1" H 2350 2450 50  0000 L CNN
+F 1 "10uF" H 2350 2250 50  0000 L CNN
+F 2 "Capacitors_SMD:C_0603_HandSoldering" H 2338 2200 50  0001 C CNN
+F 3 "~" H 2300 2350 50  0001 C CNN
+	1    2300 2350
 	1    0    0    -1
 $EndComp
@@
 L Device:C C2
 U 1 1 5C166B56
-P 3350 1750
-F 0 "C2" H 3400 1850 50  0000 L CNN
-F 1 "10uF" H 3150 1650 50  0000 L CNN
-F 2 "Capacitors_SMD:C_0603_HandSoldering" H 3388 1600 50  0001 C CNN
-F 3 "~" H 3350 1750 50  0001 C CNN
-	1    3350 1750
+P 3300 2350
+F 0 "C2" H 3350 2450 50  0000 L CNN
+F 1 "10uF" H 3100 2250 50  0000 L CNN
+F 2 "Capacitors_SMD:C_0603_HandSoldering" H 3338 2200 50  0001 C CNN
+F 3 "~" H 3300 2350 50  0001 C CNN
+	1    3300 2350
 	1    0    0    -1
 $EndComp
@@
 L power:+5V #PWR0114
 U 1 1 5C167097
-P 3350 1550
-F 0 "#PWR0114" H 3350 1400 50  0001 C CNN
-F 1 "+5V" H 3365 1723 50  0000 C CNN
-F 2 "" H 3350 1550 50  0001 C CNN
-F 3 "" H 3350 1550 50  0001 C CNN
-	1    3350 1550
-	1    0    0    -1
-$EndComp
-Connection ~ 2200 1900
-Connection ~ 2350 1900
-Wire Wire Line
-	2350 1900 2200 1900
-Connection ~ 2850 1900
-Wire Wire Line
-	2850 1900 2350 1900
-Wire Wire Line
-	3350 1900 2850 1900
-Wire Wire Line
-	2200 1600 2350 1600
-Connection ~ 2200 1600
-Connection ~ 2350 1600
-Wire Wire Line
-	2350 1600 2450 1600
-Wire Wire Line
-	3250 1600 3350 1600
-Text Notes 2950 1800 0    50   ~ 0
+P 3300 2150
+F 0 "#PWR0114" H 3300 2000 50  0001 C CNN
+F 1 "+5V" H 3315 2323 50  0000 C CNN
+F 2 "" H 3300 2150 50  0001 C CNN
+F 3 "" H 3300 2150 50  0001 C CNN
+	1    3300 2150
+	1    0    0    -1
+$EndComp
+Connection ~ 2150 2500
+Connection ~ 2300 2500
+Wire Wire Line
+	2300 2500 2150 2500
+Connection ~ 2800 2500
+Wire Wire Line
+	2800 2500 2300 2500
+Wire Wire Line
+	3300 2500 2800 2500
+Wire Wire Line
+	2150 2200 2300 2200
+Connection ~ 2150 2200
+Connection ~ 2300 2200
+Wire Wire Line
+	2300 2200 2400 2200
+Wire Wire Line
+	3200 2200 3300 2200
+Text Notes 2900 2400 0    50   ~ 0
 5V
 Wire Wire Line
-	3350 1550 3350 1600
-Connection ~ 3350 1600
+	3300 2150 3300 2200
+Connection ~ 3300 2200
 $EndSCHEMATC

Commit message: Updated to Rev 2 Libraries
Parts:
- Conn1: footprint MRDT_Connectors:Anderson_2_Horisontal_Side_by_Side -> MRDT_Connectors:Anderson_2_Horizontal_Side_by_Side
- J1, J2: footprint BNC-75-Ohm-HORIZONTAL:BNC-75-Ohm-HORIZONTAL-1-1478032-0 -> MRDT_Connectors:BNC_THT_Horizontal; symbol BNC-75-Ohm-HORIZONTAL:BNC_75_OHM_HORIZ -> Connector:Conn_Coaxial
- U1: footprint MRDT_Shields:TM4C129E_Launchpad_X9_THT -> MRDT_Shields:TM4C129E_Launchpad_X9_THT_BOTTOM
- U3, U4: footprint MAX4314:MAX4314ESD&plus_ -> MRDT_ICs:MAX4314ESD+; symbol MAX4314ESD+:MAX4314ESD+ -> MRDT_ICs:MAX4314ESD+
Connections:
- wire segments 108 -> 109
