File: PowerBoard_Hardware_Rev_2/PowerBoard_Hardware.kicad_pcb (KiCad board)
At the start: 4 copper layers, 279.4 x 126.9 mm, 153 parts, among them Q1 BSS138PW.115, Q10 Q_NMOS_GDS, Q11 Q_NMOS_GDS, Q12 Q_NMOS_GDS, Q13 Q_NMOS_GDS, Q2 BSS138PW.115, Q3 IPT020N10N3, Q4 IPT020N10N3, Q5 IPT020N10N3, Q6 Q_NMOS_GDS, Q7 Q_NMOS_GDS, Q8 Q_NMOS_GDS, Q9 Q_NMOS_GDS, U1 TM4C129E_Launchpad, U10 OKI, U11 LT1910, U12 LT1910, U13 LT1910, U14 LT1910, U15 ATC_FUSE_BLOCK, U16 ATC_FUSE_BLOCK, U17 ATC_FUSE_BLOCK, U18 ATC_FUSE_BLOCK, U19 ACS722xLCTR-40AU, U2 ATC_FUSE_BLOCK, U20 ACS722xLCTR-40AU, U21 ACS722xLCTR-40AU, U22 ACS722xLCTR-40AU, U23 LT1910, U24 LT1910, U25 LT1910, U26 LT1910, U27 ATC_FUSE_BLOCK, U28 ATC_FUSE_BLOCK, U29 ATC_FUSE_BLOCK, U3 ATC_FUSE_BLOCK, U30 ATC_FUSE_BLOCK, U31 ACS722xLCTR-40AU, U32 ACS722xLCTR-40AU, U33 ACS722xLCTR-40AU, U34 ACS722xLCTR-40AU, U4 ATC_FUSE_BLOCK, U5 LT1910, U6 LT1910, U7 ACS722xLCTR-40AU, U8 ACS722xLCTR-40AU, U9 ACS722xLCTR-40AU

Commit message: Started Slimming down the board
The lefthand side of the board has gotten trimmed as to fit in our reflow oven
Parts:
- moved G*** 65.1 mm to (88.9, 31.1)
- moved G*** 63.3 mm to (91.4, 46.4)
- moved R14 18.0 mm to (52.1, 137.2)
- moved D8 15.3 mm to (47.0, 137.2)
- moved C43 14.9 mm to (89.5, 137.8)
- moved U29 14.6 mm to (91.4, 119.4)
- moved Q10 14.2 mm to (63.1, 129.9)
- moved C41 14.0 mm to (76.8, 80.6)
- moved Q11 14.0 mm to (62.9, 112.2)
- moved U28 14.0 mm to (91.4, 102.2)
- moved U27 14.0 mm to (91.4, 135.3)
- moved U31 14.0 mm to (83.2, 132.7)
- moved Q13 13.8 mm to (62.6, 94.0)
- moved U32 13.7 mm to (82.9, 116.7)
- moved C47 13.7 mm to (84.8, 124.1)
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Routing:
- net M3_IMEAS: track 170.7 -> 56.6 mm, vias 2 -> 1
- net M2_IMEAS: track 164.2 -> 58.7 mm, vias 2 -> 1
- net M3_CTL: track 125.9 -> 40.1 mm, vias 3 -> 1
- net M1_IMEAS: track 144.6 -> 59.7 mm, vias 1 -> 0
- net M2_CTL: track 110.0 -> 41.0 mm, vias 3 -> 1
- net M1_CTL: track 91.6 -> 41.7 mm, vias 3 -> 1
- net AUX_IMEAS: track 70.4 -> 24.2 mm, vias 3 -> 1
- net +3.3VA: track 650.8 -> 632.2 mm, vias 13 -> 9
- net AUX_CTL: track 7.21 -> 22.9 mm
- net Net-(C44-Pad2): track 10.2 -> 0.00 mm
- net FAN_CTL: track 121.1 -> 112.2 mm
- net Net-(C41-Pad1): track 20.3 -> 12.6 mm
- net Net-(C38-Pad1): track 20.8 -> 14.0 mm
- net GND: track 222.7 -> 217.2 mm, vias 47 -> 50
- net Net-(C39-Pad1): track 21.2 -> 16.8 mm
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Other:
- board size 279.4 x 126.9 mm -> 266.7 x 126.9 mm

Commit message: Squeezed board even more
The board is now about 10 inches wide and the board now has a much tighter fit.
Parts:
- moved Q3 22.4 mm to (64.8, 52.7)
- moved 3V3FAN1 17.2 mm to (52.8, 53.1)
- moved C45 14.5 mm to (96.0, 91.2)
- moved C48 14.4 mm to (98.6, 91.3)
- moved U30 14.2 mm to (105.4, 85.7)
- moved U33 14.1 mm to (96.6, 82.5)
- moved REF** 14.0 mm to (39.4, 139.5)
- moved C42 14.0 mm to (96.3, 125.1)
- moved C47 14.0 mm to (98.8, 125.1)
- moved C40 14.0 mm to (90.8, 98.4)
- moved R14 14.0 mm to (66.0, 136.5)
- moved C38 14.0 mm to (90.2, 131.8)
- moved C39 14.0 mm to (91.4, 116.2)
- moved C43 14.0 mm to (103.5, 137.2)
- moved C44 14.0 mm to (91.8, 137.2)
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Routing:
- net M3_IMEAS: track 56.6 -> 174.7 mm, vias 1 -> 2
- net M2_IMEAS: track 58.7 -> 160.3 mm, vias 1 -> 2
- net M3_CTL: track 40.1 -> 129.4 mm, vias 1 -> 3
- net M1_IMEAS: track 59.7 -> 146.7 mm, vias 0 -> 1
- net M2_CTL: track 41.0 -> 116.8 mm, vias 1 -> 3
- net M1_CTL: track 41.7 -> 88.2 mm
- net +3.3VA: track 632.2 -> 665.3 mm, vias 9 -> 15
- net FAN_CTL: track 112.2 -> 94.3 mm
- net AUX_IMEAS: track 24.2 -> 40.5 mm
- net AUX_CTL: track 22.9 -> 36.6 mm
- net VMEAS_VBATT: track 76.4 -> 83.4 mm
- net Net-(3V3FAN1-Pad1): track 4.91 -> 11.3 mm, vias 0 -> 1
- net Net-(C44-Pad2): track 0.00 -> 5.47 mm
- net Net-(C42-Pad2): track 0.00 -> 5.37 mm
- net Net-(C45-Pad2): track 0.00 -> 5.23 mm
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Other:
- board size 266.7 x 126.9 mm -> 252.7 x 127.1 mm

Commit message: Minor Silkscreen update
Parts:
- moved C9 2.30 mm to (154.6, 34.9), turned to 0 degrees
Other:
- board text added: "Power Board Rev 2 2019 Mars Rover Design Team Missouri S&T Evan Hite"
- board text removed: "Power Board Rev 1 2019 Mars Rover Design Team Missouri S&T Evan Hite"
Changed lines of the file:
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@@
     (tags "resistor 0603")
     (attr smd)
-    (fp_text reference R5 (at 0 -1.45 90) (layer F.SilkS)
+    (fp_text reference R5 (at 0 1.905 90) (layer F.SilkS)
       (effects (font (size 1 1) (thickness 0.15)))
     )
@@
   )
   (module Capacitors_THT:CP_Radial_D8.0mm_P3.50mm (layer F.Cu)
-    (at 152.4 34.29 180)
+    (at 154.615 34.925)
     (descr "CP, Radial series, Radial, pin pitch=3.50mm, , diameter=8mm, Electrolytic Capacitor")
     (tags "CP Radial series Radial pin pitch 3.50mm  diameter 8mm Electrolytic Capacitor")
-    (fp_text reference C9 (at 1.75 -5.31 180) (layer F.SilkS)
+    (fp_text reference C9 (at 1.75 -5.31) (layer F.SilkS)
       (effects (font (size 1 1) (thickness 0.15)))
     )
-    (fp_text value 330u (at 1.75 5.31 180) (layer F.Fab)
+    (fp_text value 330u (at 1.75 5.31) (layer F.Fab)
       (effects (font (size 1 1) (thickness 0.15)))
     )
@@
     (fp_line (start 6.1 4.35) (end 6.1 -4.35) (layer F.CrtYd) (width 0.05))
     (fp_line (start 6.1 -4.35) (end -2.6 -4.35) (layer F.CrtYd) (width 0.05))
-    (fp_text user %R (at 1.75 0 180) (layer F.Fab)
+    (fp_text user %R (at 1.75 0) (layer F.Fab)
       (effects (font (size 1 1) (thickness 0.15)))
     )
-    (pad 1 thru_hole rect (at 0 0 180) (size 1.6 1.6) (drill 0.8) (layers *.Cu *.Mask)
+    (pad 1 thru_hole rect (at 0 0) (size 1.6 1.6) (drill 0.8) (layers *.Cu *.Mask)
       (net 81 "Net-(C10-Pad1)"))
-    (pad 2 thru_hole circle (at 3.5 0 180) (size 1.6 1.6) (drill 0.8) (layers *.Cu *.Mask)
+    (pad 2 thru_hole circle (at 3.5 0) (size 1.6 1.6) (drill 0.8) (layers *.Cu *.Mask)
       (net 76 GND))
     (model ${KISYS3DMOD}/Capacitors_THT.3dshapes/CP_Radial_D8.0mm_P3.50mm.wrl
@@
     (effects (font (size 2.54 2.54) (thickness 0.3)))
   )
-  (gr_text - (at 226.06 124.46) (layer F.SilkS)
+  (gr_text - (at 227.33 123.19) (layer F.SilkS)
     (effects (font (size 12.7 12.7) (thickness 1.27)))
   )
-  (gr_text + (at 127 124.46) (layer F.SilkS)
+  (gr_text + (at 127 122.555) (layer F.SilkS)
     (effects (font (size 12.7 12.7) (thickness 1.27)))
   )
@@
   (gr_arc (start 288.010731 135.513092) (end 287.8836 139.573) (angle -94.10571235) (layer Edge.Cuts) (width 0.2))
   (gr_arc (start 288.1376 16.6624) (end 292.1 16.77) (angle -87.7888971) (layer Edge.Cuts) (width 0.2))
-  (gr_text "Power Board Rev 1 2019\nMars Rover Design Team\nMissouri S&T\nEvan Hite" (at 87.376 24.13) (layer F.SilkS)
+  (gr_text "Power Board Rev 2 2019\nMars Rover Design Team\nMissouri S&T\nEvan Hite" (at 87.376 24.13) (layer F.SilkS)
     (effects (font (size 1.5 1.5) (thickness 0.3)))
   )
-  (gr_text Ethernet (at 30.48 23.495) (layer F.SilkS)
+  (gr_text Ethernet (at 44.45 28.575) (layer F.SilkS)
     (effects (font (size 1.5 1.5) (thickness 0.3)))
   )
-  (gr_line (start 35.56 22.225) (end 25.4 22.225) (layer F.SilkS) (width 0.2))
-  (gr_line (start 35.56 28.575) (end 35.56 22.225) (layer F.SilkS) (width 0.2))
-  (gr_line (start 25.4 28.575) (end 35.56 28.575) (layer F.SilkS) (width 0.2))
+  (gr_line (start 49.53 25.4) (end 39.37 25.4) (layer F.SilkS) (width 0.2))
+  (gr_line (start 49.53 31.75) (end 49.53 25.4) (layer F.SilkS) (width 0.2))
+  (gr_line (start 39.37 31.75) (end 49.53 31.75) (layer F.SilkS) (width 0.2))
   (gr_text M4 (at 286.512 124.968) (layer F.SilkS)
     (effects (font (size 5.08 5.08) (thickness 0.635)))
@@
     (effects (font (size 5.08 5.08) (thickness 0.635)))
   )
-  (gr_text "Fan Control" (at 32.385 37.465) (layer F.SilkS)
+  (gr_text "Fan Control" (at 46.355 46.99) (layer F.SilkS)
     (effects (font (size 1.5 1.5) (thickness 0.3)))
   )
@@
   (gr_line (start 39.37 16.51) (end 39.37 135.636) (layer Edge.Cuts) (width 0.2))
   (gr_line (start 133.35 17.78) (end 133.35 19.05) (layer F.SilkS) (width 0.2))
-  (gr_line (start 25.4 17.78) (end 133.35 17.78) (layer F.SilkS) (width 0.2))
+  (gr_line (start 39.37 17.78) (end 133.35 17.78) (layer F.SilkS) (width 0.2))
   (gr_line (start 133.35 73.66) (end 133.35 19.05) (layer F.SilkS) (width 0.2))
   (gr_line (start 147.32 73.025) (end 39.37 73.025) (layer F.SilkS) (width 0.2))
-  (gr_line (start 25.4 19.05) (end 25.4 17.78) (layer F.SilkS) (width 0.2))
-  (gr_line (start 25.4 73.66) (end 25.4 19.05) (layer F.SilkS) (width 0.2))
+  (gr_line (start 39.37 19.685) (end 39.37 17.78) (layer F.SilkS) (width 0.2))
+  (gr_line (start 39.37 73.025) (end 39.37 19.685) (layer F.SilkS) (width 0.2))
   (gr_line (start 43.307 139.573) (end 95.09 139.573) (layer Edge.Cuts) (width 0.2))
   (segment (start 63.44 52.705) (end 61.750501 52.705) (width 0.381) (layer F.Cu) (net 1))

Commit message: Completed Board Review. Minor Changes to Motor Bus Layout
Deleted Motor 7 from Board. Renamed Motors 1-6 for other uses and easier reading. Auxillary is now on the right hand side of the board, As well as non motor busses. Front Middle, Back and Extra are all on one side to fit with Motor Controller Specs. Added Extra Silkscreen for a more beautiful look.
Parts:
- removed C26, C34: 0.1u, Capacitors_SMD:C_0603_HandSoldering
- removed C31: 1n, Capacitors_SMD:C_0603_HandSoldering
- removed Conn4: AndersonPP, MRDT-Connectors:Anderson_2_Vertical
- removed D14: D_Schottky, Diodes_SMD:D_0603
- removed D4: LED, LEDs:LED_0603_HandSoldering
- removed the G*** at (88.9, 31.1)
- removed the G*** at (91.4, 46.4)
- removed GND: GND, MRDT-Drill_Holes:BATT_PWR_VIA
- removed Q8: Q_NMOS_GDS, TO_SOT_Packages_SMD:TO-263-2
- removed R11: 1.5k, Resistors_SMD:R_0603_HandSoldering
- removed R5: 100k, Resistors_SMD:R_0603_HandSoldering
- removed R6: 10k, Resistors_SMD:R_0603_HandSoldering
- removed the REF** at (39.4, 139.5)
- removed the REF** at (292.0, 139.6)
- removed the REF** at (138.4, 17.1)
- removed the REF** at (279.7, 17.1)
- removed the REF** at (279.7, 83.8)
- removed the REF** at (177.8, 83.8)
- removed U12: LT1910, Housings_SOIC:SOIC-8_3.9x4.9mm_Pitch1.27mm
- removed U16: ATC_FUSE_BLOCK, MRDT-Passives:ATC_Fuse_Block
- removed U20: ACS722xLCTR-40AU, Housings_SOIC:SOIC-8_3.9x4.9mm_Pitch1.27mm
- added G***: LOGO, MRDT-Silkscreen:0_MRDT_Logo_40mm, F.Cu at (94.0, 46.4)
- added G***: LOGO, MRDT-Silkscreen:z_sig_Evan_Hite_Sig_15mm, F.Cu at (89.5, 31.1)
- added G***: LOGO, MRDT-Silkscreen:2_Dahlbot_2.0, F.Cu at (177.2, 96.5)
- added G***: LOGO, MRDT-Silkscreen:0_MRDT_Retro_Logo_40mmX25.3mm, F.Cu at (272.4, 45.1)
- added REF**: 4_40_Hole, MRDT-Drill_Holes:4_40_Hole_Corner, F.Cu at (292.0, 139.7)
- added REF**: 4_40_Hole, MRDT-Drill_Holes:4_40_Hole_Corner, F.Cu at (39.5, 139.6)
- added REF**: 6_32_Hole, MRDT-Drill_Holes:6_32_Hole, F.Cu at (279.7, 17.1)
- added REF**: 6_32_Hole, MRDT-Drill_Holes:6_32_Hole, F.Cu at (177.8, 83.8)
- added REF**: 6_32_Hole, MRDT-Drill_Holes:6_32_Hole, F.Cu at (279.7, 83.8)
- added REF**: 6_32_Hole, MRDT-Drill_Holes:6_32_Hole, F.Cu at (138.4, 17.1)
- added REF**: BATT_PWR_VIA, MRDT-Drill_Holes:BATT_PWR_VIA, F.Cu at (210.8, 125.1)
- Q3: value IPT020N10N3 -> N_Fet
- Q4, Q5: value IPT020N10N3 -> FDD8780
- The Van: renamed from CONV2
- moved D5 7.70 mm to (286.1, 129.5)
- moved D6 6.33 mm to (285.0, 78.2)
- moved D7 6.25 mm to (285.0, 104.8)
- renumbered CONV1 to Dahlbot
Connections:
- net M1_CTL renamed FM_CTL
- net M1_IMEAS renamed FM_IMEAS
- net M2_CTL renamed MM_CTL
- net M2_IMEAS renamed MM_IMEAS
- net M3_CTL renamed BM_CTL
- net M3_IMEAS renamed BM_IMEAS
- net M5_CTL renamed ROCKET_CTL
- net M5_IMEAS renamed ROCKET_IMEAS
- net M6_CTL renamed GE_CTL
- net M6_IMEAS renamed GE_IMEAS
- Dahlbot pad 6: Net-(CONV1-Pad6) -> (no net)
- The Van pad 6: Net-(CONV2-Pad6) -> (no net)
- U1 pad PA4: Net-(U1-PadPA4) -> (no net)
- U1 pad PA5: Net-(U1-PadPA5) -> (no net)
- U1 pad PA6: Net-(U1-PadPA6) -> (no net)
- U1 pad PA7: Net-(U1-PadPA7) -> (no net)
- U1 pad PB2: Net-(U1-PadPB2) -> (no net)
- U1 pad PB3: Net-(U1-PadPB3) -> (no net)
- U1 pad PC4: Net-(U1-PadPC4) -> (no net)
- U1 pad PC5: Net-(U1-PadPC5) -> (no net)
- U1 pad PC6: Net-(U1-PadPC6) -> (no net)
- U1 pad PC7: Net-(U1-PadPC7) -> (no net)
- U1 pad PD0: AUX_IMEAS -> EM_IMEAS
- U1 pad PD2: Net-(U1-PadPD2) -> (no net)
- U1 pad PD3: Net-(U1-PadPD3) -> (no net)
- U1 pad PD4: Net-(U1-PadPD4) -> (no net)
- U1 pad PD5: Net-(U1-PadPD5) -> (no net)
- U1 pad PD7: Net-(U1-PadPD7) -> (no net)
- U1 pad PE3: M7_IMEAS -> (no net)
- U1 pad PE4: Net-(U1-PadPE4) -> (no net)
- U1 pad PE5: VMEAS_VBATT -> (no net)
- U1 pad PF1: Net-(U1-PadPF1) -> (no net)
- U1 pad PF2: Net-(U1-PadPF2) -> (no net)
- U1 pad PF3: Net-(U1-PadPF3) -> (no net)
- U1 pad PG0: Net-(U1-PadPG0) -> (no net)
- U1 pad PG1: Net-(U1-PadPG1) -> (no net)
- U1 pad PH0: M4_CTL -> AUX_CTL
- U1 pad PH3: Net-(U1-PadPH3) -> (no net)
- U1 pad PK0: M4_IMEAS -> AUX_IMEAS
- U1 pad PK4: Net-(U1-PadPK4) -> (no net)
- U1 pad PK5: AUX_CTL -> EM_CTL
- U1 pad PL0: Net-(U1-PadPL0) -> (no net)
- U1 pad PL1: Net-(U1-PadPL1) -> (no net)
- U1 pad PL2: Net-(U1-PadPL2) -> (no net)
- U1 pad PL3: Net-(U1-PadPL3) -> (no net)
- U1 pad PL4: Net-(U1-PadPL4) -> (no net)
- U1 pad PL5: Net-(U1-PadPL5) -> (no net)
- U1 pad PM0: M7_CTL -> (no net)
- U1 pad PM4: Net-(U1-PadPM4) -> (no net)
- U1 pad PM5: Net-(U1-PadPM5) -> (no net)
- U1 pad PM6: Net-(U1-PadPM6) -> (no net)
- U1 pad PM7: Net-(U1-PadPM7) -> (no net)
- U1 pad PN2: Net-(U1-PadPN2) -> (no net)
- U1 pad PN4: Net-(U1-PadPN4) -> (no net)
- U1 pad PN5: Net-(U1-PadPN5) -> (no net)
- U1 pad PP0: Net-(U1-PadPP0) -> (no net)
- U1 pad PP1: Net-(U1-PadPP1) -> (no net)
- U1 pad PP3: Net-(U1-PadPP3) -> (no net)
- U1 pad PP4: Net-(U1-PadPP4) -> (no net)
- U1 pad PP5: Net-(U1-PadPP5) -> (no net)
- U1 pad PQ0: Net-(U1-PadPQ0) -> (no net)
- U1 pad PQ1: Net-(U1-PadPQ1) -> (no net)
- U1 pad PQ2: Net-(U1-PadPQ2) -> (no net)
- U1 pad PQ3: Net-(U1-PadPQ3) -> (no net)
- U11 pad 2: Net-(U11-Pad2) -> (no net)
- U11 pad 3: Net-(U11-Pad3) -> (no net)
- U13 pad 2: Net-(U13-Pad2) -> (no net)
- U13 pad 3: Net-(U13-Pad3) -> (no net)
- U14 pad 2: Net-(U14-Pad2) -> (no net)
- U14 pad 3: Net-(U14-Pad3) -> (no net)
- U14 pad 4: M4_CTL -> AUX_CTL
- U22 pad 7: M4_IMEAS -> AUX_IMEAS
- U23 pad 2: Net-(U23-Pad2) -> (no net)
- U23 pad 3: Net-(U23-Pad3) -> (no net)
- U24 pad 2: Net-(U24-Pad2) -> (no net)
- U24 pad 3: Net-(U24-Pad3) -> (no net)
- U25 pad 2: Net-(U25-Pad2) -> (no net)
- U25 pad 3: Net-(U25-Pad3) -> (no net)
- U26 pad 2: Net-(U26-Pad2) -> (no net)
- U26 pad 3: Net-(U26-Pad3) -> (no net)
- U26 pad 4: AUX_CTL -> EM_CTL
- U33 pad 7: AUX_IMEAS -> EM_IMEAS
- U5 pad 2: Net-(U5-Pad2) -> (no net)
- U5 pad 3: Net-(U5-Pad3) -> (no net)
- U6 pad 2: Net-(U6-Pad2) -> (no net)
- U6 pad 3: Net-(U6-Pad3) -> (no net)
Routing:
- net M4_CTL: track 306.4 -> 0.00 mm, vias 2 -> 0
- net M4_IMEAS: track 296.1 -> 0.00 mm, vias 2 -> 0
- net AUX_CTL: track 36.6 -> 306.4 mm, vias 0 -> 2
- net AUX_IMEAS: track 40.5 -> 296.1 mm, vias 1 -> 2
- net M7_CTL: track 229.4 -> 0.00 mm, vias 2 -> 0
- net M7_IMEAS: track 162.4 -> 0.00 mm, vias 2 -> 0
- net VMEAS_VBATT: track 83.4 -> 0.00 mm, vias 2 -> 0
- net EM_IMEAS: track 0.00 -> 40.5 mm, vias 0 -> 1
- net +3.3VA: track 665.3 -> 628.5 mm, vias 15 -> 13
- net EM_CTL: track 0.00 -> 36.6 mm
- net GND: track 221.4 -> 191.4 mm, vias 51 -> 47
- net Net-(Q8-Pad1): track 17.5 -> 0.00 mm
- net Net-(C26-Pad1): track 16.3 -> 0.00 mm
- net Net-(Conn4-Pad2): track 4.56 -> 0.00 mm
- net Net-(C31-Pad2): track 3.34 -> 0.00 mm
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- removed copper zone on F.Cu, net Net-(C26-Pad1)
- removed copper zone on F.Cu, net Net-(Conn4-Pad2)
- removed copper zone on F.Cu, net Net-(U16-Pad1)
Other:
- outline, holes or cut-outs redrawn
- board text added: "(?)A"
- board text added: "40A"
- board text added: "BM"
- board text added: "EM"
- board text added: "FM"
- board text added: "GE"
- board text added: "MM"
- board text added: "ROCKETS"
- board text removed: "30A"
- board text removed: "M1"
- board text removed: "M2"
- board text removed: "M3"
- board text removed: "M4"
- board text removed: "M5"
- board text removed: "M6"
- board text removed: "M7"
