File: PowerBoard_Hardware_Rev_2/PowerBoard_Hardware.kicad_pcb (KiCad board)
At the start: 4 copper layers, 252.7 x 127.1 mm, 142 parts, among them Q1 BSS138PW.115, Q10 Q_NMOS_GDS, Q11 Q_NMOS_GDS, Q12 Q_NMOS_GDS, Q13 Q_NMOS_GDS, Q2 BSS138PW.115, Q3 N_Fet, Q4 FDD8780, Q5 FDD8780, Q6 Q_NMOS_GDS, Q7 Q_NMOS_GDS, Q9 Q_NMOS_GDS, U1 TM4C129E_Launchpad, U10 OKI, U11 LT1910, U13 LT1910, U14 LT1910, U15 ATC_FUSE_BLOCK, U17 ATC_FUSE_BLOCK, U18 ATC_FUSE_BLOCK, U19 ACS722xLCTR-40AU, U2 ATC_FUSE_BLOCK, U21 ACS722xLCTR-40AU, U22 ACS722xLCTR-40AU, U23 LT1910, U24 LT1910, U25 LT1910, U26 LT1910, U27 ATC_FUSE_BLOCK, U28 ATC_FUSE_BLOCK, U29 ATC_FUSE_BLOCK, U3 ATC_FUSE_BLOCK, U30 ATC_FUSE_BLOCK, U31 ACS722xLCTR-40AU, U32 ACS722xLCTR-40AU, U33 ACS722xLCTR-40AU, U34 ACS722xLCTR-40AU, U4 ATC_FUSE_BLOCK, U5 LT1910, U6 LT1910, U7 ACS722xLCTR-40AU, U8 ACS722xLCTR-40AU, U9 ACS722xLCTR-40AU

Commit message: Updated Silkscreen
Parts:
- added G***: LOGO, MRDT-Silkscreen:zz_Valkyrie_Logo_Full_100mmx100mm, B.Cu at (166.1, 74.9)
- moved D8 8.64 mm to (52.3, 136.9)
- moved R14 6.78 mm to (59.3, 136.9)
- moved R16 5.35 mm to (59.0, 103.6)
- moved R15 5.21 mm to (57.9, 121.4)
- moved R17 3.92 mm to (59.4, 87.4)
- moved D9 3.56 mm to (52.3, 121.4)
- moved D10 2.79 mm to (53.3, 103.6)
- moved D11 2.31 mm to (53.3, 87.4)
Routing:
- net Net-(Conn10-Pad2): track 4.24 -> 7.56 mm
- net Net-(Conn9-Pad2): track 3.98 -> 6.99 mm
- net Net-(Conn11-Pad2): track 3.25 -> 6.22 mm
- net Net-(D8-Pad2): track 2.88 -> 4.74 mm
- net GND: track 191.4 -> 189.9 mm
- net Net-(D11-Pad2): track 2.61 -> 3.90 mm
- net Net-(Conn8-Pad2): track 4.24 -> 5.16 mm
Other:
- board text added: "Back Motor"
- board text added: "Extra Motor"
- board text added: "Full Motor"
- board text added: "Gen. Extra"
- board text added: "Middle Motor"
- board text removed: "BM"
- board text removed: "EM"
- board text removed: "FM"
- board text removed: "GE"
- board text removed: "MM"

Commit message: Updated Silkscreen
Again
Other:
- board text added: "Front Motor"
- board text removed: "Full Motor"
Changed lines of the file:
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@@
     (effects (font (size 2.54 2.54) (thickness 0.381)))
   )
-  (gr_text "Full Motor" (at 49.276 99.06) (layer F.SilkS)
+  (gr_text "Front Motor" (at 50.546 98.806) (layer F.SilkS)
     (effects (font (size 2.54 2.54) (thickness 0.381)))
   )
