File: PowerBoard_Hardware_Rev_2/PowerBoard_Hardware.sch (KiCad schematic (older format))
At the start: 141 parts, among them Q1 BSS138PW.115, Q10 Q_NMOS_GDS, Q11 Q_NMOS_GDS, Q12 Q_NMOS_GDS, Q13 Q_NMOS_GDS, Q2 BSS138PW.115, Q3 N_Fet, Q4 FDD8780, Q5 FDD8780, Q6 Q_NMOS_GDS, Q7 Q_NMOS_GDS, Q8 Q_NMOS_GDS, Q9 Q_NMOS_GDS, U1 TM4C129E_Launchpad, U10 OKI, U11 LT1910, U12 LT1910, U13 LT1910, U14 LT1910, U15 ATC_FUSE_BLOCK, U16 ATC_FUSE_BLOCK, U17 ATC_FUSE_BLOCK, U18 ATC_FUSE_BLOCK, U19 ACS722xLCTR-40AU, U2 ATC_FUSE_BLOCK, U20 ACS722xLCTR-40AU, U21 ACS722xLCTR-40AU, U22 ACS722xLCTR-40AU, U23 LT1910, U24 LT1910, U25 LT1910, U26 LT1910, U27 ATC_FUSE_BLOCK, U28 ATC_FUSE_BLOCK, U29 ATC_FUSE_BLOCK, U3 ATC_FUSE_BLOCK, U30 ATC_FUSE_BLOCK, U31 ACS722xLCTR-40AU, U32 ACS722xLCTR-40AU, U33 ACS722xLCTR-40AU, U34 ACS722xLCTR-40AU, U4 ATC_FUSE_BLOCK, U5 LT1910, U6 LT1910, U7 ACS722xLCTR-40AU, U8 ACS722xLCTR-40AU, U9 ACS722xLCTR-40AU

Commit message: Completed Board Review. Minor Changes to Motor Bus Layout
Deleted Motor 7 from Board. Renamed Motors 1-6 for other uses and easier reading. Auxillary is now on the right hand side of the board, As well as non motor busses. Front Middle, Back and Extra are all on one side to fit with Motor Controller Specs. Added Extra Silkscreen for a more beautiful look.
Parts:
- removed C26, C34: 0.1u, Capacitors_SMD:C_0603_HandSoldering, symbol Device:C_Small
- removed C31: 1n, Capacitors_SMD:C_0603_HandSoldering, symbol Device:C_Small
- removed Conn4: AndersonPP, MRDT-Connectors:Anderson_2_Vertical, symbol MRDT_Connectors:AndersonPP
- removed D14: D_Schottky, Diodes_SMD:D_0603, symbol Device:D_Schottky
- removed D4: LED, LEDs:LED_0603_HandSoldering, symbol Device:LED
- removed Q8: Q_NMOS_GDS, TO_SOT_Packages_SMD:TO-263-2, symbol Device:Q_NMOS_GDS
- removed R11: 1.5k, Resistors_SMD:R_0603_HandSoldering, symbol Device:R_US
- removed R5: 100k, Resistors_SMD:R_0603_HandSoldering, symbol Device:R_US
- removed R6: 10k, Resistors_SMD:R_0603_HandSoldering, symbol Device:R_US
- removed U12: LT1910, Housings_SOIC:SOIC-8_3.9x4.9mm_Pitch1.27mm, symbol MRDT_ICs:LT1910
- removed U16: ATC_FUSE_BLOCK, MRDT-Passives:ATC_Fuse_Block, symbol Device:Fuse
- removed U20: ACS722xLCTR-40AU, Housings_SOIC:SOIC-8_3.9x4.9mm_Pitch1.27mm, symbol Sensor_Current:ACS722xLCTR-40AU
Connections:
- net labels added: BM_CTL, BM_IMEAS, EM_CTL, EM_IMEAS, FM_CTL, FM_IMEAS, GE_CTL, GE_IMEAS, MM_CTL, MM_IMEAS, ROCKET_CTL, ROCKET_IMEAS
- net labels removed: M1_CTL, M1_IMEAS, M2_CTL, M2_IMEAS, M3_CTL, M3_IMEAS, M4_CTL, M4_IMEAS, M5_CTL, M5_IMEAS, M6_CTL, M6_IMEAS, M7_CTL, M7_IMEAS, VMEAS_VBATT
- wire segments 550 -> 499
- no-connect marks 55 -> 58
Other:
- note added: "Auxillary"
- note added: "Back"
- note added: "Extra"
- note added: "Front"
- note added: "General Extra"
- note added: "MOTORS"
- note added: "Middle"
- note added: "OTHER PVDD BUSSES"
- note added: "Rockets"
- note removed: "A0"
- note removed: "A8"
- note removed: "Auxillary\n"
- note removed: "MOTORS 1-7 AND AUX"
- note removed: "Motor 1"
- note removed: "Motor 2"
- note removed: "Motor 3"
- note removed: "Motor 4"
- note removed: "Motor 5"
- note removed: "Motor 6"
- note removed: "Motor 7"
- note removed: "Primary Voltage Measuring\n<---------------"
- moved on the sheet: Q3, U19, U21, U22, U31, U32, U33
